File: FPGA_Board_BA/FPGA_Board_BA.kicad_sch (KiCad schematic)
At the start: 0 parts

Commit message: starting schematic + added kicad lib
Parts:
- added R1, R2, R3: 0R100_2512, Resistor_SMD:R_2512_6332Metric_Pad1.40x3.35mm_HandSolder, symbol MYLIB_R:0R100_2512
Connections:
- new net Current measure/Ph_A+: R1.1
- new net Current measure/Ph_A-: R1.2
- new net Current measure/Ph_B+: R2.1
- new net Current measure/Ph_B-: R2.2
- new net Current measure/Ph_C+: R3.1
- new net Current measure/Ph_C-: R3.2
Other:
- added sheet ADC (adc.kicad_sch)
- added sheet Current measure (current_measure.kicad_sch)
- added sheet FPGA (fpga.kicad_sch)
