File: FPGA_Board_BA/PCB/FPGA_Board_BA.kicad_sch (KiCad schematic)
At the start: 4 parts

Commit message: lot of work
Other:
- added sheet ADC power (adc_power.kicad_sch)
- sheet ADC for B6: file adc.kicad_sch -> adc_for_b6.kicad_sch
- sheet Main_DCDC ports: added Vout_5V; removed Vout
- note added: "- DCDC for Differential-amplifier [X] ADC power supply (1.8V ... 2.5V) - Breakout for all unused pins - ESD Diode Array for unused pins [X] Add another ADC for B6 - CHB Rx En Err -> 10 pin (wie base board) - Poti an Analog Input - ADC Datenbatt Recherche LVDS/CMOS ob 24pin + 2pins für comversion start frei sind [X] FPGA falsche pin namen an Hersteller + BA - Level shifter für Tx Rx und Fault pins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"
- note removed: "- DCDC for Differential-amplifier - ADC power supply (1.8V ... 2.5V) - Breakout for all unused pins - ESD Diode Array for unused pins [X] Add another ADC for B6 - CHB Rx En Err -> 10 pin (wie base board) - Poti an Analog Input - ADC Datenbatt Recherche LVDS/CMOS ob 24pin + 2pins für comversion start frei sind - FPGA falsche pin namen an Hersteller + BA - Level shifter für Tx Rx und Fault pins (CH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"
Changed lines of the file:
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@@
 	(generator_version "9.0")
 	(paper "A3")
-	(text "- DCDC for Differential-amplifier\n- ADC power supply (1.8V ... 2.5V)\n- Breakout for all unused pins\n- ESD Diode Array for unused pins\n[X] Add another ADC for B6\n- CHB Rx En Err -> 10 pin (wie base board)\n- Poti an Analog Input\n- ADC Datenbatt Recherche LVDS/CMOS ob 24pin + 2pins für comversion start frei sind\n- FPGA falsche pin namen an Hersteller + BA \n- Level shifter für Tx Rx und Fault pins (CHB -> FPGA)\n- Pullup Resistor für Tx der CHB und auch Rx\n- Latex dokumentation beginnen\n- Diff Eingang für ADC (mit OP-Amps)\n[X] CMOS Fest, DDR mit 2 Widerstände\n[X] HV-Probe hinzufügen"
+	(text "- DCDC for Differential-amplifier\n[X] ADC power supply (1.8V ... 2.5V)\n- Breakout for all unused pins\n- ESD Diode Array for unused pins\n[X] Add another ADC for B6\n- CHB Rx En Err -> 10 pin (wie base board)\n- Poti an Analog Input\n- ADC Datenbatt Recherche LVDS/CMOS ob 24pin + 2pins für comversion start frei sind\n[X] FPGA falsche pin namen an Hersteller + BA \n- Level shifter für Tx Rx und Fault pins (CHB -> FPGA)\n- Pullup Resistor für Tx der CHB und auch Rx\n- Latex dokumentation beginnen\n[X] Diff Eingang für ADC (mit OP-Amps)\n[X] CMOS Fest, DDR mit 2 Widerstände\n[X] HV-Probe hinzufügen\n[X] 26 pin wannenstecker\n- RapidHarness Verkabelung"
 		(exclude_from_sim no)
 		(at 302.26 230.378 0)
@@
 	)
 	(junction
+		(at 96.52 40.64)
+		(diameter 0)
+		(color 0 0 0 0)
+	)
+	(junction
 		(at 332.74 73.66)
 		(diameter 0)
@@
 	(wire
 		(pts
-			(xy 92.71 38.1) (xy 100.33 38.1)
+			(xy 96.52 43.18) (xy 100.33 43.18)
 		)
 		(stroke
@@
 	(wire
 		(pts
+			(xy 96.52 40.64) (xy 92.71 40.64)
+		)
+		(stroke
+			(width 0)
+			(type default)
+		)
+	)
+	(wire
+		(pts
 			(xy 363.22 36.83) (xy 363.22 64.77)
 		)
@@
 	(wire
 		(pts
-			(xy 259.08 127) (xy 284.48 127)
+			(xy 256.54 127) (xy 284.48 127)
 		)
 		(stroke
@@
 	(wire
 		(pts
-			(xy 259.08 129.54) (xy 284.48 129.54)
+			(xy 256.54 129.54) (xy 284.48 129.54)
 		)
 		(stroke
@@
 	(wire
 		(pts
-			(xy 198.12 72.39) (xy 224.79 72.39)
+			(xy 198.12 72.39) (xy 222.25 72.39)
 		)
 		(stroke
@@
 	(wire
 		(pts
+			(xy 67.31 38.1) (xy 58.42 38.1)
+		)
+		(stroke
+			(width 0)
+			(type default)
+		)
+	)
+	(wire
+		(pts
 			(xy 307.34 74.93) (xy 317.5 74.93)
 		)
@@
 	(wire
 		(pts
-			(xy 198.12 86.36) (xy 224.79 86.36)
+			(xy 198.12 86.36) (xy 222.25 86.36)
 		)
 		(stroke
@@
 	(wire
 		(pts
-			(xy 198.12 67.31) (xy 224.79 67.31)
+			(xy 198.12 67.31) (xy 222.25 67.31)
 		)
 		(stroke
@@
 	(wire
 		(pts
-			(xy 259.08 124.46) (xy 284.48 124.46)
+			(xy 256.54 124.46) (xy 284.48 124.46)
 		)
 		(stroke
@@
 	(wire
 		(pts
-			(xy 198.12 81.28) (xy 224.79 81.28)
+			(xy 198.12 81.28) (xy 222.25 81.28)
 		)
 		(stroke
@@
 	(wire
 		(pts
-			(xy 198.12 78.74) (xy 224.79 78.74)
+			(xy 198.12 78.74) (xy 222.25 78.74)
 		)
 		(stroke
@@
 	(wire
 		(pts
-			(xy 198.12 96.52) (xy 224.79 96.52)
+			(xy 198.12 96.52) (xy 222.25 96.52)
+		)
+		(stroke
+			(width 0)
+			(type default)
+		)
+	)
+	(wire
+		(pts
+			(xy 96.52 26.67) (xy 96.52 40.64)
 		)
 		(stroke
@@
 	(wire
 		(pts
-			(xy 198.12 88.9) (xy 224.79 88.9)
+			(xy 198.12 88.9) (xy 222.25 88.9)
 		)
 		(stroke
@@
 	(wire
 		(pts
-			(xy 198.12 91.44) (xy 224.79 91.44)
+			(xy 198.12 91.44) (xy 222.25 91.44)
 		)
 		(stroke
@@
 	(wire
 		(pts
-			(xy 198.12 83.82) (xy 224.79 83.82)
+			(xy 198.12 83.82) (xy 222.25 83.82)
 		)
 		(stroke
@@
 	(wire
 		(pts
-			(xy 198.12 69.85) (xy 224.79 69.85)
+			(xy 198.12 69.85) (xy 222.25 69.85)
 		)
 		(stroke
@@
 	(wire
 		(pts
-			(xy 198.12 93.98) (xy 224.79 93.98)
+			(xy 198.12 93.98) (xy 222.25 93.98)
 		)
 		(stroke
@@
 	(wire
 		(pts
-			(xy 58.42 38.1) (xy 68.58 38.1)
+			(xy 67.31 40.64) (xy 68.58 40.64)
 		)
 		(stroke
@@
 	(wire
 		(pts
+			(xy 96.52 43.18) (xy 96.52 40.64)
+		)
+		(stroke
+			(width 0)
+			(type default)
+		)
+	)
+	(wire
+		(pts
 			(xy 313.69 130.81) (xy 358.14 130.81)
 		)
@@
 	(wire
 		(pts
+			(xy 100.33 26.67) (xy 96.52 26.67)
+		)
+		(stroke
+			(width 0)
+			(type default)
+		)
+	)
+	(wire
+		(pts
 			(xy 110.49 266.7) (xy 156.21 266.7)
 		)
@@
 	(wire
 		(pts
-			(xy 259.08 121.92) (xy 284.48 121.92)
+			(xy 256.54 121.92) (xy 284.48 121.92)
 		)
 		(stroke
@@
 	(wire
 		(pts
+			(xy 67.31 40.64) (xy 67.31 38.1)
+		)
+		(stroke
+			(width 0)
+			(type default)
+		)
+	)
+	(wire
+		(pts
 			(xy 363.22 101.6) (xy 363.22 133.35)
 		)
@@
 	)
 	(sheet
-		(at 100.33 33.02)
+		(at 100.33 38.1)
 		(size 27.94 12.7)
 		(exclude_from_sim no)
@@
 		)
 		(property "Sheetname" "Analog Voltage"
-			(at 100.33 32.3084 0)
+			(at 100.33 37.3884 0)
 			(effects
 				(font
@@
 		)
 		(property "Sheetfile" "analog_voltage.kicad_sch"
-			(at 100.33 46.3046 0)
+			(at 100.33 51.3846 0)
 			(effects
 				(font
@@
 		)
 		(pin "Vin_A" input
-			(at 100.33 38.1 180)
+			(at 100.33 43.18 180)
 			(effects
 				(font
@@
 	)
 	(sheet
-		(at 224.79 59.69)
+		(at 222.25 59.69)
 		(size 34.29 83.82)
 		(exclude_from_sim no)
@@
 		)
 		(property "Sheetname" "ADC for Machine"
-			(at 224.79 58.9784 0)
+			(at 222.25 58.9784 0)
 			(effects
 				(font
@@
 		)
 		(property "Sheetfile" "adc_machine.kicad_sch"
-			(at 224.79 144.0946 0)
+			(at 222.25 144.0946 0)
 			(effects
 				(font
@@
 		)
 		(pin "CLK_IN_1" input
-			(at 224.79 67.31 180)
+			(at 222.25 67.31 180)
 			(effects
 				(font
@@
 		)
 		(pin "CLK_OUT_1" input
-			(at 224.79 69.85 180)
+			(at 222.25 69.85 180)
 			(effects
 				(font
@@
 		)
 		(pin "SDO1_1" output
-			(at 224.79 78.74 180)
+			(at 222.25 78.74 180)
 			(effects
 				(font
@@
 		)
 		(pin "SDO2_1" output
-			(at 224.79 81.28 180)
+			(at 222.25 81.28 180)
 			(effects
 				(font
@@
 		)
 		(pin "SDO3_1" output
-			(at 224.79 83.82 180)
+			(at 222.25 83.82 180)
 			(effects
 				(font
@@
 		)
 		(pin "SDO4_1" output
-			(at 224.79 86.36 180)
+			(at 222.25 86.36 180)
 			(effects
 				(font
@@
 		)
 		(pin "SDO5_1" output
-			(at 224.79 88.9 180)
+			(at 222.25 88.9 180)
 			(effects
 				(font
@@
 		)
 		(pin "SDO6_1" output
-			(at 224.79 91.44 180)
+			(at 222.25 91.44 180)
 			(effects
 				(font
@@
 		)
 		(pin "SDO7_1" output
-			(at 224.79 93.98 180)
+			(at 222.25 93.98 180)
 			(effects
 				(font
@@
 		)
 		(pin "SDO8_1" output
-			(at 224.79 96.52 180)
+			(at 222.25 96.52 180)
 			(effects
 				(font
@@
 		)
 		(pin "~{CNV}_1" input
-			(at 224.79 72.39 180)
+			(at 222.25 72.39 180)
 			(effects
 				(font
@@
 		)
 		(pin "Vout_1" input
-			(at 259.08 121.92 0)
+			(at 256.54 121.92 0)
 			(effects
 				(font
@@
 		)
 		(pin "Vout_2" input
-			(at 259.08 124.46 0)
+			(at 256.54 124.46 0)
 			(effects
 				(font
@@
 		)
 		(pin "Vout_3" input
-			(at 259.08 127 0)
+			(at 256.54 127 0)
 			(effects
 				(font
@@
 		)
 		(pin "Vout_4" input
-			(at 259.08 129.54 0)
+			(at 256.54 129.54 0)
 			(effects
 				(font
@@
 	)
 	(sheet
+		(at 100.33 20.32)
+		(size 27.94 11.43)
+		(exclude_from_sim no)
+		(in_bom yes)
+		(on_board yes)
+		(dnp no)
+		(fields_autoplaced yes)
+		(stroke
+			(width 0.1524)
+			(type solid)
+		)
+		(fill
+			(color 0 0 0 0.0000)
+		)
+		(property "Sheetname" "ADC power"
+			(at 100.33 19.6084 0)
+			(effects
+				(font
+					(size 1.27 1.27)
+				)
+				(justify left bottom)
+			)
+		)
+		(property "Sheetfile" "adc_power.kicad_sch"
+			(at 100.33 32.3346 0)
+			(effects
+				(font
+					(size 1.27 1.27)
+				)
+				(justify left top)
+			)
+		)
+		(pin "Vin" input
+			(at 100.33 26.67 180)
+			(effects
+				(font
+					(size 1.27 1.27)
+				)
+				(justify left)
+			)
+		)
+		(instances
+			(project "FPGA_Board_BA"
+				(path "/fd7503bc-e7fc-4766-b224-3d1c3d7de5ff"
+					(page "32")
+				)
+			)
+		)
+	)
+	(sheet
 		(at 83.82 93.98)
 		(size 25.4 13.97)
@@
 			)
 		)
-		(property "Sheetfile" "adc.kicad_sch"
+		(property "Sheetfile" "adc_for_b6.kicad_sch"
 			(at 223.52 163.83 0)
 			(effects
@@
 	)
 	(sheet
-		(at 68.58 33.02)
+		(at 68.58 35.56)
 		(size 24.13 12.7)
 		(exclude_from_sim no)
@@
 		)
 		(property "Sheetname" "Main_DCDC"
-			(at 68.58 32.3084 0)
+			(at 68.58 34.8484 0)
 			(effects
 				(font
@@
 		)
 		(property "Sheetfile" "main_dcdc.kicad_sch"
-			(at 68.58 46.3046 0)
+			(at 68.58 48.8446 0)
 			(effects
 				(font
@@
 		)
 		(pin "Vin" input
-			(at 68.58 38.1 180)
+			(at 68.58 40.64 180)
 			(effects
 				(font
@@
 			)
 		)
-		(pin "Vout" output
-			(at 92.71 38.1 0)
+		(pin "Vout_5V" output
+			(at 92.71 40.64 0)
 			(effects
 				(font
