File: FPGA_Board_BA/PCB/main_dcdc.kicad_sch (KiCad schematic)
At the start: 27 parts, among them Q501 IPT017N12NM6, Q502 IPT017N12NM6, Q503 IPT017N12NM6, Q504 IPT017N12NM6, U501 LM5143

Commit message: some work on the schematics
Parts:
- removed D503: SBR10U200P5-13, Diode_SMD:D_PowerDI-5, symbol MYLIB_Misc:SBR10U200P5-13
- added D502: SBR10U200P5-13, MYLIB_Misc:SBR10U200P5, symbol MYLIB_Misc:SBR10U200P5-13
- D501: footprint Diode_SMD:D_PowerDI-5 -> MYLIB_Misc:SBR10U200P5
Connections:
- net at C504.1, C512.1, D501.2 (A)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: now also D502.2 (A)
- net at C503.1, U501.20 (HB1): now also D502.1 (K)
Changed lines of the file:
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@@
 	(wire
 		(pts
-			(xy 173.99 67.31) (xy 173.99 74.93)
-		)
-		(stroke
-			(width 0)
-			(type default)
-		)
-	)
-	(wire
-		(pts
 			(xy 78.74 38.1) (xy 78.74 71.12)
 		)
@@
 	(wire
 		(pts
+			(xy 173.99 67.31) (xy 173.99 74.93)
+		)
+		(stroke
+			(width 0)
+			(type default)
+		)
+	)
+	(wire
+		(pts
 			(xy 110.49 99.06) (xy 110.49 76.2)
 		)
@@
 	)
 	(symbol
+		(lib_name "SBR10U200P5-13_1")
+		(lib_id "MYLIB_Misc:SBR10U200P5-13")
+		(at 115.57 59.69 270)
+		(unit 1)
+		(exclude_from_sim no)
+		(in_bom yes)
+		(on_board yes)
+		(dnp no)
+		(fields_autoplaced yes)
+		(property "Reference" "D502"
+			(at 118.11 58.7374 90)
+			(effects
+				(font
+					(size 1.27 1.27)
+				)
+				(justify left)
+			)
+		)
+		(property "Value" "SBR10U200P5-13"
+			(at 118.11 61.2774 90)
+			(effects
+				(font
+					(size 1.27 1.27)
+				)
+				(justify left)
+			)
+		)
+		(property "Footprint" "MYLIB_Misc:SBR10U200P5"
+			(at 130.048 59.944 0)
+			(effects
+				(font
+					(size 1.27 1.27)
+				)
+				(hide yes)
+			)
+		)
+		(property "Datasheet" "https://eu.mouser.com/datasheet/3/175/1/SBR10U200P5.pdf"
+			(at 127.762 59.69 0)
+			(effects
+				(font
+					(size 1.27 1.27)
+				)
+				(hide yes)
+			)
+		)
+		(property "Description" "Ultra Low Forward Voltage Drop Power Diode"
+			(at 124.968 59.182 0)
+			(effects
+				(font
+					(size 1.27 1.27)
+				)
+				(hide yes)
+			)
+		)
+		(property "Mouser nr" " 621-SBR10U200P5-13 "
+			(at 132.08 60.452 0)
+			(effects
+				(font
+					(size 1.27 1.27)
+				)
+				(hide yes)
+			)
+		)
+		(pin "2"
+		)
+		(pin "1"
+		)
+		(instances
+			(project ""
+				(path "/fd7503bc-e7fc-4766-b224-3d1c3d7de5ff/c363a192-a091-4a49-a77c-8a6e46625814"
+					(reference "D502")
+					(unit 1)
+				)
+			)
+		)
+	)
+	(symbol
 		(lib_id "power:GND")
 		(at 60.96 55.88 0)
@@
 			)
 		)
-		(property "Footprint" "Diode_SMD:D_PowerDI-5"
+		(property "Footprint" "MYLIB_Misc:SBR10U200P5"
 			(at 188.468 63.754 0)
 			(effects
@@
 		)
 		(instances
-			(project "FPGA_Board_BA"
+			(project ""
 				(path "/fd7503bc-e7fc-4766-b224-3d1c3d7de5ff/c363a192-a091-4a49-a77c-8a6e46625814"
 					(reference "D501")
@@
 					(unit 1)
 				)
-			)
-		)
-	)
-	(symbol
-		(lib_id "MYLIB_Misc:SBR10U200P5-13")
-		(at 115.57 59.69 270)
-		(unit 1)
-		(exclude_from_sim no)
-		(in_bom yes)
-		(on_board yes)
-		(dnp no)
-		(fields_autoplaced yes)
-		(property "Reference" "D503"
-			(at 118.11 58.7374 90)
-			(effects
-				(font
-					(size 1.27 1.27)
-				)
-				(justify left)
-			)
-		)
-		(property "Value" "SBR10U200P5-13"
-			(at 118.11 61.2774 90)
-			(effects
-				(font
-					(size 1.27 1.27)
-				)
-				(justify left)
-			)
-		)
-		(property "Footprint" "Diode_SMD:D_PowerDI-5"
-			(at 130.048 59.944 0)
-			(effects
-				(font
-					(size 1.27 1.27)
-				)
-				(hide yes)
-			)
-		)
-		(property "Datasheet" "https://eu.mouser.com/datasheet/3/175/1/SBR10U200P5.pdf"
-			(at 127.762 59.69 0)
-			(effects
-				(font
-					(size 1.27 1.27)
-				)
-				(hide yes)
-			)
-		)
-		(property "Description" "Ultra Low Forward Voltage Drop Power Diode"
-			(at 124.968 59.182 0)
-			(effects
-				(font
-					(size 1.27 1.27)
-				)
-				(hide yes)
-			)
-		)
-		(property "Mouser nr" " 621-SBR10U200P5-13 "
-			(at 132.08 60.452 0)
-			(effects
-				(font
-					(size 1.27 1.27)
-				)
-				(hide yes)
-			)
-		)
-		(pin "2"
-		)
-		(pin "1"
-		)
-		(instances
-			(project ""
-				(path "/fd7503bc-e7fc-4766-b224-3d1c3d7de5ff/c363a192-a091-4a49-a77c-8a6e46625814"
-					(reference "D503")
-					(unit 1)
-				)

Commit message: schematic almost ready
Changed lines of the file:
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@@
-		)
-	)
-	(label "Vout"
-		(at 269.24 92.71 180)
-		(effects
-			(font
-				(size 1.27 1.27)
-			)
-			(justify right bottom)
 		)
 	)
@@
 		)
 	)
+	(hierarchical_label "Vout"
+		(shape output)
+		(at 269.24 92.71 0)
+		(effects
+			(font
+				(size 1.27 1.27)
+			)
+			(justify left)
+		)
+	)

Commit message: schematic almost ready pt2
Parts:
- added D503: LED_G_0603, WLIB_DO:LED_0603_1608Metric, symbol WLIB_D:LED_G_0603
- added R507: 10k_0603, Resistor_SMD:R_0603_1608Metric, symbol WLIB_R:10k_0603
Connections:
- net +5V: now also R507.1
- net GND: now also D503.1 (K)
- new net: D503.2 (A), R507.2
Other:
- note added: "Status LED for active 5V"

Commit message: lot of work
Connections:
- net +5V: no longer R501.1, U501.26 (VOUT1)
- new net Vout: R501.1, U501.26 (VOUT1)
Changed lines of the file:
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@@
 		)
 	)
-	(hierarchical_label "Vout"
+	(hierarchical_label "Vout_5V"
 		(shape output)
 		(at 269.24 92.71 0)

Commit message: work
Parts:
- renumbered C511 to C16, C505 to C17, C501 to C18, C507 to C19, C504 to C20, C503 to C21, C502 to C22, C508 to C23, C509 to C24, C506 to C25, C512 to C26, C510 to C27, D502 to D1, D501 to D2, D503 to D3, L501 to L1, L502 to L2, Q501 to Q2, Q502 to Q3, Q503 to Q4, Q504 to Q5, R502 to R10, R506 to R11, R504 to R12, R503 to R13, R507 to R14, R501 to R8, R505 to R9, U501 to U7
