File: FPGA_Board_BA/PCB/adc_power.kicad_sch (KiCad schematic)
At the start: 9 parts, among them U3203 TPS6282518

Commit message: work
Parts:
- renumbered C3203 to C144, C3201 to C145, C3205 to C146, C3211 to C147, C3212 to C148, F3201 to F1, L3201 to L4, R3201 to R159, U3203 to U38
Changed lines of the file:
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@@
 		(dnp no)
 		(fields_autoplaced yes)
-		(property "Reference" "#PWR03211"
+		(property "Reference" "#PWR0201"
 			(at 212.09 110.49 0)
 			(effects
@@
 			(project "FPGA_Board_BA"
 				(path "/fd7503bc-e7fc-4766-b224-3d1c3d7de5ff/723da5aa-073c-46b3-9d44-c3664aff4ac6"
-					(reference "#PWR03211")
+					(reference "#PWR0201")
 					(unit 1)
 				)
@@
 		(on_board yes)
 		(dnp no)
-		(property "Reference" "R3201"
+		(property "Reference" "R159"
 			(at 113.03 94.234 90)
 			(effects
@@
 			(project ""
 				(path "/fd7503bc-e7fc-4766-b224-3d1c3d7de5ff/723da5aa-073c-46b3-9d44-c3664aff4ac6"
-					(reference "R3201")
+					(reference "R159")
 					(unit 1)
 				)
@@
 		(dnp no)
 		(fields_autoplaced yes)
-		(property "Reference" "C3212"
+		(property "Reference" "C148"
 			(at 219.71 93.9799 0)
 			(effects
@@
 			(project "FPGA_Board_BA"
 				(path "/fd7503bc-e7fc-4766-b224-3d1c3d7de5ff/723da5aa-073c-46b3-9d44-c3664aff4ac6"
-					(reference "C3212")
+					(reference "C148")
 					(unit 1)
 				)
@@
 		(dnp no)
 		(fields_autoplaced yes)
-		(property "Reference" "#PWR03212"
+		(property "Reference" "#PWR0200"
 			(at 212.09 80.01 0)
 			(effects
@@
 			(project ""
 				(path "/fd7503bc-e7fc-4766-b224-3d1c3d7de5ff/723da5aa-073c-46b3-9d44-c3664aff4ac6"
-					(reference "#PWR03212")
+					(reference "#PWR0200")
 					(unit 1)
 				)
@@
 		(dnp no)
 		(fields_autoplaced yes)
-		(property "Reference" "#PWR03205"
+		(property "Reference" "#PWR0199"
 			(at 173.99 109.22 0)
 			(effects
@@
 			(project ""
 				(path "/fd7503bc-e7fc-4766-b224-3d1c3d7de5ff/723da5aa-073c-46b3-9d44-c3664aff4ac6"
-					(reference "#PWR03205")
+					(reference "#PWR0199")
 					(unit 1)
 				)
@@
 		(on_board yes)
 		(dnp no)
-		(property "Reference" "C3201"
+		(property "Reference" "C145"
 			(at 166.37 90.1699 0)
 			(effects
@@
 			(project ""
 				(path "/fd7503bc-e7fc-4766-b224-3d1c3d7de5ff/723da5aa-073c-46b3-9d44-c3664aff4ac6"
-					(reference "C3201")
+					(reference "C145")
 					(unit 1)
 				)
@@
 		(dnp no)
 		(fields_autoplaced yes)
-		(property "Reference" "U3203"
+		(property "Reference" "U38"
 			(at 133.35 78.74 0)
 			(effects
@@
 			(project ""
 				(path "/fd7503bc-e7fc-4766-b224-3d1c3d7de5ff/723da5aa-073c-46b3-9d44-c3664aff4ac6"
-					(reference "U3203")
+					(reference "U38")
 					(unit 1)
 				)
@@
 		(dnp no)
 		(fields_autoplaced yes)
-		(property "Reference" "C3205"
+		(property "Reference" "C146"
 			(at 181.61 90.1699 0)
 			(effects
@@
 			(project "FPGA_Board_BA"
 				(path "/fd7503bc-e7fc-4766-b224-3d1c3d7de5ff/723da5aa-073c-46b3-9d44-c3664aff4ac6"
-					(reference "C3205")
+					(reference "C146")
 					(unit 1)
 				)
@@
 		(on_board yes)
 		(dnp no)
-		(property "Reference" "C3211"
+		(property "Reference" "C147"
 			(at 204.47 93.9799 0)
 			(effects
@@
 			(project "FPGA_Board_BA"
 				(path "/fd7503bc-e7fc-4766-b224-3d1c3d7de5ff/723da5aa-073c-46b3-9d44-c3664aff4ac6"
-					(reference "C3211")
+					(reference "C147")
 					(unit 1)
 				)
@@
 		(dnp no)
 		(fields_autoplaced yes)
-		(property "Reference" "#PWR03202"
+		(property "Reference" "#PWR0197"
 			(at 87.63 113.03 0)
 			(effects
@@
 			(project ""
 				(path "/fd7503bc-e7fc-4766-b224-3d1c3d7de5ff/723da5aa-073c-46b3-9d44-c3664aff4ac6"
-					(reference "#PWR03202")
+					(reference "#PWR0197")
 					(unit 1)
 				)
@@
 		(dnp no)
 		(fields_autoplaced yes)
-		(property "Reference" "F3201"
+		(property "Reference" "F1"
 			(at 189.1792 73.66 0)
 			(effects
@@
 			(project ""
 				(path "/fd7503bc-e7fc-4766-b224-3d1c3d7de5ff/723da5aa-073c-46b3-9d44-c3664aff4ac6"
-					(reference "F3201")
+					(reference "F1")
 					(unit 1)
 				)
@@
 		(on_board yes)
 		(dnp no)
-		(property "Reference" "L3201"
+		(property "Reference" "L4"
 			(at 157.48 76.2 0)
 			(effects
@@
 			(project ""
 				(path "/fd7503bc-e7fc-4766-b224-3d1c3d7de5ff/723da5aa-073c-46b3-9d44-c3664aff4ac6"
-					(reference "L3201")
+					(reference "L4")
 					(unit 1)
 				)
@@
 		(dnp no)
 		(fields_autoplaced yes)
-		(property "Reference" "#PWR03204"
+		(property "Reference" "#PWR0198"
 			(at 146.05 107.95 0)
 			(effects
@@
 			(project "FPGA_Board_BA"
 				(path "/fd7503bc-e7fc-4766-b224-3d1c3d7de5ff/723da5aa-073c-46b3-9d44-c3664aff4ac6"
-					(reference "#PWR03204")
+					(reference "#PWR0198")
 					(unit 1)
 				)
@@
 		(dnp no)
 		(fields_autoplaced yes)
-		(property "Reference" "C3203"
+		(property "Reference" "C144"
 			(at 91.44 97.7899 0)
 			(effects
@@
 			(project ""
 				(path "/fd7503bc-e7fc-4766-b224-3d1c3d7de5ff/723da5aa-073c-46b3-9d44-c3664aff4ac6"
-					(reference "C3203")
-					(unit 1)
-				)
+					(reference "C144")
+					(unit 1)
+				)

Commit message: 18.11 Bib Session
Parts:
- added D9: LED_G_0603, LED_SMD:LED_0603_1608Metric, symbol WLIB_D:LED_G_0603
- added R54, R7: 5k1_0603, Resistor_SMD:R_0603_1608Metric, symbol WLIB_R:5k1_0603
Connections:
- net +1V8: now also R54.1, R7.1
- net GND: now also D9.1 (K)
- new net: D9.2 (A), R54.2, R7.2
