File: FPGA_Board_BA/PCB/fpga.kicad_sch (KiCad schematic)
At the start: 0 parts

Commit message: some changes + lib
Parts:
- added U5: Zynq7020, MYLIB_Misc:Zynq7020, symbol MYLIB_Misc:Zynq7020

Commit message: schematic almost ready
Parts:
- removed U5: Zynq7020, MYLIB_Misc:Zynq7020, symbol MYLIB_Misc:Zynq7020
- added U301: Zynq7020, MYLIB_Misc:Zynq7020, symbol MYLIB_Misc:Zynq7020
Connections:
- new net: U301.a3 (VDD_3V), U301.b3 (VDD_3V)
- new net +5V: U301.a1 (VDD_5V), U301.b1 (VDD_5V)
- new net CLK_IN: U301.a20 (IO_L21P_T3_13)
- new net CLK_OUT: U301.a22 (IO_L21N_T3_13)
- new net GND: U301.a2 (GND), U301.a24 (GND), U301.a25 (GND), U301.a34 (GND), U301.a35 (GND), U301.a4 (GND), U301.a44 (GND), U301.a54 (GND), U301.a67 (GND), U301.a68 (GND), U301.b10 (GND), U301.b2 (GND), U301.b20 (GND), U301.b21 (GND), U301.b30 (GND), U301.b31 (GND), U301.b4 (GND), U301.b40 (GND), U301.b41 (GND), U301.b50 (GND), U301.b60 (GND), U301.b61 (GND), U301.b70 (GND), U301.b71 (GND), U301.b80 (GND)
- new net Ph_A_Tx1: U301.a26 (IO_L1P_T0_34)
- new net Ph_A_Tx2: U301.a28 (IO_L1N_T0_34)
- new net Ph_A_Tx3: U301.a27 (IO_L2P_T0_34)
- new net Ph_A_Tx4: U301.a29 (IO_L2N_T0_34)
- new net Ph_A_Tx5: U301.a30 (IO_L3P_T0_34)
- new net Ph_A_Tx6: U301.a32 (IO_L3N_T0_34)
- new net Ph_A_Tx7: U301.a31 (IO_L4P_T0_34)
- new net Ph_A_Tx8: U301.a33 (IO_L4N_T0_34)
- new net SDO1: U301.a7 (IO_L11P_T1_13)
- new net SDO2: U301.a9 (IO_L11N_T1_13)
- new net SDO3: U301.a11 (IO_L12P_T1_13)
- new net SDO4: U301.a13 (IO_L12N_T1_13)
- new net SDO5: U301.a17 (IO_L13P_T2_13)
- new net SDO6: U301.a19 (IO_L13N_T2_13)
- new net SDO7: U301.a16 (IO_L14P_T2_13)
- new net SDO8: U301.a18 (IO_L14N_T2_13)
- new net ~{CNV}: U301.a21 (IO_L15P_T2_13)
- no-connect marks 0 -> 6

Commit message: schematic almost ready pt2
Parts:
- U301: Mouser nr Connector 200-TFM14002LDWT -> (none); Mouser nr connector (none) -> 200-TFM14002LDWT
Connections:
- net B6_En: now also U301.b42 (IO_L10P_T1_35)
- net CLK_IN: now also U301.a21 (IO_L15P_T2_13); no longer U301.a20 (IO_L21P_T3_13)
- net CLK_OUT: now also U301.a23 (IO_L15N_T2_13); no longer U301.a22 (IO_L21N_T3_13)
- net ENC_A_in: now also U301.b47 (IO_L11P_T1_35)
- net ENC_B_in: now also U301.b49 (IO_L11N_T1_35)
- net ENC_I_in: now also U301.b46 (IO_L12P_T1_35)
- net OT: now also U301.b44 (IO_L10N_T1_35)
- net PWM_AH: now also U301.b37 (IO_L7P_T1_35)
- net PWM_AL: now also U301.b39 (IO_L7N_T1_35)
- net PWM_BH: now also U301.b36 (IO_L8P_T1_35)
- net PWM_BL: now also U301.b38 (IO_L8N_T1_35)
- net PWM_CH: now also U301.b43 (IO_L9P_T1_35)
- net PWM_CL: now also U301.b45 (IO_L9N_T1_35)
- net Ph_A_En: now also U301.b27 (IO_L3P_T0_35)
- net Ph_A_Err: now also U301.b23 (IO_L1P_T0_35)
- net Ph_A_Rx: now also U301.b33 (IO_L5P_T0_35)
- net Ph_A_Tx10: now also U301.a38 (IO_L5N_T0_34)
- net Ph_A_Tx11: now also U301.a37 (IO_L6P_T0_34)
- net Ph_A_Tx12: now also U301.a39 (IO_L6N_T0_34)
- net Ph_A_Tx9: now also U301.a36 (IO_L5P_T0_34)
- net Ph_B_En: now also U301.b29 (IO_L3N_T0_35)
- net Ph_B_Err: now also U301.b25 (IO_L1N_T0_35)
- net Ph_B_Rx: now also U301.b35 (IO_L5N_T0_35)
- net Ph_B_Tx1: now also U301.a40 (IO_L7P_T1_34)
- net Ph_B_Tx10: now also U301.a47 (IO_L11N_T1_34)
- net Ph_B_Tx11: now also U301.a55 (IO_L12P_T1_34)
- net Ph_B_Tx12: now also U301.a57 (IO_L12N_T1_34)
- net Ph_B_Tx2: now also U301.a42 (IO_L7N_T1_34)
- net Ph_B_Tx3: now also U301.a41 (IO_L8P_T1_34)
- net Ph_B_Tx4: now also U301.a43 (IO_L8N_T1_34)
- net Ph_B_Tx5: now also U301.a51 (IO_L9P_T1_34)
- net Ph_B_Tx6: now also U301.a53 (IO_L9N_T2_34)
- net Ph_B_Tx7: now also U301.a46 (IO_L10P_T1_34)
- net Ph_B_Tx8: now also U301.a48 (IO_L10N_T1_34)
- net Ph_B_Tx9: now also U301.a45 (IO_L11P_T1_34)
- net Ph_C_En: now also U301.b26 (IO_L4P_T0_35)
- net Ph_C_Err: now also U301.b22 (IO_L2P_T0_35)
- net Ph_C_Rx: now also U301.b32 (IO_L6P_T0_35)
- net Ph_C_Tx1: now also U301.a50 (IO_L13P_T2_34)
- net Ph_C_Tx10: now also U301.a62 (IO_L17N_T2_34)
- net Ph_C_Tx11: now also U301.a70 (IO_L18P_T2_34)
- net Ph_C_Tx12: now also U301.a69 (IO_L18N_T2_34)
- net Ph_C_Tx2: now also U301.a52 (IO_L13N_T2_34)
- net Ph_C_Tx3: now also U301.a59 (IO_L14P_T2_34)
- net Ph_C_Tx4: now also U301.a61 (IO_L14N_T2_34)
- net Ph_C_Tx5: now also U301.a56 (IO_L15P_T2_34)
- net Ph_C_Tx6: now also U301.a58 (IO_L15N_T2_34)
- net Ph_C_Tx7: now also U301.a63 (IO_L16P_T2_34)
- net Ph_C_Tx8: now also U301.a65 (IO_L16N_T2_34)
- net Ph_C_Tx9: now also U301.a60 (IO_L17P_T2_34)
- net Ph_D_En: now also U301.b28 (IO_L4N_T0_35)
- net Ph_D_Err: now also U301.b24 (IO_L2N_T0_35)
- net Ph_D_Rx: now also U301.b34 (IO_L6N_T0_35)
- net Ph_D_Tx1: now also U301.a64 (IO_L19P_T3_34)
- net Ph_D_Tx10: now also U301.a80 (IO_L23N_T3_34)
- net Ph_D_Tx11: now also U301.a76 (IO_L24P_T3_34)
- net Ph_D_Tx12: now also U301.a78 (IO_L24N_T3_34)
- net Ph_D_Tx2: now also U301.a66 (IO_L19N_T3_34)
- net Ph_D_Tx3: now also U301.a72 (IO_L20N_T3_34)
- net Ph_D_Tx4: now also U301.a71 (IO_L20P_T3_34)
- net Ph_D_Tx5: now also U301.a74 (IO_L21P_T3_34)
- net Ph_D_Tx6: now also U301.a73 (IO_L21N_T3_34)
- net Ph_D_Tx7: now also U301.a75 (IO_L22P_T3_34)
- net Ph_D_Tx8: now also U301.a77 (IO_L22N_T3_34)
- net Ph_D_Tx9: now also U301.a79 (IO_L23P_T3_34)
- net ~{CNV}: now also U301.a20 (IO_L21P_T3_13); no longer U301.a21 (IO_L15P_T2_13)
- net LED1: now reaches U301.b48 (IO_L12N_T1_35)
- net Button1: now reaches U301.b52 (IO_L14P_T2_35)
- net LED2: now reaches U301.b53 (IO_L13P_35)
- net Button2: now reaches U301.b54 (IO_L14N_T2_35)
- net Poti: now reaches U301.b55 (IO_L13N_35)
Other:
- note added: "Bank 13: Total 12 pins -> ADC (11pins) oder 13 Bank 34: Total 48 pins -> Tx Phase A,B,C,D (48 pins) Bank 35: Total 48 pins -> B6 (8pins) + CHB En/Err/Rx (12pins) + User Interactions (5 pins)"

Commit message: some schematic changes + Misc
Other:
- note added: "Bank 13: Total 12 pins -> ADC (11pins) oder 13 Bank 34: Total 48 pins -> Tx Phase A,B,C,D (48 pins) Bank 35: Total 48 pins -> B6 (8pins) + CHB En/Err/Rx (12pins) + User Interactions (5 pins) + ADC_Machine (11pin)"
- note removed: "Bank 13: Total 12 pins -> ADC (11pins) oder 13 Bank 34: Total 48 pins -> Tx Phase A,B,C,D (48 pins) Bank 35: Total 48 pins -> B6 (8pins) + CHB En/Err/Rx (12pins) + User Interactions (5 pins)"
Changed lines of the file:
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@@
 	(generator_version "9.0")
 	(paper "A3")
-	(text "Bank 13: Total 12 pins -> ADC (11pins) oder 13\nBank 34: Total 48 pins -> Tx Phase A,B,C,D (48 pins)\nBank 35: Total 48 pins -> B6 (8pins) + CHB En/Err/Rx (12pins)\n+ User Interactions (5 pins)\n"
+	(text "Bank 13: Total 12 pins -> ADC (11pins) oder 13\nBank 34: Total 48 pins -> Tx Phase A,B,C,D (48 pins)\nBank 35: Total 48 pins -> B6 (8pins) + CHB En/Err/Rx (12pins)\n+ User Interactions (5 pins) + ADC_Machine (11pin)\n"
 		(exclude_from_sim no)
 		(at 280.924 76.454 0)
@@
 		)
 	)
+	(hierarchical_label "SDO3_1"
+		(shape input)
+		(at 314.96 162.56 180)
+		(effects
+			(font
+				(size 1.27 1.27)
+			)
+			(justify right)
+		)
+	)
 	(hierarchical_label "Ph_C_Rx"
 		(shape output)
@@
 		)
 	)
+	(hierarchical_label "SDO1_1"
+		(shape input)
+		(at 314.96 156.21 180)
+		(effects
+			(font
+				(size 1.27 1.27)
+			)
+			(justify right)
+		)
+	)
 	(hierarchical_label "Ph_B_Err"
 		(shape input)
@@
 		)
 	)
+	(hierarchical_label "SDO8_1"
+		(shape input)
+		(at 314.96 177.8 180)
+		(effects
+			(font
+				(size 1.27 1.27)
+			)
+			(justify right)
+		)
+	)
 	(hierarchical_label "SDO8"
 		(shape input)
@@
 		)
 	)
+	(hierarchical_label "~{CNV}_1"
+		(shape output)
+		(at 317.5 187.96 180)
+		(effects
+			(font
+				(size 1.27 1.27)
+			)
+			(justify right)
+		)
+	)
 	(hierarchical_label "Ph_C_En"
 		(shape output)
@@
 		)
 	)
+	(hierarchical_label "CLK_IN_1"
+		(shape output)
+		(at 317.5 185.42 180)
+		(effects
+			(font
+				(size 1.27 1.27)
+			)
+			(justify right)
+		)
+	)
 	(hierarchical_label "Ph_C_Tx2"
 		(shape input)
@@
 		)
 	)
+	(hierarchical_label "SDO4_1"
+		(shape input)
+		(at 314.96 165.1 180)
+		(effects
+			(font
+				(size 1.27 1.27)
+			)
+			(justify right)
+		)
+	)
+	(hierarchical_label "SDO6_1"
+		(shape input)
+		(at 314.96 171.45 180)
+		(effects
+			(font
+				(size 1.27 1.27)
+			)
+			(justify right)
+		)
+	)
 	(hierarchical_label "Ph_B_Tx3"
 		(shape input)
@@
 		)
 	)
+	(hierarchical_label "SDO7_1"
+		(shape input)
+		(at 314.96 175.26 180)
+		(effects
+			(font
+				(size 1.27 1.27)
+			)
+			(justify right)
+		)
+	)
 	(hierarchical_label "PWM_BL"
 		(shape output)
@@
 		)
 	)
+	(hierarchical_label "CLK_OUT_1"
+		(shape output)
+		(at 317.5 182.88 180)
+		(effects
+			(font
+				(size 1.27 1.27)
+			)
+			(justify right)
+		)
+	)
 	(hierarchical_label "Ph_B_Tx6"
 		(shape input)
@@
 		)
 	)
+	(hierarchical_label "SDO2_1"
+		(shape input)
+		(at 314.96 158.75 180)
+		(effects
+			(font
+				(size 1.27 1.27)
+			)
+			(justify right)
+		)
+	)
 	(hierarchical_label "Ph_B_Tx9"
 		(shape input)
@@
 		)
 	)
+	(hierarchical_label "SDO5_1"
+		(shape input)
+		(at 314.96 168.91 180)
+		(effects
+			(font
+				(size 1.27 1.27)
+			)
+			(justify right)
+		)
+	)

Commit message: work
Parts:
- U2: renamed from U301; Chip electrical info (none) -> https://docs.amd.com/v/u/en-US/ds187-XC7Z010-XC7Z020-Data-S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; Chip pinout datasheet (none) -> https://cdn.hackaday.io/files/19354828041536/ug865-Zynq-700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
Connections:
- net Button1: now also U2.b55 (IO_L13N_35); no longer U2.b52 (IO_L14P_T2_35)
- net Button2: now also U2.b52 (IO_L14P_T2_35); no longer U2.b54 (IO_L14N_T2_35)
- net CLK_IN_1: now also U2.b67 (IO_L19P_T3_35)
- net CLK_OUT_1: now also U2.b64 (IO_L18N_T2_35)
- net GND: now also U2.b7 (XADC_INN0)
- net Poti: now also U2.b5 (XADC_INP0); no longer U2.b55 (IO_L13N_35)
- net SDO1_1: now also U2.b54 (IO_L14N_T2_35)
- net SDO2_1: now also U2.b57 (IO_L15P_T2_35)
- net SDO3_1: now also U2.b59 (IO_L15N_T2_35)
- net SDO4_1: now also U2.b56 (IO_L16P_T2_35)
- net SDO5_1: now also U2.b58 (IO_L16N_T2_35)
- net SDO6_1: now also U2.b63 (IO_L17P_T2_35)
- net SDO7_1: now also U2.b65 (IO_L17N_T2_35)
- net SDO8_1: now also U2.b62 (IO_L18P_T2_35)
- net +3.3V: now reaches U2.a3 (VDD_3V), U2.b3 (VDD_3V)
- net CNV_1: now reaches U2.b69 (IO_L19N_T3_35)
- net ~{CNV} renamed CNV
- no-connect marks 6 -> 10
Other:
- note added: "Bank 13: Total 12 pins -> ADC (11pins) Bank 34: Total 48 pins -> Tx Phase A,B,C,D (48 pins) Bank 35: Total 48 pins -> B6 (8pins) + CHB En/Err/Rx (12pins) + User Interactions (4 pins) + ADC_Machine (11pin) XADC: Poti"
- note removed: "Bank 13: Total 12 pins -> ADC (11pins) oder 13 Bank 34: Total 48 pins -> Tx Phase A,B,C,D (48 pins) Bank 35: Total 48 pins -> B6 (8pins) + CHB En/Err/Rx (12pins) + User Interactions (5 pins) + ADC_Machine (11pin)"

Commit message: 18.11 Bib Session
Parts:
- U2: AC,DC Characteristics (none) -> https://docs.amd.com/v/u/en-US/ds187-XC7Z010-XC7Z020-Data-S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; Chip electrical info https://docs.amd.com/v/u/en-US/ds187-XC7Z010-XC7Z020-Data-S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 -> (none)
Connections:
- net CNV renamed ~{CNV}
- net CNV_1 renamed ~{CNV}_1
- no-connect marks 10 -> 21
Changed lines of the file:
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@@
 	)
 	(no_connect
+		(at 279.4 134.62)
+	)
+	(no_connect
 		(at 342.9 115.57)
 	)
@@
 	)
 	(no_connect
+		(at 231.14 127)
+	)
+	(no_connect
 		(at 342.9 118.11)
 	)
@@
 	)
 	(no_connect
+		(at 231.14 142.24)
+	)
+	(no_connect
+		(at 231.14 121.92)
+	)
+	(no_connect
 		(at 279.4 127)
 	)
@@
 	)
 	(no_connect
+		(at 231.14 137.16)
+	)
+	(no_connect
+		(at 231.14 134.62)
+	)
+	(no_connect
+		(at 231.14 139.7)
+	)
+	(no_connect
+		(at 279.4 137.16)
+	)
+	(no_connect
+		(at 231.14 119.38)
+	)
+	(no_connect
+		(at 231.14 124.46)
+	)
+	(no_connect
 		(at 342.9 123.19)
 	)
+	(no_connect
+		(at 231.14 129.54)
+	)
 	(wire
 		(pts
@@
 	)
 	(hierarchical_label "CLK_OUT"
-		(shape output)
+		(shape input)
 		(at 285.75 109.22 0)
 		(effects
@@
 		)
 	)
-	(hierarchical_label "CNV"
+	(hierarchical_label "~{CNV}"
 		(shape output)
 		(at 285.75 111.76 0)
@@
 		)
 	)
-	(hierarchical_label "CNV_1"
+	(hierarchical_label "~{CNV}_1"
 		(shape output)
 		(at 201.93 156.21 0)
@@
 	)
 	(hierarchical_label "CLK_OUT_1"
-		(shape output)
+		(shape input)
 		(at 140.97 151.13 180)
 		(effects
@@
 			)
 		)
-		(property "Chip electrical info" "https://docs.amd.com/v/u/en-US/ds187-XC7Z010-XC7Z020-Data-Sheet"
+		(property "AC,DC Characteristics" "https://docs.amd.com/v/u/en-US/ds187-XC7Z010-XC7Z020-Data-Sheet"
 			(at 76.2 114.3 0)
 			(effects
@@
 			)
 		)
-		(property "Chip electrical info" "https://docs.amd.com/v/u/en-US/ds187-XC7Z010-XC7Z020-Data-Sheet"
+		(property "AC,DC Characteristics" "https://docs.amd.com/v/u/en-US/ds187-XC7Z010-XC7Z020-Data-Sheet"
 			(at 255.27 124.46 0)
 			(effects
@@
 			)
 		)
-		(property "Chip electrical info" "https://docs.amd.com/v/u/en-US/ds187-XC7Z010-XC7Z020-Data-Sheet"
+		(property "AC,DC Characteristics" "https://docs.amd.com/v/u/en-US/ds187-XC7Z010-XC7Z020-Data-Sheet"
 			(at 328.93 119.38 0)
 			(effects
@@
 			)
 		)
-		(property "Chip electrical info" "https://docs.amd.com/v/u/en-US/ds187-XC7Z010-XC7Z020-Data-Sheet"
+		(property "AC,DC Characteristics" "https://docs.amd.com/v/u/en-US/ds187-XC7Z010-XC7Z020-Data-Sheet"
 			(at 173.99 121.92 0)
 			(effects
