File: FPGA_Board_BA/PCB/fpga.kicad_sch (KiCad schematic)
At the start: 1 part, among them U2 Zynq7020

Commit message: 22.11
Parts:
- added D1, D2, D3, D4: B72590D50H160, Capacitor_SMD:C_0402_1005Metric_Pad0.74x0.62mm_HandSolder, symbol MYLIB_Misc:ESD_Diode_5V6
- added J2: PinHeader_16_male, Connector_PinHeader_2.54mm:PinHeader_1x16_P2.54mm_Vertical, symbol WLIB_J:PinHeader_16_male
Connections:
- net +5V: now also D1.1 (A1), J2.6 (Pin_6)
- net GND: now also U2.b8 (DXN_0), D1.2 (A2), D2.2 (A2), D3.2 (A2), D4.2 (A2), J2.1 (Pin_1), J2.2 (Pin_2)
- net LED3: now reaches U2.a22 (IO_L21N_T3_13)
- net Poti2: now reaches U2.b6 (DXP_0)
- net +1V8: now reaches U2.b9 (XADC_VCC)
- net +1V8: now also D4.1 (A1), J2.3 (Pin_3)
- net at U2.b66 (IO_L20P_T3_35): now also J2.16 (Pin_16)
- net at U2.b68 (IO_L20N_T3_35): now also J2.15 (Pin_15)
- net at U2.b72 (IO_L22P_T3_35): now also J2.14 (Pin_14)
- net at U2.b73 (IO_L21P_T3_35): now also J2.7 (Pin_7)
- net at U2.b75 (IO_L21N_T3_35): now also J2.8 (Pin_8)
- net at U2.b76 (IO_L24P_T3_35): now also J2.12 (Pin_12)
- net at U2.b77 (IO_L23P_T3_35): now also J2.9 (Pin_9)
- net at U2.b78 (IO_L24N_T3_35): now also J2.11 (Pin_11)
- net at U2.b79 (IO_L23N_T3_35): now also J2.10 (Pin_10)
- new net +3V3: D3.1 (A1), J2.4 (Pin_4)
- new net +5VA: D2.1 (A1), J2.5 (Pin_5)
- no-connect marks 21 -> 18
Other:
- note added: "Bank 0: 3.3V Bank 13: 3.3V Bank 34: 3.3V Bank 35: 3.3V Bank 500: 3.3V Bank 501: 1.8V AUX: 1.8V PLL: 1.8V XADC: 1.8V Vref for it is 1.25V"
- note added: "Bank 13: Total 12 pins -> ADC (11pins) Bank 34: Total 48 pins -> Tx Phase A,B,C,D (48 pins) Bank 35: Total 48 pins -> B6 (8pins) + CHB En/Err/Rx (12pins) + User Interactions (5 pins) + ADC_Machine (11pin) + encoder (3pins) XADC: 2 Potis Free pins left: 10"
- note added: "Min - Typ - Max"
- note added: "PinHeader for the free pins"
- note added: "Source: https://docs.amd.com/v/u/en-US/ds187-XC7Z010-XC7Z020-Data-Sheet"
- note removed: "Bank 13: Total 12 pins -> ADC (11pins) Bank 34: Total 48 pins -> Tx Phase A,B,C,D (48 pins) Bank 35: Total 48 pins -> B6 (8pins) + CHB En/Err/Rx (12pins) + User Interactions (4 pins) + ADC_Machine (11pin) XADC: Poti Free pins left: 14"

Commit message: exported stuff
Parts:
- D1, D2: now not fitted
- U2: Chip pinout (none) -> https://cdn.hackaday.io/files/19354828041536/ug865-Zynq-700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
Connections:
- net +3V3 is gone; now on net +3.3V: D3.1 (A1), J2.4 (Pin_4)
- net esd_diodes/Pin7: now reaches J2.10 (Pin_10), U2.b79 (IO_L23N_T3_35)
- net esd_diodes/Pin6: now reaches J2.11 (Pin_11), U2.b78 (IO_L24N_T3_35)
- net esd_diodes/Pin5: now reaches J2.12 (Pin_12), U2.b76 (IO_L24P_T3_35)
- net esd_diodes/Pin4: now reaches J2.13 (Pin_13)
- net esd_diodes/Pin4: now also U2.b74 (IO_L22N_T3_35)
- net esd_diodes/Pin3: now reaches J2.14 (Pin_14), U2.b72 (IO_L22P_T3_35)
- net esd_diodes/Pin2: now reaches J2.15 (Pin_15), U2.b68 (IO_L20N_T3_35)
- net esd_diodes/Pin1: now reaches J2.16 (Pin_16), U2.b66 (IO_L20P_T3_35)
- net esd_diodes/Pin10: now reaches J2.7 (Pin_7), U2.b73 (IO_L21P_T3_35)
- net esd_diodes/Pin9: now reaches J2.8 (Pin_8), U2.b75 (IO_L21N_T3_35)
- net esd_diodes/Pin8: now reaches J2.9 (Pin_9), U2.b77 (IO_L23P_T3_35)
Other:
- added sheet esd_diodes (esd_diodes.kicad_sch)
- note added: "V_dc_max = 5.6 V"

Commit message: schematic fixes after Leo Meeting
Parts:
- removed D2: B72590D50H160, Capacitor_SMD:C_0402_1005Metric_Pad0.74x0.62mm_HandSolder, symbol MYLIB_Misc:ESD_Diode_5V6
- removed J2: PinHeader_16_male, Connector_PinHeader_2.54mm:PinHeader_1x16_P2.54mm_Vertical, symbol WLIB_J:PinHeader_16_male
- added J9: Box_Header_26pin, Connector_IDC:IDC-Header_2x13_P2.54mm_Vertical, symbol MYLIB_Misc:Box_Header_26pin
- D1: now fitted
Connections:
- net +1V8: now also J9.26 (Pin_26)
- net +3.3V: now also J9.24 (Pin_24)
- net +5V: now also J9.22 (Pin_22)
- net GND: now also J9.1 (Pin_1), J9.11 (Pin_11), J9.13 (Pin_13), J9.15 (Pin_15), J9.17 (Pin_17), J9.19 (Pin_19), J9.21 (Pin_21), J9.23 (Pin_23), J9.25 (Pin_25), J9.3 (Pin_3), J9.5 (Pin_5), J9.7 (Pin_7), J9.9 (Pin_9)
- net esd_diodes/Pin1: now also J9.2 (Pin_2)
- net esd_diodes/Pin10: now also J9.20 (Pin_20)
- net esd_diodes/Pin2: now also J9.4 (Pin_4)
- net esd_diodes/Pin3: now also J9.6 (Pin_6)
- net esd_diodes/Pin4: now also J9.8 (Pin_8)
- net esd_diodes/Pin5: now also J9.10 (Pin_10)
- net esd_diodes/Pin6: now also J9.12 (Pin_12)
- net esd_diodes/Pin7: now also J9.14 (Pin_14)
- net esd_diodes/Pin8: now also J9.16 (Pin_16)
- net esd_diodes/Pin9: now also J9.18 (Pin_18)
Other:
- moved on the sheet: D3, D4

Commit message: started component placement
Parts:
- U2: now not fitted
Changed lines of the file:
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@@
 		(in_bom yes)
 		(on_board yes)
-		(dnp no)
+		(dnp yes)
 		(fields_autoplaced yes)
 		(property "Reference" "U2"
@@
 		(in_bom yes)
 		(on_board yes)
-		(dnp no)
+		(dnp yes)
 		(fields_autoplaced yes)
 		(property "Reference" "U2"
@@
 		(in_bom yes)
 		(on_board yes)
-		(dnp no)
+		(dnp yes)
 		(fields_autoplaced yes)
 		(property "Reference" "U2"
@@
 		(in_bom yes)
 		(on_board yes)
-		(dnp no)
+		(dnp yes)
 		(fields_autoplaced yes)
 		(property "Reference" "U2"

Commit message: placement of Power DCDC and Buffers ready
Parts:
- U2: now fitted
Changed lines of the file:
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@@
 		(in_bom yes)
 		(on_board yes)
-		(dnp yes)
+		(dnp no)
 		(fields_autoplaced yes)
 		(property "Reference" "U2"
@@
 		(in_bom yes)
 		(on_board yes)
-		(dnp yes)
+		(dnp no)
 		(fields_autoplaced yes)
 		(property "Reference" "U2"
@@
 		(in_bom yes)
 		(on_board yes)
-		(dnp yes)
+		(dnp no)
 		(fields_autoplaced yes)
 		(property "Reference" "U2"
@@
 		(in_bom yes)
 		(on_board yes)
-		(dnp yes)
+		(dnp no)
 		(fields_autoplaced yes)
 		(property "Reference" "U2"

Commit message: Component placement ready. Waiting to meet with Leo
Parts:
- J9: now not fitted
Changed lines of the file:
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@@
 		(in_bom yes)
 		(on_board yes)
-		(dnp no)
+		(dnp yes)
 		(fields_autoplaced yes)
 		(property "Reference" "J9"

Commit message: Placement optimised
Parts:
- J9: now fitted
Connections:
- net B6_En: now also U2.a18 (IO_L14N_T2_13); no longer U2.b42 (IO_L10P_T1_35)
- net CLK_IN: no longer U2.a21 (IO_L15P_T2_13)
- net CLK_OUT: no longer U2.a23 (IO_L15N_T2_13)
- net LED3: no longer U2.a22 (IO_L21N_T3_13)
- net OT: now also U2.a16 (IO_L14P_T2_13); no longer U2.b44 (IO_L10N_T1_35)
- net PWM_AH: now also U2.a19 (IO_L13N_T2_13); no longer U2.b37 (IO_L7P_T1_35)
- net PWM_AL: now also U2.a17 (IO_L13P_T2_13); no longer U2.b39 (IO_L7N_T1_35)
- net PWM_BH: now also U2.a13 (IO_L12N_T1_13); no longer U2.b36 (IO_L8P_T1_35)
- net PWM_BL: now also U2.a11 (IO_L12P_T1_13); no longer U2.b38 (IO_L8N_T1_35)
- net PWM_CH: now also U2.a9 (IO_L11N_T1_13); no longer U2.b43 (IO_L9P_T1_35)
- net PWM_CL: now also U2.a7 (IO_L11P_T1_13); no longer U2.b45 (IO_L9N_T1_35)
- net SDO1: no longer U2.a7 (IO_L11P_T1_13)
- net SDO2: no longer U2.a9 (IO_L11N_T1_13)
- net SDO3: no longer U2.a11 (IO_L12P_T1_13)
- net SDO4: no longer U2.a13 (IO_L12N_T1_13)
- net SDO5: no longer U2.a17 (IO_L13P_T2_13)
- net SDO6: no longer U2.a19 (IO_L13N_T2_13)
- net SDO7: no longer U2.a16 (IO_L14P_T2_13)
- net SDO8: no longer U2.a18 (IO_L14N_T2_13)
- net ~{CNV}: no longer U2.a20 (IO_L21P_T3_13)
Changed lines of the file:
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@@
 	(wire
 		(pts
-			(xy 279.4 101.6) (xy 285.75 101.6)
+			(xy 279.4 101.6) (xy 289.56 101.6)
 		)
 		(stroke
@@
 	(wire
 		(pts
-			(xy 279.4 104.14) (xy 285.75 104.14)
+			(xy 279.4 104.14) (xy 289.56 104.14)
 		)
 		(stroke
@@
 	(hierarchical_label "CLK_IN"
 		(shape output)
-		(at 285.75 106.68 0)
+		(at 238.76 77.47 0)
 		(effects
 			(font
@@
 	(hierarchical_label "SDO2"
 		(shape input)
-		(at 224.79 104.14 180)
+		(at 226.06 74.93 180)
 		(effects
 			(font
@@
 	(hierarchical_label "PWM_AH"
 		(shape output)
-		(at 201.93 115.57 0)
+		(at 224.79 114.3 180)
 		(effects
 			(font
 				(size 1.27 1.27)
 			)
-			(justify left)
+			(justify right)
 		)
 	)
 	(hierarchical_label "CLK_OUT"
 		(shape input)
-		(at 285.75 109.22 0)
+		(at 238.76 80.01 0)
 		(effects
 			(font
@@
 	(hierarchical_label "LED3"
 		(shape output)
-		(at 285.75 114.3 0)
+		(at 238.76 85.09 0)
 		(effects
 			(font
@@
 	(hierarchical_label "SDO7"
 		(shape input)
-		(at 285.75 101.6 0)
+		(at 238.76 72.39 0)
 		(effects
 			(font
@@
 	(hierarchical_label "SDO8"
 		(shape input)
-		(at 285.75 104.14 0)
+		(at 238.76 74.93 0)
 		(effects
 			(font
@@
 	(hierarchical_label "PWM_BH"
 		(shape output)
-		(at 140.97 115.57 180)
+		(at 224.79 109.22 180)
 		(effects
 			(font
@@
 	(hierarchical_label "SDO6"
 		(shape input)
-		(at 224.79 114.3 180)
+		(at 226.06 85.09 180)
 		(effects
 			(font
@@
 	(hierarchical_label "SDO3"
 		(shape input)
-		(at 224.79 106.68 180)
+		(at 226.06 77.47 180)
 		(effects
 			(font
@@
 	(hierarchical_label "SDO4"
 		(shape input)
-		(at 224.79 109.22 180)
+		(at 226.06 80.01 180)
 		(effects
 			(font
@@
 	(hierarchical_label "~{CNV}"
 		(shape output)
-		(at 285.75 111.76 0)
+		(at 238.76 82.55 0)
 		(effects
 			(font
@@
 	(hierarchical_label "OT"
 		(shape input)
-		(at 140.97 125.73 180)
+		(at 289.56 101.6 0)
 		(effects
 			(font
 				(size 1.27 1.27)
 			)
-			(justify right)
+			(justify left)
 		)
 	)
@@
 	(hierarchical_label "SDO1"
 		(shape input)
-		(at 224.79 101.6 180)
+		(at 226.06 72.39 180)
 		(effects
 			(font
@@
 	(hierarchical_label "SDO5"
 		(shape input)
-		(at 224.79 111.76 180)
+		(at 226.06 82.55 180)
 		(effects
 			(font
@@
 	(hierarchical_label "PWM_CL"
 		(shape output)
-		(at 201.93 125.73 0)
+		(at 224.79 101.6 180)
 		(effects
 			(font
 				(size 1.27 1.27)
 			)
-			(justify left)
+			(justify right)
 		)
 	)
@@
 	(hierarchical_label "PWM_BL"
 		(shape output)
-		(at 140.97 118.11 180)
+		(at 224.79 106.68 180)
 		(effects
 			(font
@@
 	(hierarchical_label "PWM_CH"
 		(shape output)
-		(at 201.93 123.19 0)
+		(at 224.79 104.14 180)
 		(effects
 			(font
 				(size 1.27 1.27)
 			)
-			(justify left)
+			(justify right)
 		)
 	)
@@
 	(hierarchical_label "PWM_AL"
 		(shape output)
-		(at 201.93 118.11 0)
+		(at 224.79 111.76 180)
 		(effects
 			(font
 				(size 1.27 1.27)
 			)
-			(justify left)
+			(justify right)
 		)
 	)
@@
 	(hierarchical_label "B6_En"
 		(shape output)
-		(at 140.97 123.19 180)
+		(at 289.56 104.14 0)
 		(effects
 			(font
 				(size 1.27 1.27)
 			)
-			(justify right)
+			(justify left)
 		)
 	)
@@
 		(in_bom yes)
 		(on_board yes)
-		(dnp yes)
+		(dnp no)
 		(fields_autoplaced yes)
 		(property "Reference" "J9"

Commit message: some changes in the PCB
Connections:
- net Button1: no longer U2.b55 (IO_L13N_35)
- net Button2: no longer U2.b52 (IO_L14P_T2_35)
- net CLK_IN_1: no longer U2.b67 (IO_L19P_T3_35)
- net CLK_OUT_1: no longer U2.b64 (IO_L18N_T2_35)
- net ENC_A_in: no longer U2.b47 (IO_L11P_T1_35)
- net ENC_B_in: no longer U2.b49 (IO_L11N_T1_35)
- net ENC_I_in: no longer U2.b46 (IO_L12P_T1_35)
- net LED1: no longer U2.b48 (IO_L12N_T1_35)
- net LED2: no longer U2.b53 (IO_L13P_35)
- net Ph_A_En: no longer U2.b27 (IO_L3P_T0_35)
- net Ph_A_Err: no longer U2.b23 (IO_L1P_T0_35)
- net Ph_A_Rx: no longer U2.b33 (IO_L5P_T0_35)
- net Ph_A_Tx1: now also U2.b23 (IO_L1P_T0_35); no longer U2.a26 (IO_L1P_T0_34)
- net Ph_A_Tx10: now also U2.b35 (IO_L5N_T0_35); no longer U2.a38 (IO_L5N_T0_34)
- net Ph_A_Tx11: now also U2.b32 (IO_L6P_T0_35); no longer U2.a37 (IO_L6P_T0_34)
- net Ph_A_Tx12: now also U2.b34 (IO_L6N_T0_35); no longer U2.a39 (IO_L6N_T0_34)
- net Ph_A_Tx2: now also U2.b25 (IO_L1N_T0_35); no longer U2.a28 (IO_L1N_T0_34)
- net Ph_A_Tx3: now also U2.b22 (IO_L2P_T0_35); no longer U2.a27 (IO_L2P_T0_34)
- net Ph_A_Tx4: now also U2.b24 (IO_L2N_T0_35); no longer U2.a29 (IO_L2N_T0_34)
- net Ph_A_Tx5: now also U2.b27 (IO_L3P_T0_35); no longer U2.a30 (IO_L3P_T0_34)
- net Ph_A_Tx6: now also U2.b29 (IO_L3N_T0_35); no longer U2.a32 (IO_L3N_T0_34)
- net Ph_A_Tx7: now also U2.b26 (IO_L4P_T0_35); no longer U2.a31 (IO_L4P_T0_34)
- net Ph_A_Tx8: now also U2.b28 (IO_L4N_T0_35); no longer U2.a33 (IO_L4N_T0_34)
- net Ph_A_Tx9: now also U2.b33 (IO_L5P_T0_35); no longer U2.a36 (IO_L5P_T0_34)
- net Ph_B_En: no longer U2.b29 (IO_L3N_T0_35)
- net Ph_B_Err: no longer U2.b25 (IO_L1N_T0_35)
- net Ph_B_Rx: no longer U2.b35 (IO_L5N_T0_35)
- net Ph_B_Tx1: now also U2.b37 (IO_L7P_T1_35); no longer U2.a40 (IO_L7P_T1_34)
- net Ph_B_Tx10: now also U2.b49 (IO_L11N_T1_35); no longer U2.a47 (IO_L11N_T1_34)
- net Ph_B_Tx11: now also U2.b46 (IO_L12P_T1_35); no longer U2.a55 (IO_L12P_T1_34)
- net Ph_B_Tx12: now also U2.b48 (IO_L12N_T1_35); no longer U2.a57 (IO_L12N_T1_34)
- net Ph_B_Tx2: now also U2.b39 (IO_L7N_T1_35); no longer U2.a42 (IO_L7N_T1_34)
- net Ph_B_Tx3: now also U2.b36 (IO_L8P_T1_35); no longer U2.a41 (IO_L8P_T1_34)
- net Ph_B_Tx4: now also U2.b38 (IO_L8N_T1_35); no longer U2.a43 (IO_L8N_T1_34)
- net Ph_B_Tx5: now also U2.b43 (IO_L9P_T1_35); no longer U2.a51 (IO_L9P_T1_34)
- net Ph_B_Tx6: now also U2.b45 (IO_L9N_T1_35); no longer U2.a53 (IO_L9N_T2_34)
- net Ph_B_Tx7: now also U2.b42 (IO_L10P_T1_35); no longer U2.a46 (IO_L10P_T1_34)
- net Ph_B_Tx8: now also U2.b44 (IO_L10N_T1_35); no longer U2.a48 (IO_L10N_T1_34)
- net Ph_B_Tx9: now also U2.b47 (IO_L11P_T1_35); no longer U2.a45 (IO_L11P_T1_34)
- net Ph_C_En: no longer U2.b26 (IO_L4P_T0_35)
- net Ph_C_Err: no longer U2.b22 (IO_L2P_T0_35)
- net Ph_C_Rx: no longer U2.b32 (IO_L6P_T0_35)
- net Ph_C_Tx1: now also U2.b53 (IO_L13P_35); no longer U2.a50 (IO_L13P_T2_34)
- net Ph_C_Tx10: now also U2.b65 (IO_L17N_T2_35); no longer U2.a62 (IO_L17N_T2_34)
- net Ph_C_Tx11: now also U2.b62 (IO_L18P_T2_35); no longer U2.a70 (IO_L18P_T2_34)
- net Ph_C_Tx12: now also U2.b64 (IO_L18N_T2_35); no longer U2.a69 (IO_L18N_T2_34)
- net Ph_C_Tx2: now also U2.b55 (IO_L13N_35); no longer U2.a52 (IO_L13N_T2_34)
- net Ph_C_Tx3: now also U2.b52 (IO_L14P_T2_35); no longer U2.a59 (IO_L14P_T2_34)
- net Ph_C_Tx4: now also U2.b54 (IO_L14N_T2_35); no longer U2.a61 (IO_L14N_T2_34)
- net Ph_C_Tx5: now also U2.b57 (IO_L15P_T2_35); no longer U2.a56 (IO_L15P_T2_34)
- net Ph_C_Tx6: now also U2.b59 (IO_L15N_T2_35); no longer U2.a58 (IO_L15N_T2_34)
- net Ph_C_Tx7: now also U2.b56 (IO_L16P_T2_35); no longer U2.a63 (IO_L16P_T2_34)
- net Ph_C_Tx8: now also U2.b58 (IO_L16N_T2_35); no longer U2.a65 (IO_L16N_T2_34)
- net Ph_C_Tx9: now also U2.b63 (IO_L17P_T2_35); no longer U2.a60 (IO_L17P_T2_34)
- net Ph_D_En: no longer U2.b28 (IO_L4N_T0_35)
- net Ph_D_Err: no longer U2.b24 (IO_L2N_T0_35)
- net Ph_D_Rx: no longer U2.b34 (IO_L6N_T0_35)
- net Ph_D_Tx1: now also U2.b67 (IO_L19P_T3_35); no longer U2.a64 (IO_L19P_T3_34)
- net Ph_D_Tx10: now also U2.b79 (IO_L23N_T3_35); no longer U2.a80 (IO_L23N_T3_34)
- net Ph_D_Tx11: now also U2.b76 (IO_L24P_T3_35); no longer U2.a76 (IO_L24P_T3_34)
- net Ph_D_Tx12: now also U2.b78 (IO_L24N_T3_35); no longer U2.a78 (IO_L24N_T3_34)
- net Ph_D_Tx2: now also U2.b69 (IO_L19N_T3_35); no longer U2.a66 (IO_L19N_T3_34)
- net Ph_D_Tx3: now also U2.b66 (IO_L20P_T3_35); no longer U2.a72 (IO_L20N_T3_34)
- net Ph_D_Tx4: now also U2.b68 (IO_L20N_T3_35); no longer U2.a71 (IO_L20P_T3_34)
- net Ph_D_Tx5: now also U2.b73 (IO_L21P_T3_35); no longer U2.a74 (IO_L21P_T3_34)
- net Ph_D_Tx6: now also U2.b75 (IO_L21N_T3_35); no longer U2.a73 (IO_L21N_T3_34)
- net Ph_D_Tx7: now also U2.b72 (IO_L22P_T3_35); no longer U2.a75 (IO_L22P_T3_34)
- net Ph_D_Tx8: now also U2.b74 (IO_L22N_T3_35); no longer U2.a77 (IO_L22N_T3_34)
- net Ph_D_Tx9: now also U2.b77 (IO_L23P_T3_35); no longer U2.a79 (IO_L23P_T3_34)
- net SDO1_1: no longer U2.b54 (IO_L14N_T2_35)
- net SDO2_1: no longer U2.b57 (IO_L15P_T2_35)
- net SDO3_1: no longer U2.b59 (IO_L15N_T2_35)
- net SDO4_1: no longer U2.b56 (IO_L16P_T2_35)
- net SDO5_1: no longer U2.b58 (IO_L16N_T2_35)
- net SDO6_1: no longer U2.b63 (IO_L17P_T2_35)
- net SDO7_1: no longer U2.b65 (IO_L17N_T2_35)
- net SDO8_1: no longer U2.b62 (IO_L18P_T2_35)
- net esd_diodes/Pin1: no longer U2.b66 (IO_L20P_T3_35)
- net esd_diodes/Pin10: no longer U2.b73 (IO_L21P_T3_35)
- net esd_diodes/Pin2: no longer U2.b68 (IO_L20N_T3_35)
- net esd_diodes/Pin3: no longer U2.b72 (IO_L22P_T3_35)
- net esd_diodes/Pin4: no longer U2.b74 (IO_L22N_T3_35)
- net esd_diodes/Pin5: no longer U2.b76 (IO_L24P_T3_35)
- net esd_diodes/Pin6: no longer U2.b78 (IO_L24N_T3_35)
- net esd_diodes/Pin7: no longer U2.b79 (IO_L23N_T3_35)
- net esd_diodes/Pin8: no longer U2.b77 (IO_L23P_T3_35)
- net esd_diodes/Pin9: no longer U2.b75 (IO_L21N_T3_35)
- net ~{CNV}_1: no longer U2.b69 (IO_L19N_T3_35)
Other:
- moved on the sheet: U2B
