File: FPGA_Board_BA/PCB/chb_com.kicad_sch (KiCad schematic)
At the start: 4 parts, among them J1401 Plug_Terminal_2x12pin, J1402 Plug_Terminal_2x12pin, J1403 Plug_Terminal_2x12pin, J1404 Plug_Terminal_2x12pin

Commit message: schematic almost ready
Parts:
- added J1201, J1202: Plug_Terminal_2x12pin, MYLIB_Misc:DMCV 1,5_12-G1F-3,5-LR P20THR, symbol MYLIB_Misc:Plug_Terminal_2x12pin
- added J1203, J1204, J1205, J1206: Box_Header_6pin, Connector_IDC:IDC-Header_2x03_P2.54mm_Vertical, symbol MYLIB_Misc:Box_Header_6pin
Connections:
- net +5V: now also J1403.1, J1403.11, J1403.13, J1403.15, J1403.17, J1403.19, J1403.21, J1403.23, J1403.3, J1403.5, J1403.7, J1403.9, J1201.1, J1201.10, J1201.11, J1201.12, J1201.13, J1201.14, J1201.15, J1201.16, J1201.17, J1201.18, J1201.19, J1201.2, J1201.20, J1201.21, J1201.22, J1201.23, J1201.24, J1201.3, J1201.4, J1201.5, J1201.6, J1201.7, J1201.8, J1201.9; no longer J1404.10, J1404.12, J1404.14, J1404.16, J1404.18, J1404.2, J1404.20, J1404.22, J1404.24, J1404.4, J1404.6, J1404.8
- net GND: now also J1404.10, J1404.12, J1404.14, J1404.16, J1404.18, J1404.2, J1404.20, J1404.22, J1404.24, J1404.4, J1404.6, J1404.8, J1202.1, J1202.10, J1202.11, J1202.12, J1202.13, J1202.14, J1202.15, J1202.16, J1202.17, J1202.18, J1202.19, J1202.2, J1202.20, J1202.21, J1202.22, J1202.23, J1202.24, J1202.3, J1202.4, J1202.5, J1202.6, J1202.7, J1202.8, J1202.9, J1203.2 (Pin_2), J1203.4 (Pin_4), J1203.6 (Pin_6), J1204.2 (Pin_2), J1204.4 (Pin_4), J1204.6 (Pin_6), J1205.2 (Pin_2), J1205.4 (Pin_4), J1205.6 (Pin_6), J1206.2 (Pin_2), J1206.4 (Pin_4), J1206.6 (Pin_6); no longer J1403.1, J1403.11, J1403.13, J1403.15, J1403.17, J1403.19, J1403.21, J1403.23, J1403.3, J1403.5, J1403.7, J1403.9
- net Ph_C_Tx1: now reaches J1402.1
- net Ph_C_Tx10: now reaches J1402.10
- net Ph_C_Tx11: now reaches J1402.11
- net Ph_C_Tx12: now reaches J1402.12
- net Ph_D_Tx1: now reaches J1402.13
- net Ph_D_Tx2: now reaches J1402.14
- net Ph_D_Tx3: now reaches J1402.15
- net Ph_D_Tx4: now reaches J1402.16
- net Ph_D_Tx5: now reaches J1402.17
- net Ph_D_Tx6: now reaches J1402.18
- net Ph_D_Tx7: now reaches J1402.19
- net Ph_C_Tx2: now reaches J1402.2
- net Ph_D_Tx8: now reaches J1402.20
- net Ph_D_Tx9: now reaches J1402.21
- net Ph_D_Tx10: now reaches J1402.22
- net Ph_D_Tx11: now reaches J1402.23
- net Ph_D_Tx12: now reaches J1402.24
- net Ph_C_Tx3: now reaches J1402.3
- net Ph_C_Tx4: now reaches J1402.4
- net Ph_C_Tx5: now reaches J1402.5
- net Ph_C_Tx6: now reaches J1402.6
- net Ph_C_Tx7: now reaches J1402.7
- net Ph_C_Tx8: now reaches J1402.8
- net Ph_C_Tx9: now reaches J1402.9
- new net Ph_A_En: J1203.3 (Pin_3)
- new net Ph_A_Err: J1203.1 (Pin_1)
- new net Ph_A_Rx: J1203.5 (Pin_5)
- new net Ph_B_En: J1204.3 (Pin_3)
- new net Ph_B_Err: J1204.1 (Pin_1)
- new net Ph_B_Rx: J1204.5 (Pin_5)
- new net Ph_C_En: J1205.3 (Pin_3)
- new net Ph_C_Err: J1205.1 (Pin_1)
- new net Ph_C_Rx: J1205.5 (Pin_5)
- new net Ph_D_En: J1206.3 (Pin_3)
- new net Ph_D_Err: J1206.1 (Pin_1)
- new net Ph_D_Rx: J1206.5 (Pin_5)
Other:
- note added: "12 CHBs on 4 Phases -> 48 in total"
- note added: "En, Err, Rx (for the CHB)"
- moved on the sheet: J1401, J1402, J1403, J1404

Commit message: schematic almost ready pt2
Parts:
- added D1203, D1204, D1205, D1206, D1207, D1208, D1209, D1210, D1211, D1212, D1213, D1214, D1215, D1216, D1217, D1218, D1219, D1220, D1221, D1222, D1223, D1224, D1225, D1226, D1227, D1228, D1229, D1230, D1231, D1232, D1233, D1234, D1235, D1236, D1237, D1238, D1239, D1240, D1241, D1242, D1243, D1244, D1245, D1246, D1247, D1248, D1249, D1250: B72590D50H160, Capacitor_SMD:C_0402_1005Metric_Pad0.74x0.62mm_HandSolder, symbol MYLIB_Misc:ESD_Diode_5V6
Other:
- note added: "48 ESD Diodes"

Commit message: Besprechung mit Leo
Other:
- note added: "8 Pin Wannenstecker und 3 module gleichzeitig versorgt Eine Plug terminal reicht für alle 48 CHBs"
- note added: "Artikel nr Reichelt: WSL 26G 26 pin WAnnenstecker -> 4 St. (GND-Tx gekoppelt)"
- note added: "One side 5V Other GND for better EMV"
Changed lines of the file:
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@@
+		)
+	)
+	(text "One side 5V\nOther GND for better EMV"
+		(exclude_from_sim no)
+		(at 96.266 33.528 0)
+		(effects
+			(font
+				(size 1.27 1.27)
+			)
 		)
 	)
@@
 		)
 	)
+	(text "Artikel nr Reichelt: WSL 26G\n26 pin WAnnenstecker -> 4 St. (GND-Tx gekoppelt)"
+		(exclude_from_sim no)
+		(at 84.9673 130.7909 0)
+		(effects
+			(font
+				(size 1.27 1.27)
+			)
+		)
+	)
 	(text "En, Err, Rx (for the CHB)"
 		(exclude_from_sim no)
@@
 		(effects
 			(font
+				(size 1.27 1.27)
+			)
+		)
+	)
+	(text "8 Pin Wannenstecker und 3 module gleichzeitig versorgt\nEine Plug terminal reicht für alle 48 CHBs"
+		(exclude_from_sim no)
+		(at 83.82 92.964 0)
+		(effects
+			(font

Commit message: lot of work
Parts:
- removed J1201, J1202, J1401, J1402, J1404: Plug_Terminal_2x12pin, MYLIB_Misc:DMCV 1,5_12-G1F-3,5-LR P20THR, symbol MYLIB_Misc:Plug_Terminal_2x12pin
- added J1201, J1202, J1207, J1208: Box_Header_26pin, Connector_IDC:IDC-Header_2x13_P2.54mm_Vertical, symbol MYLIB_Misc:Box_Header_26pin
Connections:
- net +5V: no longer J1403.1, J1403.11, J1403.13, J1403.15, J1403.17, J1403.19, J1403.21, J1403.23, J1403.3, J1403.5, J1403.7, J1403.9
- net GND: now also J1403.1, J1403.11, J1403.13, J1403.15, J1403.17, J1403.19, J1403.21, J1403.23, J1403.3, J1403.5, J1403.7, J1403.9, J1201.1 (Pin_1), J1201.11 (Pin_11), J1201.13 (Pin_13), J1201.15 (Pin_15), J1201.17 (Pin_17), J1201.19 (Pin_19), J1201.21 (Pin_21), J1201.23 (Pin_23), J1201.25 (Pin_25), J1201.26 (Pin_26), J1201.3 (Pin_3), J1201.5 (Pin_5), J1201.7 (Pin_7), J1201.9 (Pin_9), J1202.1 (Pin_1), J1202.11 (Pin_11), J1202.13 (Pin_13), J1202.15 (Pin_15), J1202.17 (Pin_17), J1202.19 (Pin_19), J1202.21 (Pin_21), J1202.23 (Pin_23), J1202.25 (Pin_25), J1202.26 (Pin_26), J1202.3 (Pin_3), J1202.5 (Pin_5), J1202.7 (Pin_7), J1202.9 (Pin_9), J1207.1 (Pin_1), J1207.11 (Pin_11), J1207.13 (Pin_13), J1207.15 (Pin_15), J1207.17 (Pin_17), J1207.19 (Pin_19), J1207.21 (Pin_21), J1207.23 (Pin_23), J1207.25 (Pin_25), J1207.26 (Pin_26), J1207.3 (Pin_3), J1207.5 (Pin_5), J1207.7 (Pin_7), J1207.9 (Pin_9), J1208.1 (Pin_1), J1208.11 (Pin_11), J1208.13 (Pin_13), J1208.15 (Pin_15), J1208.17 (Pin_17), J1208.19 (Pin_19), J1208.21 (Pin_21), J1208.23 (Pin_23), J1208.25 (Pin_25), J1208.26 (Pin_26), J1208.3 (Pin_3), J1208.5 (Pin_5), J1208.7 (Pin_7), J1208.9 (Pin_9)
- net Ph_A_Tx1: now also J1201.2 (Pin_2)
- net Ph_A_Tx10: now also J1201.20 (Pin_20)
- net Ph_A_Tx11: now also J1201.22 (Pin_22)
- net Ph_A_Tx12: now also J1201.24 (Pin_24)
- net Ph_A_Tx2: now also J1201.4 (Pin_4)
- net Ph_A_Tx3: now also J1201.6 (Pin_6)
- net Ph_A_Tx4: now also J1201.8 (Pin_8)
- net Ph_A_Tx5: now also J1201.10 (Pin_10)
- net Ph_A_Tx6: now also J1201.12 (Pin_12)
- net Ph_A_Tx7: now also J1201.14 (Pin_14)
- net Ph_A_Tx8: now also J1201.16 (Pin_16)
- net Ph_A_Tx9: now also J1201.18 (Pin_18)
- net Ph_B_Tx1: now also J1202.2 (Pin_2)
- net Ph_B_Tx10: now also J1202.20 (Pin_20)
- net Ph_B_Tx11: now also J1202.22 (Pin_22)
- net Ph_B_Tx12: now also J1202.24 (Pin_24)
- net Ph_B_Tx2: now also J1202.4 (Pin_4)
- net Ph_B_Tx3: now also J1202.6 (Pin_6)
- net Ph_B_Tx4: now also J1202.8 (Pin_8)
- net Ph_B_Tx5: now also J1202.10 (Pin_10)
- net Ph_B_Tx6: now also J1202.12 (Pin_12)
- net Ph_B_Tx7: now also J1202.14 (Pin_14)
- net Ph_B_Tx8: now also J1202.16 (Pin_16)
- net Ph_B_Tx9: now also J1202.18 (Pin_18)
- net Ph_C_Tx1: now also J1207.2 (Pin_2)
- net Ph_C_Tx10: now also J1207.20 (Pin_20)
- net Ph_C_Tx11: now also J1207.22 (Pin_22)
- net Ph_C_Tx12: now also J1207.24 (Pin_24)
- net Ph_C_Tx2: now also J1207.4 (Pin_4)
- net Ph_C_Tx3: now also J1207.6 (Pin_6)
- net Ph_C_Tx4: now also J1207.8 (Pin_8)
- net Ph_C_Tx5: now also J1207.10 (Pin_10)
- net Ph_C_Tx6: now also J1207.12 (Pin_12)
- net Ph_C_Tx7: now also J1207.14 (Pin_14)
- net Ph_C_Tx8: now also J1207.16 (Pin_16)
- net Ph_C_Tx9: now also J1207.18 (Pin_18)
- net Ph_D_Tx1: now also J1208.2 (Pin_2)
- net Ph_D_Tx10: now also J1208.20 (Pin_20)
- net Ph_D_Tx11: now also J1208.22 (Pin_22)
- net Ph_D_Tx12: now also J1208.24 (Pin_24)
- net Ph_D_Tx2: now also J1208.4 (Pin_4)
- net Ph_D_Tx3: now also J1208.6 (Pin_6)
- net Ph_D_Tx4: now also J1208.8 (Pin_8)
- net Ph_D_Tx5: now also J1208.10 (Pin_10)
- net Ph_D_Tx6: now also J1208.12 (Pin_12)
- net Ph_D_Tx7: now also J1208.14 (Pin_14)
- net Ph_D_Tx8: now also J1208.16 (Pin_16)
- net Ph_D_Tx9: now also J1208.18 (Pin_18)
Other:
- note added: "+5V: 12 pins -> 4 module in each GND: 12 pins -> -||-"
- note added: "Tx lines coupled with GND Phase A-D"
- note removed: "12 CHBs on 4 Phases -> 48 in total"
- note removed: "8 Pin Wannenstecker und 3 module gleichzeitig versorgt Eine Plug terminal reicht für alle 48 CHBs"
- note removed: "Artikel nr Reichelt: WSL 26G 26 pin WAnnenstecker -> 4 St. (GND-Tx gekoppelt)"
- note removed: "One side 5V Other GND for better EMV"
- note removed: "Plug Terminals for Tx of CHB MCU Phase A: Ph_A_Tx1...Ph_A_Tx12 Phase B: analog"
- moved on the sheet: D1203, D1204, D1205, D1206, D1207, D1208, D1209, D1210, D1211, D1212, D1213, D1214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

Commit message: lots of work
Parts:
- removed D1203, D1204, D1205, D1206, D1207, D1208, D1209, D1210, D1211, D1212, D1213, D1214, D1215, D1216, D1217, D1218, D1219, D1220, D1221, D1222, D1223, D1224, D1225, D1226, D1227, D1228, D1229, D1230, D1231, D1232, D1233, D1234, D1235, D1236, D1237, D1238, D1239, D1240, D1241, D1242, D1243, D1244, D1245, D1246, D1247, D1248, D1249, D1250: B72590D50H160, Capacitor_SMD:C_0402_1005Metric_Pad0.74x0.62mm_HandSolder, symbol MYLIB_Misc:ESD_Diode_5V6
- removed J1203, J1204, J1205, J1206: Box_Header_6pin, Connector_IDC:IDC-Header_2x03_P2.54mm_Vertical, symbol MYLIB_Misc:Box_Header_6pin
- added J1601, J1602, J1603, J1604: Box_Header_2x05_THT, Connector_IDC:IDC-Header_2x05_P2.54mm_Vertical, symbol MYLIB_Misc:Box_Header_10pin
Connections:
- net +5V: now also J1601.10 (Pin_10), J1601.9 (Pin_9), J1602.10 (Pin_10), J1602.9 (Pin_9), J1603.10 (Pin_10), J1603.9 (Pin_9), J1604.10 (Pin_10), J1604.9 (Pin_9)
- net GND: now also J1601.2 (Pin_2), J1601.4 (Pin_4), J1601.6 (Pin_6), J1601.8 (Pin_8), J1602.2 (Pin_2), J1602.4 (Pin_4), J1602.6 (Pin_6), J1602.8 (Pin_8), J1603.2 (Pin_2), J1603.4 (Pin_4), J1603.6 (Pin_6), J1603.8 (Pin_8), J1604.2 (Pin_2), J1604.4 (Pin_4), J1604.6 (Pin_6), J1604.8 (Pin_8)
- net Ph_A_Tx1: now also J1601.3 (Pin_3); no longer J1201.2 (Pin_2)
- net Ph_A_Tx10: no longer J1201.20 (Pin_20)
- net Ph_A_Tx11: no longer J1201.22 (Pin_22)
- net Ph_A_Tx12: no longer J1201.24 (Pin_24)
- net Ph_A_Tx2: no longer J1201.4 (Pin_4)
- net Ph_A_Tx3: no longer J1201.6 (Pin_6)
- net Ph_A_Tx4: no longer J1201.8 (Pin_8)
- net Ph_A_Tx5: no longer J1201.10 (Pin_10)
- net Ph_A_Tx6: no longer J1201.12 (Pin_12)
- net Ph_A_Tx7: no longer J1201.14 (Pin_14)
- net Ph_A_Tx8: no longer J1201.16 (Pin_16)
- net Ph_A_Tx9: no longer J1201.18 (Pin_18)
- net Ph_B_Tx1: now also J1604.3 (Pin_3); no longer J1202.2 (Pin_2)
- net Ph_B_Tx10: no longer J1202.20 (Pin_20)
- net Ph_B_Tx11: no longer J1202.22 (Pin_22)
- net Ph_B_Tx12: no longer J1202.24 (Pin_24)
- net Ph_B_Tx2: no longer J1202.4 (Pin_4)
- net Ph_B_Tx3: no longer J1202.6 (Pin_6)
- net Ph_B_Tx4: no longer J1202.8 (Pin_8)
- net Ph_B_Tx5: no longer J1202.10 (Pin_10)
- net Ph_B_Tx6: no longer J1202.12 (Pin_12)
- net Ph_B_Tx7: no longer J1202.14 (Pin_14)
- net Ph_B_Tx8: no longer J1202.16 (Pin_16)
- net Ph_B_Tx9: no longer J1202.18 (Pin_18)
- net Ph_C_Tx1: now also J1602.3 (Pin_3); no longer J1207.2 (Pin_2)
- net Ph_C_Tx10: no longer J1207.20 (Pin_20)
- net Ph_C_Tx11: no longer J1207.22 (Pin_22)
- net Ph_C_Tx12: no longer J1207.24 (Pin_24)
- net Ph_C_Tx2: no longer J1207.4 (Pin_4)
- net Ph_C_Tx3: no longer J1207.6 (Pin_6)
- net Ph_C_Tx4: no longer J1207.8 (Pin_8)
- net Ph_C_Tx5: no longer J1207.10 (Pin_10)
- net Ph_C_Tx6: no longer J1207.12 (Pin_12)
- net Ph_C_Tx7: no longer J1207.14 (Pin_14)
- net Ph_C_Tx8: no longer J1207.16 (Pin_16)
- net Ph_C_Tx9: no longer J1207.18 (Pin_18)
- net Ph_D_Tx1: now also J1603.3 (Pin_3); no longer J1208.2 (Pin_2)
- net Ph_D_Tx10: no longer J1208.20 (Pin_20)
- net Ph_D_Tx11: no longer J1208.22 (Pin_22)
- net Ph_D_Tx12: no longer J1208.24 (Pin_24)
- net Ph_D_Tx2: no longer J1208.4 (Pin_4)
- net Ph_D_Tx3: no longer J1208.6 (Pin_6)
- net Ph_D_Tx4: no longer J1208.8 (Pin_8)
- net Ph_D_Tx5: no longer J1208.10 (Pin_10)
- net Ph_D_Tx6: no longer J1208.12 (Pin_12)
- net Ph_D_Tx7: no longer J1208.14 (Pin_14)
- net Ph_D_Tx8: no longer J1208.16 (Pin_16)
- net Ph_D_Tx9: no longer J1208.18 (Pin_18)
- new net Level_Shifter_8bit_1/A1: J1201.2 (Pin_2)
- new net Level_Shifter_8bit_1/A2: J1201.4 (Pin_4)
- new net Level_Shifter_8bit_1/A3: J1201.6 (Pin_6)
- new net Level_Shifter_8bit_1/A4: J1201.8 (Pin_8)
- new net Level_Shifter_8bit_1/A5: J1201.10 (Pin_10)
- new net Level_Shifter_8bit_1/A6: J1201.12 (Pin_12)
- new net Level_Shifter_8bit_1/A7: J1201.14 (Pin_14)
- new net Level_Shifter_8bit_1/A8: J1201.16 (Pin_16)
- new net Level_Shifter_8bit_2/A1: J1201.18 (Pin_18)
- new net Level_Shifter_8bit_2/A2: J1201.20 (Pin_20)
- new net Level_Shifter_8bit_2/A3: J1201.22 (Pin_22)
- new net Level_Shifter_8bit_2/A4: J1201.24 (Pin_24)
- new net Level_Shifter_8bit_2/A5: J1202.2 (Pin_2)
- new net Level_Shifter_8bit_2/A6: J1202.4 (Pin_4)
- new net Level_Shifter_8bit_2/A7: J1202.6 (Pin_6)
- new net Level_Shifter_8bit_2/A8: J1202.8 (Pin_8)
- new net Level_Shifter_8bit_3/A1: J1202.10 (Pin_10)
- new net Level_Shifter_8bit_3/A2: J1202.12 (Pin_12)
- new net Level_Shifter_8bit_3/A3: J1202.14 (Pin_14)
- new net Level_Shifter_8bit_3/A4: J1202.16 (Pin_16)
- new net Level_Shifter_8bit_3/A5: J1202.18 (Pin_18)
- new net Level_Shifter_8bit_3/A6: J1202.20 (Pin_20)
- new net Level_Shifter_8bit_3/A7: J1202.22 (Pin_22)
- new net Level_Shifter_8bit_3/A8: J1202.24 (Pin_24)
- new net Level_Shifter_8bit_4/A1: J1207.2 (Pin_2)
- new net Level_Shifter_8bit_4/A2: J1207.4 (Pin_4)
- new net Level_Shifter_8bit_4/A3: J1207.6 (Pin_6)
- new net Level_Shifter_8bit_4/A4: J1207.8 (Pin_8)
- new net Level_Shifter_8bit_4/A5: J1207.10 (Pin_10)
- new net Level_Shifter_8bit_4/A6: J1207.12 (Pin_12)
- new net Level_Shifter_8bit_4/A7: J1207.14 (Pin_14)
- new net Level_Shifter_8bit_4/A8: J1207.16 (Pin_16)
- new net Level_Shifter_8bit_5/A1: J1207.18 (Pin_18)
- new net Level_Shifter_8bit_5/A2: J1207.20 (Pin_20)
- new net Level_Shifter_8bit_5/A3: J1207.22 (Pin_22)
- new net Level_Shifter_8bit_5/A4: J1207.24 (Pin_24)
- new net Level_Shifter_8bit_5/A5: J1208.2 (Pin_2)
- new net Level_Shifter_8bit_5/A6: J1208.4 (Pin_4)
- new net Level_Shifter_8bit_5/A7: J1208.6 (Pin_6)
- new net Level_Shifter_8bit_5/A8: J1208.8 (Pin_8)
- new net Level_Shifter_8bit_6/A1: J1208.10 (Pin_10)
- new net Level_Shifter_8bit_6/A2: J1208.12 (Pin_12)
- new net Level_Shifter_8bit_6/A3: J1208.14 (Pin_14)
- new net Level_Shifter_8bit_6/A4: J1208.16 (Pin_16)
- new net Level_Shifter_8bit_6/A5: J1208.18 (Pin_18)
- new net Level_Shifter_8bit_6/A6: J1208.20 (Pin_20)
- new net Level_Shifter_8bit_6/A7: J1208.22 (Pin_22)
- new net Level_Shifter_8bit_6/A8: J1208.24 (Pin_24)
- new net Level_shifter_Rx_En/B1: J1601.7 (Pin_7)
- new net Level_shifter_Rx_En/B2: J1601.5 (Pin_5)
- new net Level_shifter_Rx_En/B3: J1604.7 (Pin_7)
- new net Level_shifter_Rx_En/B4: J1604.5 (Pin_5)
- new net Level_shifter_Rx_En/B5: J1602.7 (Pin_7)
- new net Level_shifter_Rx_En/B6: J1602.5 (Pin_5)
- new net Level_shifter_Rx_En/B7: J1603.7 (Pin_7)
- new net Level_shifter_Rx_En/B8: J1603.5 (Pin_5)
- new net Level_shifter_error_1/A1: J1601.1 (Pin_1)
- new net Level_shifter_error_1/A2: J1604.1 (Pin_1)
- new net Level_shifter_error_2/A1: J1602.1 (Pin_1)
- new net Level_shifter_error_2/A2: J1603.1 (Pin_1)
Other:
- added sheet Level_Shifter_8bit_1 (level_shifter_8bit.kicad_sch)
- added sheet Level_Shifter_8bit_2 (level_shifter_8bit.kicad_sch)
- added sheet Level_Shifter_8bit_3 (level_shifter_8bit.kicad_sch)
- added sheet Level_Shifter_8bit_4 (level_shifter_8bit.kicad_sch)
- added sheet Level_Shifter_8bit_5 (level_shifter_8bit.kicad_sch)
- added sheet Level_Shifter_8bit_6 (level_shifter_8bit.kicad_sch)
- added sheet Level_shifter_Rx_En (ls_rx_en.kicad_sch)
- added sheet Level_shifter_error_1 (ls_error.kicad_sch)
- added sheet Level_shifter_error_2 (ls_error.kicad_sch)
- note removed: "48 ESD Diodes"
- moved on the sheet: J1201, J1202, J1207, J1208, J1403

Commit message: work
Parts:
- renumbered J1201 to J10, J1202 to J11, J1601 to J12, J1604 to J13, J1602 to J14, J1603 to J15, J1207 to J16, J1208 to J17, J1403 to J18
Changed lines of the file:
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@@
 		(dnp no)
 		(fields_autoplaced yes)
-		(property "Reference" "J1201"
+		(property "Reference" "J10"
 			(at 40.64 26.67 0)
 			(effects
@@
 			(project ""
 				(path "/fd7503bc-e7fc-4766-b224-3d1c3d7de5ff/1b181806-12f4-40c8-bf91-78ac0d892dab"
-					(reference "J1201")
+					(reference "J10")
 					(unit 1)
 				)
@@
 		(dnp no)
 		(fields_autoplaced yes)
-		(property "Reference" "J1604"
+		(property "Reference" "J13"
 			(at 53.34 185.42 0)
 			(effects
@@
 			(project "FPGA_Board_BA"
 				(path "/fd7503bc-e7fc-4766-b224-3d1c3d7de5ff/1b181806-12f4-40c8-bf91-78ac0d892dab"
-					(reference "J1604")
+					(reference "J13")
 					(unit 1)
 				)
@@
 		(dnp no)
 		(fields_autoplaced yes)
-		(property "Reference" "#PWR01212"
+		(property "Reference" "#PWR074"
 			(at 140.97 76.2 0)
 			(effects
@@
 			(project "FPGA_Board_BA"
 				(path "/fd7503bc-e7fc-4766-b224-3d1c3d7de5ff/1b181806-12f4-40c8-bf91-78ac0d892dab"
-					(reference "#PWR01212")
+					(reference "#PWR074")
 					(unit 1)
 				)
@@
 		(dnp no)
 		(fields_autoplaced yes)
-		(property "Reference" "J1601"
+		(property "Reference" "J12"
 			(at 53.34 158.75 0)
 			(effects
@@
 			(project ""
 				(path "/fd7503bc-e7fc-4766-b224-3d1c3d7de5ff/1b181806-12f4-40c8-bf91-78ac0d892dab"
-					(reference "J1601")
+					(reference "J12")
 					(unit 1)
 				)
@@
 		(dnp no)
 		(fields_autoplaced yes)
-		(property "Reference" "#PWR01210"
+		(property "Reference" "#PWR068"
 			(at 27.94 76.2 0)
 			(effects
@@
 			(project ""
 				(path "/fd7503bc-e7fc-4766-b224-3d1c3d7de5ff/1b181806-12f4-40c8-bf91-78ac0d892dab"
-					(reference "#PWR01210")
+					(reference "#PWR068")
 					(unit 1)
 				)
@@
 		(dnp no)
 		(fields_autoplaced yes)
-		(property "Reference" "J1208"
+		(property "Reference" "J17"
 			(at 151.13 76.2 0)
 			(effects
@@
 			(project "FPGA_Board_BA"
 				(path "/fd7503bc-e7fc-4766-b224-3d1c3d7de5ff/1b181806-12f4-40c8-bf91-78ac0d892dab"
-					(reference "J1208")
+					(reference "J17")
 					(unit 1)
 				)
@@
 		(dnp no)
 		(fields_autoplaced yes)
-		(property "Reference" "J1202"
+		(property "Reference" "J11"
 			(at 40.64 77.47 0)
 			(effects
@@
 			(project "FPGA_Board_BA"
 				(path "/fd7503bc-e7fc-4766-b224-3d1c3d7de5ff/1b181806-12f4-40c8-bf91-78ac0d892dab"
-					(reference "J1202")
+					(reference "J11")
 					(unit 1)
 				)
@@
 		(dnp no)
 		(fields_autoplaced yes)
-		(property "Reference" "J1207"
+		(property "Reference" "J16"
 			(at 151.13 25.4 0)
 			(effects
@@
 			(project "FPGA_Board_BA"
 				(path "/fd7503bc-e7fc-4766-b224-3d1c3d7de5ff/1b181806-12f4-40c8-bf91-78ac0d892dab"
-					(reference "J1207")
+					(reference "J16")
 					(unit 1)
 				)
@@
 		(dnp no)
 		(fields_autoplaced yes)
-		(property "Reference" "#PWR01610"
+		(property "Reference" "#PWR072"
 			(at 40.64 237.49 0)
 			(effects
@@
 			(project "FPGA_Board_BA"
 				(path "/fd7503bc-e7fc-4766-b224-3d1c3d7de5ff/1b181806-12f4-40c8-bf91-78ac0d892dab"
-					(reference "#PWR01610")
+					(reference "#PWR072")
 					(unit 1)
 				)
@@
 		(dnp no)
 		(fields_autoplaced yes)
-		(property "Reference" "#PWR01211"
+		(property "Reference" "#PWR069"
 			(at 34.29 128.27 0)
 			(effects
@@
 			(project "FPGA_Board_BA"
 				(path "/fd7503bc-e7fc-4766-b224-3d1c3d7de5ff/1b181806-12f4-40c8-bf91-78ac0d892dab"
-					(reference "#PWR01211")
+					(reference "#PWR069")
 					(unit 1)
 				)
@@
 		(dnp no)
 		(fields_autoplaced yes)
-		(property "Reference" "J1603"
+		(property "Reference" "J15"
 			(at 53.34 237.49 0)
 			(effects
@@
 			(project "FPGA_Board_BA"
 				(path "/fd7503bc-e7fc-4766-b224-3d1c3d7de5ff/1b181806-12f4-40c8-bf91-78ac0d892dab"
-					(reference "J1603")
+					(reference "J15")
 					(unit 1)
 				)
@@
 		(dnp no)
 		(fields_autoplaced yes)
-		(property "Reference" "#PWR01213"
+		(property "Reference" "#PWR075"
 			(at 142.24 125.73 0)
 			(effects
@@
 			(project "FPGA_Board_BA"
 				(path "/fd7503bc-e7fc-4766-b224-3d1c3d7de5ff/1b181806-12f4-40c8-bf91-78ac0d892dab"
-					(reference "#PWR01213")
+					(reference "#PWR075")
 					(unit 1)
 				)
@@
 		(on_board yes)
 		(dnp no)
-		(property "Reference" "#PWR01612"
+		(property "Reference" "#PWR071"
 			(at 40.64 210.82 0)
 			(effects
@@
 			(project "FPGA_Board_BA"
 				(path "/fd7503bc-e7fc-4766-b224-3d1c3d7de5ff/1b181806-12f4-40c8-bf91-78ac0d892dab"
-					(reference "#PWR01612")
+					(reference "#PWR071")
 					(unit 1)
 				)
@@
 		(dnp no)
 		(fields_autoplaced yes)
-		(property "Reference" "#PWR01209"
+		(property "Reference" "#PWR076"
 			(at 224.79 241.3 0)
 			(effects
@@
 			(project ""
 				(path "/fd7503bc-e7fc-4766-b224-3d1c3d7de5ff/1b181806-12f4-40c8-bf91-78ac0d892dab"
-					(reference "#PWR01209")
+					(reference "#PWR076")
 					(unit 1)
 				)
@@
 		(dnp no)
 		(fields_autoplaced yes)
-		(property "Reference" "#PWR01401"
+		(property "Reference" "#PWR077"
 			(at 256.54 204.47 0)
 			(effects
@@
 			(project ""
 				(path "/fd7503bc-e7fc-4766-b224-3d1c3d7de5ff/1b181806-12f4-40c8-bf91-78ac0d892dab"
-					(reference "#PWR01401")
+					(reference "#PWR077")
 					(unit 1)
 				)
@@
 		(dnp no)
 		(fields_autoplaced yes)
-		(property "Reference" "J1602"
+		(property "Reference" "J14"
 			(at 53.34 212.09 0)
 			(effects
@@
 			(project "FPGA_Board_BA"
 				(path "/fd7503bc-e7fc-4766-b224-3d1c3d7de5ff/1b181806-12f4-40c8-bf91-78ac0d892dab"
-					(reference "J1602")
+					(reference "J14")
 					(unit 1)
 				)
@@
 		(dnp no)
 		(fields_autoplaced yes)
-		(property "Reference" "#PWR01611"
+		(property "Reference" "#PWR073"
 			(at 40.64 262.89 0)
 			(effects
@@
 			(project "FPGA_Board_BA"
 				(path "/fd7503bc-e7fc-4766-b224-3d1c3d7de5ff/1b181806-12f4-40c8-bf91-78ac0d892dab"
-					(reference "#PWR01611")
+					(reference "#PWR073")
 					(unit 1)
 				)
@@
 		(on_board yes)
 		(dnp no)
-		(property "Reference" "#PWR01609"
+		(property "Reference" "#PWR070"
 			(at 40.64 184.15 0)
 			(effects
@@
 			(project "FPGA_Board_BA"
 				(path "/fd7503bc-e7fc-4766-b224-3d1c3d7de5ff/1b181806-12f4-40c8-bf91-78ac0d892dab"
-					(reference "#PWR01609")
+					(reference "#PWR070")
 					(unit 1)
 				)
@@
 		(dnp no)
 		(fields_autoplaced yes)
-		(property "Reference" "J1403"
+		(property "Reference" "J18"
 			(at 237.49 198.12 0)
 			(effects
@@
 			(project "FPGA_Board_BA"
 				(path "/fd7503bc-e7fc-4766-b224-3d1c3d7de5ff/1b181806-12f4-40c8-bf91-78ac0d892dab"
-					(reference "J1403")
-					(unit 1)
-				)
+					(reference "J18")
+					(unit 1)
+				)

Commit message: 22.11
Other:
- note added: "En"
- note added: "Err"
- note added: "Rx"
- note added: "Theoretisch braucht man kein level Shifter für Rx, weil 3.3V schon als High erkannt wird"
- note added: "Tx"
