File: FPGA_Board_BA/PCB/connectors.kicad_sch (KiCad schematic)
At the start: 2 parts, among them J601 Banana_Socket_Black, J602 Banana_Socket_Red

Commit message: schematic almost ready pt2
Parts:
- added D601: LED_G_0603, WLIB_DO:LED_0603_1608Metric, symbol WLIB_D:LED_G_0603
- added R601: 100k_0603, Resistor_SMD:R_0603_1608Metric, symbol WLIB_R:100k_0603
Connections:
- net GND: now also D601.1 (K)
- net Power_in: now also R601.1
- new net: D601.2 (A), R601.2
Other:
- note added: "Status LED for plugged in power"

Commit message: work
Parts:
- renumbered D601 to D4, J602 to J2, J601 to J3, R601 to R15
Changed lines of the file:
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@@
 		(dnp no)
 		(fields_autoplaced yes)
-		(property "Reference" "R601"
+		(property "Reference" "R15"
 			(at 110.49 86.3599 0)
 			(effects
@@
 			(project ""
 				(path "/fd7503bc-e7fc-4766-b224-3d1c3d7de5ff/0e4170b7-c04b-49af-9f71-fb64eba9da72"
-					(reference "R601")
+					(reference "R15")
 					(unit 1)
 				)
@@
 		(dnp no)
 		(fields_autoplaced yes)
-		(property "Reference" "#PWR0601"
+		(property "Reference" "#PWR031"
 			(at 91.44 101.6 0)
 			(effects
@@
 			(project ""
 				(path "/fd7503bc-e7fc-4766-b224-3d1c3d7de5ff/0e4170b7-c04b-49af-9f71-fb64eba9da72"
-					(reference "#PWR0601")
+					(reference "#PWR031")
 					(unit 1)
 				)
@@
 		(dnp no)
 		(fields_autoplaced yes)
-		(property "Reference" "J602"
+		(property "Reference" "J2"
 			(at 73.66 72.39 0)
 			(effects
@@
 			(project ""
 				(path "/fd7503bc-e7fc-4766-b224-3d1c3d7de5ff/0e4170b7-c04b-49af-9f71-fb64eba9da72"
-					(reference "J602")
+					(reference "J2")
 					(unit 1)
 				)
@@
 		(dnp no)
 		(fields_autoplaced yes)
-		(property "Reference" "J601"
+		(property "Reference" "J3"
 			(at 73.66 83.82 0)
 			(effects
@@
 			(project ""
 				(path "/fd7503bc-e7fc-4766-b224-3d1c3d7de5ff/0e4170b7-c04b-49af-9f71-fb64eba9da72"
-					(reference "J601")
+					(reference "J3")
 					(unit 1)
 				)
@@
 		(dnp no)
 		(fields_autoplaced yes)
-		(property "Reference" "#PWR0602"
+		(property "Reference" "#PWR032"
 			(at 107.95 113.03 0)
 			(effects
@@
 			(project "FPGA_Board_BA"
 				(path "/fd7503bc-e7fc-4766-b224-3d1c3d7de5ff/0e4170b7-c04b-49af-9f71-fb64eba9da72"
-					(reference "#PWR0602")
+					(reference "#PWR032")
 					(unit 1)
 				)
@@
 		(dnp no)
 		(fields_autoplaced yes)
-		(property "Reference" "D601"
+		(property "Reference" "D4"
 			(at 111.76 98.1074 90)
 			(effects
@@
 			(project ""
 				(path "/fd7503bc-e7fc-4766-b224-3d1c3d7de5ff/0e4170b7-c04b-49af-9f71-fb64eba9da72"
-					(reference "D601")
-					(unit 1)
-				)
+					(reference "D4")
+					(unit 1)
+				)

Commit message: 22.11
Parts:
- renumbered D4 to D8, J2 to J3, J3 to J4, R15 to R8
Changed lines of the file:
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@@
 		(dnp no)
 		(fields_autoplaced yes)
-		(property "Reference" "R15"
+		(property "Reference" "R8"
 			(at 110.49 86.3599 0)
 			(effects
@@
 			(project ""
 				(path "/fd7503bc-e7fc-4766-b224-3d1c3d7de5ff/0e4170b7-c04b-49af-9f71-fb64eba9da72"
-					(reference "R15")
+					(reference "R8")
 					(unit 1)
 				)
@@
 		(dnp no)
 		(fields_autoplaced yes)
-		(property "Reference" "#PWR031"
+		(property "Reference" "#PWR036"
 			(at 91.44 101.6 0)
 			(effects
@@
 			(project ""
 				(path "/fd7503bc-e7fc-4766-b224-3d1c3d7de5ff/0e4170b7-c04b-49af-9f71-fb64eba9da72"
-					(reference "#PWR031")
+					(reference "#PWR036")
 					(unit 1)
 				)
@@
 		(dnp no)
 		(fields_autoplaced yes)
-		(property "Reference" "J2"
+		(property "Reference" "J3"
 			(at 73.66 72.39 0)
 			(effects
@@
 			(project ""
 				(path "/fd7503bc-e7fc-4766-b224-3d1c3d7de5ff/0e4170b7-c04b-49af-9f71-fb64eba9da72"
-					(reference "J2")
+					(reference "J3")
 					(unit 1)
 				)
@@
 		(dnp no)
 		(fields_autoplaced yes)
-		(property "Reference" "J3"
+		(property "Reference" "J4"
 			(at 73.66 83.82 0)
 			(effects
@@
 			(project ""
 				(path "/fd7503bc-e7fc-4766-b224-3d1c3d7de5ff/0e4170b7-c04b-49af-9f71-fb64eba9da72"
-					(reference "J3")
+					(reference "J4")
 					(unit 1)
 				)
@@
 		(dnp no)
 		(fields_autoplaced yes)
-		(property "Reference" "#PWR032"
+		(property "Reference" "#PWR037"
 			(at 107.95 113.03 0)
 			(effects
@@
 			(project "FPGA_Board_BA"
 				(path "/fd7503bc-e7fc-4766-b224-3d1c3d7de5ff/0e4170b7-c04b-49af-9f71-fb64eba9da72"
-					(reference "#PWR032")
+					(reference "#PWR037")
 					(unit 1)
 				)
@@
 		(dnp no)
 		(fields_autoplaced yes)
-		(property "Reference" "D4"
+		(property "Reference" "D8"
 			(at 111.76 98.1074 90)
 			(effects
@@
 			(project ""
 				(path "/fd7503bc-e7fc-4766-b224-3d1c3d7de5ff/0e4170b7-c04b-49af-9f71-fb64eba9da72"
-					(reference "D4")
-					(unit 1)
-				)
+					(reference "D8")
+					(unit 1)
+				)

Commit message: exported stuff
Parts:
- D8: footprint WLIB_DO:LED_0603_1608Metric -> LED_SMD:LED_0603_1608Metric
Changed lines of the file:
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@@
 		(dnp no)
 		(fields_autoplaced yes)
-		(property "Reference" "#PWR036"
+		(property "Reference" "#PWR037"
 			(at 91.44 101.6 0)
 			(effects
@@
 			(project ""
 				(path "/fd7503bc-e7fc-4766-b224-3d1c3d7de5ff/0e4170b7-c04b-49af-9f71-fb64eba9da72"
-					(reference "#PWR036")
+					(reference "#PWR037")
 					(unit 1)
 				)
@@
 		(dnp no)
 		(fields_autoplaced yes)
-		(property "Reference" "#PWR037"
+		(property "Reference" "#PWR038"
 			(at 107.95 113.03 0)
 			(effects
@@
 			(project "FPGA_Board_BA"
 				(path "/fd7503bc-e7fc-4766-b224-3d1c3d7de5ff/0e4170b7-c04b-49af-9f71-fb64eba9da72"
-					(reference "#PWR037")
+					(reference "#PWR038")
 					(unit 1)
 				)
@@
 			)
 		)
-		(property "Footprint" "WLIB_DO:LED_0603_1608Metric"
+		(property "Footprint" "LED_SMD:LED_0603_1608Metric"
 			(at 97.79 97.79 0)
 			(effects
