File: FPGA_Board_BA/PCB/level_shifter_8bit.kicad_sch (KiCad schematic)
At the start: 3 parts, among them U3301 SN74LXCH8T245RHLR

Commit message: work
Parts:
- added R127, R128, R129, R130, R131, R132, R133, R134: 10k_0603, Resistor_SMD:R_0603_1608Metric, symbol WLIB_R:10k_0603
- renumbered C3303 to C136, C3304 to C137, U3301 to U34
Connections:
- net +3.3V: now also R127.1, R128.1, R129.1, R130.1, R131.1, R132.1, R133.1, R134.1
- net B1: now also R127.2
- net B2: now also R128.2
- net B3: now also R129.2
- net B4: now also R130.2
- net B5: now also R131.2
- net B6: now also R132.2
- net B7: now also R133.2
- net B8: now also R134.2

Commit message: 22.11
Parts:
- renumbered C136 to C133, C137 to C134, R127 to R126, R128 to R127, R129 to R128, R130 to R129, R131 to R130, R132 to R131, R133 to R132, R134 to R133, U34 to U28
Connections:
- net +3.3V: no longer R126.1, R127.1, R128.1, R129.1, R130.1, R131.1, R132.1, R133.1
- net +5V: now also R126.1, R127.1, R128.1, R129.1, R130.1, R131.1, R132.1, R133.1
- net A1: now also R126.2
- net A2: now also R127.2
- net A3: now also R128.2
- net A4: now also R129.2
- net A5: now also R130.2
- net A6: now also R131.2
- net A7: now also R132.2
- net A8: now also R133.2
- net B1: no longer R126.2
- net B2: no longer R127.2
- net B3: no longer R128.2
- net B4: no longer R129.2
- net B5: no longer R130.2
- net B6: no longer R131.2
- net B7: no longer R132.2
- net B8: no longer R133.2
Other:
- moved on the sheet: C133, C134, R126, R127, R128, R129, R130, R131, R132, R133, U28

Commit message: exported stuff
Parts:
- renumbered C133 to C128, C134 to C129, R126 to R165, R127 to R166, R128 to R167, R129 to R168, R130 to R169, R131 to R170, R132 to R171, R133 to R172, U28 to U27
