File: FPGA_Board_BA/PCB/ls_rx_en.kicad_sch (KiCad schematic)
At the start: 3 parts, among them U3901 SN74LXCH8T245RHLR

Commit message: work
Parts:
- added R178, R179, R180, R181, R182, R183, R184, R185: 10k_0603, Resistor_SMD:R_0603_1608Metric, symbol WLIB_R:10k_0603
- renumbered C3901 to C155, C3902 to C156, U3901 to U42
Connections:
- net +5V: now also R178.1, R179.1, R180.1, R181.1, R182.1, R183.1, R184.1, R185.1
- net B1: now also R178.2
- net B2: now also R179.2
- net B3: now also R180.2
- net B4: now also R181.2
- net B5: now also R182.2
- net B6: now also R183.2
- net B7: now also R184.2
- net B8: now also R185.2
Other:
- moved on the sheet: C155, C156, U42

Commit message: 22.11
Parts:
- renumbered C155 to C153, C156 to C154, R178 to R186, R179 to R187, R180 to R188, R181 to R189, R182 to R190, R183 to R191, R184 to R192, R185 to R193, U42 to U39
Connections:
- net +3.3V: now also R186.1, R187.1, R188.1, R189.1, R190.1, R191.1, R192.1, R193.1
- net +5V: no longer R186.1, R187.1, R188.1, R189.1, R190.1, R191.1, R192.1, R193.1
- net A1: now also R186.2
- net A2: now also R187.2
- net A3: now also R188.2
- net A4: now also R189.2
- net A5: now also R190.2
- net A6: now also R191.2
- net A7: now also R192.2
- net A8: now also R193.2
- net B1: no longer R186.2
- net B2: no longer R187.2
- net B3: no longer R188.2
- net B4: no longer R189.2
- net B5: no longer R190.2
- net B6: no longer R191.2
- net B7: no longer R192.2
- net B8: no longer R193.2
Other:
- moved on the sheet: C153, C154, R186, R187, R188, R189, R190, R191, R192, R193, U39

Commit message: exported stuff
Parts:
- renumbered C153 to C148, C154 to C149, R186 to R225, R187 to R226, R188 to R227, R189 to R228, R190 to R229, R191 to R230, R192 to R231, R193 to R232, U39 to U38
Changed lines of the file:
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@@
 		(on_board yes)
 		(dnp no)
-		(property "Reference" "R189"
+		(property "Reference" "R228"
 			(at 101.346 66.04 90)
 			(effects
@@
 			(project "FPGA_Board_BA"
 				(path "/fd7503bc-e7fc-4766-b224-3d1c3d7de5ff/1b181806-12f4-40c8-bf91-78ac0d892dab/d6c6031d-c1b3-49bb-af8f-093ee0f25456"
-					(reference "R189")
+					(reference "R228")
 					(unit 1)
 				)
@@
 		(on_board yes)
 		(dnp no)
-		(property "Reference" "R190"
+		(property "Reference" "R229"
 			(at 110.236 66.04 90)
 			(effects
@@
 			(project "FPGA_Board_BA"
 				(path "/fd7503bc-e7fc-4766-b224-3d1c3d7de5ff/1b181806-12f4-40c8-bf91-78ac0d892dab/d6c6031d-c1b3-49bb-af8f-093ee0f25456"
-					(reference "R190")
+					(reference "R229")
 					(unit 1)
 				)
@@
 		(on_board yes)
 		(dnp no)
-		(property "Reference" "R193"
+		(property "Reference" "R232"
 			(at 135.636 66.04 90)
 			(effects
@@
 			(project "FPGA_Board_BA"
 				(path "/fd7503bc-e7fc-4766-b224-3d1c3d7de5ff/1b181806-12f4-40c8-bf91-78ac0d892dab/d6c6031d-c1b3-49bb-af8f-093ee0f25456"
-					(reference "R193")
+					(reference "R232")
 					(unit 1)
 				)
@@
 		(dnp no)
 		(fields_autoplaced yes)
-		(property "Reference" "#PWR0235"
+		(property "Reference" "#PWR0247"
 			(at 203.2 60.96 0)
 			(effects
@@
 			(project "FPGA_Board_BA"
 				(path "/fd7503bc-e7fc-4766-b224-3d1c3d7de5ff/1b181806-12f4-40c8-bf91-78ac0d892dab/d6c6031d-c1b3-49bb-af8f-093ee0f25456"
-					(reference "#PWR0235")
+					(reference "#PWR0247")
 					(unit 1)
 				)
@@
 		(dnp no)
 		(fields_autoplaced yes)
-		(property "Reference" "#PWR0233"
+		(property "Reference" "#PWR0245"
 			(at 175.26 129.54 0)
 			(effects
@@
 			(project "FPGA_Board_BA"
 				(path "/fd7503bc-e7fc-4766-b224-3d1c3d7de5ff/1b181806-12f4-40c8-bf91-78ac0d892dab/d6c6031d-c1b3-49bb-af8f-093ee0f25456"
-					(reference "#PWR0233")
+					(reference "#PWR0245")
 					(unit 1)
 				)
@@
 		(on_board yes)
 		(dnp no)
-		(property "Reference" "R191"
+		(property "Reference" "R230"
 			(at 117.856 66.04 90)
 			(effects
@@
 			(project "FPGA_Board_BA"
 				(path "/fd7503bc-e7fc-4766-b224-3d1c3d7de5ff/1b181806-12f4-40c8-bf91-78ac0d892dab/d6c6031d-c1b3-49bb-af8f-093ee0f25456"
-					(reference "R191")
+					(reference "R230")
 					(unit 1)
 				)
@@
 		(dnp no)
 		(fields_autoplaced yes)
-		(property "Reference" "#PWR0234"
+		(property "Reference" "#PWR0246"
 			(at 185.42 60.96 0)
 			(effects
@@
 			(project "FPGA_Board_BA"
 				(path "/fd7503bc-e7fc-4766-b224-3d1c3d7de5ff/1b181806-12f4-40c8-bf91-78ac0d892dab/d6c6031d-c1b3-49bb-af8f-093ee0f25456"
-					(reference "#PWR0234")
+					(reference "#PWR0246")
 					(unit 1)
 				)
@@
 		(on_board yes)
 		(dnp no)
-		(property "Reference" "R188"
+		(property "Reference" "R227"
 			(at 92.456 66.04 90)
 			(effects
@@
 			(project "FPGA_Board_BA"
 				(path "/fd7503bc-e7fc-4766-b224-3d1c3d7de5ff/1b181806-12f4-40c8-bf91-78ac0d892dab/d6c6031d-c1b3-49bb-af8f-093ee0f25456"
-					(reference "R188")
+					(reference "R227")
 					(unit 1)
 				)
@@
 		(dnp no)
 		(fields_autoplaced yes)
-		(property "Reference" "#PWR0232"
+		(property "Reference" "#PWR0244"
 			(at 152.4 73.66 0)
 			(effects
@@
 			(project "FPGA_Board_BA"
 				(path "/fd7503bc-e7fc-4766-b224-3d1c3d7de5ff/1b181806-12f4-40c8-bf91-78ac0d892dab/d6c6031d-c1b3-49bb-af8f-093ee0f25456"
-					(reference "#PWR0232")
+					(reference "#PWR0244")
 					(unit 1)
 				)
@@
 		(on_board yes)
 		(dnp no)
-		(property "Reference" "R192"
+		(property "Reference" "R231"
 			(at 126.746 66.04 90)
 			(effects
@@
 			(project "FPGA_Board_BA"
 				(path "/fd7503bc-e7fc-4766-b224-3d1c3d7de5ff/1b181806-12f4-40c8-bf91-78ac0d892dab/d6c6031d-c1b3-49bb-af8f-093ee0f25456"
-					(reference "R192")
+					(reference "R231")
 					(unit 1)
 				)
@@
 		(on_board yes)
 		(dnp no)
-		(property "Reference" "R187"
+		(property "Reference" "R226"
 			(at 83.566 66.04 90)
 			(effects
@@
 			(project "FPGA_Board_BA"
 				(path "/fd7503bc-e7fc-4766-b224-3d1c3d7de5ff/1b181806-12f4-40c8-bf91-78ac0d892dab/d6c6031d-c1b3-49bb-af8f-093ee0f25456"
-					(reference "R187")
+					(reference "R226")
 					(unit 1)
 				)
@@
 		(on_board yes)
 		(dnp no)
-		(property "Reference" "R186"
+		(property "Reference" "R225"
 			(at 74.676 66.04 90)
 			(effects
@@
 			(project "FPGA_Board_BA"
 				(path "/fd7503bc-e7fc-4766-b224-3d1c3d7de5ff/1b181806-12f4-40c8-bf91-78ac0d892dab/d6c6031d-c1b3-49bb-af8f-093ee0f25456"
-					(reference "R186")
+					(reference "R225")
 					(unit 1)
 				)
@@
 		(dnp no)
 		(fields_autoplaced yes)
-		(property "Reference" "U39"
+		(property "Reference" "U38"
 			(at 194.31 121.92 0)
 			(effects
@@
 			(project "FPGA_Board_BA"
 				(path "/fd7503bc-e7fc-4766-b224-3d1c3d7de5ff/1b181806-12f4-40c8-bf91-78ac0d892dab/d6c6031d-c1b3-49bb-af8f-093ee0f25456"
-					(reference "U39")
+					(reference "U38")
 					(unit 1)
 				)
@@
 		(dnp no)
 		(fields_autoplaced yes)
-		(property "Reference" "C153"
+		(property "Reference" "C148"
 			(at 171.45 54.61 90)
 			(effects
@@
 			(project "FPGA_Board_BA"
 				(path "/fd7503bc-e7fc-4766-b224-3d1c3d7de5ff/1b181806-12f4-40c8-bf91-78ac0d892dab/d6c6031d-c1b3-49bb-af8f-093ee0f25456"
-					(reference "C153")
+					(reference "C148")
 					(unit 1)
 				)
@@
 		(dnp no)
 		(fields_autoplaced yes)
-		(property "Reference" "#PWR0237"
+		(property "Reference" "#PWR0249"
 			(at 229.87 73.66 0)
 			(effects
@@
 			(project "FPGA_Board_BA"
 				(path "/fd7503bc-e7fc-4766-b224-3d1c3d7de5ff/1b181806-12f4-40c8-bf91-78ac0d892dab/d6c6031d-c1b3-49bb-af8f-093ee0f25456"
-					(reference "#PWR0237")
+					(reference "#PWR0249")
 					(unit 1)
 				)
@@
 		(dnp no)
 		(fields_autoplaced yes)
-		(property "Reference" "C154"
+		(property "Reference" "C149"
 			(at 212.09 54.61 90)
 			(effects
@@
 			(project "FPGA_Board_BA"
 				(path "/fd7503bc-e7fc-4766-b224-3d1c3d7de5ff/1b181806-12f4-40c8-bf91-78ac0d892dab/d6c6031d-c1b3-49bb-af8f-093ee0f25456"
-					(reference "C154")
+					(reference "C149")
 					(unit 1)
 				)
@@
 		(dnp no)
 		(fields_autoplaced yes)
-		(property "Reference" "#PWR0231"
+		(property "Reference" "#PWR0243"
 			(at 110.49 43.18 0)
 			(effects
@@
 			(project "FPGA_Board_BA"
 				(path "/fd7503bc-e7fc-4766-b224-3d1c3d7de5ff/1b181806-12f4-40c8-bf91-78ac0d892dab/d6c6031d-c1b3-49bb-af8f-093ee0f25456"
-					(reference "#PWR0231")
+					(reference "#PWR0243")
 					(unit 1)
 				)
@@
 		(dnp no)
 		(fields_autoplaced yes)
-		(property "Reference" "#PWR0236"
+		(property "Reference" "#PWR0248"
 			(at 214.63 127 0)
 			(effects
@@
 			(project "FPGA_Board_BA"
 				(path "/fd7503bc-e7fc-4766-b224-3d1c3d7de5ff/1b181806-12f4-40c8-bf91-78ac0d892dab/d6c6031d-c1b3-49bb-af8f-093ee0f25456"
-					(reference "#PWR0236")
-					(unit 1)
-				)
+					(reference "#PWR0248")
+					(unit 1)
+				)
