File: FPGA_Board_BA/PCB/power_from_chb.kicad_sch (KiCad schematic)
At the start: 0 parts

Commit message: some stuff
Parts:
- added J716, J717, J718, J720: Plug_Terminal_2x12pin, MYLIB_Misc:DMCV 1,5_12-G1F-3,5-LR P20THR, symbol MYLIB_Misc:Plug_Terminal_2x12pin
Connections:
- net PH_B1: now also J716.1
- net Ph_A1: now also J720.1
- net Ph_A2: now also J720.24
- net Ph_B2: now also J716.24
- net Ph_C2: now also J717.24
- net Ph_D2: now also J718.24
- new net: J720.10, J720.11
- new net: J720.12, J720.13
- new net: J720.14, J720.15
- new net: J720.16, J720.17
- new net: J720.18, J720.19
- new net: J720.2, J720.3
- new net: J720.20, J720.21
- new net: J720.22, J720.23
- new net: J720.4, J720.5
- new net: J720.6, J720.7
- new net: J720.8, J720.9
- new net: J718.10, J718.11
- new net: J718.12, J718.13
- new net: J718.14, J718.15
- new net: J718.16, J718.17
- new net: J718.18, J718.19
- new net: J718.2, J718.3
- new net: J718.20, J718.21
- new net: J718.22, J718.23
- new net: J718.4, J718.5
- new net: J718.6, J718.7
- new net: J718.8, J718.9
- new net: J717.10, J717.11
- new net: J717.12, J717.13
- new net: J717.14, J717.15
- new net: J717.16, J717.17
- new net: J717.18, J717.19
- new net: J717.2, J717.3
- new net: J717.20, J717.21
- new net: J717.22, J717.23
- new net: J717.4, J717.5
- new net: J717.6, J717.7
- new net: J717.8, J717.9
- new net: J716.10, J716.11
- new net: J716.12, J716.13
- new net: J716.14, J716.15
- new net: J716.16, J716.17
- new net: J716.18, J716.19
- new net: J716.2, J716.3
- new net: J716.20, J716.21
- new net: J716.22, J716.23
- new net: J716.4, J716.5
- new net: J716.6, J716.7
- new net: J716.8, J716.9
- new net PH_C1: J717.1
- new net PH_D1: J718.1
Other:
- removed sheet CHB Phase B
- removed sheet CHB Phase C
- removed sheet CHB Phase D
- removed sheet CHB_Phase_A
- note added: "Even side: Out1 Odd side: Out2"

Commit message: Besprechung mit Leo
Parts:
- added J701: Box_Header_6pin, Connector_IDC:IDC-Header_2x03_P2.54mm_Vertical, symbol MYLIB_Misc:Box_Header_6pin
Changed lines of the file:
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@@
+		)
+	)
+	(symbol
+		(lib_id "MYLIB_Misc:Box_Header_6pin")
+		(at 193.04 69.85 0)
+		(unit 1)
+		(exclude_from_sim no)
+		(in_bom yes)
+		(on_board yes)
+		(dnp no)
+		(fields_autoplaced yes)
+		(property "Reference" "J701"
+			(at 193.04 59.69 0)
+			(effects
+				(font
+					(size 1.27 1.27)
+				)
+			)
+		)
+		(property "Value" "Box_Header_6pin"
+			(at 193.04 62.23 0)
+			(effects
+				(font
+					(size 1.27 1.27)
+				)
+			)
+		)
+		(property "Footprint" "Connector_IDC:IDC-Header_2x03_P2.54mm_Vertical"
+			(at 189.484 52.832 0)
+			(effects
+				(font
+					(size 1.27 1.27)
+				)
+				(hide yes)
+			)
+		)
+		(property "Datasheet" "https://www.reichelt.de/de/de/shop/produkt/wannenstecker_6-polig_gewinkelt-105978"
+			(at 193.04 55.626 0)
+			(effects
+				(font
+					(size 1.27 1.27)
+				)
+				(hide yes)
+			)
+		)
+		(property "Description" "Wannenstecker 6pin, THT Vertikal"
+			(at 193.802 57.912 0)
+			(effects
+				(font
+					(size 1.27 1.27)
+				)
+				(hide yes)
+			)
+		)
+		(pin "4"
+		)
+		(pin "2"
+		)
+		(pin "5"
+		)
+		(pin "3"
+		)
+		(pin "1"
+		)
+		(pin "6"
+		)
+		(instances
+			(project ""
+				(path "/fd7503bc-e7fc-4766-b224-3d1c3d7de5ff/e884b539-4fb2-499d-8c9d-64645c35288e"
+					(reference "J701")
+					(unit 1)
+				)
+			)
 		)
 	)

Commit message: work
Parts:
- renumbered J720 to J4, J717 to J5, J716 to J6, J718 to J7, J701 to J8
Changed lines of the file:
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@@
 		(dnp no)
 		(fields_autoplaced yes)
-		(property "Reference" "J720"
+		(property "Reference" "J4"
 			(at 105.41 49.53 0)
 			(effects
@@
 			(project ""
 				(path "/fd7503bc-e7fc-4766-b224-3d1c3d7de5ff/e884b539-4fb2-499d-8c9d-64645c35288e"
-					(reference "J720")
+					(reference "J4")
 					(unit 1)
 				)
@@
 		(dnp no)
 		(fields_autoplaced yes)
-		(property "Reference" "J718"
+		(property "Reference" "J7"
 			(at 154.94 90.17 0)
 			(effects
@@
 			(project "FPGA_Board_BA"
 				(path "/fd7503bc-e7fc-4766-b224-3d1c3d7de5ff/e884b539-4fb2-499d-8c9d-64645c35288e"
-					(reference "J718")
+					(reference "J7")
 					(unit 1)
 				)
@@
 		(dnp no)
 		(fields_autoplaced yes)
-		(property "Reference" "J717"
+		(property "Reference" "J5"
 			(at 105.41 90.17 0)
 			(effects
@@
 			(project "FPGA_Board_BA"
 				(path "/fd7503bc-e7fc-4766-b224-3d1c3d7de5ff/e884b539-4fb2-499d-8c9d-64645c35288e"
-					(reference "J717")
+					(reference "J5")
 					(unit 1)
 				)
@@
 		(dnp no)
 		(fields_autoplaced yes)
-		(property "Reference" "J716"
+		(property "Reference" "J6"
 			(at 154.94 49.53 0)
 			(effects
@@
 			(project "FPGA_Board_BA"
 				(path "/fd7503bc-e7fc-4766-b224-3d1c3d7de5ff/e884b539-4fb2-499d-8c9d-64645c35288e"
-					(reference "J716")
+					(reference "J6")
 					(unit 1)
 				)
@@
 		(dnp no)
 		(fields_autoplaced yes)
-		(property "Reference" "J701"
+		(property "Reference" "J8"
 			(at 193.04 59.69 0)
 			(effects
@@
 			(project ""
 				(path "/fd7503bc-e7fc-4766-b224-3d1c3d7de5ff/e884b539-4fb2-499d-8c9d-64645c35288e"
-					(reference "J701")
+					(reference "J8")
 					(unit 1)
 				)

Commit message: 22.11
Parts:
- removed J4, J5, J6, J7: Plug_Terminal_2x12pin, MYLIB_Misc:DMCV 1,5_12-G1F-3,5-LR P20THR, symbol MYLIB_Misc:Plug_Terminal_2x12pin
- added J6, J7, J8: Box_Header_6pin, Connector_IDC:IDC-Header_2x03_P2.54mm_Vertical, symbol MYLIB_Misc:Box_Header_6pin
- renumbered J8 to J5
Connections:
- net PH_B1: now also J6.1 (Pin_1), J6.3 (Pin_3), J6.5 (Pin_5)
- net PH_C1: now also J7.1 (Pin_1), J7.3 (Pin_3), J7.5 (Pin_5)
- net PH_D1: now also J8.1 (Pin_1), J8.3 (Pin_3), J8.5 (Pin_5)
- net Ph_A2: now also J5.2 (Pin_2), J5.4 (Pin_4), J5.6 (Pin_6)
- net Ph_B2: now also J6.2 (Pin_2), J6.4 (Pin_4), J6.6 (Pin_6)
- net Ph_C2: now also J7.2 (Pin_2), J7.4 (Pin_4), J7.6 (Pin_6)
- net Ph_D2: now also J8.2 (Pin_2), J8.4 (Pin_4), J8.6 (Pin_6)
- net PH_A1: now reaches J5.1 (Pin_1)
- net PH_A1: now also J5.3 (Pin_3), J5.5 (Pin_5)
Other:
- note added: "Wannenstecker für CHB outputs"
- note removed: "Even side: Out1 Odd side: Out2"
- moved on the sheet: J5
