File: FPGA_Board_BA/PCB/FPGA_Board_BA.kicad_pcb (KiCad board)
At the start: 2 copper layers, 140 parts, among them J103 Plug_Termincal_8pin, J1101 Molex_Mini_Fit_Jr_2x08pin, J1201 Plug_Terminal_2x12pin, J1202 Plug_Terminal_2x12pin, J1203 Box_Header_6pin, J1204 Box_Header_6pin, J1205 Box_Header_6pin, J1206 Box_Header_6pin, J1401 Plug_Terminal_2x12pin, J1402 Plug_Terminal_2x12pin, J1403 Plug_Terminal_2x12pin, J1404 Plug_Terminal_2x12pin, J601 Banana_Socket_Black, J602 Banana_Socket_Red, J716 Plug_Terminal_2x12pin, J717 Plug_Terminal_2x12pin, J718 Plug_Terminal_2x12pin, J720 Plug_Terminal_2x12pin, Q501 IPT017N12NM6, Q502 IPT017N12NM6, Q503 IPT017N12NM6, Q504 IPT017N12NM6, SW1201 TL3305BF100QG, SW1202 TL3305BF100QG, U1001 BOOSTXL-3PHGANINV, U201 LTC2320-16_LVDS, U301 Zynq7020, U401 AMC0300D, U402 AMC0300D, U403 AMC0300D, U501 LM5143, U801 TPS61022, U802 MCP1703AT-5002EDB

Commit message: lot of work
Parts:
- removed D901, D902: B72590D50H160, Capacitor_SMD:C_0402_1005Metric_Pad0.74x0.62mm_HandSolder
- removed J1401, J1402, J1404: Plug_Terminal_2x12pin, MYLIB_Misc:DMCV 1,5_12-G1F-3,5-LR P20THR
- removed R903: 100k_0603, Resistor_SMD:R_0603_1608Metric
- added C1301: 10u_1210, WLIB_Capacitor:C_1210, F.Cu at (141.6, 173.9)
- added C1302: 10u_1210, WLIB_Capacitor:C_1210, F.Cu at (141.6, 178.1)
- added C1303: 10u_1210, WLIB_Capacitor:C_1210, F.Cu at (141.6, 182.4)
- added C1304: 10u_1210, WLIB_Capacitor:C_1210, F.Cu at (141.6, 186.6)
- added C1601: 15p_0603, WLIB_Capacitor:C_0603, F.Cu at (216.4, 116.4)
- added C1602: 15p_0603, WLIB_Capacitor:C_0603, F.Cu at (131.4, 193.3)
- added C1603: 15p_0603, WLIB_Capacitor:C_0603, F.Cu at (131.4, 195.8)
- added C1604: 15p_0603, WLIB_Capacitor:C_0603, F.Cu at (216.4, 118.9)
- added C1605: 100n_0603, WLIB_Capacitor:C_0603, F.Cu at (131.4, 198.3)
- added C1606: 15p_0603, WLIB_Capacitor:C_0603, F.Cu at (216.4, 121.4)
- added C1607: 100n_0603, WLIB_Capacitor:C_0603, F.Cu at (216.4, 123.9)
- added C1608: 100n_0603, WLIB_Capacitor:C_0603, F.Cu at (216.4, 126.4)
- added C1701: 15p_0603, WLIB_Capacitor:C_0603, F.Cu at (216.4, 167.6)
- added C1702: 15p_0603, WLIB_Capacitor:C_0603, F.Cu at (216.4, 170.1)
- added C1703: 15p_0603, WLIB_Capacitor:C_0603, F.Cu at (216.4, 172.6)
- added C1704: 100n_0603, WLIB_Capacitor:C_0603, F.Cu at (216.4, 175.1)
- added C1705: 100n_0603, WLIB_Capacitor:C_0603, F.Cu at (216.4, 177.6)
- added C1706: 15p_0603, WLIB_Capacitor:C_0603, F.Cu at (161.3, 92.8)
- added C1707: 15p_0603, WLIB_Capacitor:C_0603, F.Cu at (161.3, 95.3)
- added C1708: 15p_0603, WLIB_Capacitor:C_0603, F.Cu at (161.3, 97.8)
- added C1709: 100n_0603, WLIB_Capacitor:C_0603, F.Cu at (161.3, 100.3)
- added C1710: 100n_0603, WLIB_Capacitor:C_0603, F.Cu at (161.3, 102.8)
- added C1801: 15p_0603, WLIB_Capacitor:C_0603, F.Cu at (142.4, 92.8)
- added C1801: 15p_0603, WLIB_Capacitor:C_0603, F.Cu at (254.1, 116.4)
- added C1802: 15p_0603, WLIB_Capacitor:C_0603, F.Cu at (142.4, 95.3)
- added C1802: 15p_0603, WLIB_Capacitor:C_0603, F.Cu at (254.1, 118.9)
- added C1803: 15p_0603, WLIB_Capacitor:C_0603, F.Cu at (142.4, 97.8)
- added C1803: 15p_0603, WLIB_Capacitor:C_0603, F.Cu at (254.1, 121.4)
- added C1804: 100n_0603, WLIB_Capacitor:C_0603, F.Cu at (254.1, 123.9)
- added C1804: 100n_0603, WLIB_Capacitor:C_0603, F.Cu at (142.4, 100.3)
- added C1805: 100n_0603, WLIB_Capacitor:C_0603, F.Cu at (142.4, 102.8)
- added C1805: 100n_0603, WLIB_Capacitor:C_0603, F.Cu at (254.1, 126.4)
- added C1901: 15p_0603, WLIB_Capacitor:C_0603, F.Cu at (235.3, 116.4)
- added C1902: 15p_0603, WLIB_Capacitor:C_0603, F.Cu at (235.3, 118.9)
- added C1903: 15p_0603, WLIB_Capacitor:C_0603, F.Cu at (235.3, 121.4)
- added C1904: 100n_0603, WLIB_Capacitor:C_0603, F.Cu at (235.3, 123.9)
- added C1905: 100n_0603, WLIB_Capacitor:C_0603, F.Cu at (235.3, 126.4)
- added C2001: 15p_0603, WLIB_Capacitor:C_0603, F.Cu at (273.0, 116.4)
- added C2002: 15p_0603, WLIB_Capacitor:C_0603, F.Cu at (273.0, 118.9)
- added C2003: 15p_0603, WLIB_Capacitor:C_0603, F.Cu at (273.0, 121.4)
- added C2004: 100n_0603, WLIB_Capacitor:C_0603, F.Cu at (273.0, 123.9)
- added C2005: 100n_0603, WLIB_Capacitor:C_0603, F.Cu at (273.0, 126.4)
- added C2006: 15p_0603, WLIB_Capacitor:C_0603, F.Cu at (216.4, 133.5)
- added C2007: 15p_0603, WLIB_Capacitor:C_0603, F.Cu at (216.4, 136.0)
- added C2008: 15p_0603, WLIB_Capacitor:C_0603, F.Cu at (216.4, 138.5)
- added C2009: 100n_0603, WLIB_Capacitor:C_0603, F.Cu at (216.4, 141.0)
- added C2010: 100n_0603, WLIB_Capacitor:C_0603, F.Cu at (216.4, 143.5)
- added C2011: 15p_0603, WLIB_Capacitor:C_0603, F.Cu at (216.4, 150.5)
- added C2012: 15p_0603, WLIB_Capacitor:C_0603, F.Cu at (216.4, 153.0)
- added C2013: 15p_0603, WLIB_Capacitor:C_0603, F.Cu at (216.4, 155.5)
- added C2014: 100n_0603, WLIB_Capacitor:C_0603, F.Cu at (216.4, 158.0)
- added C2015: 100n_0603, WLIB_Capacitor:C_0603, F.Cu at (216.4, 160.6)
- added C2501: 15p_0603, WLIB_Capacitor:C_0603, F.Cu at (235.3, 133.5)
- added C2502: 15p_0603, WLIB_Capacitor:C_0603, F.Cu at (235.3, 136.0)
- added C2503: 15p_0603, WLIB_Capacitor:C_0603, F.Cu at (235.3, 138.5)
- added C2504: 100n_0603, WLIB_Capacitor:C_0603, F.Cu at (235.3, 141.0)
- added C2505: 100n_0603, WLIB_Capacitor:C_0603, F.Cu at (235.3, 143.5)
- added C2601: 15p_0603, WLIB_Capacitor:C_0603, F.Cu at (273.0, 133.5)
- added C2602: 15p_0603, WLIB_Capacitor:C_0603, F.Cu at (273.0, 136.0)
- added C2603: 15p_0603, WLIB_Capacitor:C_0603, F.Cu at (273.0, 138.5)
- added C2604: 100n_0603, WLIB_Capacitor:C_0603, F.Cu at (273.0, 141.0)
- added C2605: 100n_0603, WLIB_Capacitor:C_0603, F.Cu at (273.0, 143.5)
- added C2701: 15p_0603, WLIB_Capacitor:C_0603, F.Cu at (235.3, 150.5)
- added C2702: 15p_0603, WLIB_Capacitor:C_0603, F.Cu at (235.3, 153.0)
- added C2703: 15p_0603, WLIB_Capacitor:C_0603, F.Cu at (235.3, 155.5)
- added C2704: 100n_0603, WLIB_Capacitor:C_0603, F.Cu at (235.3, 158.0)
- added C2705: 100n_0603, WLIB_Capacitor:C_0603, F.Cu at (235.3, 160.6)
- added C2801: 15p_0603, WLIB_Capacitor:C_0603, F.Cu at (254.1, 133.5)
- added C2802: 15p_0603, WLIB_Capacitor:C_0603, F.Cu at (254.1, 136.0)
- added C2803: 15p_0603, WLIB_Capacitor:C_0603, F.Cu at (254.1, 138.5)
- added C2804: 100n_0603, WLIB_Capacitor:C_0603, F.Cu at (254.1, 141.0)
- added C2805: 100n_0603, WLIB_Capacitor:C_0603, F.Cu at (254.1, 143.5)
- added C2901: 15p_0603, WLIB_Capacitor:C_0603, F.Cu at (273.0, 150.5)
- added C2902: 15p_0603, WLIB_Capacitor:C_0603, F.Cu at (273.0, 153.0)
- added C2903: 15p_0603, WLIB_Capacitor:C_0603, F.Cu at (273.0, 155.5)
- added C2904: 100n_0603, WLIB_Capacitor:C_0603, F.Cu at (273.0, 158.0)
- added C2905: 100n_0603, WLIB_Capacitor:C_0603, F.Cu at (273.0, 160.6)
- added C3001: 15p_0603, WLIB_Capacitor:C_0603, F.Cu at (235.3, 167.6)
- added C3002: 15p_0603, WLIB_Capacitor:C_0603, F.Cu at (235.3, 170.1)
- added C3003: 15p_0603, WLIB_Capacitor:C_0603, F.Cu at (235.3, 172.6)
- added C3004: 100n_0603, WLIB_Capacitor:C_0603, F.Cu at (235.3, 175.1)
- added C3005: 100n_0603, WLIB_Capacitor:C_0603, F.Cu at (235.3, 177.6)
- added C3101: 15p_0603, WLIB_Capacitor:C_0603, F.Cu at (254.1, 150.5)
- added C3102: 15p_0603, WLIB_Capacitor:C_0603, F.Cu at (254.1, 153.0)
- added C3103: 15p_0603, WLIB_Capacitor:C_0603, F.Cu at (254.1, 155.5)
- added C3104: 100n_0603, WLIB_Capacitor:C_0603, F.Cu at (254.1, 158.0)
- added C3105: 100n_0603, WLIB_Capacitor:C_0603, F.Cu at (254.1, 160.6)
- added C3202: 15p_0603, WLIB_Capacitor:C_0603, F.Cu at (131.4, 200.9)
- added C3204: 100n_0603, WLIB_Capacitor:C_0603, F.Cu at (131.4, 203.4)
- added C3206: 15p_0603, WLIB_Capacitor:C_0603, F.Cu at (254.1, 167.6)
- added C3207: 15p_0603, WLIB_Capacitor:C_0603, F.Cu at (254.1, 170.1)
- added C3208: 15p_0603, WLIB_Capacitor:C_0603, F.Cu at (254.1, 172.6)
- added C3209: 100n_0603, WLIB_Capacitor:C_0603, F.Cu at (254.1, 175.1)
- added C3210: 100n_0603, WLIB_Capacitor:C_0603, F.Cu at (254.1, 177.6)
- added J1207: Box_Header_26pin, Connector_IDC:IDC-Header_2x13_P2.54mm_Vertical, F.Cu at (165.4, 52.9)
- added J1208: Box_Header_26pin, Connector_IDC:IDC-Header_2x13_P2.54mm_Vertical, F.Cu at (177.4, 52.9)
- added J1301: PinHeader_03_male, Connector_PinHeader_2.54mm:PinHeader_1x03_P2.54mm_Vertical, F.Cu at (156.0, 174.1)
- added J201: PinHeader_03_male, Connector_PinHeader_2.54mm:PinHeader_1x03_P2.54mm_Vertical, F.Cu at (134.2, 174.1)
- added J701: Box_Header_6pin, Connector_IDC:IDC-Header_2x03_P2.54mm_Vertical, F.Cu at (71.3, 129.0)
- added R101: 0R100_2512, Resistor_SMD:R_2512_6332Metric_Pad1.40x3.35mm_HandSolder, F.Cu at (197.6, 176.0)
- added R1601: 30R_0603, Resistor_SMD:R_0603_1608Metric, F.Cu at (212.2, 116.4)
- added R1602: 500R_0603, Resistor_SMD:R_0603_1608Metric, F.Cu at (127.2, 193.3)
- added R1603: 30R_0603, Resistor_SMD:R_0603_1608Metric, F.Cu at (212.2, 118.9)
- added R1604: 30R_0603, Resistor_SMD:R_0603_1608Metric, F.Cu at (127.2, 195.8)
- added R1605: 500R_0603, Resistor_SMD:R_0603_1608Metric, F.Cu at (212.2, 121.4)
- added R1606: 5k1_0603, Resistor_SMD:R_0603_1608Metric, F.Cu at (127.2, 198.3)
- added R1607: 5k1_0603, Resistor_SMD:R_0603_1608Metric, F.Cu at (212.2, 123.9)
- added R1608: 500R_0603, Resistor_SMD:R_0603_1608Metric, F.Cu at (212.2, 126.4)
- added R1609: 5k1_0603, Resistor_SMD:R_0603_1608Metric, F.Cu at (212.2, 128.9)
- added R1701: 30R_0603, Resistor_SMD:R_0603_1608Metric, F.Cu at (212.2, 167.6)
- added R1702: 30R_0603, Resistor_SMD:R_0603_1608Metric, F.Cu at (212.2, 170.1)
- added R1703: 500R_0603, Resistor_SMD:R_0603_1608Metric, F.Cu at (212.2, 172.6)
- added R1704: 5k1_0603, Resistor_SMD:R_0603_1608Metric, F.Cu at (212.2, 175.1)
- added R1705: 500R_0603, Resistor_SMD:R_0603_1608Metric, F.Cu at (212.2, 177.6)
- added R1706: 5k1_0603, Resistor_SMD:R_0603_1608Metric, F.Cu at (212.2, 180.1)
- added R1707: 30R_0603, Resistor_SMD:R_0603_1608Metric, F.Cu at (157.1, 92.8)
- added R1708: 30R_0603, Resistor_SMD:R_0603_1608Metric, F.Cu at (157.1, 95.3)
- added R1709: 500R_0603, Resistor_SMD:R_0603_1608Metric, F.Cu at (157.1, 97.8)
- added R1710: 5k1_0603, Resistor_SMD:R_0603_1608Metric, F.Cu at (157.1, 100.3)
- added R1711: 500R_0603, Resistor_SMD:R_0603_1608Metric, F.Cu at (157.1, 102.8)
- added R1712: 5k1_0603, Resistor_SMD:R_0603_1608Metric, F.Cu at (157.1, 105.3)
- added R1801: 30R_0603, Resistor_SMD:R_0603_1608Metric, F.Cu at (138.2, 92.8)
- added R1801: 30R_0603, Resistor_SMD:R_0603_1608Metric, F.Cu at (249.9, 116.4)
- added R1802: 30R_0603, Resistor_SMD:R_0603_1608Metric, F.Cu at (249.9, 118.9)
- added R1802: 30R_0603, Resistor_SMD:R_0603_1608Metric, F.Cu at (138.2, 95.3)
- added R1803: 500R_0603, Resistor_SMD:R_0603_1608Metric, F.Cu at (138.2, 97.8)
- added R1803: 500R_0603, Resistor_SMD:R_0603_1608Metric, F.Cu at (249.9, 121.4)
- added R1804: 5k1_0603, Resistor_SMD:R_0603_1608Metric, F.Cu at (138.2, 100.3)
- added R1804: 5k1_0603, Resistor_SMD:R_0603_1608Metric, F.Cu at (249.9, 123.9)
- added R1805: 500R_0603, Resistor_SMD:R_0603_1608Metric, F.Cu at (138.2, 102.8)
- added R1805: 500R_0603, Resistor_SMD:R_0603_1608Metric, F.Cu at (249.9, 126.4)
- added R1806: 5k1_0603, Resistor_SMD:R_0603_1608Metric, F.Cu at (249.9, 128.9)
- added R1806: 5k1_0603, Resistor_SMD:R_0603_1608Metric, F.Cu at (138.2, 105.3)
- added R1901: 30R_0603, Resistor_SMD:R_0603_1608Metric, F.Cu at (231.1, 116.4)
- added R1902: 30R_0603, Resistor_SMD:R_0603_1608Metric, F.Cu at (231.1, 118.9)
- added R1903: 500R_0603, Resistor_SMD:R_0603_1608Metric, F.Cu at (231.1, 121.4)
- added R1904: 5k1_0603, Resistor_SMD:R_0603_1608Metric, F.Cu at (231.1, 123.9)
- added R1905: 500R_0603, Resistor_SMD:R_0603_1608Metric, F.Cu at (231.1, 126.4)
- added R1906: 5k1_0603, Resistor_SMD:R_0603_1608Metric, F.Cu at (231.1, 128.9)
- added R2001: 30R_0603, Resistor_SMD:R_0603_1608Metric, F.Cu at (268.8, 116.4)
- added R2002: 30R_0603, Resistor_SMD:R_0603_1608Metric, F.Cu at (268.8, 118.9)
- added R2003: 500R_0603, Resistor_SMD:R_0603_1608Metric, F.Cu at (268.8, 121.4)
- added R2004: 5k1_0603, Resistor_SMD:R_0603_1608Metric, F.Cu at (268.8, 123.9)
- added R2005: 500R_0603, Resistor_SMD:R_0603_1608Metric, F.Cu at (268.8, 126.4)
- added R2006: 5k1_0603, Resistor_SMD:R_0603_1608Metric, F.Cu at (268.8, 128.9)
- added R2007: 30R_0603, Resistor_SMD:R_0603_1608Metric, F.Cu at (212.2, 133.5)
- added R2008: 30R_0603, Resistor_SMD:R_0603_1608Metric, F.Cu at (212.2, 136.0)
- added R2009: 500R_0603, Resistor_SMD:R_0603_1608Metric, F.Cu at (212.2, 138.5)
- added R2010: 5k1_0603, Resistor_SMD:R_0603_1608Metric, F.Cu at (212.2, 141.0)
- added R2011: 500R_0603, Resistor_SMD:R_0603_1608Metric, F.Cu at (212.2, 143.5)
- added R2012: 5k1_0603, Resistor_SMD:R_0603_1608Metric, F.Cu at (212.2, 146.0)
- added R2013: 30R_0603, Resistor_SMD:R_0603_1608Metric, F.Cu at (212.2, 150.5)
- added R2014: 30R_0603, Resistor_SMD:R_0603_1608Metric, F.Cu at (212.2, 153.0)
- added R2015: 500R_0603, Resistor_SMD:R_0603_1608Metric, F.Cu at (212.2, 155.5)
- added R2016: 5k1_0603, Resistor_SMD:R_0603_1608Metric, F.Cu at (212.2, 158.0)
- added R2017: 500R_0603, Resistor_SMD:R_0603_1608Metric, F.Cu at (212.2, 160.6)
- added R2018: 5k1_0603, Resistor_SMD:R_0603_1608Metric, F.Cu at (212.2, 163.1)
- added R2501: 30R_0603, Resistor_SMD:R_0603_1608Metric, F.Cu at (231.1, 133.5)
- added R2502: 30R_0603, Resistor_SMD:R_0603_1608Metric, F.Cu at (231.1, 136.0)
- added R2503: 500R_0603, Resistor_SMD:R_0603_1608Metric, F.Cu at (231.1, 138.5)
- added R2504: 5k1_0603, Resistor_SMD:R_0603_1608Metric, F.Cu at (231.1, 141.0)
- added R2505: 500R_0603, Resistor_SMD:R_0603_1608Metric, F.Cu at (231.1, 143.5)
- added R2506: 5k1_0603, Resistor_SMD:R_0603_1608Metric, F.Cu at (231.1, 146.0)
- added R2601: 30R_0603, Resistor_SMD:R_0603_1608Metric, F.Cu at (268.8, 133.5)
- added R2602: 30R_0603, Resistor_SMD:R_0603_1608Metric, F.Cu at (268.8, 136.0)
- added R2603: 500R_0603, Resistor_SMD:R_0603_1608Metric, F.Cu at (268.8, 138.5)
- added R2604: 5k1_0603, Resistor_SMD:R_0603_1608Metric, F.Cu at (268.8, 141.0)
- added R2605: 500R_0603, Resistor_SMD:R_0603_1608Metric, F.Cu at (268.8, 143.5)
- added R2606: 5k1_0603, Resistor_SMD:R_0603_1608Metric, F.Cu at (268.8, 146.0)
- added R2701: 30R_0603, Resistor_SMD:R_0603_1608Metric, F.Cu at (231.1, 150.5)
- added R2702: 30R_0603, Resistor_SMD:R_0603_1608Metric, F.Cu at (231.1, 153.0)
- added R2703: 500R_0603, Resistor_SMD:R_0603_1608Metric, F.Cu at (231.1, 155.5)
- added R2704: 5k1_0603, Resistor_SMD:R_0603_1608Metric, F.Cu at (231.1, 158.0)
- added R2705: 500R_0603, Resistor_SMD:R_0603_1608Metric, F.Cu at (231.1, 160.6)
- added R2706: 5k1_0603, Resistor_SMD:R_0603_1608Metric, F.Cu at (231.1, 163.1)
- added R2801: 30R_0603, Resistor_SMD:R_0603_1608Metric, F.Cu at (249.9, 133.5)
- added R2802: 30R_0603, Resistor_SMD:R_0603_1608Metric, F.Cu at (249.9, 136.0)
- added R2803: 500R_0603, Resistor_SMD:R_0603_1608Metric, F.Cu at (249.9, 138.5)
- added R2804: 5k1_0603, Resistor_SMD:R_0603_1608Metric, F.Cu at (249.9, 141.0)
- added R2805: 500R_0603, Resistor_SMD:R_0603_1608Metric, F.Cu at (249.9, 143.5)
- added R2806: 5k1_0603, Resistor_SMD:R_0603_1608Metric, F.Cu at (249.9, 146.0)
- added R2901: 30R_0603, Resistor_SMD:R_0603_1608Metric, F.Cu at (268.8, 150.5)
- added R2902: 30R_0603, Resistor_SMD:R_0603_1608Metric, F.Cu at (268.8, 153.0)
- added R2903: 500R_0603, Resistor_SMD:R_0603_1608Metric, F.Cu at (268.8, 155.5)
- added R2904: 5k1_0603, Resistor_SMD:R_0603_1608Metric, F.Cu at (268.8, 158.0)
- added R2905: 500R_0603, Resistor_SMD:R_0603_1608Metric, F.Cu at (268.8, 160.6)
- added R2906: 5k1_0603, Resistor_SMD:R_0603_1608Metric, F.Cu at (268.8, 163.1)
- added R3001: 30R_0603, Resistor_SMD:R_0603_1608Metric, F.Cu at (231.1, 167.6)
- added R3002: 30R_0603, Resistor_SMD:R_0603_1608Metric, F.Cu at (231.1, 170.1)
- added R3003: 500R_0603, Resistor_SMD:R_0603_1608Metric, F.Cu at (231.1, 172.6)
- added R3004: 5k1_0603, Resistor_SMD:R_0603_1608Metric, F.Cu at (231.1, 175.1)
- added R3005: 500R_0603, Resistor_SMD:R_0603_1608Metric, F.Cu at (231.1, 177.6)
- added R3006: 5k1_0603, Resistor_SMD:R_0603_1608Metric, F.Cu at (231.1, 180.1)
- added R3101: 30R_0603, Resistor_SMD:R_0603_1608Metric, F.Cu at (249.9, 150.5)
- added R3102: 30R_0603, Resistor_SMD:R_0603_1608Metric, F.Cu at (249.9, 153.0)
- added R3103: 500R_0603, Resistor_SMD:R_0603_1608Metric, F.Cu at (249.9, 155.5)
- added R3104: 5k1_0603, Resistor_SMD:R_0603_1608Metric, F.Cu at (249.9, 158.0)
- added R3105: 500R_0603, Resistor_SMD:R_0603_1608Metric, F.Cu at (249.9, 160.6)
- added R3106: 5k1_0603, Resistor_SMD:R_0603_1608Metric, F.Cu at (249.9, 163.1)
- added R3202: 30R_0603, Resistor_SMD:R_0603_1608Metric, F.Cu at (127.2, 200.9)
- added R3203: 500R_0603, Resistor_SMD:R_0603_1608Metric, F.Cu at (127.2, 203.4)
- added R3206: 5k1_0603, Resistor_SMD:R_0603_1608Metric, F.Cu at (127.2, 205.9)
- added R3207: 30R_0603, Resistor_SMD:R_0603_1608Metric, F.Cu at (249.9, 167.6)
- added R3208: 30R_0603, Resistor_SMD:R_0603_1608Metric, F.Cu at (249.9, 170.1)
- added R3209: 500R_0603, Resistor_SMD:R_0603_1608Metric, F.Cu at (249.9, 172.6)
- added R3210: 5k1_0603, Resistor_SMD:R_0603_1608Metric, F.Cu at (249.9, 175.1)
- added R3211: 500R_0603, Resistor_SMD:R_0603_1608Metric, F.Cu at (249.9, 177.6)
- added R3212: 5k1_0603, Resistor_SMD:R_0603_1608Metric, F.Cu at (249.9, 180.1)
- added R904: 100R_0603, Resistor_SMD:R_0603_1608Metric, F.Cu at (16.0, 183.2)
- added R905: 100R_0603, Resistor_SMD:R_0603_1608Metric, F.Cu at (16.0, 185.8)
- added U101: HV_Probe, MYLIB_Misc:HV_Probe, F.Cu at (107.3, 27.3)
- added U1301: LTC2320-16_LVDS, MYLIB_chips:UKG_52_7mm_8mm, F.Cu at (148.9, 172.5)
- added U1501: HV_Probe, MYLIB_Misc:HV_Probe, F.Cu at (107.3, 50.5)
- added U1502: HV_Probe, MYLIB_Misc:HV_Probe, F.Cu at (107.3, 73.6)
- added U1503: HV_Probe, MYLIB_Misc:HV_Probe, F.Cu at (107.3, 96.7)
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Connections:
- net /ADC/CLK_IN renamed /ADC for B6/CLK_IN
- net /ADC/CLK_OUT renamed /ADC for B6/CLK_OUT
- net /ADC/SDO1 renamed /ADC for B6/SDO1
- net /ADC/SDO2 renamed /ADC for B6/SDO2
- net /ADC/SDO3 renamed /ADC for B6/SDO3
- net /ADC/SDO4 renamed /ADC for B6/SDO4
- net /ADC/SDO5 renamed /ADC for B6/SDO5
- net /ADC/SDO6 renamed /ADC for B6/SDO6
- net /ADC/SDO7 renamed /ADC for B6/SDO7
- net /ADC/SDO8 renamed /ADC for B6/SDO8
- net /ADC/~{CNV} renamed /ADC for B6/~{CNV}
- J1201 pad 1: +5V -> GND
- J1201 pad 10: +5V -> /CHB Communication/Ph_A_Tx5
- J1201 pad 11: +5V -> GND
- J1201 pad 12: +5V -> /CHB Communication/Ph_A_Tx6
- J1201 pad 13: +5V -> GND
- J1201 pad 14: +5V -> /CHB Communication/Ph_A_Tx7
- J1201 pad 15: +5V -> GND
- J1201 pad 16: +5V -> /CHB Communication/Ph_A_Tx8
- J1201 pad 17: +5V -> GND
- J1201 pad 18: +5V -> /CHB Communication/Ph_A_Tx9
- J1201 pad 19: +5V -> GND
- J1201 pad 2: +5V -> /CHB Communication/Ph_A_Tx1
- J1201 pad 20: +5V -> /CHB Communication/Ph_A_Tx10
- J1201 pad 21: +5V -> GND
- J1201 pad 22: +5V -> /CHB Communication/Ph_A_Tx11
- J1201 pad 23: +5V -> GND
- J1201 pad 24: +5V -> /CHB Communication/Ph_A_Tx12
- J1201 pad 3: +5V -> GND
- J1201 pad 4: +5V -> /CHB Communication/Ph_A_Tx2
- J1201 pad 5: +5V -> GND
- J1201 pad 6: +5V -> /CHB Communication/Ph_A_Tx3
- J1201 pad 7: +5V -> GND
- J1201 pad 8: +5V -> /CHB Communication/Ph_A_Tx4
- J1201 pad 9: +5V -> GND
- J1202 pad 10: GND -> /CHB Communication/Ph_B_Tx5
- J1202 pad 12: GND -> /CHB Communication/Ph_B_Tx6
- J1202 pad 14: GND -> /CHB Communication/Ph_B_Tx7
- J1202 pad 16: GND -> /CHB Communication/Ph_B_Tx8
- J1202 pad 18: GND -> /CHB Communication/Ph_B_Tx9
- J1202 pad 2: GND -> /CHB Communication/Ph_B_Tx1
- J1202 pad 20: GND -> /CHB Communication/Ph_B_Tx10
- J1202 pad 22: GND -> /CHB Communication/Ph_B_Tx11
- J1202 pad 24: GND -> /CHB Communication/Ph_B_Tx12
- J1202 pad 4: GND -> /CHB Communication/Ph_B_Tx2
- J1202 pad 6: GND -> /CHB Communication/Ph_B_Tx3
- J1202 pad 8: GND -> /CHB Communication/Ph_B_Tx4
- J1403 pad 1: +5V -> GND
- J1403 pad 11: +5V -> GND
- J1403 pad 13: +5V -> GND
- J1403 pad 15: +5V -> GND
- J1403 pad 17: +5V -> GND
- J1403 pad 19: +5V -> GND
- J1403 pad 21: +5V -> GND
- J1403 pad 23: +5V -> GND
- J1403 pad 3: +5V -> GND
- J1403 pad 5: +5V -> GND
- J1403 pad 7: +5V -> GND
- J1403 pad 9: +5V -> GND
- R902 pad 4: Net-(D901-A2) -> GND
- R902 pad 5: Net-(D901-A2) -> GND
- SW1201 pad 1: /FPGA/Button1 -> Net-(R904-Pad1)
- SW1202 pad 1: /FPGA/Button2 -> Net-(R905-Pad1)
- U1001 pad 23: /ADC/V_DC -> /ADC for B6/V_DC
- U1001 pad 24: /ADC/V_A -> /ADC for B6/V_A
- U1001 pad 25: /ADC/V_B -> /ADC for B6/V_B
- U1001 pad 26: /ADC/V_C -> /ADC for B6/V_C
- U1001 pad 27: /ADC/I_A -> /ADC for B6/I_A
- U1001 pad 28: /ADC/I_B -> /ADC for B6/I_B
- U1001 pad 29: /ADC/I_C -> /ADC for B6/I_C
- U201 pad 1: /ADC/V_B -> /ADC for B6/Diffamp6/Ain-
- U201 pad 10: unconnected-(U201-Ain4--Pad10) -> /ADC for B6/Diffamp4/Ain-
- U201 pad 11: unconnected-(U201-Ain4+-Pad11) -> /ADC for B6/Diffamp4/Ain+
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
Commit message: lots of work
Parts:
- removed D1203, D1204, D1205, D1206, D1207, D1208, D1209, D1210, D1211, D1212, D1213, D1214, D1215, D1216, D1217, D1218, D1219, D1220, D1221, D1222, D1223, D1224, D1225, D1226, D1227, D1228, D1229, D1230, D1231, D1232, D1233, D1234, D1235, D1236, D1237, D1238, D1239, D1240, D1241, D1242, D1243, D1244, D1245, D1246, D1247, D1248, D1249, D1250: B72590D50H160, Capacitor_SMD:C_0402_1005Metric_Pad0.74x0.62mm_HandSolder
- removed J1101: Molex_Mini_Fit_Jr_2x08pin, MYLIB_Misc:Molex_2x8pin_vertical_tht
- added C1806: 100n_0603, WLIB_Capacitor:C_0603, F.Cu at (218.6, 16.8)
- added C1807: 100n_0603, WLIB_Capacitor:C_0603, F.Cu at (218.6, 19.3)
- added C1808: 100n_0603, WLIB_Capacitor:C_0603, F.Cu at (218.6, 21.8)
- added C1809: 100n_0603, WLIB_Capacitor:C_0603, F.Cu at (218.6, 24.3)
- added C3201: 10u_1210, WLIB_Capacitor:C_1210, F.Cu at (198.7, 74.7)
- added C3203: 10u_1210, WLIB_Capacitor:C_1210, F.Cu at (198.7, 79.0)
- added C3205: 10u_1210, WLIB_Capacitor:C_1210, F.Cu at (198.7, 83.2)
- added C3211: 10u_1210, WLIB_Capacitor:C_1210, F.Cu at (198.7, 87.5)
- added C3212: 10u_1210, WLIB_Capacitor:C_1210, F.Cu at (198.7, 91.7)
- added C3213: 100n_0603, WLIB_Capacitor:C_0603, F.Cu at (249.1, 16.8)
- added C3214: 100n_0603, WLIB_Capacitor:C_0603, F.Cu at (249.1, 19.3)
- added C3301: 100n_0603, WLIB_Capacitor:C_0603, F.Cu at (249.1, 39.7)
- added C3302: 100n_0603, WLIB_Capacitor:C_0603, F.Cu at (249.1, 42.2)
- added C3303: 100n_0603, WLIB_Capacitor:C_0603, F.Cu at (249.1, 28.3)
- added C3304: 100n_0603, WLIB_Capacitor:C_0603, F.Cu at (249.1, 30.8)
- added C3305: 100n_0603, WLIB_Capacitor:C_0603, F.Cu at (233.9, 16.8)
- added C3306: 100n_0603, WLIB_Capacitor:C_0603, F.Cu at (233.9, 19.3)
- added C3401: 100n_0603, WLIB_Capacitor:C_0603, F.Cu at (233.9, 39.7)
- added C3402: 100n_0603, WLIB_Capacitor:C_0603, F.Cu at (233.9, 42.2)
- added C3403: 100n_0603, WLIB_Capacitor:C_0603, F.Cu at (233.9, 28.3)
- added C3404: 100n_0603, WLIB_Capacitor:C_0603, F.Cu at (233.9, 30.8)
- added F3201: BLM18SP221SZ1D, MYLIB_Misc:BLM18SP221SZ1D, F.Cu at (203.7, 83.3)
- added J1601: Box_Header_2x05_THT, Connector_IDC:IDC-Header_2x05_P2.54mm_Vertical, F.Cu at (223.0, 89.6)
- added J1602: Box_Header_2x05_THT, Connector_IDC:IDC-Header_2x05_P2.54mm_Vertical, F.Cu at (235.0, 89.6)
- added J1603: Box_Header_2x05_THT, Connector_IDC:IDC-Header_2x05_P2.54mm_Vertical, F.Cu at (247.0, 89.6)
- added J1604: Box_Header_2x05_THT, Connector_IDC:IDC-Header_2x05_P2.54mm_Vertical, F.Cu at (259.0, 89.6)
- added J1801: Molex_Mini_Fit_Jr_2x08pin, MYLIB_Misc:Molex_2x8pin_vertical_tht, F.Cu at (235.7, 60.0)
- added L3201: WE_Inductor_470nH, MYLIB_Misc:WE_74479275147, F.Cu at (203.9, 74.2)
- added R3201: 1k_0603, Resistor_SMD:R_0603_1608Metric, F.Cu at (203.7, 80.7)
- added U1602: SN74LXCH8T245RHLR, MYLIB_Misc:SN74LXCH8T245, F.Cu at (242.6, 43.2)
- added U1802: SN74LXC2T45Q1, MYLIB_Misc:SN74LXC2T45QDCURQ1, F.Cu at (220.2, 68.9)
- added U1803: SN74LXC2T45Q1, MYLIB_Misc:SN74LXC2T45QDCURQ1, F.Cu at (220.2, 72.5)
- added U3203: TPS6282518, MYLIB_Misc:TPS6282518DMQR, F.Cu at (203.8, 77.6)
- added U3204: SN74LXCH8T245RHLR, MYLIB_Misc:SN74LXCH8T245, F.Cu at (242.6, 20.3)
- added U3301: SN74LXCH8T245RHLR, MYLIB_Misc:SN74LXCH8T245, F.Cu at (242.6, 31.8)
- added U3302: SN74LXCH8T245RHLR, MYLIB_Misc:SN74LXCH8T245, F.Cu at (227.3, 20.3)
- added U3401: SN74LXCH8T245RHLR, MYLIB_Misc:SN74LXCH8T245, F.Cu at (227.3, 43.2)
- added U3402: SN74LXCH8T245RHLR, MYLIB_Misc:SN74LXCH8T245, F.Cu at (227.3, 31.8)
Connections:
- net /CHB to 3Ph/Ph_A1_out renamed M_PHA
- net /CHB to 3Ph/Ph_B1_out renamed M_PHB
- net /CHB to 3Ph/Ph_C1_out renamed M_PHC
- net OVDD renamed +1V8
- J1201 pad 10: /CHB Communication/Ph_A_Tx5 -> /CHB Communication/Level_Shifter_8bit_1/A5
- J1201 pad 12: /CHB Communication/Ph_A_Tx6 -> /CHB Communication/Level_Shifter_8bit_1/A6
- J1201 pad 14: /CHB Communication/Ph_A_Tx7 -> /CHB Communication/Level_Shifter_8bit_1/A7
- J1201 pad 16: /CHB Communication/Ph_A_Tx8 -> /CHB Communication/Level_Shifter_8bit_1/A8
- J1201 pad 18: /CHB Communication/Ph_A_Tx9 -> /CHB Communication/Level_Shifter_8bit_2/A1
- J1201 pad 2: /CHB Communication/Ph_A_Tx1 -> /CHB Communication/Level_Shifter_8bit_1/A1
- J1201 pad 20: /CHB Communication/Ph_A_Tx10 -> /CHB Communication/Level_Shifter_8bit_2/A2
- J1201 pad 22: /CHB Communication/Ph_A_Tx11 -> /CHB Communication/Level_Shifter_8bit_2/A3
- J1201 pad 24: /CHB Communication/Ph_A_Tx12 -> /CHB Communication/Level_Shifter_8bit_2/A4
- J1201 pad 4: /CHB Communication/Ph_A_Tx2 -> /CHB Communication/Level_Shifter_8bit_1/A2
- J1201 pad 6: /CHB Communication/Ph_A_Tx3 -> /CHB Communication/Level_Shifter_8bit_1/A3
- J1201 pad 8: /CHB Communication/Ph_A_Tx4 -> /CHB Communication/Level_Shifter_8bit_1/A4
- J1202 pad 10: /CHB Communication/Ph_B_Tx5 -> /CHB Communication/Level_Shifter_8bit_3/A1
- J1202 pad 12: /CHB Communication/Ph_B_Tx6 -> /CHB Communication/Level_Shifter_8bit_3/A2
- J1202 pad 14: /CHB Communication/Ph_B_Tx7 -> /CHB Communication/Level_Shifter_8bit_3/A3
- J1202 pad 16: /CHB Communication/Ph_B_Tx8 -> /CHB Communication/Level_Shifter_8bit_3/A4
- J1202 pad 18: /CHB Communication/Ph_B_Tx9 -> /CHB Communication/Level_Shifter_8bit_3/A5
- J1202 pad 2: /CHB Communication/Ph_B_Tx1 -> /CHB Communication/Level_Shifter_8bit_2/A5
- J1202 pad 20: /CHB Communication/Ph_B_Tx10 -> /CHB Communication/Level_Shifter_8bit_3/A6
- J1202 pad 22: /CHB Communication/Ph_B_Tx11 -> /CHB Communication/Level_Shifter_8bit_3/A7
- J1202 pad 24: /CHB Communication/Ph_B_Tx12 -> /CHB Communication/Level_Shifter_8bit_3/A8
- J1202 pad 4: /CHB Communication/Ph_B_Tx2 -> /CHB Communication/Level_Shifter_8bit_2/A6
- J1202 pad 6: /CHB Communication/Ph_B_Tx3 -> /CHB Communication/Level_Shifter_8bit_2/A7
- J1202 pad 8: /CHB Communication/Ph_B_Tx4 -> /CHB Communication/Level_Shifter_8bit_2/A8
- J1207 pad 10: /CHB Communication/Ph_C_Tx5 -> /CHB Communication/Level_Shifter_8bit_4/A5
- J1207 pad 12: /CHB Communication/Ph_C_Tx6 -> /CHB Communication/Level_Shifter_8bit_4/A6
- J1207 pad 14: /CHB Communication/Ph_C_Tx7 -> /CHB Communication/Level_Shifter_8bit_4/A7
- J1207 pad 16: /CHB Communication/Ph_C_Tx8 -> /CHB Communication/Level_Shifter_8bit_4/A8
- J1207 pad 18: /CHB Communication/Ph_C_Tx9 -> /CHB Communication/Level_Shifter_8bit_5/A1
- J1207 pad 2: /CHB Communication/Ph_C_Tx1 -> /CHB Communication/Level_Shifter_8bit_4/A1
- J1207 pad 20: /CHB Communication/Ph_C_Tx10 -> /CHB Communication/Level_Shifter_8bit_5/A2
- J1207 pad 22: /CHB Communication/Ph_C_Tx11 -> /CHB Communication/Level_Shifter_8bit_5/A3
- J1207 pad 24: /CHB Communication/Ph_C_Tx12 -> /CHB Communication/Level_Shifter_8bit_5/A4
- J1207 pad 4: /CHB Communication/Ph_C_Tx2 -> /CHB Communication/Level_Shifter_8bit_4/A2
- J1207 pad 6: /CHB Communication/Ph_C_Tx3 -> /CHB Communication/Level_Shifter_8bit_4/A3
- J1207 pad 8: /CHB Communication/Ph_C_Tx4 -> /CHB Communication/Level_Shifter_8bit_4/A4
- J1208 pad 10: /CHB Communication/Ph_D_Tx5 -> /CHB Communication/Level_Shifter_8bit_6/A1
- J1208 pad 12: /CHB Communication/Ph_D_Tx6 -> /CHB Communication/Level_Shifter_8bit_6/A2
- J1208 pad 14: /CHB Communication/Ph_D_Tx7 -> /CHB Communication/Level_Shifter_8bit_6/A3
- J1208 pad 16: /CHB Communication/Ph_D_Tx8 -> /CHB Communication/Level_Shifter_8bit_6/A4
- J1208 pad 18: /CHB Communication/Ph_D_Tx9 -> /CHB Communication/Level_Shifter_8bit_6/A5
- J1208 pad 2: /CHB Communication/Ph_D_Tx1 -> /CHB Communication/Level_Shifter_8bit_5/A5
- J1208 pad 20: /CHB Communication/Ph_D_Tx10 -> /CHB Communication/Level_Shifter_8bit_6/A6
- J1208 pad 22: /CHB Communication/Ph_D_Tx11 -> /CHB Communication/Level_Shifter_8bit_6/A7
- J1208 pad 24: /CHB Communication/Ph_D_Tx12 -> /CHB Communication/Level_Shifter_8bit_6/A8
- J1208 pad 4: /CHB Communication/Ph_D_Tx2 -> /CHB Communication/Level_Shifter_8bit_5/A6
- J1208 pad 6: /CHB Communication/Ph_D_Tx3 -> /CHB Communication/Level_Shifter_8bit_5/A7
- J1208 pad 8: /CHB Communication/Ph_D_Tx4 -> /CHB Communication/Level_Shifter_8bit_5/A8
- R501 pad 1: +5V -> /Main_DCDC/Vout
- U301 pad a29: /FPGA/Ph_A_Tx4 -> /CHB Communication/Ph_A_Tx4
- U301 pad a30: /FPGA/Ph_A_Tx5 -> /CHB Communication/Ph_A_Tx5
- U301 pad a31: /FPGA/Ph_A_Tx7 -> /CHB Communication/Ph_A_Tx7
- U301 pad a32: /FPGA/Ph_A_Tx6 -> /CHB Communication/Ph_A_Tx6
- U301 pad a33: /FPGA/Ph_A_Tx8 -> /CHB Communication/Ph_A_Tx8
- U301 pad a36: /FPGA/Ph_A_Tx9 -> /CHB Communication/Ph_A_Tx9
- U301 pad a37: /FPGA/Ph_A_Tx11 -> /CHB Communication/Ph_A_Tx11
- U301 pad a38: /FPGA/Ph_A_Tx10 -> /CHB Communication/Ph_A_Tx10
- U301 pad a39: /FPGA/Ph_A_Tx12 -> /CHB Communication/Ph_A_Tx12
- U301 pad a40: /FPGA/Ph_B_Tx1 -> /CHB Communication/Ph_B_Tx1
- U301 pad a41: /FPGA/Ph_B_Tx3 -> /CHB Communication/Ph_B_Tx3
- U301 pad a42: /FPGA/Ph_B_Tx2 -> /CHB Communication/Ph_B_Tx2
- U301 pad a43: /FPGA/Ph_B_Tx4 -> /CHB Communication/Ph_B_Tx4
- U301 pad a45: /FPGA/Ph_B_Tx9 -> /CHB Communication/Ph_B_Tx9
- U301 pad a46: /FPGA/Ph_B_Tx7 -> /CHB Communication/Ph_B_Tx7
- U301 pad a47: /FPGA/Ph_B_Tx10 -> /CHB Communication/Ph_B_Tx10
- U301 pad a48: /FPGA/Ph_B_Tx8 -> /CHB Communication/Ph_B_Tx8
- U301 pad a50: /FPGA/Ph_C_Tx1 -> /CHB Communication/Ph_C_Tx1
- U301 pad a51: /FPGA/Ph_B_Tx5 -> /CHB Communication/Ph_B_Tx5
- U301 pad a52: /FPGA/Ph_C_Tx2 -> /CHB Communication/Ph_C_Tx2
- U301 pad a53: /FPGA/Ph_B_Tx6 -> /CHB Communication/Ph_B_Tx6
- U301 pad a55: /FPGA/Ph_B_Tx11 -> /CHB Communication/Ph_B_Tx11
- U301 pad a56: /FPGA/Ph_C_Tx5 -> /CHB Communication/Ph_C_Tx5
- U301 pad a57: /FPGA/Ph_B_Tx12 -> /CHB Communication/Ph_B_Tx12
- U301 pad a58: /FPGA/Ph_C_Tx6 -> /CHB Communication/Ph_C_Tx6
- U301 pad a59: /FPGA/Ph_C_Tx3 -> /CHB Communication/Ph_C_Tx3
- U301 pad a60: /FPGA/Ph_C_Tx9 -> /CHB Communication/Ph_C_Tx9
- U301 pad a61: /FPGA/Ph_C_Tx4 -> /CHB Communication/Ph_C_Tx4
- U301 pad a62: /FPGA/Ph_C_Tx10 -> /CHB Communication/Ph_C_Tx10
- U301 pad a63: /FPGA/Ph_C_Tx7 -> /CHB Communication/Ph_C_Tx7
- U301 pad a64: /FPGA/Ph_D_Tx1 -> /CHB Communication/Ph_D_Tx1
- U301 pad a65: /FPGA/Ph_C_Tx8 -> /CHB Communication/Ph_C_Tx8
- U301 pad a66: /FPGA/Ph_D_Tx2 -> /CHB Communication/Ph_D_Tx2
- U301 pad a69: /FPGA/Ph_C_Tx12 -> /CHB Communication/Ph_C_Tx12
- U301 pad a70: /FPGA/Ph_C_Tx11 -> /CHB Communication/Ph_C_Tx11
- U301 pad a71: /FPGA/Ph_D_Tx4 -> /CHB Communication/Ph_D_Tx4
- U301 pad a72: /FPGA/Ph_D_Tx3 -> /CHB Communication/Ph_D_Tx3
- U301 pad a73: /FPGA/Ph_D_Tx6 -> /CHB Communication/Ph_D_Tx6
- U301 pad a74: /FPGA/Ph_D_Tx5 -> /CHB Communication/Ph_D_Tx5
- U301 pad a75: /FPGA/Ph_D_Tx7 -> /CHB Communication/Ph_D_Tx7
- U301 pad a76: /FPGA/Ph_D_Tx11 -> /CHB Communication/Ph_D_Tx11
- U301 pad a77: /FPGA/Ph_D_Tx8 -> /CHB Communication/Ph_D_Tx8
- U301 pad a78: /FPGA/Ph_D_Tx12 -> /CHB Communication/Ph_D_Tx12
- U301 pad a79: /FPGA/Ph_D_Tx9 -> /CHB Communication/Ph_D_Tx9
- U301 pad a80: /FPGA/Ph_D_Tx10 -> /CHB Communication/Ph_D_Tx10
- U501 pad 26: +5V -> /Main_DCDC/Vout

Commit message: work
Parts:
- removed C1706, C1707, C1708: 15p_0603, WLIB_Capacitor:C_0603
- removed C1709, C1710: 100n_0603, WLIB_Capacitor:C_0603
- removed the C1801 at (142.4, 92.8)
- removed the C1801 at (254.1, 116.4)
- removed the C1802 at (142.4, 95.3)
- removed the C1802 at (254.1, 118.9)
- removed the C1803 at (142.4, 97.8)
- removed the C1803 at (254.1, 121.4)
- removed the C1804 at (254.1, 123.9)
- removed the C1804 at (142.4, 100.3)
- removed the C1805 at (142.4, 102.8)
- removed the C1805 at (254.1, 126.4)
- removed J1203, J1204, J1205, J1206: Box_Header_6pin, Connector_IDC:IDC-Header_2x03_P2.54mm_Vertical
- removed R1707, R1708: 30R_0603, Resistor_SMD:R_0603_1608Metric
- removed R1709, R1711: 500R_0603, Resistor_SMD:R_0603_1608Metric
- removed R1710, R1712: 5k1_0603, Resistor_SMD:R_0603_1608Metric
- removed the R1801 at (138.2, 92.8)
- removed the R1801 at (249.9, 116.4)
- removed the R1802 at (249.9, 118.9)
- removed the R1802 at (138.2, 95.3)
- removed the R1803 at (138.2, 97.8)
- removed the R1803 at (249.9, 121.4)
- removed the R1804 at (138.2, 100.3)
- removed the R1804 at (249.9, 123.9)
- removed the R1805 at (138.2, 102.8)
- removed the R1805 at (249.9, 126.4)
- removed the R1806 at (249.9, 128.9)
- removed the R1806 at (138.2, 105.3)
- removed U1702: 1819_IS8, MYLIB_Misc:LT1819
- removed the U1801 at (148.7, 94.8)
- removed the U1801 at (260.5, 118.4)
- added C1801: 15p_0603, WLIB_Capacitor:C_0603, F.Cu at (103.4, 34.3)
- added C1802: 15p_0603, WLIB_Capacitor:C_0603, F.Cu at (103.4, 36.8)
- added C1803: 15p_0603, WLIB_Capacitor:C_0603, F.Cu at (103.4, 39.3)
- added C1804: 100n_0603, WLIB_Capacitor:C_0603, F.Cu at (103.4, 41.8)
- added C1805: 100n_0603, WLIB_Capacitor:C_0603, F.Cu at (103.4, 44.3)
- added C3901: 100n_0603, WLIB_Capacitor:C_0603, F.Cu at (205.8, 31.7)
- added C3902: 100n_0603, WLIB_Capacitor:C_0603, F.Cu at (205.8, 34.2)
- added C4001: 100n_0603, WLIB_Capacitor:C_0603, F.Cu at (216.2, 48.0)
- added C4002: 100n_0603, WLIB_Capacitor:C_0603, F.Cu at (216.2, 50.5)
- added C4101: 100n_0603, WLIB_Capacitor:C_0603, F.Cu at (205.8, 48.0)
- added C4102: 100n_0603, WLIB_Capacitor:C_0603, F.Cu at (205.8, 50.5)
- added R1801: 30R_0603, Resistor_SMD:R_0603_1608Metric, F.Cu at (99.2, 34.3)
- added R1802: 30R_0603, Resistor_SMD:R_0603_1608Metric, F.Cu at (99.2, 36.8)
- added R1803: 500R_0603, Resistor_SMD:R_0603_1608Metric, F.Cu at (99.2, 39.3)
- added R1804: 5k1_0603, Resistor_SMD:R_0603_1608Metric, F.Cu at (99.2, 41.8)
- added R1805: 500R_0603, Resistor_SMD:R_0603_1608Metric, F.Cu at (99.2, 44.3)
- added R1806: 5k1_0603, Resistor_SMD:R_0603_1608Metric, F.Cu at (99.2, 46.8)
- added R3204: 10k_0603, Resistor_SMD:R_0603_1608Metric, F.Cu at (186.7, 22.2)
- added R3205: 10k_0603, Resistor_SMD:R_0603_1608Metric, F.Cu at (186.7, 24.7)
- added R3213: 10k_0603, Resistor_SMD:R_0603_1608Metric, F.Cu at (186.7, 27.2)
- added R3214: 10k_0603, Resistor_SMD:R_0603_1608Metric, F.Cu at (186.7, 29.8)
- added R3215: 10k_0603, Resistor_SMD:R_0603_1608Metric, F.Cu at (186.7, 32.3)
- added R3216: 10k_0603, Resistor_SMD:R_0603_1608Metric, F.Cu at (186.7, 34.8)
- added R3217: 10k_0603, Resistor_SMD:R_0603_1608Metric, F.Cu at (186.7, 37.3)
- added R3218: 10k_0603, Resistor_SMD:R_0603_1608Metric, F.Cu at (186.7, 39.8)
- added R3301: 10k_0603, Resistor_SMD:R_0603_1608Metric, F.Cu at (155.8, 31.8)
- added R3302: 10k_0603, Resistor_SMD:R_0603_1608Metric, F.Cu at (155.8, 34.3)
- added R3303: 10k_0603, Resistor_SMD:R_0603_1608Metric, F.Cu at (155.8, 36.8)
- added R3304: 10k_0603, Resistor_SMD:R_0603_1608Metric, F.Cu at (155.8, 39.3)
- added R3305: 10k_0603, Resistor_SMD:R_0603_1608Metric, F.Cu at (155.8, 41.8)
- added R3306: 10k_0603, Resistor_SMD:R_0603_1608Metric, F.Cu at (155.8, 44.3)
- added R3307: 10k_0603, Resistor_SMD:R_0603_1608Metric, F.Cu at (155.8, 46.9)
- added R3308: 10k_0603, Resistor_SMD:R_0603_1608Metric, F.Cu at (155.8, 49.4)
- added R3401: 10k_0603, Resistor_SMD:R_0603_1608Metric, F.Cu at (171.8, 22.2)
- added R3402: 10k_0603, Resistor_SMD:R_0603_1608Metric, F.Cu at (171.8, 24.7)
- added R3403: 10k_0603, Resistor_SMD:R_0603_1608Metric, F.Cu at (171.8, 27.2)
- added R3404: 10k_0603, Resistor_SMD:R_0603_1608Metric, F.Cu at (171.8, 29.8)
- added R3405: 10k_0603, Resistor_SMD:R_0603_1608Metric, F.Cu at (171.8, 32.3)
- added R3406: 10k_0603, Resistor_SMD:R_0603_1608Metric, F.Cu at (171.8, 34.8)
- added R3407: 10k_0603, Resistor_SMD:R_0603_1608Metric, F.Cu at (171.8, 37.3)
- added R3408: 10k_0603, Resistor_SMD:R_0603_1608Metric, F.Cu at (171.8, 39.8)
- added R3501: 10k_0603, Resistor_SMD:R_0603_1608Metric, F.Cu at (201.6, 0.15)
- added R3502: 10k_0603, Resistor_SMD:R_0603_1608Metric, F.Cu at (201.6, 2.66)
- added R3503: 10k_0603, Resistor_SMD:R_0603_1608Metric, F.Cu at (201.6, 5.17)
- added R3504: 10k_0603, Resistor_SMD:R_0603_1608Metric, F.Cu at (201.6, 7.68)
- added R3505: 10k_0603, Resistor_SMD:R_0603_1608Metric, F.Cu at (201.6, 10.2)
- added R3506: 10k_0603, Resistor_SMD:R_0603_1608Metric, F.Cu at (201.6, 12.7)
- added R3507: 10k_0603, Resistor_SMD:R_0603_1608Metric, F.Cu at (201.6, 15.2)
- added R3508: 10k_0603, Resistor_SMD:R_0603_1608Metric, F.Cu at (201.6, 17.7)
- added R3701: 10k_0603, Resistor_SMD:R_0603_1608Metric, F.Cu at (171.8, 0.15)
- added R3702: 10k_0603, Resistor_SMD:R_0603_1608Metric, F.Cu at (171.8, 2.66)
- added R3703: 10k_0603, Resistor_SMD:R_0603_1608Metric, F.Cu at (171.8, 5.17)
- added R3704: 10k_0603, Resistor_SMD:R_0603_1608Metric, F.Cu at (171.8, 7.68)
- added R3705: 10k_0603, Resistor_SMD:R_0603_1608Metric, F.Cu at (171.8, 10.2)
- added R3706: 10k_0603, Resistor_SMD:R_0603_1608Metric, F.Cu at (171.8, 12.7)
- added R3707: 10k_0603, Resistor_SMD:R_0603_1608Metric, F.Cu at (171.8, 15.2)
- added R3708: 10k_0603, Resistor_SMD:R_0603_1608Metric, F.Cu at (171.8, 17.7)
- added R3801: 10k_0603, Resistor_SMD:R_0603_1608Metric, F.Cu at (186.7, 0.15)
- added R3802: 10k_0603, Resistor_SMD:R_0603_1608Metric, F.Cu at (186.7, 2.66)
- added R3803: 10k_0603, Resistor_SMD:R_0603_1608Metric, F.Cu at (186.7, 5.17)
- added R3804: 10k_0603, Resistor_SMD:R_0603_1608Metric, F.Cu at (186.7, 7.68)
- added R3805: 10k_0603, Resistor_SMD:R_0603_1608Metric, F.Cu at (186.7, 10.2)
- added R3806: 10k_0603, Resistor_SMD:R_0603_1608Metric, F.Cu at (186.7, 12.7)
- added R3807: 10k_0603, Resistor_SMD:R_0603_1608Metric, F.Cu at (186.7, 15.2)
- added R3808: 10k_0603, Resistor_SMD:R_0603_1608Metric, F.Cu at (186.7, 17.7)
- added R3901: 10k_0603, Resistor_SMD:R_0603_1608Metric, F.Cu at (201.6, 48.0)
- added R3902: 10k_0603, Resistor_SMD:R_0603_1608Metric, F.Cu at (201.6, 50.5)
- added R4001: 10k_0603, Resistor_SMD:R_0603_1608Metric, F.Cu at (201.6, 22.2)
- added R4002: 10k_0603, Resistor_SMD:R_0603_1608Metric, F.Cu at (201.6, 24.7)
- added R4003: 10k_0603, Resistor_SMD:R_0603_1608Metric, F.Cu at (201.6, 27.2)
- added R4004: 10k_0603, Resistor_SMD:R_0603_1608Metric, F.Cu at (201.6, 29.8)
- added R4005: 10k_0603, Resistor_SMD:R_0603_1608Metric, F.Cu at (201.6, 32.3)
- added R4006: 10k_0603, Resistor_SMD:R_0603_1608Metric, F.Cu at (201.6, 34.8)
- added R4007: 10k_0603, Resistor_SMD:R_0603_1608Metric, F.Cu at (201.6, 37.3)
- added R4008: 10k_0603, Resistor_SMD:R_0603_1608Metric, F.Cu at (201.6, 39.8)
- added R4101: 10k_0603, Resistor_SMD:R_0603_1608Metric, F.Cu at (212.0, 48.0)
- added R4102: 10k_0603, Resistor_SMD:R_0603_1608Metric, F.Cu at (212.0, 50.5)
- added U1801: 1819_IS8, MYLIB_Misc:LT1819, F.Cu at (109.7, 36.3)
- added U3901: SN74LXCH8T245RHLR, MYLIB_Misc:SN74LXCH8T245, F.Cu at (208.2, 25.7)
- added U4001: SN74LXC2T45Q1, MYLIB_Misc:SN74LXC2T45QDCURQ1, F.Cu at (212.8, 44.9)
- added U4101: SN74LXC2T45Q1, MYLIB_Misc:SN74LXC2T45QDCURQ1, F.Cu at (202.4, 44.9)
- moved C2001 261.9 mm to (21.4, 189.0)
- moved C2002 261.9 mm to (21.4, 191.6)
- moved C2003 261.9 mm to (21.4, 194.1)
- moved C2004 261.9 mm to (21.4, 196.6)
- moved C2005 261.9 mm to (21.4, 199.1)
- moved R2001 261.9 mm to (17.2, 189.0)
- moved R2002 261.9 mm to (17.2, 191.6)
- moved R2003 261.9 mm to (17.2, 194.1)
- moved R2004 261.9 mm to (17.2, 196.6)
- moved R2005 261.9 mm to (17.2, 199.1)
- moved R2006 261.9 mm to (17.2, 201.6)
- moved U2001 261.9 mm to (27.7, 191.1)
- moved C3103 214.9 mm to (42.1, 190.8)
- moved R2606 214.9 mm to (56.8, 181.3)
- moved R3103 214.9 mm to (38.0, 190.8)
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Connections:
- J1601 pad 1: /CHB Communication/Ph_A_Err -> /CHB Communication/Level_shifter_error_1/A1
- J1601 pad 5: /CHB Communication/Ph_A_Rx -> /CHB Communication/Level_shifter_Rx_En/B2
- J1601 pad 7: /CHB Communication/Ph_A_En -> /CHB Communication/Level_shifter_Rx_En/B1
- J1602 pad 1: /CHB Communication/Ph_C_Err -> /CHB Communication/Level_shifter_error_2/A1
- J1602 pad 5: /CHB Communication/Ph_C_Rx -> /CHB Communication/Level_shifter_Rx_En/B6
- J1602 pad 7: /CHB Communication/Ph_C_En -> /CHB Communication/Level_shifter_Rx_En/B5
- J1603 pad 1: /CHB Communication/Ph_D_Err -> /CHB Communication/Level_shifter_error_2/A2
- J1603 pad 5: /CHB Communication/Ph_D_Rx -> /CHB Communication/Level_shifter_Rx_En/B8
- J1603 pad 7: /CHB Communication/Ph_D_En -> /CHB Communication/Level_shifter_Rx_En/B7
- J1604 pad 1: /CHB Communication/Ph_B_Err -> /CHB Communication/Level_shifter_error_1/A2
- J1604 pad 5: /CHB Communication/Ph_B_Rx -> /CHB Communication/Level_shifter_Rx_En/B4
- J1604 pad 7: /CHB Communication/Ph_B_En -> /CHB Communication/Level_shifter_Rx_En/B3
- U301 pad a3: unconnected-(U301D-VDD_3V-Pada3)_1 -> +3.3V
- U301 pad b3: unconnected-(U301D-VDD_3V-Pada3) -> +3.3V
