File: FPGA_Board_BA/PCB/FPGA_Board_BA.kicad_pcb (KiCad board)
At the start: 2 copper layers, 398 parts, among them J103 Plug_Termincal_8pin, J1201 Box_Header_26pin, J1202 Box_Header_26pin, J1207 Box_Header_26pin, J1208 Box_Header_26pin, J1301 PinHeader_03_male, J1403 Plug_Terminal_2x12pin, J1601 Box_Header_2x05_THT, J1602 Box_Header_2x05_THT, J1603 Box_Header_2x05_THT, J1604 Box_Header_2x05_THT, J1801 Molex_Mini_Fit_Jr_2x08pin, J201 PinHeader_03_male, J601 Banana_Socket_Black, J602 Banana_Socket_Red, J701 Box_Header_6pin, J716 Plug_Terminal_2x12pin, J717 Plug_Terminal_2x12pin, J718 Plug_Terminal_2x12pin, J720 Plug_Terminal_2x12pin, Q501 IPT017N12NM6, Q502 IPT017N12NM6, Q503 IPT017N12NM6, Q504 IPT017N12NM6, SW1201 TL3305BF100QG, SW1202 TL3305BF100QG, U1001 BOOSTXL-3PHGANINV, U101 HV_Probe, U1301 LTC2320-16_LVDS, U1501 HV_Probe, U1502 HV_Probe, U1503 HV_Probe, U1601 1819_IS8, U1602 SN74LXCH8T245RHLR, U1701 1819_IS8, U1801 1819_IS8, U1802 SN74LXC2T45Q1, U1803 SN74LXC2T45Q1, U1901 1819_IS8, U2001 1819_IS8, U2002 1819_IS8, U2003 1819_IS8, U201 LTC2320-16_LVDS, U2501 1819_IS8, U2601 1819_IS8, U2701 1819_IS8, U2801 1819_IS8, U2901 1819_IS8, U3001 1819_IS8, U301 Zynq7020, U3101 1819_IS8, U3201 1819_IS8, U3202 1819_IS8, U3203 TPS6282518, U3204 SN74LXCH8T245RHLR, U3301 SN74LXCH8T245RHLR, U3302 SN74LXCH8T245RHLR, U3401 SN74LXCH8T245RHLR, U3402 SN74LXCH8T245RHLR, U3901 SN74LXCH8T245RHLR, U4001 SN74LXC2T45Q1, U401 AMC0300D, U402 AMC0300D, U403 AMC0300D, U404 AMC0300D, U4101 SN74LXC2T45Q1, U501 LM5143, U801 TPS61022, U802 MCP1703AT-5002EDB

Commit message: 18.11 Bib Session
Parts:
- removed C1201, C1202, C1605, C1607, C1608, C1704, C1705, C1804, C1805, C1806, C1807, C1808, C1809, C1904, C1905, C2004, C2005, C2009, C2010, C2014, C2015, C2504, C2505, C2604, C2605, C2704, C2705, C2804, C2805, C2904, C2905, C3004, C3005, C3104, C3105, C3204, C3209, C3210, C3213, C3214, C3301, C3302, C3303, C3304, C3305, C3306, C3401, C3402, C3403, C3404, C3901, C3902, C4001, C4002, C4101, C4102, C801, C901: 100n_0603, WLIB_Capacitor:C_0603
- removed C1301, C1302, C1303, C1304, C201, C202, C203, C204, C3201, C3203, C3205, C3211, C3212, C502, C504, C512, C802, C803, C804: 10u_1210, WLIB_Capacitor:C_1210
- removed C1601, C1602, C1603, C1604, C1606, C1701, C1702, C1703, C1801, C1802, C1803, C1901, C1902, C1903, C2001, C2002, C2003, C2006, C2007, C2008, C2011, C2012, C2013, C2501, C2502, C2503, C2601, C2602, C2603, C2701, C2702, C2703, C2801, C2802, C2803, C2901, C2902, C2903, C3001, C3002, C3003, C3101, C3102, C3103, C3202, C3206, C3207, C3208: 15p_0603, WLIB_Capacitor:C_0603
- removed C501: 1n_0603, WLIB_Capacitor:C_0603
- removed C503, C505, C506, C510: 4u7_0603, WLIB_Capacitor:C_0603
- removed C507: 56pF_0603, Capacitor_SMD:C_0603_1608Metric_Pad1.08x0.95mm_HandSolder
- removed C508: 120nF_0603, Capacitor_SMD:C_0603_1608Metric_Pad1.08x0.95mm_HandSolder
- removed C509, C805, C806: 1u_0603, WLIB_Capacitor:C_0603
- removed C511: 25uF_2220, Capacitor_SMD:C_2220_5650Metric_Pad1.97x5.40mm_HandSolder
- removed D1201: LED_B_0603, WLIB_DO:LED_0603_1608Metric
- removed D1202, D503, D601, D801, D802: LED_G_0603, WLIB_DO:LED_0603_1608Metric
- removed D501, D502: SBR10U200P5-13, MYLIB_Misc:SBR10U200P5
- removed F3201: BLM18SP221SZ1D, MYLIB_Misc:BLM18SP221SZ1D
- removed J103: Plug_Termincal_8pin, MYLIB_Misc:DMC 1,5_ 8-G1-3,5 P20THR
- removed J1201, J1202, J1207, J1208: Box_Header_26pin, Connector_IDC:IDC-Header_2x13_P2.54mm_Vertical
- removed J1301, J201: PinHeader_03_male, Connector_PinHeader_2.54mm:PinHeader_1x03_P2.54mm_Vertical
- removed J1403, J716, J717, J718, J720: Plug_Terminal_2x12pin, MYLIB_Misc:DMCV 1,5_12-G1F-3,5-LR P20THR
- removed J1601, J1602, J1603, J1604: Box_Header_2x05_THT, Connector_IDC:IDC-Header_2x05_P2.54mm_Vertical
- removed J1801: Molex_Mini_Fit_Jr_2x08pin, MYLIB_Misc:Molex_2x8pin_vertical_tht
- removed J601: Banana_Socket_Black, MYLIB_Misc:Banana_Socket_Aletch_Black
- removed J602: Banana_Socket_Red, MYLIB_Misc:Banana_Socket_Altech_Red
- removed J701: Box_Header_6pin, Connector_IDC:IDC-Header_2x03_P2.54mm_Vertical
- removed L3201: WE_Inductor_470nH, MYLIB_Misc:WE_74479275147
- removed L501, L502: XAL1010-152MED, Inductor_SMD:L_Coilcraft_XAL1010-XXX
- removed Q501, Q502, Q503, Q504: IPT017N12NM6, Package_TO_SOT_SMD:Infineon_PG-HSOF-8-1
- removed R1, R101, R2, R3: 0R100_2512, Resistor_SMD:R_2512_6332Metric_Pad1.40x3.35mm_HandSolder
- removed R1201, R1202, R1203, R1204, R3204, R3205, R3213, R3214, R3215, R3216, R3217, R3218, R3301, R3302, R3303, R3304, R3305, R3306, R3307, R3308, R3401, R3402, R3403, R3404, R3405, R3406, R3407, R3408, R3501, R3502, R3503, R3504, R3505, R3506, R3507, R3508, R3701, R3702, R3703, R3704, R3705, R3706, R3707, R3708, R3801, R3802, R3803, R3804, R3805, R3806, R3807, R3808, R3901, R3902, R4001, R4002, R4003, R4004, R4005, R4006, R4007, R4008, R4101, R4102, R507, R803, R804: 10k_0603, Resistor_SMD:R_0603_1608Metric
- removed R1601, R1603, R1604, R1701, R1702, R1801, R1802, R1901, R1902, R2001, R2002, R2007, R2008, R2013, R2014, R2501, R2502, R2601, R2602, R2701, R2702, R2801, R2802, R2901, R2902, R3001, R3002, R3101, R3102, R3202, R3207, R3208: 30R_0603, Resistor_SMD:R_0603_1608Metric
- removed R1602, R1605, R1608, R1703, R1705, R1803, R1805, R1903, R1905, R2003, R2005, R2009, R2011, R2015, R2017, R2503, R2505, R2603, R2605, R2703, R2705, R2803, R2805, R2903, R2905, R3003, R3005, R3103, R3105, R3203, R3209, R3211: 500R_0603, Resistor_SMD:R_0603_1608Metric
- removed R1606, R1607, R1609, R1704, R1706, R1804, R1806, R1904, R1906, R2004, R2006, R2010, R2012, R2016, R2018, R2504, R2506, R2604, R2606, R2704, R2706, R2804, R2806, R2904, R2906, R3004, R3006, R3104, R3106, R3206, R3210, R3212: 5k1_0603, Resistor_SMD:R_0603_1608Metric
- removed R3201: 1k_0603, Resistor_SMD:R_0603_1608Metric
- removed R501, R503: 0R002_1206, Resistor_SMD:R_1206_3216Metric_Pad1.30x1.75mm_HandSolder
- removed R502, R504: 2R2_0603, Resistor_SMD:R_0603_1608Metric
- removed R505: 25k5_0603, Resistor_SMD:R_0603_1608Metric_Pad0.98x0.95mm_HandSolder
- removed R506: 39k2_0603, Resistor_SMD:R_0603_1608Metric_Pad0.98x0.95mm_HandSolder
- removed R601, R801: 100k_0603, Resistor_SMD:R_0603_1608Metric
- removed R802: 820k_0603, Resistor_SMD:R_0603_1608Metric_Pad0.98x0.95mm_HandSolder
- removed R901, R904, R905: 100R_0603, Resistor_SMD:R_0603_1608Metric
- removed R902: Poti_10k, MYLIB_Misc:RK09D1130A1N
- removed SW1201, SW1202: TL3305BF100QG, WLIB_Button_Switch:TL3305BF160QG
- removed U1001: BOOSTXL-3PHGANINV, MYLIB_Misc:TI_BOOSTXL_3PH
- removed U101, U1501, U1502, U1503: HV_Probe, MYLIB_Misc:HV_Probe
- removed U1301, U201: LTC2320-16_LVDS, MYLIB_chips:UKG_52_7mm_8mm
- removed U1601, U1701, U1801, U1901, U2001, U2002, U2003, U2501, U2601, U2701, U2801, U2901, U3001, U3101, U3201, U3202: 1819_IS8, MYLIB_Misc:LT1819
- removed U1602, U3204, U3301, U3302, U3401, U3402, U3901: SN74LXCH8T245RHLR, MYLIB_Misc:SN74LXCH8T245
- removed U1802, U1803, U4001, U4101: SN74LXC2T45Q1, MYLIB_Misc:SN74LXC2T45QDCURQ1
- removed U301: Zynq7020, MYLIB_Misc:Zynq7020
- removed U3203: TPS6282518, MYLIB_Misc:TPS6282518DMQR
- removed U401, U402, U403, U404: AMC0300D, MYLIB_Misc:SOIC-8_7.5x5.85mm_P1.27mm
- removed U501: LM5143, MYLIB_chips:VQFN 40 pin 5.8mm x 5.8mm
- removed U801: TPS61022, MYLIB_Misc:TPS61022
- removed U802: MCP1703AT-5002EDB, Package_TO_SOT_SMD:SOT-223

Commit message: schematic fixes after Leo Meeting
Parts:
- added C1: 1u_0603, WLIB_Capacitor:C_0603, F.Cu at (232.6, 210.0)
- added C10: 100n_0603, WLIB_Capacitor:C_0603, F.Cu at (237.0, 217.5)
- added C100: 15p_0603, WLIB_Capacitor:C_0603, F.Cu at (104.1, 187.0)
- added C101: 100n_0603, WLIB_Capacitor:C_0603, F.Cu at (104.1, 189.5)
- added C102: 100n_0603, WLIB_Capacitor:C_0603, F.Cu at (104.1, 192.0)
- added C103: 15p_0603, WLIB_Capacitor:C_0603, F.Cu at (230.6, 235.8)
- added C104: 15p_0603, WLIB_Capacitor:C_0603, F.Cu at (230.6, 238.3)
- added C105: 15p_0603, WLIB_Capacitor:C_0603, F.Cu at (230.6, 240.8)
- added C106: 100n_0603, WLIB_Capacitor:C_0603, F.Cu at (230.6, 243.4)
- added C107: 100n_0603, WLIB_Capacitor:C_0603, F.Cu at (230.6, 245.9)
- added C108: 15p_0603, WLIB_Capacitor:C_0603, F.Cu at (104.1, 216.1)
- added C109: 15p_0603, WLIB_Capacitor:C_0603, F.Cu at (104.1, 218.6)
- added C11: 1u_0603, WLIB_Capacitor:C_0603, F.Cu at (237.0, 220.0)
- added C110: 15p_0603, WLIB_Capacitor:C_0603, F.Cu at (104.1, 221.1)
- added C111: 100n_0603, WLIB_Capacitor:C_0603, F.Cu at (104.1, 223.6)
- added C112: 100n_0603, WLIB_Capacitor:C_0603, F.Cu at (104.1, 226.2)
- added C113: 15p_0603, WLIB_Capacitor:C_0603, F.Cu at (237.9, 81.9)
- added C114: 15p_0603, WLIB_Capacitor:C_0603, F.Cu at (237.9, 84.4)
- added C115: 15p_0603, WLIB_Capacitor:C_0603, F.Cu at (237.9, 86.9)
- added C116: 100n_0603, WLIB_Capacitor:C_0603, F.Cu at (237.9, 89.4)
- added C117: 100n_0603, WLIB_Capacitor:C_0603, F.Cu at (237.9, 92.0)
- added C118: 15p_0603, WLIB_Capacitor:C_0603, F.Cu at (104.1, 233.2)
- added C119: 15p_0603, WLIB_Capacitor:C_0603, F.Cu at (104.1, 235.7)
- added C12: 10u_1210, WLIB_Capacitor:C_1210, F.Cu at (227.4, 210.8)
- added C120: 15p_0603, WLIB_Capacitor:C_0603, F.Cu at (104.1, 238.2)
- added C121: 100n_0603, WLIB_Capacitor:C_0603, F.Cu at (104.1, 240.7)
- added C122: 100n_0603, WLIB_Capacitor:C_0603, F.Cu at (104.1, 243.2)
- added C123: 1u_0603, WLIB_Capacitor:C_0603, F.Cu at (60.4, 245.6)
- added C124: 1u_0603, WLIB_Capacitor:C_0603, F.Cu at (60.4, 248.1)
- added C128: 100n_0603, WLIB_Capacitor:C_0603, F.Cu at (223.0, 69.3)
- added C129: 100n_0603, WLIB_Capacitor:C_0603, F.Cu at (223.0, 71.8)
- added C13: 10u_1210, WLIB_Capacitor:C_1210, F.Cu at (227.4, 215.1)
- added C130: 100n_0603, WLIB_Capacitor:C_0603, F.Cu at (223.0, 47.2)
- added C131: 100n_0603, WLIB_Capacitor:C_0603, F.Cu at (223.0, 49.7)
- added C132: 100n_0603, WLIB_Capacitor:C_0603, F.Cu at (208.1, 47.2)
- added C133: 100n_0603, WLIB_Capacitor:C_0603, F.Cu at (208.1, 49.7)
- added C134: 100n_0603, WLIB_Capacitor:C_0603, F.Cu at (208.1, 69.3)
- added C135: 100n_0603, WLIB_Capacitor:C_0603, F.Cu at (208.1, 71.8)
- added C136: 100n_0603, WLIB_Capacitor:C_0603, F.Cu at (212.2, 195.7)
- added C137: 100n_0603, WLIB_Capacitor:C_0603, F.Cu at (104.1, 152.3)
- added C138: 100n_0603, WLIB_Capacitor:C_0603, F.Cu at (104.1, 154.8)
- added C139: 100n_0603, WLIB_Capacitor:C_0603, F.Cu at (237.9, 47.2)
- added C14: 10u_1210, WLIB_Capacitor:C_1210, F.Cu at (227.4, 219.3)
- added C140: 100n_0603, WLIB_Capacitor:C_0603, F.Cu at (237.9, 49.7)
- added C141: 100n_0603, WLIB_Capacitor:C_0603, F.Cu at (203.3, 246.1)
- added C142: 100n_0603, WLIB_Capacitor:C_0603, F.Cu at (203.3, 248.6)
- added C143: 100n_0603, WLIB_Capacitor:C_0603, F.Cu at (223.0, 85.6)
- added C144: 100n_0603, WLIB_Capacitor:C_0603, F.Cu at (223.0, 88.1)
- added C145: 100n_0603, WLIB_Capacitor:C_0603, F.Cu at (208.1, 85.6)
- added C146: 100n_0603, WLIB_Capacitor:C_0603, F.Cu at (208.1, 88.1)
- added C147: 100n_0603, WLIB_Capacitor:C_0603, F.Cu at (184.9, 228.2)
- added C148: 100n_0603, WLIB_Capacitor:C_0603, F.Cu at (237.9, 69.3)
- added C149: 100n_0603, WLIB_Capacitor:C_0603, F.Cu at (237.9, 71.8)
- added C15: 10u_1210, WLIB_Capacitor:C_1210, F.Cu at (227.4, 223.6)
- added C150: 100n_0603, WLIB_Capacitor:C_0603, F.Cu at (217.3, 162.2)
- added C151: 100n_0603, WLIB_Capacitor:C_0603, F.Cu at (217.3, 164.7)
- added C152: 100n_0603, WLIB_Capacitor:C_0603, F.Cu at (184.9, 195.7)
- added C153: 100n_0603, WLIB_Capacitor:C_0603, F.Cu at (213.7, 246.1)
- added C154: 100n_0603, WLIB_Capacitor:C_0603, F.Cu at (213.7, 248.6)
- added C155: 100n_0603, WLIB_Capacitor:C_0603, F.Cu at (217.3, 151.5)
- added C156: 100n_0603, WLIB_Capacitor:C_0603, F.Cu at (217.3, 154.0)
- added C157: 100n_0603, WLIB_Capacitor:C_0603, F.Cu at (212.2, 228.2)
- added C158: 15p_0603, WLIB_Capacitor:C_0603, F.Cu at (104.1, 199.1)
- added C159: 15p_0603, WLIB_Capacitor:C_0603, F.Cu at (104.1, 201.6)
- added C16: 25uF_2220, Capacitor_SMD:C_2220_5650Metric_Pad1.97x5.40mm_HandSolder, F.Cu at (210.1, 134.4)
- added C160: 15p_0603, WLIB_Capacitor:C_0603, F.Cu at (104.1, 204.1)
- added C161: 100n_0603, WLIB_Capacitor:C_0603, F.Cu at (104.1, 206.6)
- added C162: 100n_0603, WLIB_Capacitor:C_0603, F.Cu at (104.1, 209.1)
- added C17: 4u7_0603, WLIB_Capacitor:C_0603, F.Cu at (197.5, 112.7)
- added C18: 1n_0603, WLIB_Capacitor:C_0603, F.Cu at (197.5, 115.2)
- added C19: 56pF_0603, Capacitor_SMD:C_0603_1608Metric_Pad1.08x0.95mm_HandSolder, F.Cu at (197.5, 117.7)
- added C2: 1u_0603, WLIB_Capacitor:C_0603, F.Cu at (232.6, 212.5)
- added C20: 10u_1210, WLIB_Capacitor:C_1210, F.Cu at (202.7, 124.8)
- added C21: 4u7_0603, WLIB_Capacitor:C_0603, F.Cu at (197.5, 120.2)
- added C22: 10u_1210, WLIB_Capacitor:C_1210, F.Cu at (202.7, 129.0)
- added C23: 120nF_0603, Capacitor_SMD:C_0603_1608Metric_Pad1.08x0.95mm_HandSolder, F.Cu at (197.5, 122.7)
- added C24: 1u_0603, WLIB_Capacitor:C_0603, F.Cu at (197.5, 125.2)
- added C25: 4u7_0603, WLIB_Capacitor:C_0603, F.Cu at (197.5, 127.8)
- added C26: 10u_1210, WLIB_Capacitor:C_1210, F.Cu at (202.7, 133.3)
- added C27: 4u7_0603, WLIB_Capacitor:C_0603, F.Cu at (197.5, 130.3)
- added C28: 15p_0603, WLIB_Capacitor:C_0603, F.Cu at (242.3, 148.4)
- added C29: 15p_0603, WLIB_Capacitor:C_0603, F.Cu at (242.3, 150.9)
- added C3: 100n_0603, WLIB_Capacitor:C_0603, F.Cu at (232.6, 215.0)
- added C30: 15p_0603, WLIB_Capacitor:C_0603, F.Cu at (242.3, 153.5)
- added C31: 100n_0603, WLIB_Capacitor:C_0603, F.Cu at (242.3, 156.0)
- added C32: 100n_0603, WLIB_Capacitor:C_0603, F.Cu at (242.3, 158.5)
- added C33: 15p_0603, WLIB_Capacitor:C_0603, F.Cu at (227.8, 123.8)
- added C34: 15p_0603, WLIB_Capacitor:C_0603, F.Cu at (227.8, 126.4)
- added C35: 15p_0603, WLIB_Capacitor:C_0603, F.Cu at (227.8, 128.9)
- added C36: 100n_0603, WLIB_Capacitor:C_0603, F.Cu at (227.8, 131.4)
- added C37: 100n_0603, WLIB_Capacitor:C_0603, F.Cu at (227.8, 133.9)
- added C38: 15p_0603, WLIB_Capacitor:C_0603, F.Cu at (227.8, 99.3)
- added C39: 15p_0603, WLIB_Capacitor:C_0603, F.Cu at (227.8, 101.8)
- added C4: 100n_0603, WLIB_Capacitor:C_0603, F.Cu at (232.6, 217.5)
- added C40: 15p_0603, WLIB_Capacitor:C_0603, F.Cu at (227.8, 104.3)
- added C41: 100n_0603, WLIB_Capacitor:C_0603, F.Cu at (227.8, 106.8)
- added C42: 100n_0603, WLIB_Capacitor:C_0603, F.Cu at (227.8, 109.3)
- added C43: 15p_0603, WLIB_Capacitor:C_0603, F.Cu at (242.3, 99.3)
- added C44: 15p_0603, WLIB_Capacitor:C_0603, F.Cu at (242.3, 101.8)
- added C45: 15p_0603, WLIB_Capacitor:C_0603, F.Cu at (242.3, 104.3)
- added C46: 100n_0603, WLIB_Capacitor:C_0603, F.Cu at (242.3, 106.8)
- added C47: 100n_0603, WLIB_Capacitor:C_0603, F.Cu at (242.3, 109.3)
- added C48: 100n_0603, WLIB_Capacitor:C_0603, F.Cu at (54.0, 242.5)
- added C49: 10u_1210, WLIB_Capacitor:C_1210, F.Cu at (44.8, 238.2)
- added C5: 100n_0603, WLIB_Capacitor:C_0603, F.Cu at (232.6, 220.0)
- added C50: 1u_0603, WLIB_Capacitor:C_0603, F.Cu at (74.8, 245.6)
- added C51: 1u_0603, WLIB_Capacitor:C_0603, F.Cu at (74.8, 248.1)
- added C52: 10u_1210, WLIB_Capacitor:C_1210, F.Cu at (44.8, 242.5)
- added C53: 10u_1210, WLIB_Capacitor:C_1210, F.Cu at (44.8, 246.7)
- added C54: 100n_0603, WLIB_Capacitor:C_0603, F.Cu at (146.0, 211.9)
- added C55: 100n_0603, WLIB_Capacitor:C_0603, F.Cu at (146.0, 214.4)
- added C56: 100n_0603, WLIB_Capacitor:C_0603, F.Cu at (146.0, 216.9)
- added C57: 100n_0603, WLIB_Capacitor:C_0603, F.Cu at (146.0, 219.4)
- added C58: 1u_0603, WLIB_Capacitor:C_0603, F.Cu at (232.6, 177.5)
- added C59: 1u_0603, WLIB_Capacitor:C_0603, F.Cu at (232.6, 180.0)
- added C6: 100n_0603, WLIB_Capacitor:C_0603, F.Cu at (232.6, 222.5)
- added C60: 100n_0603, WLIB_Capacitor:C_0603, F.Cu at (232.6, 182.5)
- added C61: 100n_0603, WLIB_Capacitor:C_0603, F.Cu at (232.6, 185.0)
- added C62: 100n_0603, WLIB_Capacitor:C_0603, F.Cu at (232.6, 187.5)
- added C63: 100n_0603, WLIB_Capacitor:C_0603, F.Cu at (232.6, 190.0)
- added C64: 100n_0603, WLIB_Capacitor:C_0603, F.Cu at (237.0, 177.5)
- added C65: 100n_0603, WLIB_Capacitor:C_0603, F.Cu at (237.0, 180.0)
- added C66: 100n_0603, WLIB_Capacitor:C_0603, F.Cu at (237.0, 182.5)
- added C67: 100n_0603, WLIB_Capacitor:C_0603, F.Cu at (237.0, 185.0)
- added C68: 1u_0603, WLIB_Capacitor:C_0603, F.Cu at (237.0, 187.5)
- added C69: 10u_1210, WLIB_Capacitor:C_1210, F.Cu at (227.4, 178.3)
- added C7: 100n_0603, WLIB_Capacitor:C_0603, F.Cu at (237.0, 210.0)
- added C70: 10u_1210, WLIB_Capacitor:C_1210, F.Cu at (227.4, 182.6)
- added C71: 10u_1210, WLIB_Capacitor:C_1210, F.Cu at (227.4, 186.8)
- added C72: 10u_1210, WLIB_Capacitor:C_1210, F.Cu at (227.4, 191.1)
- added C73: 15p_0603, WLIB_Capacitor:C_0603, F.Cu at (160.5, 229.1)
- added C74: 15p_0603, WLIB_Capacitor:C_0603, F.Cu at (160.5, 231.6)
- added C75: 15p_0603, WLIB_Capacitor:C_0603, F.Cu at (160.5, 234.1)
- added C76: 100n_0603, WLIB_Capacitor:C_0603, F.Cu at (160.5, 236.6)
- added C77: 100n_0603, WLIB_Capacitor:C_0603, F.Cu at (160.5, 239.1)
- added C78: 15p_0603, WLIB_Capacitor:C_0603, F.Cu at (159.5, 196.8)
- added C79: 15p_0603, WLIB_Capacitor:C_0603, F.Cu at (159.5, 199.3)
- added C8: 100n_0603, WLIB_Capacitor:C_0603, F.Cu at (237.0, 212.5)
- added C80: 15p_0603, WLIB_Capacitor:C_0603, F.Cu at (159.5, 201.8)
- added C81: 100n_0603, WLIB_Capacitor:C_0603, F.Cu at (159.5, 204.3)
- added C82: 100n_0603, WLIB_Capacitor:C_0603, F.Cu at (159.5, 206.8)
- added C83: 15p_0603, WLIB_Capacitor:C_0603, F.Cu at (227.8, 148.4)
- added C84: 15p_0603, WLIB_Capacitor:C_0603, F.Cu at (227.8, 150.9)
- added C85: 15p_0603, WLIB_Capacitor:C_0603, F.Cu at (227.8, 153.5)
- added C86: 100n_0603, WLIB_Capacitor:C_0603, F.Cu at (227.8, 156.0)
- added C87: 100n_0603, WLIB_Capacitor:C_0603, F.Cu at (227.8, 158.5)
- added C88: 15p_0603, WLIB_Capacitor:C_0603, F.Cu at (242.3, 123.8)
- added C89: 15p_0603, WLIB_Capacitor:C_0603, F.Cu at (242.3, 126.4)
- added C9: 100n_0603, WLIB_Capacitor:C_0603, F.Cu at (237.0, 215.0)
- added C90: 15p_0603, WLIB_Capacitor:C_0603, F.Cu at (242.3, 128.9)
- added C91: 100n_0603, WLIB_Capacitor:C_0603, F.Cu at (242.3, 131.4)
- added C92: 100n_0603, WLIB_Capacitor:C_0603, F.Cu at (242.3, 133.9)
- added C93: 15p_0603, WLIB_Capacitor:C_0603, F.Cu at (104.1, 164.9)
- added C94: 15p_0603, WLIB_Capacitor:C_0603, F.Cu at (104.1, 167.4)
- added C95: 15p_0603, WLIB_Capacitor:C_0603, F.Cu at (104.1, 170.0)
- added C96: 100n_0603, WLIB_Capacitor:C_0603, F.Cu at (104.1, 172.5)
- added C97: 100n_0603, WLIB_Capacitor:C_0603, F.Cu at (104.1, 175.0)
- added C98: 15p_0603, WLIB_Capacitor:C_0603, F.Cu at (104.1, 182.0)
- added C99: 15p_0603, WLIB_Capacitor:C_0603, F.Cu at (104.1, 184.5)
- added D1: B72590D50H160, Capacitor_SMD:C_0402_1005Metric_Pad0.74x0.62mm_HandSolder, F.Cu at (107.5, 80.2)
- added D10: LED_G_0603, LED_SMD:LED_0603_1608Metric, F.Cu at (53.9, 247.5)
- added D11: LED_B_0603, LED_SMD:LED_0603_1608Metric, F.Cu at (149.3, 196.8)
- added D12: LED_G_0603, LED_SMD:LED_0603_1608Metric, F.Cu at (149.3, 199.4)
- added D13: LED_R_0603, LED_SMD:LED_0603_1608Metric, F.Cu at (149.3, 202.0)
- added D14: B72590D50H160, Capacitor_SMD:C_0402_1005Metric_Pad0.74x0.62mm_HandSolder, F.Cu at (88.6, 237.1)
- added D15: B72590D50H160, Capacitor_SMD:C_0402_1005Metric_Pad0.74x0.62mm_HandSolder, F.Cu at (88.6, 239.1)
- added D16: B72590D50H160, Capacitor_SMD:C_0402_1005Metric_Pad0.74x0.62mm_HandSolder, F.Cu at (88.6, 241.0)
- added D17: B72590D50H160, Capacitor_SMD:C_0402_1005Metric_Pad0.74x0.62mm_HandSolder, F.Cu at (88.6, 243.0)
- added D18: B72590D50H160, Capacitor_SMD:C_0402_1005Metric_Pad0.74x0.62mm_HandSolder, F.Cu at (88.6, 245.0)
- added D19: B72590D50H160, Capacitor_SMD:C_0402_1005Metric_Pad0.74x0.62mm_HandSolder, F.Cu at (88.6, 246.9)
- added D20: B72590D50H160, Capacitor_SMD:C_0402_1005Metric_Pad0.74x0.62mm_HandSolder, F.Cu at (91.8, 237.1)
- added D21: B72590D50H160, Capacitor_SMD:C_0402_1005Metric_Pad0.74x0.62mm_HandSolder, F.Cu at (91.8, 239.1)
- added D22: B72590D50H160, Capacitor_SMD:C_0402_1005Metric_Pad0.74x0.62mm_HandSolder, F.Cu at (91.8, 241.0)
- added D23: B72590D50H160, Capacitor_SMD:C_0402_1005Metric_Pad0.74x0.62mm_HandSolder, F.Cu at (91.8, 243.0)
- added D24: LED_G_0603, LED_SMD:LED_0603_1608Metric, F.Cu at (64.6, 245.6)
- added D3: B72590D50H160, Capacitor_SMD:C_0402_1005Metric_Pad0.74x0.62mm_HandSolder, F.Cu at (107.5, 82.2)
- added D4: B72590D50H160, Capacitor_SMD:C_0402_1005Metric_Pad0.74x0.62mm_HandSolder, F.Cu at (107.5, 84.2)
- added D5: SBR10U200P5-13, MYLIB_Misc:SBR10U200P5, F.Cu at (203.8, 114.2)
- added D6: SBR10U200P5-13, MYLIB_Misc:SBR10U200P5, F.Cu at (203.8, 119.9)
- added D7: LED_G_0603, LED_SMD:LED_0603_1608Metric, F.Cu at (213.7, 139.2)
- added D8: LED_G_0603, LED_SMD:LED_0603_1608Metric, F.Cu at (207.1, 147.9)
- added D9: LED_G_0603, LED_SMD:LED_0603_1608Metric, F.Cu at (79.0, 245.6)
- added J1: PinHeader_03_male, Connector_PinHeader_2.54mm:PinHeader_1x03_P2.54mm_Vertical, F.Cu at (241.5, 225.2)
- added J10: PinHeader_2x4_SMD, Connector_PinHeader_2.54mm:PinHeader_2x04_P2.54mm_Vertical_SMD, F.Cu at (176.3, 233.1)
- added J11: PinHeader_2x4_SMD, Connector_PinHeader_2.54mm:PinHeader_2x04_P2.54mm_Vertical_SMD, F.Cu at (176.3, 200.6)
- added J12: Box_Header_2x05_THT, Connector_IDC:IDC-Header_2x05_P2.54mm_Vertical, F.Cu at (125.1, 157.9)
- added J13: Box_Header_2x05_THT, Connector_IDC:IDC-Header_2x05_P2.54mm_Vertical, F.Cu at (137.1, 157.9)
- added J14: Box_Header_2x05_THT, Connector_IDC:IDC-Header_2x05_P2.54mm_Vertical, F.Cu at (149.1, 157.9)
- added J15: Box_Header_2x05_THT, Connector_IDC:IDC-Header_2x05_P2.54mm_Vertical, F.Cu at (161.1, 157.9)
- added J16: PinHeader_2x4_SMD, Connector_PinHeader_2.54mm:PinHeader_2x04_P2.54mm_Vertical_SMD, F.Cu at (203.6, 233.1)
- added J18: Plug_Terminal_2x12pin, MYLIB_Misc:DMCV 1,5_12-G1F-3,5-LR P20THR, F.Cu at (145.9, 144.8)
- added J19: PinHeader_03_male, Connector_PinHeader_2.54mm:PinHeader_1x03_P2.54mm_Vertical, F.Cu at (241.5, 192.7)
- added J2: PinHeader_2x4_SMD, Connector_PinHeader_2.54mm:PinHeader_2x04_P2.54mm_Vertical_SMD, F.Cu at (203.6, 200.6)
- added J20: JST_XH_05_vertical, Connector_JST:JST_XH_B5B-XH-A_1x05_P2.50mm_Vertical, F.Cu at (173.3, 244.6)
- added J21: Plug_Terminal_2x4pin, MYLIB_Misc:DMC 1,5_ 8-G1-3,5 P20THR, F.Cu at (136.3, 235.5)
- added J3: Banana_Socket_Red, MYLIB_Misc:Banana_Socket_Altech_Red, F.Cu at (181.3, 153.4)
- added J4: Banana_Socket_Black, MYLIB_Misc:Banana_Socket_Aletch_Black, F.Cu at (193.0, 166.2)
- added J5: Box_Header_6pin, Connector_IDC:IDC-Header_2x03_P2.54mm_Vertical, F.Cu at (125.1, 182.3)
- added J6: Box_Header_6pin, Connector_IDC:IDC-Header_2x03_P2.54mm_Vertical, F.Cu at (137.1, 182.3)
- added J7: Box_Header_6pin, Connector_IDC:IDC-Header_2x03_P2.54mm_Vertical, F.Cu at (149.1, 182.3)
- added J8: Box_Header_6pin, Connector_IDC:IDC-Header_2x03_P2.54mm_Vertical, F.Cu at (161.1, 182.3)
- added J9: Box_Header_26pin, Connector_IDC:IDC-Header_2x13_P2.54mm_Vertical, F.Cu at (111.1, 42.6)
- added L1: XAL1010-152MED, Inductor_SMD:L_Coilcraft_XAL1010-XXX, F.Cu at (201.4, 104.7)
- added L2: XAL1010-152MED, Inductor_SMD:L_Coilcraft_XAL1010-XXX, F.Cu at (213.5, 104.7)
- added Q1: IPT017N12NM6, Package_TO_SOT_SMD:Infineon_PG-HSOF-8-1, F.Cu at (187.9, 103.8)
- added Q2: IPT017N12NM6, Package_TO_SOT_SMD:Infineon_PG-HSOF-8-1, F.Cu at (187.9, 115.5)
- added Q3: IPT017N12NM6, Package_TO_SOT_SMD:Infineon_PG-HSOF-8-1, F.Cu at (187.9, 127.1)
- added Q4: IPT017N12NM6, Package_TO_SOT_SMD:Infineon_PG-HSOF-8-1, F.Cu at (187.9, 138.8)
- added R1: 0R002_1206, Resistor_SMD:R_1206_3216Metric_Pad1.30x1.75mm_HandSolder, F.Cu at (208.7, 139.5)
- added R10: 30R_0603, Resistor_SMD:R_0603_1608Metric, F.Cu at (238.1, 150.9)
- added R100: 1k_0603, Resistor_SMD:R_0603_1608Metric, F.Cu at (238.1, 141.4)
- added R101: 9k1_0603, Resistor_SMD:R_0603_1608Metric, F.Cu at (238.1, 143.9)
- added R102: 30R_0603, Resistor_SMD:R_0603_1608Metric, F.Cu at (99.9, 164.9)
- added R103: 30R_0603, Resistor_SMD:R_0603_1608Metric, F.Cu at (99.9, 167.4)
- added R104: 500R_0603, Resistor_SMD:R_0603_1608Metric, F.Cu at (99.9, 170.0)
- added R105: 5k1_0603, Resistor_SMD:R_0603_1608Metric, F.Cu at (99.9, 172.5)
- added R106: 500R_0603, Resistor_SMD:R_0603_1608Metric, F.Cu at (99.9, 175.0)
- added R107: 5k1_0603, Resistor_SMD:R_0603_1608Metric, F.Cu at (99.9, 177.5)
- added R108: 10k_0603, Resistor_SMD:R_0603_1608Metric, F.Cu at (68.6, 245.6)
- added R11: 500R_0603, Resistor_SMD:R_0603_1608Metric, F.Cu at (238.1, 153.5)
- added R111: 30R_0603, Resistor_SMD:R_0603_1608Metric, F.Cu at (99.9, 182.0)
- added R112: 30R_0603, Resistor_SMD:R_0603_1608Metric, F.Cu at (99.9, 184.5)
- added R113: 500R_0603, Resistor_SMD:R_0603_1608Metric, F.Cu at (99.9, 187.0)
- added R114: 5k1_0603, Resistor_SMD:R_0603_1608Metric, F.Cu at (99.9, 189.5)
- added R115: 500R_0603, Resistor_SMD:R_0603_1608Metric, F.Cu at (99.9, 192.0)
- added R116: 5k1_0603, Resistor_SMD:R_0603_1608Metric, F.Cu at (99.9, 194.5)
- added R12: 5k1_0603, Resistor_SMD:R_0603_1608Metric, F.Cu at (238.1, 156.0)
- added R120: 30R_0603, Resistor_SMD:R_0603_1608Metric, F.Cu at (226.4, 235.8)
- added R121: 30R_0603, Resistor_SMD:R_0603_1608Metric, F.Cu at (226.4, 238.3)
- added R122: 500R_0603, Resistor_SMD:R_0603_1608Metric, F.Cu at (226.4, 240.8)
- added R123: 5k1_0603, Resistor_SMD:R_0603_1608Metric, F.Cu at (226.4, 243.4)
- added R124: 500R_0603, Resistor_SMD:R_0603_1608Metric, F.Cu at (226.4, 245.9)
- added R125: 5k1_0603, Resistor_SMD:R_0603_1608Metric, F.Cu at (226.4, 248.4)
- added R129: 30R_0603, Resistor_SMD:R_0603_1608Metric, F.Cu at (99.9, 216.1)
- added R13: 500R_0603, Resistor_SMD:R_0603_1608Metric, F.Cu at (238.1, 158.5)
- added R130: 30R_0603, Resistor_SMD:R_0603_1608Metric, F.Cu at (99.9, 218.6)
- added R131: 500R_0603, Resistor_SMD:R_0603_1608Metric, F.Cu at (99.9, 221.1)
- added R132: 5k1_0603, Resistor_SMD:R_0603_1608Metric, F.Cu at (99.9, 223.6)
- added R133: 500R_0603, Resistor_SMD:R_0603_1608Metric, F.Cu at (99.9, 226.2)
- added R134: 5k1_0603, Resistor_SMD:R_0603_1608Metric, F.Cu at (99.9, 228.7)
- added R138: 30R_0603, Resistor_SMD:R_0603_1608Metric, F.Cu at (233.7, 81.9)
- added R139: 30R_0603, Resistor_SMD:R_0603_1608Metric, F.Cu at (233.7, 84.4)
- added R14: 5k1_0603, Resistor_SMD:R_0603_1608Metric, F.Cu at (238.1, 161.0)
- added R140: 500R_0603, Resistor_SMD:R_0603_1608Metric, F.Cu at (233.7, 86.9)
- added R141: 5k1_0603, Resistor_SMD:R_0603_1608Metric, F.Cu at (233.7, 89.4)
- added R142: 500R_0603, Resistor_SMD:R_0603_1608Metric, F.Cu at (233.7, 92.0)
- added R143: 5k1_0603, Resistor_SMD:R_0603_1608Metric, F.Cu at (233.7, 94.5)
- added R147: 30R_0603, Resistor_SMD:R_0603_1608Metric, F.Cu at (99.9, 233.2)
- added R148: 30R_0603, Resistor_SMD:R_0603_1608Metric, F.Cu at (99.9, 235.7)
- added R149: 500R_0603, Resistor_SMD:R_0603_1608Metric, F.Cu at (99.9, 238.2)
- added R15: 9k1_0603, Resistor_SMD:R_0603_1608Metric, F.Cu at (238.1, 163.5)
- added R150: 5k1_0603, Resistor_SMD:R_0603_1608Metric, F.Cu at (99.9, 240.7)
- added R151: 500R_0603, Resistor_SMD:R_0603_1608Metric, F.Cu at (99.9, 243.2)
- added R152: 5k1_0603, Resistor_SMD:R_0603_1608Metric, F.Cu at (99.9, 245.7)
- added R16: 1k_0603, Resistor_SMD:R_0603_1608Metric, F.Cu at (238.1, 166.0)
- added R165: 10k_0603, Resistor_SMD:R_0603_1608Metric, F.Cu at (218.8, 59.8)
- added R166: 10k_0603, Resistor_SMD:R_0603_1608Metric, F.Cu at (218.8, 62.3)
- added R167: 10k_0603, Resistor_SMD:R_0603_1608Metric, F.Cu at (218.8, 64.9)
- added R168: 10k_0603, Resistor_SMD:R_0603_1608Metric, F.Cu at (218.8, 67.4)
- added R169: 10k_0603, Resistor_SMD:R_0603_1608Metric, F.Cu at (218.8, 69.9)
- added R17: 9k1_0603, Resistor_SMD:R_0603_1608Metric, F.Cu at (238.1, 168.5)
- added R170: 10k_0603, Resistor_SMD:R_0603_1608Metric, F.Cu at (218.8, 72.4)
- added R171: 10k_0603, Resistor_SMD:R_0603_1608Metric, F.Cu at (218.8, 74.9)
- added R172: 10k_0603, Resistor_SMD:R_0603_1608Metric, F.Cu at (218.8, 77.4)
- added R173: 10k_0603, Resistor_SMD:R_0603_1608Metric, F.Cu at (218.8, 37.8)
- added R174: 10k_0603, Resistor_SMD:R_0603_1608Metric, F.Cu at (218.8, 40.3)
- added R175: 10k_0603, Resistor_SMD:R_0603_1608Metric, F.Cu at (218.8, 42.8)
- added R176: 10k_0603, Resistor_SMD:R_0603_1608Metric, F.Cu at (218.8, 45.3)
- added R177: 10k_0603, Resistor_SMD:R_0603_1608Metric, F.Cu at (218.8, 47.8)
- added R178: 10k_0603, Resistor_SMD:R_0603_1608Metric, F.Cu at (218.8, 50.3)
- added R179: 10k_0603, Resistor_SMD:R_0603_1608Metric, F.Cu at (218.8, 52.8)
- added R18: 30R_0603, Resistor_SMD:R_0603_1608Metric, F.Cu at (223.6, 123.8)
- added R180: 10k_0603, Resistor_SMD:R_0603_1608Metric, F.Cu at (218.8, 55.3)
- added R181: 10k_0603, Resistor_SMD:R_0603_1608Metric, F.Cu at (203.9, 37.8)
- added R182: 10k_0603, Resistor_SMD:R_0603_1608Metric, F.Cu at (203.9, 40.3)
- added R183: 10k_0603, Resistor_SMD:R_0603_1608Metric, F.Cu at (203.9, 42.8)
- added R184: 10k_0603, Resistor_SMD:R_0603_1608Metric, F.Cu at (203.9, 45.3)
- added R185: 10k_0603, Resistor_SMD:R_0603_1608Metric, F.Cu at (203.9, 47.8)
- added R186: 10k_0603, Resistor_SMD:R_0603_1608Metric, F.Cu at (203.9, 50.3)
- added R187: 10k_0603, Resistor_SMD:R_0603_1608Metric, F.Cu at (203.9, 52.8)
- added R188: 10k_0603, Resistor_SMD:R_0603_1608Metric, F.Cu at (203.9, 55.3)
- added R189: 10k_0603, Resistor_SMD:R_0603_1608Metric, F.Cu at (203.9, 59.8)
- added R19: 30R_0603, Resistor_SMD:R_0603_1608Metric, F.Cu at (223.6, 126.4)
- added R190: 10k_0603, Resistor_SMD:R_0603_1608Metric, F.Cu at (203.9, 62.3)
- added R191: 10k_0603, Resistor_SMD:R_0603_1608Metric, F.Cu at (203.9, 64.9)
- added R192: 10k_0603, Resistor_SMD:R_0603_1608Metric, F.Cu at (203.9, 67.4)
- added R193: 10k_0603, Resistor_SMD:R_0603_1608Metric, F.Cu at (203.9, 69.9)
- added R194: 10k_0603, Resistor_SMD:R_0603_1608Metric, F.Cu at (203.9, 72.4)
- added R195: 10k_0603, Resistor_SMD:R_0603_1608Metric, F.Cu at (203.9, 74.9)
- added R196: 10k_0603, Resistor_SMD:R_0603_1608Metric, F.Cu at (203.9, 77.4)
- added R2: 25k5_0603, Resistor_SMD:R_0603_1608Metric_Pad0.98x0.95mm_HandSolder, F.Cu at (197.5, 132.8)
- added R20: 500R_0603, Resistor_SMD:R_0603_1608Metric, F.Cu at (223.6, 128.9)
- added R200: 10k_0603, Resistor_SMD:R_0603_1608Metric, F.Cu at (99.9, 142.9)
- added R201: 10k_0603, Resistor_SMD:R_0603_1608Metric, F.Cu at (99.9, 145.4)
- added R202: 10k_0603, Resistor_SMD:R_0603_1608Metric, F.Cu at (99.9, 147.9)
- added R203: 10k_0603, Resistor_SMD:R_0603_1608Metric, F.Cu at (99.9, 150.4)
- added R204: 10k_0603, Resistor_SMD:R_0603_1608Metric, F.Cu at (99.9, 152.9)
- added R205: 10k_0603, Resistor_SMD:R_0603_1608Metric, F.Cu at (99.9, 155.4)
- added R206: 10k_0603, Resistor_SMD:R_0603_1608Metric, F.Cu at (99.9, 157.9)
- added R207: 10k_0603, Resistor_SMD:R_0603_1608Metric, F.Cu at (99.9, 160.4)
- added R208: 10k_0603, Resistor_SMD:R_0603_1608Metric, F.Cu at (233.7, 37.8)
- added R209: 10k_0603, Resistor_SMD:R_0603_1608Metric, F.Cu at (233.7, 40.3)
- added R21: 5k1_0603, Resistor_SMD:R_0603_1608Metric, F.Cu at (223.6, 131.4)
- added R210: 10k_0603, Resistor_SMD:R_0603_1608Metric, F.Cu at (233.7, 42.8)
- added R211: 10k_0603, Resistor_SMD:R_0603_1608Metric, F.Cu at (233.7, 45.3)
- added R212: 10k_0603, Resistor_SMD:R_0603_1608Metric, F.Cu at (233.7, 47.8)
- added R213: 10k_0603, Resistor_SMD:R_0603_1608Metric, F.Cu at (233.7, 50.3)
- added R214: 10k_0603, Resistor_SMD:R_0603_1608Metric, F.Cu at (233.7, 52.8)
- added R215: 10k_0603, Resistor_SMD:R_0603_1608Metric, F.Cu at (233.7, 55.3)
- added R216: 10k_0603, Resistor_SMD:R_0603_1608Metric, F.Cu at (199.1, 246.1)
- added R217: 10k_0603, Resistor_SMD:R_0603_1608Metric, F.Cu at (199.1, 248.6)
- added R218: 10k_0603, Resistor_SMD:R_0603_1608Metric, F.Cu at (218.8, 85.6)
- added R219: 10k_0603, Resistor_SMD:R_0603_1608Metric, F.Cu at (218.8, 88.1)
- added R22: 500R_0603, Resistor_SMD:R_0603_1608Metric, F.Cu at (223.6, 133.9)
- added R220: 0R_0603, Resistor_SMD:R_0603_1608Metric, F.Cu at (203.9, 85.6)
- added R221: 0R_0603, Resistor_SMD:R_0603_1608Metric, F.Cu at (203.9, 88.1)
- added R225: 10k_0603, Resistor_SMD:R_0603_1608Metric, F.Cu at (233.7, 59.8)
- added R226: 10k_0603, Resistor_SMD:R_0603_1608Metric, F.Cu at (233.7, 62.3)
- added R227: 10k_0603, Resistor_SMD:R_0603_1608Metric, F.Cu at (233.7, 64.9)
- added R228: 10k_0603, Resistor_SMD:R_0603_1608Metric, F.Cu at (233.7, 67.4)
- added R229: 10k_0603, Resistor_SMD:R_0603_1608Metric, F.Cu at (233.7, 69.9)
- added R23: 5k1_0603, Resistor_SMD:R_0603_1608Metric, F.Cu at (223.6, 136.4)
- added R230: 10k_0603, Resistor_SMD:R_0603_1608Metric, F.Cu at (233.7, 72.4)
- added R231: 10k_0603, Resistor_SMD:R_0603_1608Metric, F.Cu at (233.7, 74.9)
- added R232: 10k_0603, Resistor_SMD:R_0603_1608Metric, F.Cu at (233.7, 77.4)
- added R233: 10k_0603, Resistor_SMD:R_0603_1608Metric, F.Cu at (213.1, 162.2)
- added R234: 10k_0603, Resistor_SMD:R_0603_1608Metric, F.Cu at (213.1, 164.7)
- added R238: 10k_0603, Resistor_SMD:R_0603_1608Metric, F.Cu at (209.5, 246.1)
- added R239: 10k_0603, Resistor_SMD:R_0603_1608Metric, F.Cu at (209.5, 248.6)
- added R24: 9k1_0603, Resistor_SMD:R_0603_1608Metric, F.Cu at (223.6, 138.9)
- added R240: 0R_0603, Resistor_SMD:R_0603_1608Metric, F.Cu at (213.1, 151.5)
- added R241: 0R_0603, Resistor_SMD:R_0603_1608Metric, F.Cu at (213.1, 154.0)
- added R245: 30R_0603, Resistor_SMD:R_0603_1608Metric, F.Cu at (99.9, 199.1)
- added R246: 30R_0603, Resistor_SMD:R_0603_1608Metric, F.Cu at (99.9, 201.6)
- added R247: 500R_0603, Resistor_SMD:R_0603_1608Metric, F.Cu at (99.9, 204.1)
- added R248: 5k1_0603, Resistor_SMD:R_0603_1608Metric, F.Cu at (99.9, 206.6)
- added R249: 500R_0603, Resistor_SMD:R_0603_1608Metric, F.Cu at (99.9, 209.1)
- added R25: 1k_0603, Resistor_SMD:R_0603_1608Metric, F.Cu at (223.6, 141.4)
- added R250: 5k1_0603, Resistor_SMD:R_0603_1608Metric, F.Cu at (99.9, 211.6)
- added R26: 9k1_0603, Resistor_SMD:R_0603_1608Metric, F.Cu at (223.6, 143.9)
- added R27: 30R_0603, Resistor_SMD:R_0603_1608Metric, F.Cu at (223.6, 99.3)
- added R28: 30R_0603, Resistor_SMD:R_0603_1608Metric, F.Cu at (223.6, 101.8)
- added R29: 500R_0603, Resistor_SMD:R_0603_1608Metric, F.Cu at (223.6, 104.3)
- added R3: 2R2_0603, Resistor_SMD:R_0603_1608Metric, F.Cu at (216.0, 123.9)
- added R30: 5k1_0603, Resistor_SMD:R_0603_1608Metric, F.Cu at (223.6, 106.8)
- added R31: 500R_0603, Resistor_SMD:R_0603_1608Metric, F.Cu at (223.6, 109.3)
- added R32: 5k1_0603, Resistor_SMD:R_0603_1608Metric, F.Cu at (223.6, 111.8)
- added R33: 9k1_0603, Resistor_SMD:R_0603_1608Metric, F.Cu at (223.6, 114.3)
- added R34: 1k_0603, Resistor_SMD:R_0603_1608Metric, F.Cu at (223.6, 116.8)
- added R35: 9k1_0603, Resistor_SMD:R_0603_1608Metric, F.Cu at (223.6, 119.3)
- added R36: 30R_0603, Resistor_SMD:R_0603_1608Metric, F.Cu at (238.1, 99.3)
- added R37: 30R_0603, Resistor_SMD:R_0603_1608Metric, F.Cu at (238.1, 101.8)
- added R38: 500R_0603, Resistor_SMD:R_0603_1608Metric, F.Cu at (238.1, 104.3)
- added R39: 5k1_0603, Resistor_SMD:R_0603_1608Metric, F.Cu at (238.1, 106.8)
- added R4: 39k2_0603, Resistor_SMD:R_0603_1608Metric_Pad0.98x0.95mm_HandSolder, F.Cu at (197.5, 135.3)
- added R40: 500R_0603, Resistor_SMD:R_0603_1608Metric, F.Cu at (238.1, 109.3)
- added R41: 5k1_0603, Resistor_SMD:R_0603_1608Metric, F.Cu at (238.1, 111.8)
- added R42: 9k1_0603, Resistor_SMD:R_0603_1608Metric, F.Cu at (238.1, 114.3)
- added R43: 1k_0603, Resistor_SMD:R_0603_1608Metric, F.Cu at (238.1, 116.8)
- added R44: 9k1_0603, Resistor_SMD:R_0603_1608Metric, F.Cu at (238.1, 119.3)
- added R45: 820k_0603, Resistor_SMD:R_0603_1608Metric_Pad0.98x0.95mm_HandSolder, F.Cu at (54.0, 245.0)
- added R46: 100k_0603, Resistor_SMD:R_0603_1608Metric, F.Cu at (49.8, 242.5)
- added R47: 10k_0603, Resistor_SMD:R_0603_1608Metric, F.Cu at (83.0, 245.6)
- added R48: 10k_0603, Resistor_SMD:R_0603_1608Metric, F.Cu at (49.8, 245.0)
- added R49: 10k_0603, Resistor_SMD:R_0603_1608Metric, F.Cu at (133.8, 211.9)
- added R5: 2R2_0603, Resistor_SMD:R_0603_1608Metric, F.Cu at (216.0, 126.4)
- added R50: 10k_0603, Resistor_SMD:R_0603_1608Metric, F.Cu at (133.8, 214.4)
- added R51: 10k_0603, Resistor_SMD:R_0603_1608Metric, F.Cu at (133.8, 216.9)
- added R52: 10k_0603, Resistor_SMD:R_0603_1608Metric, F.Cu at (133.8, 219.4)
- added R53: 10k_0603, Resistor_SMD:R_0603_1608Metric, F.Cu at (133.8, 221.9)
- added R54: Poti_10k, MYLIB_Misc:RK09D1130A1N, F.Cu at (126.7, 202.0)
- added R55: 10k_0603, Resistor_SMD:R_0603_1608Metric, F.Cu at (133.8, 224.5)
- added R56: 100R_0603, Resistor_SMD:R_0603_1608Metric, F.Cu at (137.8, 211.9)
- added R57: 10k_0603, Resistor_SMD:R_0603_1608Metric, F.Cu at (137.8, 214.4)
- added R58: 100R_0603, Resistor_SMD:R_0603_1608Metric, F.Cu at (137.8, 216.9)
- added R59: 100R_0603, Resistor_SMD:R_0603_1608Metric, F.Cu at (137.8, 219.4)
- added R6: 0R002_1206, Resistor_SMD:R_1206_3216Metric_Pad1.30x1.75mm_HandSolder, F.Cu at (208.7, 142.8)
- added R60: 10k_0603, Resistor_SMD:R_0603_1608Metric, F.Cu at (137.8, 221.9)
- added R61: 10k_0603, Resistor_SMD:R_0603_1608Metric, F.Cu at (137.8, 224.5)
- added R62: 10k_0603, Resistor_SMD:R_0603_1608Metric, F.Cu at (141.8, 211.9)
- added R63: Poti_10k, MYLIB_Misc:RK09D1130A1N, F.Cu at (140.4, 202.0)
- added R64: 10k_0603, Resistor_SMD:R_0603_1608Metric, F.Cu at (141.8, 214.4)
- added R65: 100R_0603, Resistor_SMD:R_0603_1608Metric, F.Cu at (141.8, 216.9)
- added R66: 30R_0603, Resistor_SMD:R_0603_1608Metric, F.Cu at (156.3, 229.1)
- added R67: 30R_0603, Resistor_SMD:R_0603_1608Metric, F.Cu at (156.3, 231.6)
- added R68: 500R_0603, Resistor_SMD:R_0603_1608Metric, F.Cu at (156.3, 234.1)
- added R69: 5k1_0603, Resistor_SMD:R_0603_1608Metric, F.Cu at (156.3, 236.6)
- added R7: 10k_0603, Resistor_SMD:R_0603_1608Metric, F.Cu at (216.0, 128.9)
- added R70: 500R_0603, Resistor_SMD:R_0603_1608Metric, F.Cu at (156.3, 239.1)
- added R71: 5k1_0603, Resistor_SMD:R_0603_1608Metric, F.Cu at (156.3, 241.7)
- added R72: 9k1_0603, Resistor_SMD:R_0603_1608Metric, F.Cu at (156.3, 244.2)
- added R73: 1k_0603, Resistor_SMD:R_0603_1608Metric, F.Cu at (156.3, 246.7)
- added R74: 9k1_0603, Resistor_SMD:R_0603_1608Metric, F.Cu at (156.3, 249.2)
- added R75: 30R_0603, Resistor_SMD:R_0603_1608Metric, F.Cu at (155.3, 196.8)
- added R76: 30R_0603, Resistor_SMD:R_0603_1608Metric, F.Cu at (155.3, 199.3)
- added R77: 500R_0603, Resistor_SMD:R_0603_1608Metric, F.Cu at (155.3, 201.8)
- added R78: 5k1_0603, Resistor_SMD:R_0603_1608Metric, F.Cu at (155.3, 204.3)
- added R79: 500R_0603, Resistor_SMD:R_0603_1608Metric, F.Cu at (155.3, 206.8)
- added R8: 100k_0603, Resistor_SMD:R_0603_1608Metric, F.Cu at (207.0, 150.4)
- added R80: 5k1_0603, Resistor_SMD:R_0603_1608Metric, F.Cu at (155.3, 209.4)
- added R81: 9k1_0603, Resistor_SMD:R_0603_1608Metric, F.Cu at (155.3, 211.9)
- added R82: 1k_0603, Resistor_SMD:R_0603_1608Metric, F.Cu at (155.3, 214.4)
- added R83: 9k1_0603, Resistor_SMD:R_0603_1608Metric, F.Cu at (155.3, 216.9)
- added R84: 30R_0603, Resistor_SMD:R_0603_1608Metric, F.Cu at (223.6, 148.4)
- added R85: 30R_0603, Resistor_SMD:R_0603_1608Metric, F.Cu at (223.6, 150.9)
- added R86: 500R_0603, Resistor_SMD:R_0603_1608Metric, F.Cu at (223.6, 153.5)
- added R87: 5k1_0603, Resistor_SMD:R_0603_1608Metric, F.Cu at (223.6, 156.0)
- added R88: 500R_0603, Resistor_SMD:R_0603_1608Metric, F.Cu at (223.6, 158.5)
- added R89: 5k1_0603, Resistor_SMD:R_0603_1608Metric, F.Cu at (223.6, 161.0)
- added R9: 30R_0603, Resistor_SMD:R_0603_1608Metric, F.Cu at (238.1, 148.4)
- added R90: 9k1_0603, Resistor_SMD:R_0603_1608Metric, F.Cu at (223.6, 163.5)
- added R91: 1k_0603, Resistor_SMD:R_0603_1608Metric, F.Cu at (223.6, 166.0)
- added R92: 9k1_0603, Resistor_SMD:R_0603_1608Metric, F.Cu at (223.6, 168.5)
- added R93: 30R_0603, Resistor_SMD:R_0603_1608Metric, F.Cu at (238.1, 123.8)
- added R94: 30R_0603, Resistor_SMD:R_0603_1608Metric, F.Cu at (238.1, 126.4)
- added R95: 500R_0603, Resistor_SMD:R_0603_1608Metric, F.Cu at (238.1, 128.9)
- added R96: 5k1_0603, Resistor_SMD:R_0603_1608Metric, F.Cu at (238.1, 131.4)
- added R97: 500R_0603, Resistor_SMD:R_0603_1608Metric, F.Cu at (238.1, 133.9)
- added R98: 5k1_0603, Resistor_SMD:R_0603_1608Metric, F.Cu at (238.1, 136.4)
- added R99: 9k1_0603, Resistor_SMD:R_0603_1608Metric, F.Cu at (238.1, 138.9)
- added SW1: TL3305BF100QG, WLIB_Button_Switch:TL3305BF160QG, F.Cu at (125.8, 214.4)
- added SW2: TL3305BF100QG, WLIB_Button_Switch:TL3305BF160QG, F.Cu at (125.8, 222.0)
- added U1: LTC2320-16_CMOS, MYLIB_chips:UKG_52_7mm_8mm, F.Cu at (243.4, 209.4)
- added U10: BOOSTXL-3PHGANINV, MYLIB_Misc:TI_BOOSTXL_3PH, F.Cu at (195.4, 41.8)
- added U11: LTC2320-16_CMOS, MYLIB_chips:UKG_52_7mm_8mm, F.Cu at (243.4, 177.0)
- added U12: HV_Probe, MYLIB_Misc:HV_Probe, F.Cu at (69.0, 153.2)
- added U13: HV_Probe, MYLIB_Misc:HV_Probe, F.Cu at (69.0, 176.3)
- added U14: HV_Probe, MYLIB_Misc:HV_Probe, F.Cu at (69.0, 199.4)
- added U15: HV_Probe, MYLIB_Misc:HV_Probe, F.Cu at (69.0, 222.5)
- added U16: 1819_IS8, MYLIB_Misc:LT1819, F.Cu at (162.5, 243.7)
- added U17: 1819_IS8, MYLIB_Misc:LT1819, F.Cu at (161.5, 211.4)
- added U18: 1819_IS8, MYLIB_Misc:LT1819, F.Cu at (229.8, 163.0)
- added U19: 1819_IS8, MYLIB_Misc:LT1819, F.Cu at (244.3, 138.4)
- added U2: Zynq7020, MYLIB_Misc:Zynq7020, F.Cu at (47.4, 89.0)
- added U20: 1819_IS8, MYLIB_Misc:LT1819, F.Cu at (110.5, 167.0)
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