File: FPGA_Board_BA/PCB/FPGA_Board_BA.kicad_pcb (KiCad board)
At the start: 2 copper layers, 470 parts, among them J1 PinHeader_03_male, J10 PinHeader_2x4_SMD, J11 PinHeader_2x4_SMD, J12 Box_Header_2x05_THT, J13 Box_Header_2x05_THT, J14 Box_Header_2x05_THT, J15 Box_Header_2x05_THT, J16 PinHeader_2x4_SMD, J18 Plug_Terminal_2x12pin, J19 PinHeader_03_male, J2 PinHeader_2x4_SMD, J20 JST_XH_05_vertical, J21 Plug_Terminal_2x4pin, J3 Banana_Socket_Red, J4 Banana_Socket_Black, J5 Box_Header_6pin, J6 Box_Header_6pin, J7 Box_Header_6pin, J8 Box_Header_6pin, J9 Box_Header_26pin, Q1 IPT017N12NM6, Q2 IPT017N12NM6, Q3 IPT017N12NM6, Q4 IPT017N12NM6, SW1 TL3305BF100QG, SW2 TL3305BF100QG, U1 LTC2320-16_CMOS, U10 BOOSTXL-3PHGANINV, U11 LTC2320-16_CMOS, U12 HV_Probe, U13 HV_Probe, U14 HV_Probe, U15 HV_Probe, U16 1819_IS8, U17 1819_IS8, U18 1819_IS8, U19 1819_IS8, U2 Zynq7020, U20 1819_IS8, U21 1819_IS8, U22 1819_IS8, U23 1819_IS8, U24 1819_IS8, U25 1819_IS8, U26 BoxHeader_24pin, U27 SN74LXCH8T245RHLR, U28 SN74LXCH8T245RHLR, U29 SN74LXCH8T245RHLR, U3 LM5143, U30 SN74LXCH8T245RHLR, U31 S22P006S05, U32 SN74LXCH8T245RHLR, U33 SN74LXCH8T245RHLR, U34 SN74LXC2T45Q1, U35 SN74LXC2T45Q1, U36 SN74LXC2T45Q1, U37 S22P006S05, U38 SN74LXCH8T245RHLR, U39 SN74LXC2T45Q1, U4 1819_IS8, U40 S22P006S05, U41 SN74LXC2T45Q1, U42 SN74LXC2T45Q1, U43 S22P006S05, U44 1819_IS8, U45 BoxHeader_24pin, U46 BoxHeader_24pin, U47 BoxHeader_24pin, U48 MCP1703AT-5002EDB, U5 1819_IS8, U6 1819_IS8, U7 1819_IS8, U8 TPS61022, U9 MCP1703AT-5002EDB

Commit message: started component placement
Parts:
- C157: moved to B.Cu
- moved U40 148.3 mm to (325.4, 225.4)
- moved U37 143.6 mm to (325.4, 202.4)
- moved C152 140.5 mm to (320.9, 230.8)
- moved C157 139.3 mm to (332.0, 157.2), turned to -90 degrees
- moved C147 136.3 mm to (319.6, 207.8)
- moved J10 134.1 mm to (306.8, 202.2), turned to 180 degrees
- moved J11 132.8 mm to (306.8, 225.2), turned to 180 degrees
- moved U43 130.8 mm to (325.4, 156.4)
- moved J16 128.6 mm to (306.8, 156.2), turned to 180 degrees
- moved C17 120.5 mm to (307.0, 62.5)
- moved C18 120.5 mm to (307.0, 65.0)
- moved C19 120.5 mm to (307.0, 67.5)
- moved C21 120.5 mm to (307.0, 70.0)
- moved C23 120.5 mm to (307.0, 72.5)
- moved C24 120.5 mm to (307.0, 75.0)
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
Commit message: placement of Power DCDC and Buffers ready
Parts:
- removed U2: Zynq7020, MYLIB_Misc:Zynq7020
- added C125: 120nF_0603, Capacitor_SMD:C_0603_1608Metric_Pad1.08x0.95mm_HandSolder, F.Cu at (370.5, 18.8)
- added C126: 25uF_2220, Capacitor_SMD:C_2220_5650Metric_Pad1.97x5.40mm_HandSolder, F.Cu at (400.5, 39.6)
- C102, C107, C112, C117, C122, C162, C29, C32, C34, C37, C39, C42, C44, C47, C74, C77, C79, C82, C84, C87, C89, C92, C97, R106, R115, R124, R13, R133, R142, R151, R22, R249, R31, R40, R70, R79, R88, R97: moved to B.Cu
- moved R149 303.2 mm to (375.5, 111.8), turned to -90 degrees
- moved R150 303.2 mm to (376.2, 116.0), turned to 180 degrees
- moved R152 301.3 mm to (372.8, 117.8), turned to 180 degrees
- moved C121 300.3 mm to (376.5, 114.2)
- moved R151 299.4 mm to (370.2, 114.5), turned to 180 degrees
- moved R148 298.7 mm to (370.2, 108.5), turned to -90 degrees
- moved C120 297.9 mm to (372.2, 108.5), turned to -90 degrees
- moved C122 296.5 mm to (370.3, 112.6), turned to 180 degrees
- moved C119 293.2 mm to (368.2, 108.5), turned to 90 degrees
- moved R147 291.1 mm to (364.2, 111.2)
- moved U25 286.8 mm to (370.2, 113.6)
- moved C118 286.4 mm to (364.2, 113.2), turned to 180 degrees
- moved R105 278.7 mm to (376.2, 136.0), turned to 180 degrees
- moved R104 278.2 mm to (375.5, 131.8), turned to -90 degrees
- moved R107 275.7 mm to (372.8, 137.8), turned to 180 degrees
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Connections:
- C23 pad 1: Net-(U3-SS1) -> Net-(U3-SS2)
- U3 pad 1: Net-(U3-SS1) -> Net-(U3-SS2)
Routing:
- net GND: track 0.00 -> 50.2 mm, vias 0 -> 9
- net /Current measure/Tamura_4/pin1: track 0.00 -> 27.8 mm
- net /Current measure/Tamura_4/pin5: track 0.00 -> 24.8 mm
- net /Current measure/Tamura_4/pin6: track 0.00 -> 22.3 mm
- net /Current measure/Tamura_4/pin3: track 0.00 -> 22.1 mm
- net /Current measure/Tamura_4/pin4: track 0.00 -> 21.2 mm
- net /Current measure/Tamura_4/pin2: track 0.00 -> 19.6 mm
- net +5VA: track 0.00 -> 16.8 mm, vias 0 -> 8
- net Net-(R85-Pad2): track 0.00 -> 7.83 mm
- net Net-(R67-Pad2): track 0.00 -> 7.83 mm
- net Net-(R19-Pad2): track 0.00 -> 7.83 mm
- net Net-(R94-Pad2): track 0.00 -> 7.83 mm
- net Net-(R76-Pad2): track 0.00 -> 7.83 mm
- net Net-(R10-Pad2): track 0.00 -> 7.83 mm
- net Net-(R28-Pad2): track 0.00 -> 7.83 mm
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Other:
- copper layers 2 -> 4

Commit message: arranged level shifters in schematic + solid progress in layout
Parts:
- removed C10, C6, C8: 100n_0603, WLIB_Capacitor:C_0603
- added U2: Zynq7020, MYLIB_Misc:Zynq7020, F.Cu at (79.2, 129.0)
- C1, C11, C12, C128, C129, C13, C130, C131, C132, C133, C134, C135, C137, C138, C139, C14, C140, C148, C149, C15, C152, C2, C3, C4, C5, C7, C9, R165, R166, R167, R168, R169, R170, R171, R172, R173, R174, R175, R176, R177, R178, R179, R180, R181, R182, R183, R184, R185, R186, R187, R188, R189, R190, R191, R192, R193, R194, R195, R196, R200, R201, R202, R203, R204, R205, R206, R207, R208, R209, R210, R211, R212, R213, R214, R215, R225, R226, R227, R228, R229, R230, R231, R232: moved to B.Cu
- moved J8 228.7 mm to (-66.1, 155.5), turned to 90 degrees
- moved J7 215.7 mm to (-66.1, 167.5), turned to 90 degrees
- moved U33 215.4 mm to (63.4, 164.2)
- moved R208 214.7 mm to (55.9, 158.0)
- moved R209 214.2 mm to (55.9, 159.8)
- moved R210 213.8 mm to (55.9, 161.5)
- moved R211 213.4 mm to (55.9, 163.2)
- moved R212 213.0 mm to (55.9, 165.0)
- moved R213 212.6 mm to (55.9, 166.8)
- moved R214 212.1 mm to (55.9, 168.5)
- moved R215 211.7 mm to (55.9, 170.2)
- moved C139 208.5 mm to (63.4, 161.2), turned to 180 degrees
- moved C140 208.1 mm to (63.4, 163.0), turned to 180 degrees
- moved J6 203.2 mm to (-66.1, 179.5), turned to 90 degrees
- moved R123 195.8 mm to (208.5, 129.0), turned to 90 degrees
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Connections:
- R106 pad 2: /ADC for B6/V_B -> Net-(U20A--)
- R115 pad 2: /ADC for B6/V_C -> Net-(U21A--)
- R124 pad 2: /ADC for B6/I_A -> Net-(U22A--)
- R133 pad 2: /ADC for B6/I_B -> Net-(U23A--)
- R142 pad 2: /ADC for B6/I_C -> Net-(U24A--)
- R151 pad 2: /ADC for B6/V_DC -> Net-(U25A--)
- R249 pad 2: /ADC for B6/V_A -> Net-(U44A--)
- U20 pad 3: /ADC for B6/V_B -> /ADC for B6/V_A
- U21 pad 3: /ADC for B6/V_C -> /ADC for B6/V_B
- U22 pad 3: /ADC for B6/I_A -> /ADC for B6/V_C
- U23 pad 3: /ADC for B6/I_B -> /ADC for B6/I_A
- U24 pad 3: /ADC for B6/I_C -> /ADC for B6/I_B
- U25 pad 3: /ADC for B6/V_DC -> /ADC for B6/I_C
- U44 pad 3: /ADC for B6/V_A -> /ADC for B6/V_DC
Routing:
- net GND: track 50.2 -> 78.3 mm, vias 9 -> 23
- net +5VA: track 16.8 -> 32.7 mm, vias 8 -> 15
- net /ADC for B6/Diffamp_7/Ain+: track 0.00 -> 8.41 mm
- net /ADC for B6/Diffamp_6/Ain+: track 0.00 -> 8.41 mm
- net /ADC for B6/Diffamp_5/Ain+: track 0.00 -> 8.41 mm
- net /ADC for B6/Diffamp_4/Ain+: track 0.00 -> 8.41 mm
- net /ADC for B6/Diffamp_3/Ain+: track 0.00 -> 8.41 mm
- net /ADC for B6/Diffamp_2/Ain+: track 0.00 -> 8.41 mm
- net /ADC for B6/Diffamp_1/Ain+: track 0.00 -> 8.41 mm
- net Net-(R246-Pad2): track 0.00 -> 8.37 mm
- net Net-(R148-Pad2): track 0.00 -> 8.37 mm
- net Net-(R139-Pad2): track 0.00 -> 8.37 mm
- net Net-(R130-Pad2): track 0.00 -> 8.37 mm
- net Net-(R121-Pad2): track 0.00 -> 8.37 mm
- net Net-(R112-Pad2): track 0.00 -> 8.37 mm
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Other:
- board text added: "5VA - 1"
- board text added: "5VA - 2"

Commit message: layout of islands is ready
Parts:
- removed C61, C63, C65: 100n_0603, WLIB_Capacitor:C_0603
- C136, C147, C58, C59, C60, C62, C64, C66, C67, C68, C69, C70, C71, C72, R221, R241: moved to B.Cu
- moved D7 385.8 mm to (22.0, 280.5)
- moved R7 385.8 mm to (18.5, 280.5)
- moved J8 369.2 mm to (296.5, 85.7), turned to -90 degrees
- moved J7 353.2 mm to (277.5, 85.5), turned to -90 degrees
- moved C125 344.0 mm to (95.8, 225.8)
- moved C126 344.0 mm to (125.8, 246.7)
- moved C16 344.0 mm to (50.5, 246.9)
- moved C17 344.0 mm to (94.0, 225.8)
- moved C18 344.0 mm to (79.8, 229.8)
- moved C19 344.0 mm to (79.8, 231.8)
- moved C20 344.0 mm to (87.0, 242.2)
- moved C21 344.0 mm to (94.8, 237.0)
- moved C22 344.0 mm to (89.5, 225.8)
- moved C23 344.0 mm to (83.2, 225.8)
- moved C24 344.0 mm to (92.2, 225.8)
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Connections:
- R1 pad 1: /Main_DCDC/Vout -> +5V
- U3 pad 26: /Main_DCDC/Vout -> +5V
Routing:
- net /Current measure/Tamura_3/pin1: track 0.00 -> 27.8 mm
- net /Current measure/Tamura_2/pin1: track 0.00 -> 27.8 mm
- net /Current measure/Tamura_1/pin1: track 0.00 -> 27.8 mm
- net /Current measure/Tamura_1/pin5: track 0.00 -> 24.8 mm
- net /Current measure/Tamura_3/pin5: track 0.00 -> 24.8 mm
- net /Current measure/Tamura_2/pin5: track 0.00 -> 24.8 mm
- net /Current measure/Tamura_3/pin6: track 0.00 -> 22.3 mm
- net /Current measure/Tamura_2/pin6: track 0.00 -> 22.3 mm
- net /Current measure/Tamura_1/pin6: track 0.00 -> 22.3 mm
- net /Current measure/Tamura_3/pin3: track 0.00 -> 22.1 mm
- net /Current measure/Tamura_2/pin3: track 0.00 -> 22.1 mm
- net /Current measure/Tamura_1/pin3: track 0.00 -> 22.1 mm
- net /Current measure/Tamura_3/pin4: track 0.00 -> 21.2 mm
- net /Current measure/Tamura_2/pin4: track 0.00 -> 21.2 mm
- net /Current measure/Tamura_1/pin4: track 0.00 -> 21.2 mm
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Other:
- board text added: "POWER 5V"
- board text added: "POWER in"

Commit message: Component placement ready. Waiting to meet with Leo
Parts:
- added L3: SMD_Inductor_1u, MYLIB_Misc:74404043010A, F.Cu at (120.7, 173.2)
- C1, C11, C12, C13, C14, C15, C2, C3, C4, C5, C7, C9: moved to F.Cu
- C43, C45, C46, C55, C56, C78, C80, C81, C83, C85, C86, C88, C90, C91, R100, R101, R36, R37, R38, R39, R41, R42, R43, R44, R56, R57, R59, R60, R75, R76, R77, R78, R80, R81, R82, R83, R84, R85, R86, R87, R89, R90, R91, R92, R93, R94, R95, R96, R98, R99, U17, U18, U19, U27, U28, U29, U30, U32, U33, U38, U7: moved to B.Cu
- moved C53 170.3 mm to (131.2, 167.2), turned to -90 degrees
- moved C50 168.1 mm to (205.3, 84.2)
- moved C51 168.1 mm to (205.3, 88.1)
- moved D9 168.1 mm to (212.2, 92.2)
- moved R47 168.1 mm to (208.7, 92.2)
- moved U9 168.1 mm to (211.2, 86.2)
- moved C154 168.0 mm to (180.7, 151.0), turned to -90 degrees
- moved C153 165.9 mm to (182.4, 151.0), turned to 90 degrees
- moved J20 162.7 mm to (140.4, 59.0), turned to -90 degrees
- moved U41 161.5 mm to (181.4, 147.5), turned to 180 degrees
- moved R238 157.7 mm to (185.7, 148.3), turned to 180 degrees
- moved R239 154.8 mm to (185.7, 146.5), turned to 180 degrees
- moved C150 154.2 mm to (184.0, 118.2)
- moved C151 154.2 mm to (185.8, 118.2)
- moved R233 154.2 mm to (180.8, 120.9)
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Routing:
- net GND: track 91.6 -> 66.0 mm, vias 25 -> 20
- net +5V: track 17.4 -> 37.5 mm, vias 2 -> 0
- net +3.3V: track 14.3 -> 34.0 mm
- net +5VA: track 32.7 -> 38.2 mm, vias 15 -> 11
- net Net-(U18B--): track 3.10 -> 7.40 mm
- net Net-(U19B--): track 3.10 -> 7.40 mm
- net Net-(U7B--): track 3.10 -> 7.40 mm
- net Net-(U17B--): track 3.10 -> 7.40 mm
- net /Main_DCDC/Comp1: track 1.81 -> 0.00 mm, vias 1 -> 0
- net Net-(U18A--): track 7.17 -> 8.77 mm, vias 1 -> 0
- net Net-(U7A--): track 7.17 -> 8.77 mm, vias 1 -> 0
- net Net-(U19A--): track 7.17 -> 8.77 mm, vias 1 -> 0
- net Net-(U17A--): track 7.17 -> 8.77 mm, vias 1 -> 0
- net /ADC for Machine/Diffamp5/Ain-: track 2.24 -> 3.83 mm, vias 1 -> 0
- net /ADC for Machine/Diffamp8/Ain-: track 2.24 -> 3.83 mm, vias 1 -> 0
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Other:
- board outline added: 272.6 x 187.2 mm
- board text added: "5.5V"
- board text added: "LED-1"
- board text added: "LED-2"
- board text added: "LED-3"
- board text added: "POTI-1"
- board text added: "POTI-2"
