File: FPGA_Board_BA/PCB/FPGA_Board_BA.kicad_pcb (KiCad board)
At the start: 4 copper layers, 272.6 x 187.2 mm, 467 parts, among them J1 PinHeader_03_male, J10 PinHeader_2x4_SMD, J11 PinHeader_2x4_SMD, J12 Box_Header_2x05_THT, J13 Box_Header_2x05_THT, J14 Box_Header_2x05_THT, J15 Box_Header_2x05_THT, J16 PinHeader_2x4_SMD, J18 Plug_Terminal_2x12pin, J19 PinHeader_03_male, J2 PinHeader_2x4_SMD, J20 JST_XH_05_vertical, J21 Plug_Terminal_2x4pin, J3 Banana_Socket_Red, J4 Banana_Socket_Black, J5 Box_Header_6pin, J6 Box_Header_6pin, J7 Box_Header_6pin, J8 Box_Header_6pin, J9 Box_Header_26pin, Q1 IPT017N12NM6, Q2 IPT017N12NM6, Q3 IPT017N12NM6, Q4 IPT017N12NM6, SW1 TL3305BF100QG, SW2 TL3305BF100QG, U1 LTC2320-16_CMOS, U10 BOOSTXL-3PHGANINV, U11 LTC2320-16_CMOS, U12 HV_Probe, U13 HV_Probe, U14 HV_Probe, U15 HV_Probe, U16 1819_IS8, U17 1819_IS8, U18 1819_IS8, U19 1819_IS8, U2 Zynq7020, U20 1819_IS8, U21 1819_IS8, U22 1819_IS8, U23 1819_IS8, U24 1819_IS8, U25 1819_IS8, U26 BoxHeader_24pin, U27 SN74LXCH8T245RHLR, U28 SN74LXCH8T245RHLR, U29 SN74LXCH8T245RHLR, U3 LM5143, U30 SN74LXCH8T245RHLR, U31 S22P006S05, U32 SN74LXCH8T245RHLR, U33 SN74LXCH8T245RHLR, U34 SN74LXC2T45Q1, U35 SN74LXC2T45Q1, U36 SN74LXC2T45Q1, U37 S22P006S05, U38 SN74LXCH8T245RHLR, U39 SN74LXC2T45Q1, U4 1819_IS8, U40 S22P006S05, U41 SN74LXC2T45Q1, U42 SN74LXC2T45Q1, U43 S22P006S05, U44 1819_IS8, U45 BoxHeader_24pin, U46 BoxHeader_24pin, U47 BoxHeader_24pin, U48 MCP1703AT-5002EDB, U5 1819_IS8, U6 1819_IS8, U7 1819_IS8, U8 TPS61022, U9 MCP1703AT-5002EDB

Commit message: Placement optimised
Parts:
- removed L2: XAL1010-152MED, Inductor_SMD:L_Coilcraft_XAL1010-XXX
- removed Q3, Q4: IPT017N12NM6, Package_TO_SOT_SMD:Infineon_PG-HSOF-8-1
- removed R6: 0R002_1206, Resistor_SMD:R_1206_3216Metric_Pad1.30x1.75mm_HandSolder
- added L4: XAL1010-152MED, Inductor_SMD:L_Coilcraft_XAL1010-XXX, F.Cu at (78.8, 211.2)
- added Q5: IPT017N12NM6, Package_TO_SOT_SMD:Infineon_PG-HSOF-8-1, F.Cu at (65.3, 197.9)
- added Q6: IPT017N12NM6, Package_TO_SOT_SMD:Infineon_PG-HSOF-8-1, F.Cu at (81.1, 198.1)
- added R109: 0R002_1206, Resistor_SMD:R_1206_3216Metric_Pad1.30x1.75mm_HandSolder, F.Cu at (78.8, 220.5)
- moved J15 151.9 mm to (303.1, 60.7)
- moved J14 151.8 mm to (279.9, 60.7)
- moved J13 151.4 mm to (256.2, 60.7)
- moved J12 150.5 mm to (231.9, 60.7)
- moved J9 102.5 mm to (145.2, 227.2), turned to 180 degrees
- moved R59 50.2 mm to (203.7, 62.5)
- moved R60 50.2 mm to (203.7, 60.8)
- moved SW2 50.2 mm to (203.7, 60.8)
- moved C56 50.2 mm to (203.5, 59.0)
- moved J1 41.2 mm to (129.2, 109.3), turned to 135 degrees
- moved J20 41.1 mm to (180.0, 70.2), turned to 0 degrees
- moved C55 40.2 mm to (203.7, 67.8)
- moved R56 40.2 mm to (203.7, 71.2)
- moved R57 40.2 mm to (203.7, 69.5)
- moved SW1 40.2 mm to (203.7, 69.5)
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Connections:
- net Net-(Q1-G) renamed /Main_DCDC/Leg-1/Gate_H
- net Net-(Q1-S) renamed /Main_DCDC/Leg-1/SW
- net Net-(Q2-G) renamed /Main_DCDC/Leg-1/Gate_L
- net Net-(Q3-G) renamed /Main_DCDC/Leg-2/Gate_H
- net Net-(Q3-S) renamed /Main_DCDC/Leg-2/SW
- net Net-(Q4-G) renamed /Main_DCDC/Leg-2/Gate_L
- net Net-(U3-CS1) renamed /Main_DCDC/Leg-1/R_I+
- U2 pad a11: /ADC for B6/SDO3 -> /FPGA/PWM_BL
- U2 pad a13: /ADC for B6/SDO4 -> /FPGA/PWM_BH
- U2 pad a16: /ADC for B6/SDO7 -> /FPGA/OT
- U2 pad a17: /ADC for B6/SDO5 -> /FPGA/PWM_AL
- U2 pad a18: /ADC for B6/SDO8 -> /FPGA/B6_En
- U2 pad a19: /ADC for B6/SDO6 -> /FPGA/PWM_AH
- U2 pad a20: /ADC for B6/~{CNV} -> unconnected-(U2C-IO_L21P_T3_13-Pada20)
- U2 pad a21: /ADC for B6/CLK_IN -> unconnected-(U2C-IO_L15P_T2_13-Pada21)
- U2 pad a22: /FPGA/LED3 -> unconnected-(U2C-IO_L21N_T3_13-Pada22)
- U2 pad a23: /ADC for B6/CLK_OUT -> unconnected-(U2C-IO_L15N_T2_13-Pada23)
- U2 pad a7: /ADC for B6/SDO1 -> /FPGA/PWM_CL
- U2 pad a9: /ADC for B6/SDO2 -> /FPGA/PWM_CH
- U2 pad b36: /FPGA/PWM_BH -> unconnected-(U2B-IO_L8P_T1_35-Padb36)
- U2 pad b37: /FPGA/PWM_AH -> unconnected-(U2B-IO_L7P_T1_35-Padb37)
- U2 pad b38: /FPGA/PWM_BL -> unconnected-(U2B-IO_L8N_T1_35-Padb38)
- U2 pad b39: /FPGA/PWM_AL -> unconnected-(U2B-IO_L7N_T1_35-Padb39)
- U2 pad b42: /FPGA/B6_En -> unconnected-(U2B-IO_L10P_T1_35-Padb42)
- U2 pad b43: /FPGA/PWM_CH -> unconnected-(U2B-IO_L9P_T1_35-Padb43)
- U2 pad b44: /FPGA/OT -> unconnected-(U2B-IO_L10N_T1_35-Padb44)
- U2 pad b45: /FPGA/PWM_CL -> unconnected-(U2B-IO_L9N_T1_35-Padb45)
- U3 pad 4: Net-(U3-CS2) -> /Main_DCDC/Leg-2/R_I+
Routing:
- net /Main_DCDC/Leg-1/R_I+: track 0.00 -> 58.8 mm, vias 0 -> 2
- net +5V: track 37.5 -> 95.7 mm, vias 0 -> 2
- added copper zone on F.Cu, net /Main_DCDC/Leg-1/R_I+
- added copper zone on F.Cu, net /Main_DCDC/Leg-1/SW
- added copper zone on B.Cu, net /Main_DCDC/Vin
- added copper zone on F.Cu, net /Main_DCDC/Vin
Other:
- outline, holes or cut-outs redrawn
