File: FPGA_Board_BA/PCB/FPGA_Board_BA.kicad_pcb (KiCad board)
At the start: 4 copper layers, 272.6 x 187.2 mm, 467 parts, among them J1 PinHeader_03_male, J10 PinHeader_2x4_SMD, J11 PinHeader_2x4_SMD, J12 Box_Header_2x05_THT, J13 Box_Header_2x05_THT, J14 Box_Header_2x05_THT, J15 Box_Header_2x05_THT, J16 PinHeader_2x4_SMD, J18 Plug_Terminal_2x12pin, J19 PinHeader_03_male, J2 PinHeader_2x4_SMD, J20 JST_XH_05_vertical, J21 Plug_Terminal_2x4pin, J3 Banana_Socket_Red, J4 Banana_Socket_Black, J5 Box_Header_6pin, J6 Box_Header_6pin, J7 Box_Header_6pin, J8 Box_Header_6pin, J9 Box_Header_26pin, Q1 IPT017N12NM6, Q2 IPT017N12NM6, Q5 IPT017N12NM6, Q6 IPT017N12NM6, SW1 TL3305BF100QG, SW2 TL3305BF100QG, U1 LTC2320-16_CMOS, U10 BOOSTXL-3PHGANINV, U11 LTC2320-16_CMOS, U12 HV_Probe, U13 HV_Probe, U14 HV_Probe, U15 HV_Probe, U16 1819_IS8, U17 1819_IS8, U18 1819_IS8, U19 1819_IS8, U2 Zynq7020, U20 1819_IS8, U21 1819_IS8, U22 1819_IS8, U23 1819_IS8, U24 1819_IS8, U25 1819_IS8, U26 BoxHeader_24pin, U27 SN74LXCH8T245RHLR, U28 SN74LXCH8T245RHLR, U29 SN74LXCH8T245RHLR, U3 LM5143, U30 SN74LXCH8T245RHLR, U31 S22P006S05, U32 SN74LXCH8T245RHLR, U33 SN74LXCH8T245RHLR, U34 SN74LXC2T45Q1, U35 SN74LXC2T45Q1, U36 SN74LXC2T45Q1, U37 S22P006S05, U38 SN74LXCH8T245RHLR, U39 SN74LXC2T45Q1, U4 1819_IS8, U40 S22P006S05, U41 SN74LXC2T45Q1, U42 SN74LXC2T45Q1, U43 S22P006S05, U44 1819_IS8, U45 BoxHeader_24pin, U46 BoxHeader_24pin, U47 BoxHeader_24pin, U48 MCP1703AT-5002EDB, U5 1819_IS8, U6 1819_IS8, U7 1819_IS8, U8 TPS61022, U9 MCP1703AT-5002EDB

Commit message: component placement with new concept is ready
Parts:
- removed C28, C29, C30, C33, C34, C35, C38, C39, C40, C73, C74, C75: 15p_0603, WLIB_Capacitor:C_0603
- removed C31, C32, C36, C37, C41, C42, C76, C77: 100n_0603, WLIB_Capacitor:C_0603
- removed J1, J19: PinHeader_03_male, Connector_PinHeader_2.54mm:PinHeader_1x03_P2.54mm_Vertical
- removed J21: Plug_Terminal_2x4pin, MYLIB_Misc:DMC 1,5_ 8-G1-3,5 P20THR
- removed R109: 0R002_1206, Resistor_SMD:R_1206_3216Metric_Pad1.30x1.75mm_HandSolder
- removed R30, R32, R69, R71: 5k1_0603, Resistor_SMD:R_0603_1608Metric
- removed R31, R68, R70: 500R_0603, Resistor_SMD:R_0603_1608Metric
- removed R33, R35, R72, R74: 9k1_0603, Resistor_SMD:R_0603_1608Metric
- removed R34, R73: 1k_0603, Resistor_SMD:R_0603_1608Metric
- removed R66, R67: 30R_0603, Resistor_SMD:R_0603_1608Metric
- removed U16, U4, U5, U6: 1819_IS8, MYLIB_Misc:LT1819
- added C10: 100n_0603, WLIB_Capacitor:C_0603, F.Cu at (287.2, 192.1)
- added C127: 100n_0603, WLIB_Capacitor:C_0603, F.Cu at (327.2, 192.1)
- added C163: 100n_0603, WLIB_Capacitor:C_0603, F.Cu at (337.3, 192.4)
- added C6: 100n_0603, WLIB_Capacitor:C_0603, F.Cu at (267.2, 192.1)
- added C61: 100n_0603, WLIB_Capacitor:C_0603, F.Cu at (297.3, 192.4)
- added C63: 100n_0603, WLIB_Capacitor:C_0603, F.Cu at (307.2, 192.1)
- added C65: 100n_0603, WLIB_Capacitor:C_0603, F.Cu at (317.3, 192.4)
- added C8: 100n_0603, WLIB_Capacitor:C_0603, F.Cu at (277.3, 192.4)
- added J17: Plug_Terminal_2x4_Vertical, MYLIB_Misc:Plug_Terminal_2x4_Vertical, F.Cu at (350.0, 170.1)
- added R110: 1k_0603, Resistor_SMD:R_0603_1608Metric, B.Cu at (131.8, 146.3)
- added R119: 1k_0603, Resistor_SMD:R_0603_1608Metric, F.Cu at (267.2, 195.6)
- added R126: 1k_0603, Resistor_SMD:R_0603_1608Metric, F.Cu at (267.2, 193.9)
- added R135: 1k_0603, Resistor_SMD:R_0603_1608Metric, F.Cu at (277.3, 195.9)
- added R136: 1k_0603, Resistor_SMD:R_0603_1608Metric, F.Cu at (277.3, 194.1)
- added R137: 1k_0603, Resistor_SMD:R_0603_1608Metric, F.Cu at (274.3, 199.8)
- added R144: 1k_0603, Resistor_SMD:R_0603_1608Metric, F.Cu at (272.3, 199.8)
- added R145: 1k_0603, Resistor_SMD:R_0603_1608Metric, F.Cu at (270.3, 199.8)
- added R156: 1k_0603, Resistor_SMD:R_0603_1608Metric, F.Cu at (287.2, 193.9)
- added R157: 1k_0603, Resistor_SMD:R_0603_1608Metric, F.Cu at (287.2, 195.6)
- added R158: 1k_0603, Resistor_SMD:R_0603_1608Metric, F.Cu at (297.3, 195.9)
- added R159: 1k_0603, Resistor_SMD:R_0603_1608Metric, F.Cu at (297.3, 194.1)
- added R160: 1k_0603, Resistor_SMD:R_0603_1608Metric, F.Cu at (290.3, 199.8)
- added R161: 1k_0603, Resistor_SMD:R_0603_1608Metric, F.Cu at (294.3, 199.8)
- added R162: 1k_0603, Resistor_SMD:R_0603_1608Metric, F.Cu at (292.3, 199.8)
- added R199: 1k_0603, Resistor_SMD:R_0603_1608Metric, F.Cu at (307.2, 193.9)
- added R222: 1k_0603, Resistor_SMD:R_0603_1608Metric, F.Cu at (307.2, 195.6)
- added R223: 1k_0603, Resistor_SMD:R_0603_1608Metric, F.Cu at (317.3, 195.9)
- added R224: 1k_0603, Resistor_SMD:R_0603_1608Metric, F.Cu at (317.3, 194.1)
- added R235: 1k_0603, Resistor_SMD:R_0603_1608Metric, F.Cu at (310.3, 199.8)
- added R236: 1k_0603, Resistor_SMD:R_0603_1608Metric, F.Cu at (314.3, 199.8)
- added R237: 1k_0603, Resistor_SMD:R_0603_1608Metric, F.Cu at (312.3, 199.8)
- added R252: 1k_0603, Resistor_SMD:R_0603_1608Metric, F.Cu at (327.2, 193.9)
- added R253: 1k_0603, Resistor_SMD:R_0603_1608Metric, F.Cu at (327.2, 195.6)
- added R254: 1k_0603, Resistor_SMD:R_0603_1608Metric, F.Cu at (337.3, 195.9)
- added R255: 1k_0603, Resistor_SMD:R_0603_1608Metric, F.Cu at (337.3, 194.1)
- added R256: 1k_0603, Resistor_SMD:R_0603_1608Metric, F.Cu at (330.3, 199.8)
- added R257: 1k_0603, Resistor_SMD:R_0603_1608Metric, F.Cu at (334.3, 199.8)
- added R258: 1k_0603, Resistor_SMD:R_0603_1608Metric, F.Cu at (332.3, 199.8)
- added R6: 1k_0603, Resistor_SMD:R_0603_1608Metric, B.Cu at (131.8, 148.1)
- added REF**: MountingHole_3.2mm_M3, MountingHole:MountingHole_3.2mm_M3, F.Cu at (59.8, 59.0)
- added REF**: MountingHole_3.2mm_M3, MountingHole:MountingHole_3.2mm_M3, F.Cu at (76.8, 113.8)
- added REF**: MountingHole_3.2mm_M3, MountingHole:MountingHole_3.2mm_M3, F.Cu at (346.5, 56.8)
- added REF**: MountingHole_3.2mm_M3, MountingHole:MountingHole_3.2mm_M3, F.Cu at (350.0, 157.2)
- added REF**: MountingHole_3.2mm_M3, MountingHole:MountingHole_3.2mm_M3, F.Cu at (350.0, 182.8)
- added REF**: MountingHole_3.2mm_M3, MountingHole:MountingHole_3.2mm_M3, F.Cu at (56.2, 206.2)
- added REF**: MountingHole_3.2mm_M3, MountingHole:MountingHole_3.2mm_M3, F.Cu at (184.5, 196.2)
- added REF**: MountingHole_3.2mm_M3, MountingHole:MountingHole_3.2mm_M3, F.Cu at (56.0, 153.5)
- added REF**: MountingHole_3.2mm_M3, MountingHole:MountingHole_3.2mm_M3, F.Cu at (256.0, 85.8)
- added REF**: MountingHole_3.2mm_M3, MountingHole:MountingHole_3.2mm_M3, F.Cu at (345.5, 84.2)
- added REF**: MountingHole_3.2mm_M3, MountingHole:MountingHole_3.2mm_M3, F.Cu at (162.5, 42.8)
- added REF**: MountingHole_3.2mm_M3, MountingHole:MountingHole_3.2mm_M3, F.Cu at (125.2, 60.2)
- added REF**: MountingHole_3.2mm_M3, MountingHole:MountingHole_3.2mm_M3, F.Cu at (255.5, 55.5)
- added REF**: MountingHole_3.2mm_M3, MountingHole:MountingHole_3.2mm_M3, F.Cu at (259.0, 171.5)
- added REF**: MountingHole_3.2mm_M3, MountingHole:MountingHole_3.2mm_M3, F.Cu at (346.8, 206.2)
- C128, C129, C130, C131, C132, C133, C134, C135, C137, C138, C139, C140, C148, C149, C43, C44, C45, C46, C47, C58, C59, C60, C62, C64, C66, C67, C68, C69, C70, C71, C72, C78, C79, C80, C81, C82, C83, C84, C85, C86, C87, C88, C89, C90, C91, C92, R100, R101, R165, R166, R167, R168, R169, R170, R171, R172, R173, R174, R175, R176, R177, R178, R179, R180, R181, R182, R183, R184, R185, R186, R187, R188, R189, R190, R191, R192, R193, R194, R195, R196, R200, R201, R202, R203, R204, R205, R206, R207, R208, R209, R210, R211, R212, R213, R214, R215, R225, R226, R227, R228, R229, R230, R231, R232, R36, R37, R38, R39, R40, R41, R42, R43, R44, R75, R76, R77, R78, R79, R80, R81, R82, R83, R84, R85, R86, R87, R88, R89, R90, R91, R92, R93, R94, R95, R96, R97, R98, R99, U17, U18, U19, U27, U28, U29, U30, U32, U33, U38, U7: moved to F.Cu
- R1: value 0R002_1206 -> 0R_0603; footprint Resistor_SMD:R_1206_3216Metric_Pad1.30x1.75mm_HandSolder -> Resistor_SMD:R_0603_1608Metric
- R10, R18, R19, R9: value 30R_0603 -> 100k_1206; footprint Resistor_SMD:R_0603_1608Metric -> Resistor_SMD:R_1206_3216Metric
- R11, R20: value 500R_0603 -> 100k_1206; footprint Resistor_SMD:R_0603_1608Metric -> Resistor_SMD:R_1206_3216Metric
- R12, R14, R21, R23: value 5k1_0603 -> 100k_1206; footprint Resistor_SMD:R_0603_1608Metric -> Resistor_SMD:R_1206_3216Metric
- R13, R22: value 500R_0603 -> 100k_1206; footprint Resistor_SMD:R_0603_1608Metric -> Resistor_SMD:R_1206_3216Metric; moved to F.Cu
- R15, R17, R24: value 9k1_0603 -> 100k_1206; footprint Resistor_SMD:R_0603_1608Metric -> Resistor_SMD:R_1206_3216Metric
- R16: value 1k_0603 -> 100k_1206; footprint Resistor_SMD:R_0603_1608Metric -> Resistor_SMD:R_1206_3216Metric
- R25: value 1k_0603 -> 0R002_2512; footprint Resistor_SMD:R_0603_1608Metric -> Resistor_SMD:R_2512_6332Metric
- R26: value 9k1_0603 -> 0R002_2512; footprint Resistor_SMD:R_0603_1608Metric -> Resistor_SMD:R_2512_6332Metric
- R27, R28: value 30R_0603 -> 0R_0603
- R29: value 500R_0603 -> 0R_0603
- U12, U13, U14, U15: value HV_Probe -> 1819_IS8; footprint MYLIB_Misc:HV_Probe -> MYLIB_Misc:LT1819
- moved U26 218.4 mm to (279.5, 61.8)
- moved U45 218.4 mm to (279.5, 76.8)
- moved U46 218.4 mm to (320.5, 61.8)
- moved U47 218.4 mm to (320.5, 76.8)
- moved R26 217.0 mm to (79.0, 75.5), turned to -90 degrees
- moved R25 189.2 mm to (112.0, 75.5), turned to -90 degrees
- moved J18 171.6 mm to (95.2, 60.0), turned to 0 degrees
- moved D7 159.5 mm to (58.8, 71.0), turned to 0 degrees
- moved R7 159.3 mm to (62.3, 71.0), turned to 180 degrees
- moved R28 155.5 mm to (141.6, 142.7)
- moved R29 148.9 mm to (143.4, 142.7)
- moved D8 148.5 mm to (58.5, 76.5), turned to 0 degrees
- moved R8 148.3 mm to (62.2, 76.5), turned to 0 degrees
- moved R1 132.8 mm to (239.9, 186.0), turned to 180 degrees
- moved L4 129.3 mm to (112.0, 86.2), turned to -90 degrees
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Connections:
- R1 pad 1: +5V -> Net-(U11-~{SDR}/DDR)
- R1 pad 2: /Main_DCDC/Leg-1/R_I+ -> +1V8
- R10 pad 1: /ADC for Machine/Diffamp2/Ain- -> /Current measure/Tamura_3/pin4
- R11 pad 1: Net-(R10-Pad2) -> /Current measure/Tamura_4/pin4
- R11 pad 2: Net-(U4B--) -> Net-(R11-Pad2)
- R12 pad 1: GND -> /Current measure/Tamura_1/pin4
- R12 pad 2: Net-(U4B-+) -> Net-(R12-Pad2)
- R13 pad 1: Net-(U4B--) -> Net-(R13-Pad1)
- R13 pad 2: Net-(U4A--) -> Net-(U12A-+)
- R14 pad 1: Net-(U4B-+) -> Net-(R10-Pad2)
- R14 pad 2: REFOUT_M -> Net-(U13A-+)
- R15 pad 1: Net-(U4A-+) -> Net-(R11-Pad2)
- R15 pad 2: GND -> Net-(U14A-+)
- R16 pad 1: /ADC for Machine/Vout_2 -> Net-(R12-Pad2)
- R16 pad 2: Net-(U4A-+) -> Net-(U15A-+)
- R17 pad 1: Net-(U4A-+) -> /CHB to 3Ph/Ph_B2_out
- R17 pad 2: GND -> Net-(R17-Pad2)
- R18 pad 1: /ADC for Machine/Diffamp3/Ain+ -> Net-(R17-Pad2)
- R18 pad 2: Net-(U5A--) -> Net-(U12A--)
- R19 pad 1: /ADC for Machine/Diffamp3/Ain- -> /CHB to 3Ph/Ph_C2_out
- R20 pad 2: Net-(U5B--) -> Net-(U13A--)
- R21 pad 1: GND -> /CHB to 3Ph/Ph_D2_out
- R21 pad 2: Net-(U5B-+) -> Net-(R21-Pad2)
- R22 pad 1: Net-(U5B--) -> Net-(R21-Pad2)
- R22 pad 2: Net-(U5A--) -> Net-(U14A--)
- R23 pad 1: Net-(U5B-+) -> /CHB to 3Ph/Ph_A2_out
- R23 pad 2: REFOUT_M -> Net-(R23-Pad2)
- R24 pad 1: Net-(U5A-+) -> Net-(R23-Pad2)
- R24 pad 2: GND -> Net-(U15A--)
- R25 pad 1: /ADC for Machine/Vout_3 -> +5V
- R25 pad 2: Net-(U5A-+) -> /Main_DCDC/Leg-2/R_I+
- R26 pad 1: Net-(U5A-+) -> +5V
- R26 pad 2: GND -> /Main_DCDC/Leg-1/R_I+
- R27 pad 1: /ADC for Machine/Diffamp4/Ain+ -> Net-(U11-~{SDR}/DDR)
- R27 pad 2: Net-(U6A--) -> GND
- R28 pad 1: /ADC for Machine/Diffamp4/Ain- -> Net-(U1-~{SDR}/DDR)
- R28 pad 2: Net-(R28-Pad2) -> +1V8
- R29 pad 1: Net-(R28-Pad2) -> Net-(U1-~{SDR}/DDR)
- R29 pad 2: Net-(U6B--) -> GND
- R9 pad 1: /ADC for Machine/Diffamp2/Ain+ -> /Current measure/Tamura_2/pin4
- R9 pad 2: Net-(U4A--) -> Net-(R13-Pad1)
- U1 pad 23: Net-(J1-Pin_2) -> Net-(U1-~{SDR}/DDR)
- U1 pad 47: unconnected-(U1-Ain8--Pad47) -> Net-(U1-Ain8-)
- U1 pad 48: unconnected-(U1-Ain8+-Pad48) -> Net-(U1-Ain8+)
- U11 pad 10: /ADC for Machine/Diffamp4/Ain- -> /ADC for Machine/Vout4-
- U11 pad 11: /ADC for Machine/Diffamp4/Ain+ -> /ADC for Machine/Vout4+
- U11 pad 13: /ADC for Machine/Diffamp3/Ain- -> /ADC for Machine/Vout3-
- U11 pad 14: /ADC for Machine/Diffamp3/Ain+ -> /ADC for Machine/Vout3+
- U11 pad 16: /ADC for Machine/Diffamp2/Ain- -> /ADC for Machine/Vout2-
- U11 pad 17: /ADC for Machine/Diffamp2/Ain+ -> /ADC for Machine/Vout2+
- U11 pad 19: /ADC for Machine/Diffamp1/Ain- -> /ADC for Machine/Vout1-
- U11 pad 20: /ADC for Machine/Diffamp1/Ain+ -> /ADC for Machine/Vout1+
- U11 pad 23: Net-(J19-Pin_2) -> Net-(U11-~{SDR}/DDR)
Routing:
- net +5V: track 95.7 -> 160.3 mm, vias 2 -> 4
- net /Main_DCDC/Leg-2/R_I+: track 0.00 -> 61.1 mm, vias 0 -> 2
- net GND: track 66.0 -> 41.4 mm, vias 20 -> 16
- net /Main_DCDC/Vin: track 0.00 -> 11.9 mm, vias 0 -> 65
- net +5VA: track 38.2 -> 29.8 mm, vias 11 -> 7
- net Net-(R67-Pad2): track 7.83 -> 0.00 mm
- net Net-(R10-Pad2): track 7.83 -> 0.00 mm
- net Net-(R28-Pad2): track 7.83 -> 0.00 mm
- net Net-(R19-Pad2): track 7.83 -> 0.00 mm
- net Net-(U4A--): track 7.17 -> 0.00 mm, vias 1 -> 0
- net Net-(U16A--): track 7.17 -> 0.00 mm, vias 1 -> 0
- net Net-(U6A--): track 7.17 -> 0.00 mm, vias 1 -> 0
- net Net-(U5A--): track 7.17 -> 0.00 mm, vias 1 -> 0
- net /Main_DCDC/Mode: track 0.00 -> 6.83 mm
- net Net-(U5B-+): track 6.17 -> 0.00 mm
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- added copper zone on F.Cu, net +5V
- added copper zone on F.Cu, net GND
- added copper zone on F.Cu, net Net-(D5-A)
Other:
- board size 272.6 x 187.2 mm -> 310.3 x 160 mm
- board text added: "A2 | B2 | C2 | D2 A1 | B1 | C1 | D1"
- board text added: "Button 1"
- board text added: "Button 2"

Commit message: started power DCDC layout
Parts:
- added C28: 15p_0603, WLIB_Capacitor:C_0603, B.Cu at (296.0, 200.0)
- added C29: 15p_0603, WLIB_Capacitor:C_0603, B.Cu at (293.4, 200.2)
- added C30: 15p_0603, WLIB_Capacitor:C_0603, B.Cu at (290.8, 200.0)
- added C31: 15p_0603, WLIB_Capacitor:C_0603, B.Cu at (316.0, 200.0)
- added C32: 15p_0603, WLIB_Capacitor:C_0603, B.Cu at (313.4, 200.2)
- added C33: 15p_0603, WLIB_Capacitor:C_0603, B.Cu at (310.8, 200.0)
- added C34: 15p_0603, WLIB_Capacitor:C_0603, B.Cu at (336.0, 200.0)
- added C35: 15p_0603, WLIB_Capacitor:C_0603, B.Cu at (333.4, 200.2)
- added C36: 15p_0603, WLIB_Capacitor:C_0603, B.Cu at (330.8, 200.0)
- added C37: 15p_0603, WLIB_Capacitor:C_0603, B.Cu at (276.0, 200.0)
- added C38: 15p_0603, WLIB_Capacitor:C_0603, B.Cu at (273.4, 200.2)
- added C39: 15p_0603, WLIB_Capacitor:C_0603, B.Cu at (270.8, 200.0)
- added C40: 100n_0603, WLIB_Capacitor:C_0603, B.Cu at (292.2, 194.0)
- added C41: 100n_0603, WLIB_Capacitor:C_0603, B.Cu at (312.2, 194.0)
- added C42: 100n_0603, WLIB_Capacitor:C_0603, B.Cu at (332.2, 194.0)
- added C73: 100n_0603, WLIB_Capacitor:C_0603, B.Cu at (272.2, 194.0)
- added R30: 30R_0603, Resistor_SMD:R_0603_1608Metric, F.Cu at (296.0, 200.0)
- added R31: 30R_0603, Resistor_SMD:R_0603_1608Metric, F.Cu at (290.8, 200.0)
- added R32: 30R_0603, Resistor_SMD:R_0603_1608Metric, F.Cu at (316.0, 200.0)
- added R33: 30R_0603, Resistor_SMD:R_0603_1608Metric, F.Cu at (310.8, 200.0)
- added R34: 30R_0603, Resistor_SMD:R_0603_1608Metric, F.Cu at (336.0, 200.0)
- added R35: 30R_0603, Resistor_SMD:R_0603_1608Metric, F.Cu at (330.8, 200.0)
- added R66: 30R_0603, Resistor_SMD:R_0603_1608Metric, F.Cu at (276.0, 200.0)
- added R67: 30R_0603, Resistor_SMD:R_0603_1608Metric, F.Cu at (270.8, 200.0)
- moved R156 1.95 mm to (287.2, 195.8)
- moved R159 1.95 mm to (297.3, 196.1)
- moved R199 1.95 mm to (307.2, 195.8)
- moved R224 1.95 mm to (317.3, 196.1)
- moved R252 1.95 mm to (327.2, 195.8)
- moved R157 1.55 mm to (287.2, 194.1)
- moved R158 1.55 mm to (297.3, 194.3)
- moved R222 1.55 mm to (307.2, 194.1)
- moved R223 1.55 mm to (317.3, 194.3)
- moved R253 1.55 mm to (327.2, 194.1)
- moved C64 1.50 mm to (248.2, 183.6)
- moved C66 1.50 mm to (246.2, 183.6)
- moved R145 1.32 mm to (269.0, 200.0)
- moved R160 1.32 mm to (289.0, 200.0)
- moved R235 1.32 mm to (309.0, 200.0)
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Connections:
- C163 pad 2: /ADC for Machine/Vout4+ -> Net-(C163-Pad2)
- C61 pad 2: /ADC for Machine/Vout2+ -> Net-(C61-Pad2)
- C65 pad 2: /ADC for Machine/Vout3+ -> Net-(C65-Pad2)
- C8 pad 2: /ADC for Machine/Vout1+ -> Net-(C8-Pad2)
- R135 pad 2: /ADC for Machine/Vout1+ -> Net-(C8-Pad2)
- R136 pad 2: /ADC for Machine/Vout1+ -> Net-(C8-Pad2)
- R137 pad 1: /ADC for Machine/Vout1+ -> Net-(C8-Pad2)
- R144 pad 2: /ADC for Machine/Vout1- -> Net-(R144-Pad2)
- R158 pad 2: /ADC for Machine/Vout2+ -> Net-(C61-Pad2)
- R159 pad 2: /ADC for Machine/Vout2+ -> Net-(C61-Pad2)
- R161 pad 1: /ADC for Machine/Vout2+ -> Net-(C61-Pad2)
- R162 pad 2: /ADC for Machine/Vout2- -> Net-(R162-Pad2)
- R223 pad 2: /ADC for Machine/Vout3+ -> Net-(C65-Pad2)
- R224 pad 2: /ADC for Machine/Vout3+ -> Net-(C65-Pad2)
- R236 pad 1: /ADC for Machine/Vout3+ -> Net-(C65-Pad2)
- R237 pad 2: /ADC for Machine/Vout3- -> Net-(R237-Pad2)
- R254 pad 2: /ADC for Machine/Vout4+ -> Net-(C163-Pad2)
- R255 pad 2: /ADC for Machine/Vout4+ -> Net-(C163-Pad2)
- R257 pad 1: /ADC for Machine/Vout4+ -> Net-(C163-Pad2)
- R258 pad 2: /ADC for Machine/Vout4- -> Net-(R258-Pad2)
- U11 pad 1: /ADC for Machine/Diffamp6/Ain- -> /ADC for Machine/Vout2-
- U11 pad 10: /ADC for Machine/Vout4- -> /ADC for Machine/Diffamp8/Ain-
- U11 pad 11: /ADC for Machine/Vout4+ -> /ADC for Machine/Diffamp8/Ain+
- U11 pad 13: /ADC for Machine/Vout3- -> /ADC for Machine/Diffamp7/Ain-
- U11 pad 14: /ADC for Machine/Vout3+ -> /ADC for Machine/Diffamp7/Ain+
- U11 pad 16: /ADC for Machine/Vout2- -> /ADC for Machine/Diffamp6/Ain-
- U11 pad 17: /ADC for Machine/Vout2+ -> /ADC for Machine/Diffamp6/Ain+
- U11 pad 19: /ADC for Machine/Vout1- -> /ADC for Machine/Diffamp5/Ain-
- U11 pad 2: /ADC for Machine/Diffamp6/Ain+ -> /ADC for Machine/Vout2+
- U11 pad 20: /ADC for Machine/Vout1+ -> /ADC for Machine/Diffamp5/Ain+
- U11 pad 4: /ADC for Machine/Diffamp5/Ain- -> /ADC for Machine/Vout1-
- U11 pad 47: /ADC for Machine/Diffamp8/Ain- -> /ADC for Machine/Vout4-
- U11 pad 48: /ADC for Machine/Diffamp8/Ain+ -> /ADC for Machine/Vout4+
- U11 pad 5: /ADC for Machine/Diffamp5/Ain+ -> /ADC for Machine/Vout1+
- U11 pad 50: /ADC for Machine/Diffamp7/Ain- -> /ADC for Machine/Vout3-
- U11 pad 51: /ADC for Machine/Diffamp7/Ain+ -> /ADC for Machine/Vout3+
- U12 pad 1: /ADC for Machine/Vout2+ -> Net-(C61-Pad2)
- U12 pad 7: /ADC for Machine/Vout2- -> Net-(R162-Pad2)
- U13 pad 1: /ADC for Machine/Vout3+ -> Net-(C65-Pad2)
- U13 pad 7: /ADC for Machine/Vout3- -> Net-(R237-Pad2)
- U14 pad 1: /ADC for Machine/Vout4+ -> Net-(C163-Pad2)
- U14 pad 7: /ADC for Machine/Vout4- -> Net-(R258-Pad2)
- U15 pad 1: /ADC for Machine/Vout1+ -> Net-(C8-Pad2)
- U15 pad 7: /ADC for Machine/Vout1- -> Net-(R144-Pad2)
Routing:
- net REFOUT_M: track 0.00 -> 41.8 mm, vias 0 -> 1
- net +5VA: track 29.8 -> 56.3 mm, vias 7 -> 11
- net GND: track 41.4 -> 61.2 mm, vias 16 -> 68
- net +5V: track 160.3 -> 175.4 mm
- net Net-(C8-Pad2): track 0.00 -> 13.7 mm
- net Net-(C65-Pad2): track 0.00 -> 13.7 mm
- net Net-(C61-Pad2): track 0.00 -> 13.7 mm
- net Net-(C163-Pad2): track 0.00 -> 13.7 mm
- net Net-(U15A-+): track 0.00 -> 11.9 mm
- net Net-(U13A-+): track 0.00 -> 11.9 mm
- net Net-(U14A-+): track 0.00 -> 11.9 mm
- net Net-(U12A-+): track 0.00 -> 11.9 mm
- net Net-(U15A--): track 0.00 -> 11.1 mm
- net Net-(U14A--): track 0.00 -> 11.1 mm
- net Net-(U13A--): track 0.00 -> 11.1 mm
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- added copper zone on F.Cu, net /Analog Voltage/5.5V
- added copper zone on B.Cu, net GND
- added copper zone on In1.Cu, net GND
- added copper zone on In2.Cu, net GND
- added copper zone on F.Cu, net Net-(U8-FB)
- added copper zone on F.Cu, net Net-(U8-SW)

Commit message: DCDC Converter layout almost ready
Parts:
- moved R48 4.71 mm to (155.6, 134.5), turned to 180 degrees
- moved D10 4.71 mm to (152.1, 134.5)
- moved C40 4.19 mm to (291.2, 198.1)
- moved C41 4.19 mm to (311.2, 198.1)
- moved C42 4.19 mm to (331.2, 198.1)
- moved C46 4.19 mm to (271.9, 113.4)
- moved C73 4.19 mm to (271.2, 198.1)
- moved C84 4.19 mm to (302.6, 119.3)
- moved C87 4.19 mm to (305.1, 114.6)
- moved C88 4.19 mm to (325.0, 122.1)
- moved C90 4.19 mm to (325.0, 116.4)
- moved J12 4.19 mm to (270.9, 100.5)
- moved J13 4.19 mm to (295.1, 100.5)
- moved R10 4.19 mm to (309.8, 186.4)
- moved R11 4.19 mm to (329.8, 186.4)
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Routing:
- net /Current measure/Tamura_4/pin1: track 27.8 -> 114.3 mm, vias 0 -> 27
- net /Current measure/Tamura_3/pin1: track 27.8 -> 114.3 mm, vias 0 -> 27
- net /Current measure/Tamura_2/pin1: track 27.8 -> 114.3 mm, vias 0 -> 27
- net /Current measure/Tamura_1/pin1: track 27.8 -> 114.3 mm, vias 0 -> 27
- net /Current measure/Tamura_4/pin5: track 24.8 -> 102.7 mm, vias 0 -> 24
- net /Current measure/Tamura_3/pin5: track 24.8 -> 102.7 mm, vias 0 -> 24
- net /Current measure/Tamura_2/pin5: track 24.8 -> 102.7 mm, vias 0 -> 24
- net /Current measure/Tamura_1/pin5: track 24.8 -> 102.7 mm, vias 0 -> 24
- net /Current measure/Tamura_4/pin6: track 22.3 -> 91.8 mm, vias 0 -> 22
- net /Current measure/Tamura_3/pin6: track 22.3 -> 91.8 mm, vias 0 -> 22
- net /Current measure/Tamura_2/pin6: track 22.3 -> 91.8 mm, vias 0 -> 22
- net /Current measure/Tamura_1/pin6: track 22.3 -> 91.8 mm, vias 0 -> 22
- net /Current measure/Tamura_4/pin3: track 22.1 -> 89.5 mm, vias 0 -> 22
- net /Current measure/Tamura_3/pin3: track 22.1 -> 89.5 mm, vias 0 -> 22
- net /Current measure/Tamura_2/pin3: track 22.1 -> 89.5 mm, vias 0 -> 22
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