File: FPGA_Board_BA/PCB/FPGA_Board_BA.kicad_pcb (KiCad board)
At the start: 4 copper layers, 310.3 x 160 mm, 502 parts, among them J10 PinHeader_2x4_SMD, J11 PinHeader_2x4_SMD, J12 Box_Header_2x05_THT, J13 Box_Header_2x05_THT, J14 Box_Header_2x05_THT, J15 Box_Header_2x05_THT, J16 PinHeader_2x4_SMD, J17 Plug_Terminal_2x4_Vertical, J18 Plug_Terminal_2x12pin, J2 PinHeader_2x4_SMD, J20 JST_XH_05_vertical, J3 Banana_Socket_Red, J4 Banana_Socket_Black, J5 Box_Header_6pin, J6 Box_Header_6pin, J7 Box_Header_6pin, J8 Box_Header_6pin, J9 Box_Header_26pin, Q1 IPT017N12NM6, Q2 IPT017N12NM6, Q5 IPT017N12NM6, Q6 IPT017N12NM6, SW1 TL3305BF100QG, SW2 TL3305BF100QG, U1 LTC2320-16_CMOS, U10 BOOSTXL-3PHGANINV, U11 LTC2320-16_CMOS, U12 1819_IS8, U13 1819_IS8, U14 1819_IS8, U15 1819_IS8, U17 1819_IS8, U18 1819_IS8, U19 1819_IS8, U2 Zynq7020, U20 1819_IS8, U21 1819_IS8, U22 1819_IS8, U23 1819_IS8, U24 1819_IS8, U25 1819_IS8, U26 BoxHeader_24pin, U27 SN74LXCH8T245RHLR, U28 SN74LXCH8T245RHLR, U29 SN74LXCH8T245RHLR, U3 LM5143, U30 SN74LXCH8T245RHLR, U31 S22P006S05, U32 SN74LXCH8T245RHLR, U33 SN74LXCH8T245RHLR, U34 SN74LXC2T45Q1, U35 SN74LXC2T45Q1, U36 SN74LXC2T45Q1, U37 S22P006S05, U38 SN74LXCH8T245RHLR, U39 SN74LXC2T45Q1, U40 S22P006S05, U41 SN74LXC2T45Q1, U42 SN74LXC2T45Q1, U43 S22P006S05, U44 1819_IS8, U45 BoxHeader_24pin, U46 BoxHeader_24pin, U47 BoxHeader_24pin, U48 MCP1703AT-5002EDB, U7 1819_IS8, U8 TPS61022, U9 MCP1703AT-5002EDB

Commit message: small changes in the PCB
Parts:
- moved R55 3.20 mm to (154.2, 77.7), turned to 90 degrees
- moved R61 2.92 mm to (135.5, 78.0), turned to 90 degrees
- moved R62 2.31 mm to (132.0, 78.0), turned to 90 degrees
- moved R52 1.86 mm to (150.8, 77.7), turned to 90 degrees
- moved C54 1.26 mm to (157.8, 77.7), turned to 90 degrees
- moved C57 1.16 mm to (139.0, 78.0), turned to -90 degrees
- moved R64 0.88 mm to (133.8, 78.0), turned to 90 degrees
- moved R53 0.85 mm to (152.5, 77.7), turned to 90 degrees
- moved C11 0.78 mm to (134.5, 157.9)
- moved C13 0.78 mm to (137.2, 158.8)
- moved C14 0.78 mm to (131.8, 158.8)
- moved R58 0.45 mm to (156.0, 77.7), turned to -90 degrees
- moved R65 0.37 mm to (137.2, 78.0)
- moved R8 0.32 mm to (61.5, 80.5), turned to 180 degrees
- moved D8 0.24 mm to (57.8, 80.5)
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Routing:
- net +5V: track 175.4 -> 182.3 mm
- net /Main_DCDC/Vin: track 11.9 -> 16.2 mm, vias 65 -> 67
- net Net-(D8-A): track 0.00 -> 2.14 mm
- net Net-(C18-Pad1): track 0.00 -> 2.01 mm
- net Net-(D7-A): track 0.00 -> 1.89 mm
- net GND: track 81.3 -> 82.6 mm, vias 70 -> 78
- added copper zone on F.Cu, net /Main_DCDC/Leg-2/R_I+
- added copper zone on F.Cu, net /Main_DCDC/Leg-2/SW

Commit message: started routing of the right side
Parts:
- C44, C79, C84, C89: moved to B.Cu
- moved C131 92.9 mm to (235.6, 155.6), turned to -90 degrees
- moved C130 92.6 mm to (237.3, 155.6), turned to 90 degrees
- moved R173 92.5 mm to (243.9, 155.7), turned to 180 degrees
- moved R207 92.4 mm to (243.9, 63.4), turned to 180 degrees
- moved R174 89.1 mm to (243.9, 153.9), turned to 180 degrees
- moved R206 88.9 mm to (243.9, 65.2), turned to 180 degrees
- moved R175 85.6 mm to (243.9, 152.2), turned to 180 degrees
- moved R205 85.4 mm to (243.9, 66.9), turned to 180 degrees
- moved R176 82.1 mm to (243.9, 150.4), turned to 180 degrees
- moved R204 81.9 mm to (243.9, 68.7), turned to 180 degrees
- moved U32 80.5 mm to (236.4, 69.5), turned to 180 degrees
- moved U28 80.5 mm to (236.4, 149.5), turned to 180 degrees
- moved R177 78.6 mm to (243.9, 148.7), turned to 180 degrees
- moved R203 78.4 mm to (243.9, 70.4), turned to 180 degrees
- moved R178 75.1 mm to (243.9, 146.9), turned to 180 degrees
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Routing:
- net /ADC for Machine/Vout4+: track 3.04 -> 103.2 mm
- net /ADC for Machine/Vout4-: track 3.49 -> 100.7 mm, vias 2 -> 3
- net /ADC for Machine/Vout3+: track 3.79 -> 81.2 mm
- net /ADC for Machine/Vout3-: track 3.54 -> 78.5 mm, vias 2 -> 3
- net /ADC for Machine/Vout2+: track 4.00 -> 60.2 mm
- net /ADC for Machine/Vout2-: track 4.55 -> 57.4 mm, vias 2 -> 3
- net /ADC for Machine/Vout1+: track 4.04 -> 40.4 mm
- net /ADC for Machine/Vout1-: track 4.05 -> 36.9 mm, vias 2 -> 3
- net Net-(U3-HO1): track 32.0 -> 1.56 mm, vias 2 -> 1
- net /Main_DCDC/Leg-1/Gate_H: track 35.4 -> 5.52 mm, vias 2 -> 1
- net Net-(U3-HO2): track 28.9 -> 2.88 mm, vias 2 -> 1
- net /Main_DCDC/Leg-2/Gate_H: track 41.2 -> 15.9 mm, vias 3 -> 1
- net /Main_DCDC/Leg-2/SW: track 23.3 -> 3.42 mm, vias 2 -> 0
- net +5VA: track 56.3 -> 75.9 mm
- net /Main_DCDC/Leg-1/SW: track 23.2 -> 3.76 mm, vias 2 -> 0
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Other:
- board size 310.3 x 160 mm -> 310.2 x 160 mm

Commit message: right side almost finished
Parts:
- moved C130 48.0 mm to (237.3, 107.6)
- moved C131 48.0 mm to (235.6, 107.6)
- moved R173 48.0 mm to (243.9, 107.7)
- moved R174 48.0 mm to (243.9, 105.9)
- moved R175 48.0 mm to (243.9, 104.2)
- moved R176 48.0 mm to (243.9, 102.4)
- moved R177 48.0 mm to (243.9, 100.7)
- moved R178 48.0 mm to (243.9, 98.9)
- moved R179 48.0 mm to (243.9, 97.2)
- moved R180 48.0 mm to (243.9, 95.4)
- moved U28 48.0 mm to (236.4, 101.5)
- moved U45 43.7 mm to (319.8, 68.4)
- moved U46 43.7 mm to (278.8, 83.4)
- moved C134 32.0 mm to (237.3, 139.6)
- moved C135 32.0 mm to (235.6, 139.6)
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Connections:
- J12 pad 3: /CHB Communication/Ph_A_Tx1 -> /CHB Communication/Ph_A_Tx1_5V
- J13 pad 3: /CHB Communication/Ph_B_Tx1 -> /CHB Communication/Ph_B_Tx1_5V
- J14 pad 3: /CHB Communication/Ph_C_Tx1 -> /CHB Communication/Ph_C_Tx1_5V
- J15 pad 3: /CHB Communication/Ph_D_Tx1 -> /CHB Communication/Ph_D_Tx1_5V
- R168 pad 2: /CHB Communication/Level_Shifter_8bit_2/A4 -> /CHB Communication/Ph_B_Tx1_5V
- R188 pad 2: /CHB Communication/Level_Shifter_8bit_4/A8 -> /CHB Communication/Ph_C_Tx1_5V
- R192 pad 2: /CHB Communication/Level_Shifter_8bit_5/A4 -> /CHB Communication/Ph_D_Tx1_5V
- R207 pad 2: /CHB Communication/Level_Shifter_8bit_1/A8 -> /CHB Communication/Ph_A_Tx1_5V
- U26 pad 10: /CHB Communication/Level_Shifter_8bit_1/A5 -> /CHB Communication/Level_Shifter_8bit_1/A4
- U26 pad 12: /CHB Communication/Level_Shifter_8bit_1/A6 -> /CHB Communication/Level_Shifter_8bit_1/A3
- U26 pad 14: /CHB Communication/Level_Shifter_8bit_1/A7 -> /CHB Communication/Level_Shifter_8bit_1/A2
- U26 pad 16: /CHB Communication/Level_Shifter_8bit_1/A8 -> /CHB Communication/Level_Shifter_8bit_1/A1
- U26 pad 18: /CHB Communication/Level_Shifter_8bit_2/A1 -> /CHB Communication/Level_Shifter_8bit_2/A8
- U26 pad 2: /CHB Communication/Level_Shifter_8bit_1/A1 -> /CHB Communication/Ph_A_Tx1_5V
- U26 pad 20: /CHB Communication/Level_Shifter_8bit_2/A2 -> /CHB Communication/Level_Shifter_8bit_2/A7
- U26 pad 22: /CHB Communication/Level_Shifter_8bit_2/A3 -> /CHB Communication/Level_Shifter_8bit_2/A6
- U26 pad 24: /CHB Communication/Level_Shifter_8bit_2/A4 -> /CHB Communication/Level_Shifter_8bit_2/A5
- U26 pad 4: /CHB Communication/Level_Shifter_8bit_1/A2 -> /CHB Communication/Level_Shifter_8bit_1/A7
- U26 pad 6: /CHB Communication/Level_Shifter_8bit_1/A3 -> /CHB Communication/Level_Shifter_8bit_1/A6
- U26 pad 8: /CHB Communication/Level_Shifter_8bit_1/A4 -> /CHB Communication/Level_Shifter_8bit_1/A5
- U27 pad 14: /CHB Communication/Ph_B_Tx4 -> /CHB Communication/Ph_A_Tx9
- U27 pad 15: /CHB Communication/Ph_B_Tx3 -> /CHB Communication/Ph_A_Tx10
- U27 pad 16: /CHB Communication/Ph_B_Tx2 -> /CHB Communication/Ph_A_Tx11
- U27 pad 17: /CHB Communication/Ph_B_Tx1 -> /CHB Communication/Ph_A_Tx12
- U27 pad 18: /CHB Communication/Ph_A_Tx12 -> /CHB Communication/Ph_B_Tx1
- U27 pad 19: /CHB Communication/Ph_A_Tx11 -> /CHB Communication/Ph_B_Tx2
- U27 pad 20: /CHB Communication/Ph_A_Tx10 -> /CHB Communication/Ph_B_Tx3
- U27 pad 21: /CHB Communication/Ph_A_Tx9 -> /CHB Communication/Ph_B_Tx4
- U27 pad 6: /CHB Communication/Level_Shifter_8bit_2/A4 -> /CHB Communication/Ph_B_Tx1_5V
- U28 pad 14: /CHB Communication/Ph_B_Tx12 -> /CHB Communication/Ph_B_Tx5
- U28 pad 15: /CHB Communication/Ph_B_Tx11 -> /CHB Communication/Ph_B_Tx6
- U28 pad 16: /CHB Communication/Ph_B_Tx10 -> /CHB Communication/Ph_B_Tx7
- U28 pad 17: /CHB Communication/Ph_B_Tx9 -> /CHB Communication/Ph_B_Tx8
- U28 pad 18: /CHB Communication/Ph_B_Tx8 -> /CHB Communication/Ph_B_Tx9
- U28 pad 19: /CHB Communication/Ph_B_Tx7 -> /CHB Communication/Ph_B_Tx10
- U28 pad 20: /CHB Communication/Ph_B_Tx6 -> /CHB Communication/Ph_B_Tx11
- U28 pad 21: /CHB Communication/Ph_B_Tx5 -> /CHB Communication/Ph_B_Tx12
- U29 pad 10: /CHB Communication/Level_Shifter_8bit_4/A8 -> /CHB Communication/Ph_C_Tx1_5V
- U29 pad 14: /CHB Communication/Ph_C_Tx8 -> /CHB Communication/Ph_C_Tx1
- U29 pad 15: /CHB Communication/Ph_C_Tx7 -> /CHB Communication/Ph_C_Tx2
- U29 pad 16: /CHB Communication/Ph_C_Tx6 -> /CHB Communication/Ph_C_Tx3
- U29 pad 17: /CHB Communication/Ph_C_Tx5 -> /CHB Communication/Ph_C_Tx4
- U29 pad 18: /CHB Communication/Ph_C_Tx4 -> /CHB Communication/Ph_C_Tx5
- U29 pad 19: /CHB Communication/Ph_C_Tx3 -> /CHB Communication/Ph_C_Tx6
- U29 pad 20: /CHB Communication/Ph_C_Tx2 -> /CHB Communication/Ph_C_Tx7
- U29 pad 21: /CHB Communication/Ph_C_Tx1 -> /CHB Communication/Ph_C_Tx8
- U30 pad 14: /CHB Communication/Ph_D_Tx4 -> /CHB Communication/Ph_C_Tx9
- U30 pad 15: /CHB Communication/Ph_D_Tx3 -> /CHB Communication/Ph_C_Tx10
- U30 pad 16: /CHB Communication/Ph_D_Tx2 -> /CHB Communication/Ph_C_Tx11
- U30 pad 17: /CHB Communication/Ph_D_Tx1 -> /CHB Communication/Ph_C_Tx12
- U30 pad 18: /CHB Communication/Ph_C_Tx12 -> /CHB Communication/Ph_D_Tx1
- U30 pad 19: /CHB Communication/Ph_C_Tx11 -> /CHB Communication/Ph_D_Tx2
- U30 pad 20: /CHB Communication/Ph_C_Tx10 -> /CHB Communication/Ph_D_Tx3
- U30 pad 21: /CHB Communication/Ph_C_Tx9 -> /CHB Communication/Ph_D_Tx4
- U30 pad 6: /CHB Communication/Level_Shifter_8bit_5/A4 -> /CHB Communication/Ph_D_Tx1_5V
- U32 pad 10: /CHB Communication/Level_Shifter_8bit_1/A8 -> /CHB Communication/Ph_A_Tx1_5V
- U32 pad 14: /CHB Communication/Ph_A_Tx8 -> /CHB Communication/Ph_A_Tx1
- U32 pad 15: /CHB Communication/Ph_A_Tx7 -> /CHB Communication/Ph_A_Tx2
- U32 pad 16: /CHB Communication/Ph_A_Tx6 -> /CHB Communication/Ph_A_Tx3
- U32 pad 17: /CHB Communication/Ph_A_Tx5 -> /CHB Communication/Ph_A_Tx4
- U32 pad 18: /CHB Communication/Ph_A_Tx4 -> /CHB Communication/Ph_A_Tx5
- U32 pad 19: /CHB Communication/Ph_A_Tx3 -> /CHB Communication/Ph_A_Tx6
- U32 pad 20: /CHB Communication/Ph_A_Tx2 -> /CHB Communication/Ph_A_Tx7
- U32 pad 21: /CHB Communication/Ph_A_Tx1 -> /CHB Communication/Ph_A_Tx8
- U33 pad 14: /CHB Communication/Ph_D_Tx12 -> /CHB Communication/Ph_D_Tx5
- U33 pad 15: /CHB Communication/Ph_D_Tx11 -> /CHB Communication/Ph_D_Tx6
- U33 pad 16: /CHB Communication/Ph_D_Tx10 -> /CHB Communication/Ph_D_Tx7
- U33 pad 17: /CHB Communication/Ph_D_Tx9 -> /CHB Communication/Ph_D_Tx8
- U33 pad 18: /CHB Communication/Ph_D_Tx8 -> /CHB Communication/Ph_D_Tx9
- U33 pad 19: /CHB Communication/Ph_D_Tx7 -> /CHB Communication/Ph_D_Tx10
- U33 pad 20: /CHB Communication/Ph_D_Tx6 -> /CHB Communication/Ph_D_Tx11
- U33 pad 21: /CHB Communication/Ph_D_Tx5 -> /CHB Communication/Ph_D_Tx12
- U45 pad 10: /CHB Communication/Level_Shifter_8bit_3/A1 -> /CHB Communication/Level_Shifter_8bit_3/A8
- U45 pad 12: /CHB Communication/Level_Shifter_8bit_3/A2 -> /CHB Communication/Level_Shifter_8bit_3/A7
- U45 pad 14: /CHB Communication/Level_Shifter_8bit_3/A3 -> /CHB Communication/Level_Shifter_8bit_3/A6
- U45 pad 16: /CHB Communication/Level_Shifter_8bit_3/A4 -> /CHB Communication/Level_Shifter_8bit_3/A5
- U45 pad 18: /CHB Communication/Level_Shifter_8bit_3/A5 -> /CHB Communication/Level_Shifter_8bit_3/A4
- U45 pad 2: /CHB Communication/Level_Shifter_8bit_2/A5 -> /CHB Communication/Ph_B_Tx1_5V
- U45 pad 20: /CHB Communication/Level_Shifter_8bit_3/A6 -> /CHB Communication/Level_Shifter_8bit_3/A3
- U45 pad 22: /CHB Communication/Level_Shifter_8bit_3/A7 -> /CHB Communication/Level_Shifter_8bit_3/A2
- U45 pad 24: /CHB Communication/Level_Shifter_8bit_3/A8 -> /CHB Communication/Level_Shifter_8bit_3/A1
- U45 pad 4: /CHB Communication/Level_Shifter_8bit_2/A6 -> /CHB Communication/Level_Shifter_8bit_2/A3
- U45 pad 6: /CHB Communication/Level_Shifter_8bit_2/A7 -> /CHB Communication/Level_Shifter_8bit_2/A2
- U45 pad 8: /CHB Communication/Level_Shifter_8bit_2/A8 -> /CHB Communication/Level_Shifter_8bit_2/A1
- U46 pad 10: /CHB Communication/Level_Shifter_8bit_4/A5 -> /CHB Communication/Level_Shifter_8bit_4/A4
- U46 pad 12: /CHB Communication/Level_Shifter_8bit_4/A6 -> /CHB Communication/Level_Shifter_8bit_4/A3
- U46 pad 14: /CHB Communication/Level_Shifter_8bit_4/A7 -> /CHB Communication/Level_Shifter_8bit_4/A2
- U46 pad 16: /CHB Communication/Level_Shifter_8bit_4/A8 -> /CHB Communication/Level_Shifter_8bit_4/A1
- U46 pad 18: /CHB Communication/Level_Shifter_8bit_5/A1 -> /CHB Communication/Level_Shifter_8bit_5/A8
- U46 pad 2: /CHB Communication/Level_Shifter_8bit_4/A1 -> /CHB Communication/Ph_C_Tx1_5V
- U46 pad 20: /CHB Communication/Level_Shifter_8bit_5/A2 -> /CHB Communication/Level_Shifter_8bit_5/A7
- U46 pad 22: /CHB Communication/Level_Shifter_8bit_5/A3 -> /CHB Communication/Level_Shifter_8bit_5/A6
- U46 pad 24: /CHB Communication/Level_Shifter_8bit_5/A4 -> /CHB Communication/Level_Shifter_8bit_5/A5
- U46 pad 4: /CHB Communication/Level_Shifter_8bit_4/A2 -> /CHB Communication/Level_Shifter_8bit_4/A7
- U46 pad 6: /CHB Communication/Level_Shifter_8bit_4/A3 -> /CHB Communication/Level_Shifter_8bit_4/A6
- U46 pad 8: /CHB Communication/Level_Shifter_8bit_4/A4 -> /CHB Communication/Level_Shifter_8bit_4/A5
- U47 pad 10: /CHB Communication/Level_Shifter_8bit_6/A1 -> /CHB Communication/Level_Shifter_8bit_6/A8
- U47 pad 12: /CHB Communication/Level_Shifter_8bit_6/A2 -> /CHB Communication/Level_Shifter_8bit_6/A7
- U47 pad 14: /CHB Communication/Level_Shifter_8bit_6/A3 -> /CHB Communication/Level_Shifter_8bit_6/A6
- U47 pad 16: /CHB Communication/Level_Shifter_8bit_6/A4 -> /CHB Communication/Level_Shifter_8bit_6/A5
- U47 pad 18: /CHB Communication/Level_Shifter_8bit_6/A5 -> /CHB Communication/Level_Shifter_8bit_6/A4
- U47 pad 2: /CHB Communication/Level_Shifter_8bit_5/A5 -> /CHB Communication/Ph_D_Tx1_5V
- U47 pad 20: /CHB Communication/Level_Shifter_8bit_6/A6 -> /CHB Communication/Level_Shifter_8bit_6/A3
- U47 pad 22: /CHB Communication/Level_Shifter_8bit_6/A7 -> /CHB Communication/Level_Shifter_8bit_6/A2
- U47 pad 24: /CHB Communication/Level_Shifter_8bit_6/A8 -> /CHB Communication/Level_Shifter_8bit_6/A1
- U47 pad 4: /CHB Communication/Level_Shifter_8bit_5/A6 -> /CHB Communication/Level_Shifter_8bit_5/A3
- U47 pad 6: /CHB Communication/Level_Shifter_8bit_5/A7 -> /CHB Communication/Level_Shifter_8bit_5/A2
- U47 pad 8: /CHB Communication/Level_Shifter_8bit_5/A8 -> /CHB Communication/Level_Shifter_8bit_5/A1
Routing:
- net /CHB Communication/Level_Shifter_8bit_6/A1: track 5.95 -> 149.0 mm, vias 0 -> 2
- net /ADC for Machine/Diffamp8/Ain-: track 3.83 -> 145.0 mm
- net /CHB Communication/Level_Shifter_8bit_6/A2: track 5.08 -> 144.2 mm, vias 0 -> 2
- net /ADC for Machine/Diffamp8/Ain+: track 3.93 -> 142.0 mm
- net /CHB Communication/Level_Shifter_8bit_6/A3: track 4.33 -> 139.9 mm, vias 0 -> 2
- net /CHB Communication/Level_Shifter_8bit_6/A4: track 3.87 -> 135.6 mm, vias 0 -> 2
- net /CHB Communication/Level_Shifter_8bit_6/A5: track 3.83 -> 131.7 mm, vias 0 -> 2
- net /CHB Communication/Level_Shifter_8bit_6/A6: track 4.29 -> 128.5 mm, vias 0 -> 2
- net /CHB Communication/Level_Shifter_8bit_6/A7: track 5.18 -> 125.6 mm, vias 0 -> 2
- net /ADC for Machine/Diffamp7/Ain-: track 4.10 -> 124.4 mm
- net /CHB Communication/Level_Shifter_8bit_3/A1: track 5.95 -> 124.5 mm, vias 0 -> 2
- net /ADC for Machine/Diffamp7/Ain+: track 4.21 -> 121.5 mm
- net /CHB Communication/Level_Shifter_8bit_6/A8: track 6.08 -> 122.6 mm, vias 0 -> 2
- net /CHB Communication/Level_Shifter_8bit_3/A2: track 5.08 -> 119.6 mm, vias 0 -> 2
- net /CHB Communication/Level_Shifter_8bit_3/A3: track 4.33 -> 115.3 mm, vias 0 -> 2
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- added copper zone on B.Cu, net /CHB to 3Ph/Ph_A2_out
- added copper zone on F.Cu, net /CHB to 3Ph/Ph_A2_out
- added copper zone on In1.Cu, net /CHB to 3Ph/Ph_A2_out
- added copper zone on In2.Cu, net /CHB to 3Ph/Ph_A2_out
- added copper zone on B.Cu, net /CHB to 3Ph/Ph_B2_out
- added copper zone on F.Cu, net /CHB to 3Ph/Ph_B2_out
- added copper zone on In1.Cu, net /CHB to 3Ph/Ph_B2_out
- added copper zone on In2.Cu, net /CHB to 3Ph/Ph_B2_out
- added copper zone on B.Cu, net /CHB to 3Ph/Ph_C2_out
- added copper zone on F.Cu, net /CHB to 3Ph/Ph_C2_out
- added copper zone on In1.Cu, net /CHB to 3Ph/Ph_C2_out
- added copper zone on In2.Cu, net /CHB to 3Ph/Ph_C2_out
- added copper zone on F.Cu, net /CHB to 3Ph/Ph_D2_out
- added copper zone on B.Cu, net /Current measure/Tamura_1/pin1
- added copper zone on F.Cu, net /Current measure/Tamura_1/pin1
- added copper zone on In1.Cu, net /Current measure/Tamura_1/pin1
- added copper zone on In2.Cu, net /Current measure/Tamura_1/pin1
- added copper zone on B.Cu, net /Current measure/Tamura_2/pin1
- added copper zone on F.Cu, net /Current measure/Tamura_2/pin1
- added copper zone on In1.Cu, net /Current measure/Tamura_2/pin1
- added copper zone on In2.Cu, net /Current measure/Tamura_2/pin1
- added copper zone on B.Cu, net /Current measure/Tamura_3/pin1
- added copper zone on F.Cu, net /Current measure/Tamura_3/pin1
- added copper zone on In1.Cu, net /Current measure/Tamura_3/pin1
- added copper zone on In2.Cu, net /Current measure/Tamura_3/pin1
- added copper zone on B.Cu, net /Current measure/Tamura_4/pin1
- added copper zone on F.Cu, net /Current measure/Tamura_4/pin1
- added copper zone on In1.Cu, net /Current measure/Tamura_4/pin1
- added copper zone on In2.Cu, net /Current measure/Tamura_4/pin1
Other:
- outline, holes or cut-outs redrawn
