File: FPGA_Board_BA/PCB/FPGA_Board_BA.kicad_pcb (KiCad board)
At the start: 4 copper layers, 310.2 x 160 mm, 502 parts, among them J10 PinHeader_2x4_SMD, J11 PinHeader_2x4_SMD, J12 Box_Header_2x05_THT, J13 Box_Header_2x05_THT, J14 Box_Header_2x05_THT, J15 Box_Header_2x05_THT, J16 PinHeader_2x4_SMD, J17 Plug_Terminal_2x4_Vertical, J18 Plug_Terminal_2x12pin, J2 PinHeader_2x4_SMD, J20 JST_XH_05_vertical, J3 Banana_Socket_Red, J4 Banana_Socket_Black, J5 Box_Header_6pin, J6 Box_Header_6pin, J7 Box_Header_6pin, J8 Box_Header_6pin, J9 Box_Header_26pin, Q1 IPT017N12NM6, Q2 IPT017N12NM6, Q5 IPT017N12NM6, Q6 IPT017N12NM6, SW1 TL3305BF100QG, SW2 TL3305BF100QG, U1 LTC2320-16_CMOS, U10 BOOSTXL-3PHGANINV, U11 LTC2320-16_CMOS, U12 1819_IS8, U13 1819_IS8, U14 1819_IS8, U15 1819_IS8, U17 1819_IS8, U18 1819_IS8, U19 1819_IS8, U2 Zynq7020, U20 1819_IS8, U21 1819_IS8, U22 1819_IS8, U23 1819_IS8, U24 1819_IS8, U25 1819_IS8, U26 BoxHeader_24pin, U27 SN74LXCH8T245RHLR, U28 SN74LXCH8T245RHLR, U29 SN74LXCH8T245RHLR, U3 LM5143, U30 SN74LXCH8T245RHLR, U31 S22P006S05, U32 SN74LXCH8T245RHLR, U33 SN74LXCH8T245RHLR, U34 SN74LXC2T45Q1, U35 SN74LXC2T45Q1, U36 SN74LXC2T45Q1, U37 S22P006S05, U38 SN74LXCH8T245RHLR, U39 SN74LXC2T45Q1, U40 S22P006S05, U41 SN74LXC2T45Q1, U42 SN74LXC2T45Q1, U43 S22P006S05, U44 1819_IS8, U45 BoxHeader_24pin, U46 BoxHeader_24pin, U47 BoxHeader_24pin, U48 MCP1703AT-5002EDB, U7 1819_IS8, U8 TPS61022, U9 MCP1703AT-5002EDB

Commit message: some changes in the PCB
Parts:
- moved U2 9.78 mm to (169.3, 136.4)
- moved C141 4.75 mm to (211.6, 108.6)
- moved C142 4.75 mm to (213.4, 108.6)
- moved C143 4.75 mm to (182.1, 100.1)
- moved C144 4.75 mm to (183.8, 100.1)
- moved C145 4.75 mm to (180.6, 85.9)
- moved C146 4.75 mm to (182.3, 85.9)
- moved C150 4.75 mm to (211.6, 118.6)
- moved C151 4.75 mm to (213.4, 118.6)
- moved C153 4.75 mm to (210.1, 151.4)
- moved C154 4.75 mm to (208.3, 151.4)
- moved C155 4.75 mm to (190.6, 85.9)
- moved C156 4.75 mm to (192.3, 85.9)
- moved D1 4.75 mm to (196.0, 171.2)
- moved D14 4.75 mm to (199.3, 170.2)
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Connections:
- U2 pad a26: /CHB Communication/Ph_A_Tx1 -> unconnected-(U2A-IO_L1P_T0_34-Pada26)
- U2 pad a27: /CHB Communication/Ph_A_Tx3 -> unconnected-(U2A-IO_L2P_T0_34-Pada27)
- U2 pad a28: /CHB Communication/Ph_A_Tx2 -> unconnected-(U2A-IO_L1N_T0_34-Pada28)
- U2 pad a29: /CHB Communication/Ph_A_Tx4 -> unconnected-(U2A-IO_L2N_T0_34-Pada29)
- U2 pad a30: /CHB Communication/Ph_A_Tx5 -> unconnected-(U2A-IO_L3P_T0_34-Pada30)
- U2 pad a31: /CHB Communication/Ph_A_Tx7 -> unconnected-(U2A-IO_L4P_T0_34-Pada31)
- U2 pad a32: /CHB Communication/Ph_A_Tx6 -> unconnected-(U2A-IO_L3N_T0_34-Pada32)
- U2 pad a33: /CHB Communication/Ph_A_Tx8 -> unconnected-(U2A-IO_L4N_T0_34-Pada33)
- U2 pad a36: /CHB Communication/Ph_A_Tx9 -> unconnected-(U2A-IO_L5P_T0_34-Pada36)
- U2 pad a37: /CHB Communication/Ph_A_Tx11 -> unconnected-(U2A-IO_L6P_T0_34-Pada37)
- U2 pad a38: /CHB Communication/Ph_A_Tx10 -> unconnected-(U2A-IO_L5N_T0_34-Pada38)
- U2 pad a39: /CHB Communication/Ph_A_Tx12 -> unconnected-(U2A-IO_L6N_T0_34-Pada39)
- U2 pad a40: /CHB Communication/Ph_B_Tx1 -> unconnected-(U2A-IO_L7P_T1_34-Pada40)
- U2 pad a41: /CHB Communication/Ph_B_Tx3 -> unconnected-(U2A-IO_L8P_T1_34-Pada41)
- U2 pad a42: /CHB Communication/Ph_B_Tx2 -> unconnected-(U2A-IO_L7N_T1_34-Pada42)
- U2 pad a43: /CHB Communication/Ph_B_Tx4 -> unconnected-(U2A-IO_L8N_T1_34-Pada43)
- U2 pad a45: /CHB Communication/Ph_B_Tx9 -> unconnected-(U2A-IO_L11P_T1_34-Pada45)
- U2 pad a46: /CHB Communication/Ph_B_Tx7 -> unconnected-(U2A-IO_L10P_T1_34-Pada46)
- U2 pad a47: /CHB Communication/Ph_B_Tx10 -> unconnected-(U2A-IO_L11N_T1_34-Pada47)
- U2 pad a48: /CHB Communication/Ph_B_Tx8 -> unconnected-(U2A-IO_L10N_T1_34-Pada48)
- U2 pad a50: /CHB Communication/Ph_C_Tx1 -> unconnected-(U2A-IO_L13P_T2_34-Pada50)
- U2 pad a51: /CHB Communication/Ph_B_Tx5 -> unconnected-(U2A-IO_L9P_T1_34-Pada51)
- U2 pad a52: /CHB Communication/Ph_C_Tx2 -> unconnected-(U2A-IO_L13N_T2_34-Pada52)
- U2 pad a53: /CHB Communication/Ph_B_Tx6 -> unconnected-(U2A-IO_L9N_T2_34-Pada53)
- U2 pad a55: /CHB Communication/Ph_B_Tx11 -> unconnected-(U2A-IO_L12P_T1_34-Pada55)
- U2 pad a56: /CHB Communication/Ph_C_Tx5 -> unconnected-(U2A-IO_L15P_T2_34-Pada56)
- U2 pad a57: /CHB Communication/Ph_B_Tx12 -> unconnected-(U2A-IO_L12N_T1_34-Pada57)
- U2 pad a58: /CHB Communication/Ph_C_Tx6 -> unconnected-(U2A-IO_L15N_T2_34-Pada58)
- U2 pad a59: /CHB Communication/Ph_C_Tx3 -> unconnected-(U2A-IO_L14P_T2_34-Pada59)
- U2 pad a60: /CHB Communication/Ph_C_Tx9 -> unconnected-(U2A-IO_L17P_T2_34-Pada60)
- U2 pad a61: /CHB Communication/Ph_C_Tx4 -> unconnected-(U2A-IO_L14N_T2_34-Pada61)
- U2 pad a62: /CHB Communication/Ph_C_Tx10 -> unconnected-(U2A-IO_L17N_T2_34-Pada62)
- U2 pad a63: /CHB Communication/Ph_C_Tx7 -> unconnected-(U2A-IO_L16P_T2_34-Pada63)
- U2 pad a64: /CHB Communication/Ph_D_Tx1 -> unconnected-(U2A-IO_L19P_T3_34-Pada64)
- U2 pad a65: /CHB Communication/Ph_C_Tx8 -> unconnected-(U2A-IO_L16N_T2_34-Pada65)
- U2 pad a66: /CHB Communication/Ph_D_Tx2 -> unconnected-(U2A-IO_L19N_T3_34-Pada66)
- U2 pad a69: /CHB Communication/Ph_C_Tx12 -> unconnected-(U2A-IO_L18N_T2_34-Pada69)
- U2 pad a70: /CHB Communication/Ph_C_Tx11 -> unconnected-(U2A-IO_L18P_T2_34-Pada70)
- U2 pad a71: /CHB Communication/Ph_D_Tx4 -> unconnected-(U2A-IO_L20P_T3_34-Pada71)
- U2 pad a72: /CHB Communication/Ph_D_Tx3 -> unconnected-(U2A-IO_L20N_T3_34-Pada72)
- U2 pad a73: /CHB Communication/Ph_D_Tx6 -> unconnected-(U2A-IO_L21N_T3_34-Pada73)
- U2 pad a74: /CHB Communication/Ph_D_Tx5 -> unconnected-(U2A-IO_L21P_T3_34-Pada74)
- U2 pad a75: /CHB Communication/Ph_D_Tx7 -> unconnected-(U2A-IO_L22P_T3_34-Pada75)
- U2 pad a76: /CHB Communication/Ph_D_Tx11 -> unconnected-(U2A-IO_L24P_T3_34-Pada76)
- U2 pad a77: /CHB Communication/Ph_D_Tx8 -> unconnected-(U2A-IO_L22N_T3_34-Pada77)
- U2 pad a78: /CHB Communication/Ph_D_Tx12 -> unconnected-(U2A-IO_L24N_T3_34-Pada78)
- U2 pad a79: /CHB Communication/Ph_D_Tx9 -> unconnected-(U2A-IO_L23P_T3_34-Pada79)
- U2 pad a80: /CHB Communication/Ph_D_Tx10 -> unconnected-(U2A-IO_L23N_T3_34-Pada80)
- U2 pad b22: /CHB Communication/Ph_C_Err -> /CHB Communication/Ph_A_Tx3
- U2 pad b23: /CHB Communication/Ph_A_Err -> /CHB Communication/Ph_A_Tx1
- U2 pad b24: /CHB Communication/Ph_D_Err -> /CHB Communication/Ph_A_Tx4
- U2 pad b25: /CHB Communication/Ph_B_Err -> /CHB Communication/Ph_A_Tx2
- U2 pad b26: /CHB Communication/Ph_C_En -> /CHB Communication/Ph_A_Tx7
- U2 pad b27: /CHB Communication/Ph_A_En -> /CHB Communication/Ph_A_Tx5
- U2 pad b28: /CHB Communication/Ph_D_En -> /CHB Communication/Ph_A_Tx8
- U2 pad b29: /CHB Communication/Ph_B_En -> /CHB Communication/Ph_A_Tx6
- U2 pad b32: /CHB Communication/Ph_C_Rx -> /CHB Communication/Ph_A_Tx11
- U2 pad b33: /CHB Communication/Ph_A_Rx -> /CHB Communication/Ph_A_Tx9
- U2 pad b34: /CHB Communication/Ph_D_Rx -> /CHB Communication/Ph_A_Tx12
- U2 pad b35: /CHB Communication/Ph_B_Rx -> /CHB Communication/Ph_A_Tx10
- U2 pad b36: unconnected-(U2B-IO_L8P_T1_35-Padb36) -> /CHB Communication/Ph_B_Tx3
- U2 pad b37: unconnected-(U2B-IO_L7P_T1_35-Padb37) -> /CHB Communication/Ph_B_Tx1
- U2 pad b38: unconnected-(U2B-IO_L8N_T1_35-Padb38) -> /CHB Communication/Ph_B_Tx4
- U2 pad b39: unconnected-(U2B-IO_L7N_T1_35-Padb39) -> /CHB Communication/Ph_B_Tx2
- U2 pad b42: unconnected-(U2B-IO_L10P_T1_35-Padb42) -> /CHB Communication/Ph_B_Tx7
- U2 pad b43: unconnected-(U2B-IO_L9P_T1_35-Padb43) -> /CHB Communication/Ph_B_Tx5
- U2 pad b44: unconnected-(U2B-IO_L10N_T1_35-Padb44) -> /CHB Communication/Ph_B_Tx8
- U2 pad b45: unconnected-(U2B-IO_L9N_T1_35-Padb45) -> /CHB Communication/Ph_B_Tx6
- U2 pad b46: /Encoder/ENC_I -> /CHB Communication/Ph_B_Tx11
- U2 pad b47: /Encoder/ENC_A -> /CHB Communication/Ph_B_Tx9
- U2 pad b48: /FPGA/LED1 -> /CHB Communication/Ph_B_Tx12
- U2 pad b49: /Encoder/ENC_B -> /CHB Communication/Ph_B_Tx10
- U2 pad b52: /FPGA/Button2 -> /CHB Communication/Ph_C_Tx3
- U2 pad b53: /FPGA/LED2 -> /CHB Communication/Ph_C_Tx1
- U2 pad b54: /ADC for Machine/SDO1_1 -> /CHB Communication/Ph_C_Tx4
- U2 pad b55: /FPGA/Button1 -> /CHB Communication/Ph_C_Tx2
- U2 pad b56: /ADC for Machine/SDO4_1 -> /CHB Communication/Ph_C_Tx7
- U2 pad b57: /ADC for Machine/SDO2_1 -> /CHB Communication/Ph_C_Tx5
- U2 pad b58: /ADC for Machine/SDO5_1 -> /CHB Communication/Ph_C_Tx8
- U2 pad b59: /ADC for Machine/SDO3_1 -> /CHB Communication/Ph_C_Tx6
- U2 pad b62: /ADC for Machine/SDO8_1 -> /CHB Communication/Ph_C_Tx11
- U2 pad b63: /ADC for Machine/SDO6_1 -> /CHB Communication/Ph_C_Tx9
- U2 pad b64: /ADC for Machine/CLK_OUT_1 -> /CHB Communication/Ph_C_Tx12
- U2 pad b65: /ADC for Machine/SDO7_1 -> /CHB Communication/Ph_C_Tx10
- U2 pad b66: /FPGA/esd_diodes/Pin1 -> /CHB Communication/Ph_D_Tx3
- U2 pad b67: /ADC for Machine/CLK_IN_1 -> /CHB Communication/Ph_D_Tx1
- U2 pad b68: /FPGA/esd_diodes/Pin2 -> /CHB Communication/Ph_D_Tx4
- U2 pad b69: /ADC for Machine/~{CNV}_1 -> /CHB Communication/Ph_D_Tx2
- U2 pad b72: /FPGA/esd_diodes/Pin3 -> /CHB Communication/Ph_D_Tx7
- U2 pad b73: /FPGA/esd_diodes/Pin10 -> /CHB Communication/Ph_D_Tx5
- U2 pad b74: /FPGA/esd_diodes/Pin4 -> /CHB Communication/Ph_D_Tx8
- U2 pad b75: /FPGA/esd_diodes/Pin9 -> /CHB Communication/Ph_D_Tx6
- U2 pad b76: /FPGA/esd_diodes/Pin5 -> /CHB Communication/Ph_D_Tx11
- U2 pad b77: /FPGA/esd_diodes/Pin8 -> /CHB Communication/Ph_D_Tx9
- U2 pad b78: /FPGA/esd_diodes/Pin6 -> /CHB Communication/Ph_D_Tx12
- U2 pad b79: /FPGA/esd_diodes/Pin7 -> /CHB Communication/Ph_D_Tx10
Routing:
- net /CHB Communication/Level_shifter_Rx_En/B8: track 0.00 -> 148.1 mm, vias 0 -> 1
- net /CHB Communication/Level_shifter_Rx_En/B7: track 0.00 -> 145.0 mm, vias 0 -> 1
- net /CHB Communication/Level_shifter_Rx_En/B6: track 0.00 -> 123.4 mm, vias 0 -> 1
- net /CHB Communication/Level_shifter_Rx_En/B5: track 0.00 -> 120.5 mm, vias 0 -> 1
- net /CHB Communication/Level_shifter_Rx_En/B4: track 0.00 -> 98.7 mm, vias 0 -> 1
- net /CHB Communication/Level_shifter_Rx_En/B3: track 0.00 -> 95.9 mm, vias 0 -> 1
- net /CHB Communication/Level_shifter_Rx_En/B2: track 0.00 -> 73.9 mm, vias 0 -> 1
- net /CHB Communication/Level_shifter_Rx_En/B1: track 0.00 -> 70.4 mm, vias 0 -> 1
- added copper zone on In1.Cu, net /CHB to 3Ph/Ph_D2_out
- removed copper zone on B.Cu, net /CHB to 3Ph/Ph_A2_out
- removed copper zone on In2.Cu, net /CHB to 3Ph/Ph_A2_out
- removed copper zone on B.Cu, net /CHB to 3Ph/Ph_B2_out
- removed copper zone on In2.Cu, net /CHB to 3Ph/Ph_B2_out
- removed copper zone on B.Cu, net /CHB to 3Ph/Ph_C2_out
- removed copper zone on In2.Cu, net /CHB to 3Ph/Ph_C2_out
Other:
- outline, holes or cut-outs redrawn

Commit message: some minimal changes on the PCB on the right side
Parts:
- moved C141 71.3 mm to (152.3, 148.1)
- moved C142 71.3 mm to (154.1, 148.1)
- moved C150 71.3 mm to (152.3, 158.1)
- moved C151 71.3 mm to (154.1, 158.1)
- moved R216 71.3 mm to (149.1, 150.8)
- moved R217 71.3 mm to (149.1, 152.6)
- moved R233 71.3 mm to (149.1, 160.8)
- moved R234 71.3 mm to (149.1, 162.6)
- moved U34 71.3 mm to (153.3, 151.6)
- moved U39 71.3 mm to (153.3, 161.6)
- moved D11 68.1 mm to (218.5, 63.9)
- moved D12 68.1 mm to (218.6, 66.9)
- moved D13 68.1 mm to (218.5, 69.9)
- moved R49 68.1 mm to (215.0, 64.1)
- moved R50 68.1 mm to (215.0, 66.9)
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Routing:
- net /CHB Communication/Ph_A_Tx8: track 0.00 -> 64.6 mm
- net /CHB Communication/Ph_A_Tx7: track 0.00 -> 64.0 mm
- net /CHB Communication/Ph_A_Tx4: track 0.00 -> 64.0 mm
- net /CHB Communication/Ph_A_Tx3: track 0.00 -> 63.5 mm
- net /CHB Communication/Ph_A_Tx12: track 0.00 -> 54.4 mm
- net /CHB Communication/Ph_B_Tx4: track 0.00 -> 53.9 mm
- net /CHB Communication/Ph_A_Tx11: track 0.00 -> 53.6 mm
- net /CHB Communication/Ph_B_Tx3: track 0.00 -> 53.3 mm
- net /CHB Communication/Ph_B_Tx8: track 0.00 -> 44.9 mm
- net /CHB Communication/Ph_B_Tx7: track 0.00 -> 44.5 mm
- net /CHB Communication/Ph_B_Tx12: track 0.00 -> 44.2 mm
- net /CHB Communication/Ph_B_Tx11: track 0.00 -> 43.6 mm
- net /CHB Communication/Ph_C_Tx4: track 0.00 -> 37.0 mm
- net /CHB Communication/Ph_C_Tx8: track 0.00 -> 36.5 mm
- net /CHB Communication/Ph_C_Tx7: track 0.00 -> 35.5 mm
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Other:
- board size 310.2 x 160 mm -> 310 x 160 mm

Commit message: added bus into schematic
Connections:
- U2 pad b32: /CHB Communication/Ph_A_Tx11 -> /CHB Communication/Ph_A_Tx10
- U2 pad b33: /CHB Communication/Ph_A_Tx9 -> /CHB Communication/Ph_A_Tx12
- U2 pad b34: /CHB Communication/Ph_A_Tx12 -> /CHB Communication/Ph_A_Tx9
- U2 pad b35: /CHB Communication/Ph_A_Tx10 -> /CHB Communication/Ph_A_Tx11
Changed lines of the file:
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@@
 			(size 0.74 2.92)
 			(layers "F.Cu" "F.Mask" "F.Paste")
-			(net 264 "/CHB Communication/Ph_A_Tx11")
+			(net 283 "/CHB Communication/Ph_A_Tx10")
 			(pinfunction "IO_L6P_T0_35")
 			(pintype "passive")
@@
 			(size 0.74 2.92)
 			(layers "F.Cu" "F.Mask" "F.Paste")
-			(net 295 "/CHB Communication/Ph_A_Tx9")
+			(net 316 "/CHB Communication/Ph_A_Tx12")
 			(pinfunction "IO_L5P_T0_35")
 			(pintype "passive")
@@
 			(size 0.74 2.92)
 			(layers "F.Cu" "F.Mask" "F.Paste")
-			(net 316 "/CHB Communication/Ph_A_Tx12")
+			(net 295 "/CHB Communication/Ph_A_Tx9")
 			(pinfunction "IO_L6N_T0_35")
 			(pintype "passive")
@@
 			(size 0.74 2.92)
 			(layers "F.Cu" "F.Mask" "F.Paste")
-			(net 283 "/CHB Communication/Ph_A_Tx10")
+			(net 264 "/CHB Communication/Ph_A_Tx11")
 			(pinfunction "IO_L5N_T0_35")
 			(pintype "passive")
@@
 	)
 	(segment
-		(start 231.750057 67.85)
-		(end 233.55 67.85)
+		(start 233.55 67.85)
+		(end 231.750057 67.85)
 		(width 0.2)
 		(layer "F.Cu")
