File: FPGA_Board_BA/PCB/ls_error.kicad_sch (KiCad schematic)
At the start: 3 parts, among them U4101 SN74LXC2T45Q1

Commit message: work
Parts:
- added R176, R177: 10k_0603, Resistor_SMD:R_0603_1608Metric, symbol WLIB_R:10k_0603
- renumbered C4101 to C153, C4102 to C154, U4101 to U41
Connections:
- net +3.3V: now also R176.1, R177.1
- net B1: now also R176.2
- net B2: now also R177.2

Commit message: 22.11
Parts:
- renumbered C153 to C146, C154 to C147, R176 to R177, R177 to R178, U41 to U35
Connections:
- net +3.3V: no longer R177.1, R178.1
- net A1: now also R177.1
- net A2: now also R178.1
- net B1: no longer R177.2
- net B2: no longer R178.2
- net GND: now also R177.2, R178.2
Other:
- moved on the sheet: R177, R178

Commit message: exported stuff
Parts:
- renumbered C146 to C141, C147 to C142, R177 to R216, R178 to R217, U35 to U34
Changed lines of the file:
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@@
 		(dnp no)
 		(fields_autoplaced yes)
-		(property "Reference" "C147"
+		(property "Reference" "C142"
 			(at 163.83 78.74 90)
 			(effects
@@
 			(project "FPGA_Board_BA"
 				(path "/fd7503bc-e7fc-4766-b224-3d1c3d7de5ff/1b181806-12f4-40c8-bf91-78ac0d892dab/195faa44-0949-4e4a-a075-cc82f959d0cf"
-					(reference "C156")
-					(unit 1)
-				)
-				(path "/fd7503bc-e7fc-4766-b224-3d1c3d7de5ff/1b181806-12f4-40c8-bf91-78ac0d892dab/e2e765af-525f-4805-b4e1-1d4694321b94"
-					(reference "C147")
+					(reference "C151")
+					(unit 1)
+				)
+				(path "/fd7503bc-e7fc-4766-b224-3d1c3d7de5ff/1b181806-12f4-40c8-bf91-78ac0d892dab/e2e765af-525f-4805-b4e1-1d4694321b94"
+					(reference "C142")
 					(unit 1)
 				)
@@
 		(dnp no)
 		(fields_autoplaced yes)
-		(property "Reference" "#PWR0211"
+		(property "Reference" "#PWR0223"
 			(at 139.7 124.46 0)
 			(effects
@@
 			(project "FPGA_Board_BA"
 				(path "/fd7503bc-e7fc-4766-b224-3d1c3d7de5ff/1b181806-12f4-40c8-bf91-78ac0d892dab/195faa44-0949-4e4a-a075-cc82f959d0cf"
-					(reference "#PWR0241")
-					(unit 1)
-				)
-				(path "/fd7503bc-e7fc-4766-b224-3d1c3d7de5ff/1b181806-12f4-40c8-bf91-78ac0d892dab/e2e765af-525f-4805-b4e1-1d4694321b94"
-					(reference "#PWR0211")
+					(reference "#PWR0253")
+					(unit 1)
+				)
+				(path "/fd7503bc-e7fc-4766-b224-3d1c3d7de5ff/1b181806-12f4-40c8-bf91-78ac0d892dab/e2e765af-525f-4805-b4e1-1d4694321b94"
+					(reference "#PWR0223")
 					(unit 1)
 				)
@@
 		(on_board yes)
 		(dnp no)
-		(property "Reference" "R177"
+		(property "Reference" "R216"
 			(at 90.17 122.174 90)
 			(effects
@@
 			(project ""
 				(path "/fd7503bc-e7fc-4766-b224-3d1c3d7de5ff/1b181806-12f4-40c8-bf91-78ac0d892dab/195faa44-0949-4e4a-a075-cc82f959d0cf"
-					(reference "R194")
-					(unit 1)
-				)
-				(path "/fd7503bc-e7fc-4766-b224-3d1c3d7de5ff/1b181806-12f4-40c8-bf91-78ac0d892dab/e2e765af-525f-4805-b4e1-1d4694321b94"
-					(reference "R177")
+					(reference "R233")
+					(unit 1)
+				)
+				(path "/fd7503bc-e7fc-4766-b224-3d1c3d7de5ff/1b181806-12f4-40c8-bf91-78ac0d892dab/e2e765af-525f-4805-b4e1-1d4694321b94"
+					(reference "R216")
 					(unit 1)
 				)
@@
 		(on_board yes)
 		(dnp no)
-		(property "Reference" "R178"
+		(property "Reference" "R217"
 			(at 105.41 122.174 90)
 			(effects
@@
 			(project "FPGA_Board_BA"
 				(path "/fd7503bc-e7fc-4766-b224-3d1c3d7de5ff/1b181806-12f4-40c8-bf91-78ac0d892dab/195faa44-0949-4e4a-a075-cc82f959d0cf"
-					(reference "R195")
-					(unit 1)
-				)
-				(path "/fd7503bc-e7fc-4766-b224-3d1c3d7de5ff/1b181806-12f4-40c8-bf91-78ac0d892dab/e2e765af-525f-4805-b4e1-1d4694321b94"
-					(reference "R178")
+					(reference "R234")
+					(unit 1)
+				)
+				(path "/fd7503bc-e7fc-4766-b224-3d1c3d7de5ff/1b181806-12f4-40c8-bf91-78ac0d892dab/e2e765af-525f-4805-b4e1-1d4694321b94"
+					(reference "R217")
 					(unit 1)
 				)
@@
 		(dnp no)
 		(fields_autoplaced yes)
-		(property "Reference" "#PWR0208"
+		(property "Reference" "#PWR0220"
 			(at 97.79 134.62 0)
 			(effects
@@
 			(project "FPGA_Board_BA"
 				(path "/fd7503bc-e7fc-4766-b224-3d1c3d7de5ff/1b181806-12f4-40c8-bf91-78ac0d892dab/195faa44-0949-4e4a-a075-cc82f959d0cf"
-					(reference "#PWR0238")
-					(unit 1)
-				)
-				(path "/fd7503bc-e7fc-4766-b224-3d1c3d7de5ff/1b181806-12f4-40c8-bf91-78ac0d892dab/e2e765af-525f-4805-b4e1-1d4694321b94"
-					(reference "#PWR0208")
+					(reference "#PWR0250")
+					(unit 1)
+				)
+				(path "/fd7503bc-e7fc-4766-b224-3d1c3d7de5ff/1b181806-12f4-40c8-bf91-78ac0d892dab/e2e765af-525f-4805-b4e1-1d4694321b94"
+					(reference "#PWR0220")
 					(unit 1)
 				)
@@
 		(dnp no)
 		(fields_autoplaced yes)
-		(property "Reference" "U35"
+		(property "Reference" "U34"
 			(at 141.8433 114.3 0)
 			(effects
@@
 			(project "FPGA_Board_BA"
 				(path "/fd7503bc-e7fc-4766-b224-3d1c3d7de5ff/1b181806-12f4-40c8-bf91-78ac0d892dab/195faa44-0949-4e4a-a075-cc82f959d0cf"
-					(reference "U40")
-					(unit 1)
-				)
-				(path "/fd7503bc-e7fc-4766-b224-3d1c3d7de5ff/1b181806-12f4-40c8-bf91-78ac0d892dab/e2e765af-525f-4805-b4e1-1d4694321b94"
-					(reference "U35")
+					(reference "U39")
+					(unit 1)
+				)
+				(path "/fd7503bc-e7fc-4766-b224-3d1c3d7de5ff/1b181806-12f4-40c8-bf91-78ac0d892dab/e2e765af-525f-4805-b4e1-1d4694321b94"
+					(reference "U34")
 					(unit 1)
 				)
@@
 		(dnp no)
 		(fields_autoplaced yes)
-		(property "Reference" "#PWR0210"
+		(property "Reference" "#PWR0222"
 			(at 133.35 88.9 0)
 			(effects
@@
 			(project "FPGA_Board_BA"
 				(path "/fd7503bc-e7fc-4766-b224-3d1c3d7de5ff/1b181806-12f4-40c8-bf91-78ac0d892dab/195faa44-0949-4e4a-a075-cc82f959d0cf"
-					(reference "#PWR0240")
-					(unit 1)
-				)
-				(path "/fd7503bc-e7fc-4766-b224-3d1c3d7de5ff/1b181806-12f4-40c8-bf91-78ac0d892dab/e2e765af-525f-4805-b4e1-1d4694321b94"
-					(reference "#PWR0210")
+					(reference "#PWR0252")
+					(unit 1)
+				)
+				(path "/fd7503bc-e7fc-4766-b224-3d1c3d7de5ff/1b181806-12f4-40c8-bf91-78ac0d892dab/e2e765af-525f-4805-b4e1-1d4694321b94"
+					(reference "#PWR0222")
 					(unit 1)
 				)
@@
 		(dnp no)
 		(fields_autoplaced yes)
-		(property "Reference" "C146"
+		(property "Reference" "C141"
 			(at 119.38 78.74 90)
 			(effects
@@
 			(project "FPGA_Board_BA"
 				(path "/fd7503bc-e7fc-4766-b224-3d1c3d7de5ff/1b181806-12f4-40c8-bf91-78ac0d892dab/195faa44-0949-4e4a-a075-cc82f959d0cf"
-					(reference "C155")
-					(unit 1)
-				)
-				(path "/fd7503bc-e7fc-4766-b224-3d1c3d7de5ff/1b181806-12f4-40c8-bf91-78ac0d892dab/e2e765af-525f-4805-b4e1-1d4694321b94"
-					(reference "C146")
+					(reference "C150")
+					(unit 1)
+				)
+				(path "/fd7503bc-e7fc-4766-b224-3d1c3d7de5ff/1b181806-12f4-40c8-bf91-78ac0d892dab/e2e765af-525f-4805-b4e1-1d4694321b94"
+					(reference "C141")
 					(unit 1)
 				)
@@
 		(dnp no)
 		(fields_autoplaced yes)
-		(property "Reference" "#PWR0209"
+		(property "Reference" "#PWR0221"
 			(at 110.49 96.52 0)
 			(effects
@@
 			(project "FPGA_Board_BA"
 				(path "/fd7503bc-e7fc-4766-b224-3d1c3d7de5ff/1b181806-12f4-40c8-bf91-78ac0d892dab/195faa44-0949-4e4a-a075-cc82f959d0cf"
-					(reference "#PWR0239")
-					(unit 1)
-				)
-				(path "/fd7503bc-e7fc-4766-b224-3d1c3d7de5ff/1b181806-12f4-40c8-bf91-78ac0d892dab/e2e765af-525f-4805-b4e1-1d4694321b94"
-					(reference "#PWR0209")
+					(reference "#PWR0251")
+					(unit 1)
+				)
+				(path "/fd7503bc-e7fc-4766-b224-3d1c3d7de5ff/1b181806-12f4-40c8-bf91-78ac0d892dab/e2e765af-525f-4805-b4e1-1d4694321b94"
+					(reference "#PWR0221")
 					(unit 1)
 				)
@@
 		(dnp no)
 		(fields_autoplaced yes)
-		(property "Reference" "#PWR0213"
+		(property "Reference" "#PWR0225"
 			(at 171.45 97.79 0)
 			(effects
@@
 			(project "FPGA_Board_BA"
 				(path "/fd7503bc-e7fc-4766-b224-3d1c3d7de5ff/1b181806-12f4-40c8-bf91-78ac0d892dab/195faa44-0949-4e4a-a075-cc82f959d0cf"
-					(reference "#PWR0243")
-					(unit 1)
-				)
-				(path "/fd7503bc-e7fc-4766-b224-3d1c3d7de5ff/1b181806-12f4-40c8-bf91-78ac0d892dab/e2e765af-525f-4805-b4e1-1d4694321b94"
-					(reference "#PWR0213")
+					(reference "#PWR0255")
+					(unit 1)
+				)
+				(path "/fd7503bc-e7fc-4766-b224-3d1c3d7de5ff/1b181806-12f4-40c8-bf91-78ac0d892dab/e2e765af-525f-4805-b4e1-1d4694321b94"
+					(reference "#PWR0225")
 					(unit 1)
 				)
@@
 		(dnp no)
 		(fields_autoplaced yes)
-		(property "Reference" "#PWR0212"
+		(property "Reference" "#PWR0224"
 			(at 146.05 88.9 0)
 			(effects
@@
 			(project "FPGA_Board_BA"
 				(path "/fd7503bc-e7fc-4766-b224-3d1c3d7de5ff/1b181806-12f4-40c8-bf91-78ac0d892dab/195faa44-0949-4e4a-a075-cc82f959d0cf"
-					(reference "#PWR0242")
-					(unit 1)
-				)
-				(path "/fd7503bc-e7fc-4766-b224-3d1c3d7de5ff/1b181806-12f4-40c8-bf91-78ac0d892dab/e2e765af-525f-4805-b4e1-1d4694321b94"
-					(reference "#PWR0212")
-					(unit 1)
-				)
+					(reference "#PWR0254")
+					(unit 1)
+				)
+				(path "/fd7503bc-e7fc-4766-b224-3d1c3d7de5ff/1b181806-12f4-40c8-bf91-78ac0d892dab/e2e765af-525f-4805-b4e1-1d4694321b94"
+					(reference "#PWR0224")
+					(unit 1)
+				)

Commit message: schematic fixes after Leo Meeting
Connections:
- net +5V: now also R216.1, R217.1
- net A1: now also R216.2; no longer R216.1
- net A2: now also R217.2; no longer R217.1
- net GND: no longer R216.2, R217.2
Other:
- moved on the sheet: R216, R217
Changed lines of the file:
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@@
 	(paper "A4")
 	(junction
-		(at 100.33 104.14)
+		(at 87.63 99.06)
+		(diameter 0)
+		(color 0 0 0 0)
+	)
+	(junction
+		(at 92.71 104.14)
 		(diameter 0)
 		(color 0 0 0 0)
@@
 	)
 	(junction
+		(at 90.17 78.74)
+		(diameter 0)
+		(color 0 0 0 0)
+	)
+	(junction
 		(at 139.7 116.84)
 		(diameter 0)
 		(color 0 0 0 0)
 	)
-	(junction
-		(at 97.79 124.46)
-		(diameter 0)
-		(color 0 0 0 0)
-	)
-	(junction
-		(at 95.25 99.06)
-		(diameter 0)
-		(color 0 0 0 0)
-	)
-	(wire
-		(pts
-			(xy 95.25 99.06) (xy 129.54 99.06)
+	(wire
+		(pts
+			(xy 87.63 83.82) (xy 87.63 78.74)
+		)
+		(stroke
+			(width 0)
+			(type default)
+		)
+	)
+	(wire
+		(pts
+			(xy 92.71 104.14) (xy 129.54 104.14)
+		)
+		(stroke
+			(width 0)
+			(type default)
+		)
+	)
+	(wire
+		(pts
+			(xy 92.71 91.44) (xy 92.71 104.14)
+		)
+		(stroke
+			(width 0)
+			(type default)
+		)
+	)
+	(wire
+		(pts
+			(xy 90.17 74.93) (xy 90.17 78.74)
 		)
 		(stroke
@@
 	(wire
 		(pts
-			(xy 97.79 124.46) (xy 100.33 124.46)
+			(xy 90.17 78.74) (xy 92.71 78.74)
 		)
 		(stroke
@@
 	(wire
 		(pts
-			(xy 95.25 113.03) (xy 95.25 99.06)
+			(xy 87.63 91.44) (xy 87.63 99.06)
 		)
 		(stroke
@@
 	(wire
 		(pts
+			(xy 87.63 99.06) (xy 129.54 99.06)
+		)
+		(stroke
+			(width 0)
+			(type default)
+		)
+	)
+	(wire
+		(pts
 			(xy 149.86 104.14) (xy 160.02 104.14)
 		)
@@
 	(wire
 		(pts
-			(xy 83.82 104.14) (xy 100.33 104.14)
+			(xy 74.93 104.14) (xy 92.71 104.14)
 		)
 		(stroke
@@
 	(wire
 		(pts
-			(xy 97.79 124.46) (xy 95.25 124.46)
-		)
-		(stroke
-			(width 0)
-			(type default)
-		)
-	)
-	(wire
-		(pts
 			(xy 137.16 86.36) (xy 137.16 88.9)
 		)
@@
 	(wire
 		(pts
+			(xy 92.71 78.74) (xy 92.71 83.82)
+		)
+		(stroke
+			(width 0)
+			(type default)
+		)
+	)
+	(wire
+		(pts
 			(xy 146.05 86.36) (xy 142.24 86.36)
 		)
@@
 	(wire
 		(pts
-			(xy 100.33 104.14) (xy 100.33 113.03)
+			(xy 87.63 78.74) (xy 90.17 78.74)
 		)
 		(stroke
@@
 	(wire
 		(pts
-			(xy 83.82 99.06) (xy 95.25 99.06)
+			(xy 74.93 99.06) (xy 87.63 99.06)
 		)
 		(stroke
@@
 	(wire
 		(pts
-			(xy 100.33 104.14) (xy 129.54 104.14)
-		)
-		(stroke
-			(width 0)
-			(type default)
-		)
-	)
-	(wire
-		(pts
 			(xy 139.7 118.11) (xy 139.7 116.84)
 		)
@@
 	(wire
 		(pts
-			(xy 97.79 128.27) (xy 97.79 124.46)
-		)
-		(stroke
-			(width 0)
-			(type default)
-		)
-	)
-	(wire
-		(pts
-			(xy 95.25 120.65) (xy 95.25 124.46)
-		)
-		(stroke
-			(width 0)
-			(type default)
-		)
-	)
-	(wire
-		(pts
 			(xy 110.49 86.36) (xy 110.49 90.17)
-		)
-		(stroke
-			(width 0)
-			(type default)
-		)
-	)
-	(wire
-		(pts
-			(xy 100.33 120.65) (xy 100.33 124.46)
 		)
 		(stroke
@@
 	(hierarchical_label "A1"
 		(shape input)
-		(at 83.82 99.06 180)
+		(at 74.93 99.06 180)
 		(effects
 			(font
@@
 	(hierarchical_label "A2"
 		(shape input)
-		(at 83.82 104.14 180)
+		(at 74.93 104.14 180)
 		(effects
 			(font
@@
 	(symbol
 		(lib_id "WLIB_R:10k_0603")
-		(at 95.25 116.84 0)
+		(at 87.63 87.63 0)
 		(unit 1)
 		(exclude_from_sim no)
@@
 		(dnp no)
 		(property "Reference" "R216"
-			(at 90.17 122.174 90)
+			(at 82.55 92.964 90)
 			(effects
 				(font
@@
 		)
 		(property "Value" "10k_0603"
-			(at 92.71 122.174 90)
+			(at 85.09 92.964 90)
 			(effects
 				(font
@@
 		)
 		(property "Footprint" "Resistor_SMD:R_0603_1608Metric"
-			(at 95.25 97.79 0)
+			(at 87.63 68.58 0)
 			(effects
 				(font
@@
 		)
 		(property "Datasheet" "https://www.farnell.com/datasheets/2860681.pdf"
-			(at 95.25 95.25 0)
+			(at 87.63 66.04 0)
 			(effects
 				(font
@@
 		)
 		(property "Description" "Resistor"
-			(at 95.25 116.84 0)
+			(at 87.63 87.63 0)
 			(effects
 				(font
@@
 		)
 		(property "FARNELL" "2447230"
-			(at 95.25 100.33 0)
+			(at 87.63 71.12 0)
 			(effects
 				(font
@@
 		)
 		(property "Rated Power" "100mW"
-			(at 95.25 102.87 0)
+			(at 87.63 73.66 0)
 			(effects
 				(font
@@
 		)
 		(property "JLCPCB" "C25804"
-			(at 95.25 105.41 0)
+			(at 87.63 76.2 0)
 			(effects
 				(font
@@
 	(symbol
 		(lib_id "WLIB_R:10k_0603")
-		(at 100.33 116.84 0)
+		(at 92.71 87.63 0)
 		(mirror y)
 		(unit 1)
@@
 		(dnp no)
 		(property "Reference" "R217"
-			(at 105.41 122.174 90)
+			(at 97.79 92.964 90)
 			(effects
 				(font
@@
 		)
 		(property "Value" "10k_0603"
-			(at 102.87 122.174 90)
+			(at 95.25 92.964 90)
 			(effects
 				(font
@@
 		)
 		(property "Footprint" "Resistor_SMD:R_0603_1608Metric"
-			(at 100.33 97.79 0)
+			(at 92.71 68.58 0)
 			(effects
 				(font
@@
 		)
 		(property "Datasheet" "https://www.farnell.com/datasheets/2860681.pdf"
-			(at 100.33 95.25 0)
+			(at 92.71 66.04 0)
 			(effects
 				(font
@@
 		)
 		(property "Description" "Resistor"
-			(at 100.33 116.84 0)
+			(at 92.71 87.63 0)
 			(effects
 				(font
@@
 		)
 		(property "FARNELL" "2447230"
-			(at 100.33 100.33 0)
+			(at 92.71 71.12 0)
 			(effects
 				(font
@@
 		)
 		(property "Rated Power" "100mW"
-			(at 100.33 102.87 0)
+			(at 92.71 73.66 0)
 			(effects
 				(font
@@
 		)
 		(property "JLCPCB" "C25804"
-			(at 100.33 105.41 0)
+			(at 92.71 76.2 0)
 			(effects
 				(font
@@
 				(path "/fd7503bc-e7fc-4766-b224-3d1c3d7de5ff/1b181806-12f4-40c8-bf91-78ac0d892dab/e2e765af-525f-4805-b4e1-1d4694321b94"
 					(reference "R217")
-					(unit 1)
-				)
-			)
-		)
-	)
-	(symbol
-		(lib_id "power:GND")
-		(at 97.79 128.27 0)
-		(unit 1)
-		(exclude_from_sim no)
-		(in_bom yes)
-		(on_board yes)
-		(dnp no)
-		(fields_autoplaced yes)
-		(property "Reference" "#PWR0220"
-			(at 97.79 134.62 0)
-			(effects
-				(font
-					(size 1.27 1.27)
-				)
-				(hide yes)
-			)
-		)
-		(property "Value" "GND"
-			(at 97.79 133.35 0)
-			(effects
-				(font
-					(size 1.27 1.27)
-				)
-			)
-		)
-		(property "Footprint" ""
-			(at 97.79 128.27 0)
-			(effects
-				(font
-					(size 1.27 1.27)
-				)
-				(hide yes)
-			)
-		)
-		(property "Datasheet" ""
-			(at 97.79 128.27 0)
-			(effects
-				(font
-					(size 1.27 1.27)
-				)
-				(hide yes)
-			)
-		)
-		(property "Description" "Power symbol creates a global label with name \"GND\" , ground"
-			(at 97.79 128.27 0)
-			(effects
-				(font
-					(size 1.27 1.27)
-				)
-				(hide yes)
-			)
-		)
-		(pin "1"
-		)
-		(instances
-			(project "FPGA_Board_BA"
-				(path "/fd7503bc-e7fc-4766-b224-3d1c3d7de5ff/1b181806-12f4-40c8-bf91-78ac0d892dab/195faa44-0949-4e4a-a075-cc82f959d0cf"
-					(reference "#PWR0250")
-					(unit 1)
-				)
-				(path "/fd7503bc-e7fc-4766-b224-3d1c3d7de5ff/1b181806-12f4-40c8-bf91-78ac0d892dab/e2e765af-525f-4805-b4e1-1d4694321b94"
-					(reference "#PWR0220")
 					(unit 1)
 				)
@@
 					(unit 1)
 				)
+			)
+		)
+	)
+	(symbol
+		(lib_id "power:+5V")
+		(at 90.17 74.93 0)
+		(unit 1)
+		(exclude_from_sim no)
+		(in_bom yes)
+		(on_board yes)
+		(dnp no)
+		(fields_autoplaced yes)
+		(property "Reference" "#PWR013"
+			(at 90.17 78.74 0)
+			(effects
+				(font
+					(size 1.27 1.27)
+				)
+				(hide yes)
+			)
+		)
+		(property "Value" "+5V"
+			(at 90.17 69.85 0)
+			(effects
+				(font
+					(size 1.27 1.27)
+				)
+			)
+		)
+		(property "Footprint" ""
+			(at 90.17 74.93 0)
+			(effects
+				(font
+					(size 1.27 1.27)
+				)
+				(hide yes)
+			)
+		)
+		(property "Datasheet" ""
+			(at 90.17 74.93 0)
+			(effects
+				(font
+					(size 1.27 1.27)
+				)
+				(hide yes)
+			)
+		)
+		(property "Description" "Power symbol creates a global label with name \"+5V\""
+			(at 90.17 74.93 0)
+			(effects
+				(font
+					(size 1.27 1.27)
+				)
+				(hide yes)
+			)
+		)
+		(pin "1"
+		)
+		(instances
+			(project "FPGA_Board_BA"
+				(path "/fd7503bc-e7fc-4766-b224-3d1c3d7de5ff/1b181806-12f4-40c8-bf91-78ac0d892dab/195faa44-0949-4e4a-a075-cc82f959d0cf"
+					(reference "#PWR041")
+					(unit 1)
+				)
+				(path "/fd7503bc-e7fc-4766-b224-3d1c3d7de5ff/1b181806-12f4-40c8-bf91-78ac0d892dab/e2e765af-525f-4805-b4e1-1d4694321b94"
+					(reference "#PWR013")
+					(unit 1)
+				)
