File: FPGA_Board_BA/PCB/tamura.kicad_sch (KiCad schematic)
At the start: 5 parts, among them U32 S22P006S05

Commit message: exported stuff
Parts:
- renumbered C141 to C136, R158 to R197, R159 to R198, R160 to R199, U32 to U31

Commit message: schematic fixes after Leo Meeting
Parts:
- removed R197, R199: 9k1_0603, Resistor_SMD:R_0603_1608Metric, symbol WLIB_R:9k1_0603
- removed R198: 1k_0603, Resistor_SMD:R_0603_1608Metric, symbol WLIB_R:1k_0603
- added J2: PinHeader_2x4_SMD, Connector_PinHeader_2.54mm:PinHeader_2x04_P2.54mm_Vertical_SMD, symbol MYLIB_Misc:PinHeader_2x4_SMD
Connections:
- net I_in: now also J2.1 (Pin_1), J2.2 (Pin_2); no longer U31.2 (In_2)
- net I_out: now also J2.7 (Pin_7), J2.8 (Pin_8)
- net Vout: now also U31.7 (Vout)
- net +5VA renamed +5VA_2
- new net pin2: J2.3 (Pin_3), U31.2 (In_2)
- new net pin3: J2.4 (Pin_4), U31.3 (In_3)
- new net pin5: J2.6 (Pin_6), U31.5 (Out_2)
- new net pin6: J2.5 (Pin_5), U31.6 (Out_3)
Other:
- note removed: "ADC Reference is 4.096V Vout = V * R1 / (R1 + R2) 4.096V = 5V * R1 / (R1 + R2) 0.8192 = R1 / (R1 + R2) 0.8192 * R1 + 0.8192 * R2 = R1 0.1808 * R1 = 0.8192 * R2 R1 / R2 = 4.53097 R1 := 9.1k || 9.1k = 4.55k R2 = 1k R1/R2 = 4.55 Vout_max = 5V * 4.55 / 5.55 = 4.099V -> very little saturation"
- note removed: "R1"
- note removed: "R2"
