File: FPGA_Board_BA/PCB/analog_voltage.kicad_sch (KiCad schematic)
At the start: 11 parts, among them U801 TPS61022, U802 MCP1703AT-5002EDB

Commit message: schematic almost ready pt2
Parts:
- added D801, D802: LED_G_0603, WLIB_DO:LED_0603_1608Metric, symbol WLIB_D:LED_G_0603
- added R803, R804: 10k_0603, Resistor_SMD:R_0603_1608Metric, symbol WLIB_R:10k_0603
Connections:
- net +5VA: now also R803.1
- net 5.5V: now also R804.1
- net GND: now also D801.1 (K), D802.1 (K)
- new net: D802.2 (A), R804.2
- new net: D801.2 (A), R803.2
Other:
- note added: "Status LED for active boost converter"
- note added: "Status LED for active low-noise 5V"

Commit message: work
Parts:
- renumbered C801 to C48, C802 to C49, C805 to C50, C806 to C51, C803 to C52, C804 to C53, D801 to D5, D802 to D6, L801 to L3, R802 to R40, R801 to R41, R803 to R42, R804 to R43, U801 to U12, U802 to U13
Changed lines of the file:
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@@
 		(dnp no)
 		(fields_autoplaced yes)
-		(property "Reference" "U802"
+		(property "Reference" "U13"
 			(at 129.54 119.38 0)
 			(effects
@@
 			(project ""
 				(path "/fd7503bc-e7fc-4766-b224-3d1c3d7de5ff/01163162-2dd3-462f-91a6-fa3b981b9fc9"
-					(reference "U802")
+					(reference "U13")
 					(unit 1)
 				)
@@
 		(on_board yes)
 		(dnp no)
-		(property "Reference" "C801"
+		(property "Reference" "C48"
 			(at 71.12 80.264 90)
 			(effects
@@
 			(project ""
 				(path "/fd7503bc-e7fc-4766-b224-3d1c3d7de5ff/01163162-2dd3-462f-91a6-fa3b981b9fc9"
-					(reference "C801")
+					(reference "C48")
 					(unit 1)
 				)
@@
 		(dnp no)
 		(fields_autoplaced yes)
-		(property "Reference" "R804"
+		(property "Reference" "R43"
 			(at 193.04 78.7399 0)
 			(effects
@@
 			(project "FPGA_Board_BA"
 				(path "/fd7503bc-e7fc-4766-b224-3d1c3d7de5ff/01163162-2dd3-462f-91a6-fa3b981b9fc9"
-					(reference "R804")
+					(reference "R43")
 					(unit 1)
 				)
@@
 		(on_board yes)
 		(dnp no)
-		(property "Reference" "C805"
+		(property "Reference" "C50"
 			(at 98.806 139.954 90)
 			(effects
@@
 			(project ""
 				(path "/fd7503bc-e7fc-4766-b224-3d1c3d7de5ff/01163162-2dd3-462f-91a6-fa3b981b9fc9"
-					(reference "C805")
+					(reference "C50")
 					(unit 1)
 				)
@@
 		(dnp no)
 		(fields_autoplaced yes)
-		(property "Reference" "D801"
+		(property "Reference" "D5"
 			(at 175.26 142.5574 90)
 			(effects
@@
 			(project ""
 				(path "/fd7503bc-e7fc-4766-b224-3d1c3d7de5ff/01163162-2dd3-462f-91a6-fa3b981b9fc9"
-					(reference "D801")
+					(reference "D5")
 					(unit 1)
 				)
@@
 		(dnp no)
 		(fields_autoplaced yes)
-		(property "Reference" "#PWR0804"
+		(property "Reference" "#PWR055"
 			(at 129.54 152.4 0)
 			(effects
@@
 			(project ""
 				(path "/fd7503bc-e7fc-4766-b224-3d1c3d7de5ff/01163162-2dd3-462f-91a6-fa3b981b9fc9"
-					(reference "#PWR0804")
+					(reference "#PWR055")
 					(unit 1)
 				)
@@
 		(dnp no)
 		(fields_autoplaced yes)
-		(property "Reference" "D802"
+		(property "Reference" "D6"
 			(at 194.31 89.2174 90)
 			(effects
@@
 			(project "FPGA_Board_BA"
 				(path "/fd7503bc-e7fc-4766-b224-3d1c3d7de5ff/01163162-2dd3-462f-91a6-fa3b981b9fc9"
-					(reference "D802")
+					(reference "D6")
 					(unit 1)
 				)
@@
 		(dnp no)
 		(fields_autoplaced yes)
-		(property "Reference" "#PWR0802"
+		(property "Reference" "#PWR053"
 			(at 67.31 92.71 0)
 			(effects
@@
 			(project "FPGA_Board_BA"
 				(path "/fd7503bc-e7fc-4766-b224-3d1c3d7de5ff/01163162-2dd3-462f-91a6-fa3b981b9fc9"
-					(reference "#PWR0802")
+					(reference "#PWR053")
 					(unit 1)
 				)
@@
 		(dnp no)
 		(fields_autoplaced yes)
-		(property "Reference" "R802"
+		(property "Reference" "R40"
 			(at 147.32 76.1999 0)
 			(effects
@@
 			(project ""
 				(path "/fd7503bc-e7fc-4766-b224-3d1c3d7de5ff/01163162-2dd3-462f-91a6-fa3b981b9fc9"
-					(reference "R802")
+					(reference "R40")
 					(unit 1)
 				)
@@
 		(on_board yes)
 		(dnp no)
-		(property "Reference" "C802"
+		(property "Reference" "C49"
 			(at 83.566 79.756 90)
 			(effects
@@
 			(project ""
 				(path "/fd7503bc-e7fc-4766-b224-3d1c3d7de5ff/01163162-2dd3-462f-91a6-fa3b981b9fc9"
-					(reference "C802")
+					(reference "C49")
 					(unit 1)
 				)
@@
 		(dnp no)
 		(fields_autoplaced yes)
-		(property "Reference" "R803"
+		(property "Reference" "R42"
 			(at 173.99 132.0799 0)
 			(effects
@@
 			(project ""
 				(path "/fd7503bc-e7fc-4766-b224-3d1c3d7de5ff/01163162-2dd3-462f-91a6-fa3b981b9fc9"
-					(reference "R803")
+					(reference "R42")
 					(unit 1)
 				)
@@
 		(on_board yes)
 		(dnp no)
-		(property "Reference" "C806"
+		(property "Reference" "C51"
 			(at 147.066 139.954 90)
 			(effects
@@
 			(project "FPGA_Board_BA"
 				(path "/fd7503bc-e7fc-4766-b224-3d1c3d7de5ff/01163162-2dd3-462f-91a6-fa3b981b9fc9"
-					(reference "C806")
+					(reference "C51")
 					(unit 1)
 				)
@@
 		(on_board yes)
 		(dnp no)
-		(property "Reference" "C804"
+		(property "Reference" "C53"
 			(at 173.736 82.296 90)
 			(effects
@@
 			(project "FPGA_Board_BA"
 				(path "/fd7503bc-e7fc-4766-b224-3d1c3d7de5ff/01163162-2dd3-462f-91a6-fa3b981b9fc9"
-					(reference "C804")
+					(reference "C53")
 					(unit 1)
 				)
@@
 		(on_board yes)
 		(dnp no)
-		(property "Reference" "C803"
+		(property "Reference" "C52"
 			(at 163.576 82.296 90)
 			(effects
@@
 			(project "FPGA_Board_BA"
 				(path "/fd7503bc-e7fc-4766-b224-3d1c3d7de5ff/01163162-2dd3-462f-91a6-fa3b981b9fc9"
-					(reference "C803")
+					(reference "C52")
 					(unit 1)
 				)
@@
 		(dnp no)
 		(fields_autoplaced yes)
-		(property "Reference" "#PWR0805"
+		(property "Reference" "#PWR058"
 			(at 171.45 154.94 0)
 			(effects
@@
 			(project "FPGA_Board_BA"
 				(path "/fd7503bc-e7fc-4766-b224-3d1c3d7de5ff/01163162-2dd3-462f-91a6-fa3b981b9fc9"
-					(reference "#PWR0805")
+					(reference "#PWR058")
 					(unit 1)
 				)
@@
 		(dnp no)
 		(fields_autoplaced yes)
-		(property "Reference" "L801"
+		(property "Reference" "L3"
 			(at 118.11 43.18 0)
 			(effects
@@
 			(project ""
 				(path "/fd7503bc-e7fc-4766-b224-3d1c3d7de5ff/01163162-2dd3-462f-91a6-fa3b981b9fc9"
-					(reference "L801")
+					(reference "L3")
 					(unit 1)
 				)
@@
 		(dnp no)
 		(fields_autoplaced yes)
-		(property "Reference" "#PWR0803"
+		(property "Reference" "#PWR056"
 			(at 144.78 102.87 0)
 			(effects
@@
 			(project "FPGA_Board_BA"
 				(path "/fd7503bc-e7fc-4766-b224-3d1c3d7de5ff/01163162-2dd3-462f-91a6-fa3b981b9fc9"
-					(reference "#PWR0803")
+					(reference "#PWR056")
 					(unit 1)
 				)
@@
 		(dnp no)
 		(fields_autoplaced yes)
-		(property "Reference" "#PWR0807"
+		(property "Reference" "#PWR057"
 			(at 153.67 123.19 0)
 			(effects
@@
 			(project ""
 				(path "/fd7503bc-e7fc-4766-b224-3d1c3d7de5ff/01163162-2dd3-462f-91a6-fa3b981b9fc9"
-					(reference "#PWR0807")
+					(reference "#PWR057")
 					(unit 1)
 				)
@@
 		(dnp no)
 		(fields_autoplaced yes)
-		(property "Reference" "R801"
+		(property "Reference" "R41"
 			(at 147.32 88.8999 0)
 			(effects
@@
 			(project ""
 				(path "/fd7503bc-e7fc-4766-b224-3d1c3d7de5ff/01163162-2dd3-462f-91a6-fa3b981b9fc9"
-					(reference "R801")
+					(reference "R41")
 					(unit 1)
 				)
@@
 		(dnp no)
 		(fields_autoplaced yes)
-		(property "Reference" "#PWR0808"
+		(property "Reference" "#PWR060"
 			(at 190.5 101.6 0)
 			(effects
@@
 			(project "FPGA_Board_BA"
 				(path "/fd7503bc-e7fc-4766-b224-3d1c3d7de5ff/01163162-2dd3-462f-91a6-fa3b981b9fc9"
-					(reference "#PWR0808")
+					(reference "#PWR060")
 					(unit 1)
 				)
@@
 		(dnp no)
 		(fields_autoplaced yes)
-		(property "Reference" "U801"
+		(property "Reference" "U12"
 			(at 121.92 58.42 0)
 			(effects
@@
 			(project ""
 				(path "/fd7503bc-e7fc-4766-b224-3d1c3d7de5ff/01163162-2dd3-462f-91a6-fa3b981b9fc9"
-					(reference "U801")
+					(reference "U12")
 					(unit 1)
 				)
@@
 		(dnp no)
 		(fields_autoplaced yes)
-		(property "Reference" "#PWR0806"
+		(property "Reference" "#PWR059"
 			(at 173.99 96.52 0)
 			(effects
@@
 			(project "FPGA_Board_BA"
 				(path "/fd7503bc-e7fc-4766-b224-3d1c3d7de5ff/01163162-2dd3-462f-91a6-fa3b981b9fc9"
-					(reference "#PWR0806")
+					(reference "#PWR059")
 					(unit 1)
 				)
@@
 		(dnp no)
 		(fields_autoplaced yes)
-		(property "Reference" "#PWR0801"
+		(property "Reference" "#PWR054"
 			(at 121.92 96.52 0)
 			(effects
@@
 			(project ""
 				(path "/fd7503bc-e7fc-4766-b224-3d1c3d7de5ff/01163162-2dd3-462f-91a6-fa3b981b9fc9"
-					(reference "#PWR0801")
-					(unit 1)
-				)
+					(reference "#PWR054")
+					(unit 1)
+				)

Commit message: 22.11
Parts:
- renumbered D6 to D10, D5 to D9, R40 to R33, R41 to R34, R42 to R35, R43 to R36, U12 to U8, U13 to U9
Other:
- note added: "Driven loads: - Tamura Current Sensor 50mA - 150mA (4x, typ:12.5mA, max:37.5mA) - HV-Probe (4x, (TLV197 typ:1mA)) 4mA - ADC (2x, typ: 31mA) 62mA - OpAmp for ADC (16x, Typ:9mA) 144mA - Potentiometer (2x, max:1.5mA) 3mA Sum: 263mA - 363mA Maximal Current: 250mA Frage: sollte der Tamura auch von 5VA versorgt werden?"
Changed lines of the file:
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@@
 	(text "Status LED for active low-noise 5V"
 		(exclude_from_sim no)
-		(at 181.61 123.444 0)
+		(at 175.514 123.444 0)
 		(effects
 			(font
@@
 		(exclude_from_sim no)
 		(at 146.558 64.262 0)
+		(effects
+			(font
+				(size 1.27 1.27)
+			)
+			(justify left)
+		)
+	)
+	(text "Driven loads:\n- Tamura Current Sensor					50mA - 150mA\n(4x, typ:12.5mA, max:37.5mA)			\n- HV-Probe (4x, (TLV197 typ:1mA))		4mA\n- ADC (2x, typ: 31mA)					62mA\n- OpAmp for ADC (16x, Typ:9mA)			144mA\n- Potentiometer (2x, max:1.5mA)			3mA\n\nSum:									263mA - 363mA\nMaximal Current:						250mA\n\nFrage: sollte der Tamura auch von 5VA versorgt werden?"
+		(exclude_from_sim no)
+		(at 98.806 168.656 0)
 		(effects
 			(font
@@
 		(dnp no)
 		(fields_autoplaced yes)
-		(property "Reference" "U13"
+		(property "Reference" "U9"
 			(at 129.54 119.38 0)
 			(effects
@@
 			(project ""
 				(path "/fd7503bc-e7fc-4766-b224-3d1c3d7de5ff/01163162-2dd3-462f-91a6-fa3b981b9fc9"
-					(reference "U13")
+					(reference "U9")
 					(unit 1)
 				)
@@
 		(dnp no)
 		(fields_autoplaced yes)
-		(property "Reference" "R43"
+		(property "Reference" "R36"
 			(at 193.04 78.7399 0)
 			(effects
@@
 			(project "FPGA_Board_BA"
 				(path "/fd7503bc-e7fc-4766-b224-3d1c3d7de5ff/01163162-2dd3-462f-91a6-fa3b981b9fc9"
-					(reference "R43")
+					(reference "R36")
 					(unit 1)
 				)
@@
 		(dnp no)
 		(fields_autoplaced yes)
-		(property "Reference" "D5"
+		(property "Reference" "D9"
 			(at 175.26 142.5574 90)
 			(effects
@@
 			(project ""
 				(path "/fd7503bc-e7fc-4766-b224-3d1c3d7de5ff/01163162-2dd3-462f-91a6-fa3b981b9fc9"
-					(reference "D5")
+					(reference "D9")
 					(unit 1)
 				)
@@
 		(dnp no)
 		(fields_autoplaced yes)
-		(property "Reference" "#PWR055"
+		(property "Reference" "#PWR060"
 			(at 129.54 152.4 0)
 			(effects
@@
 			(project ""
 				(path "/fd7503bc-e7fc-4766-b224-3d1c3d7de5ff/01163162-2dd3-462f-91a6-fa3b981b9fc9"
-					(reference "#PWR055")
+					(reference "#PWR060")
 					(unit 1)
 				)
@@
 		(dnp no)
 		(fields_autoplaced yes)
-		(property "Reference" "D6"
+		(property "Reference" "D10"
 			(at 194.31 89.2174 90)
 			(effects
@@
 			(project "FPGA_Board_BA"
 				(path "/fd7503bc-e7fc-4766-b224-3d1c3d7de5ff/01163162-2dd3-462f-91a6-fa3b981b9fc9"
-					(reference "D6")
+					(reference "D10")
 					(unit 1)
 				)
@@
 		(dnp no)
 		(fields_autoplaced yes)
-		(property "Reference" "#PWR053"
+		(property "Reference" "#PWR058"
 			(at 67.31 92.71 0)
 			(effects
@@
 			(project "FPGA_Board_BA"
 				(path "/fd7503bc-e7fc-4766-b224-3d1c3d7de5ff/01163162-2dd3-462f-91a6-fa3b981b9fc9"
-					(reference "#PWR053")
+					(reference "#PWR058")
 					(unit 1)
 				)
@@
 		(dnp no)
 		(fields_autoplaced yes)
-		(property "Reference" "R40"
+		(property "Reference" "R33"
 			(at 147.32 76.1999 0)
 			(effects
@@
 			(project ""
 				(path "/fd7503bc-e7fc-4766-b224-3d1c3d7de5ff/01163162-2dd3-462f-91a6-fa3b981b9fc9"
-					(reference "R40")
+					(reference "R33")
 					(unit 1)
 				)
@@
 		(dnp no)
 		(fields_autoplaced yes)
-		(property "Reference" "R42"
+		(property "Reference" "R35"
 			(at 173.99 132.0799 0)
 			(effects
@@
 			(project ""
 				(path "/fd7503bc-e7fc-4766-b224-3d1c3d7de5ff/01163162-2dd3-462f-91a6-fa3b981b9fc9"
-					(reference "R42")
+					(reference "R35")
 					(unit 1)
 				)
@@
 		(dnp no)
 		(fields_autoplaced yes)
-		(property "Reference" "#PWR058"
+		(property "Reference" "#PWR063"
 			(at 171.45 154.94 0)
 			(effects
@@
 			(project "FPGA_Board_BA"
 				(path "/fd7503bc-e7fc-4766-b224-3d1c3d7de5ff/01163162-2dd3-462f-91a6-fa3b981b9fc9"
-					(reference "#PWR058")
+					(reference "#PWR063")
 					(unit 1)
 				)
@@
 		(dnp no)
 		(fields_autoplaced yes)
-		(property "Reference" "#PWR056"
+		(property "Reference" "#PWR061"
 			(at 144.78 102.87 0)
 			(effects
@@
 			(project "FPGA_Board_BA"
 				(path "/fd7503bc-e7fc-4766-b224-3d1c3d7de5ff/01163162-2dd3-462f-91a6-fa3b981b9fc9"
-					(reference "#PWR056")
+					(reference "#PWR061")
 					(unit 1)
 				)
@@
 		(dnp no)
 		(fields_autoplaced yes)
-		(property "Reference" "#PWR057"
+		(property "Reference" "#PWR062"
 			(at 153.67 123.19 0)
 			(effects
@@
 			(project ""
 				(path "/fd7503bc-e7fc-4766-b224-3d1c3d7de5ff/01163162-2dd3-462f-91a6-fa3b981b9fc9"
-					(reference "#PWR057")
+					(reference "#PWR062")
 					(unit 1)
 				)
@@
 		(dnp no)
 		(fields_autoplaced yes)
-		(property "Reference" "R41"
+		(property "Reference" "R34"
 			(at 147.32 88.8999 0)
 			(effects
@@
 			(project ""
 				(path "/fd7503bc-e7fc-4766-b224-3d1c3d7de5ff/01163162-2dd3-462f-91a6-fa3b981b9fc9"
-					(reference "R41")
+					(reference "R34")
 					(unit 1)
 				)
@@
 		(dnp no)
 		(fields_autoplaced yes)
-		(property "Reference" "#PWR060"
+		(property "Reference" "#PWR065"
 			(at 190.5 101.6 0)
 			(effects
@@
 			(project "FPGA_Board_BA"
 				(path "/fd7503bc-e7fc-4766-b224-3d1c3d7de5ff/01163162-2dd3-462f-91a6-fa3b981b9fc9"
-					(reference "#PWR060")
+					(reference "#PWR065")
 					(unit 1)
 				)
@@
 		(dnp no)
 		(fields_autoplaced yes)
-		(property "Reference" "U12"
+		(property "Reference" "U8"
 			(at 121.92 58.42 0)
 			(effects
@@
 			(project ""
 				(path "/fd7503bc-e7fc-4766-b224-3d1c3d7de5ff/01163162-2dd3-462f-91a6-fa3b981b9fc9"
-					(reference "U12")
+					(reference "U8")
 					(unit 1)
 				)
@@
 		(dnp no)
 		(fields_autoplaced yes)
-		(property "Reference" "#PWR059"
+		(property "Reference" "#PWR064"
 			(at 173.99 96.52 0)
 			(effects
@@
 			(project "FPGA_Board_BA"
 				(path "/fd7503bc-e7fc-4766-b224-3d1c3d7de5ff/01163162-2dd3-462f-91a6-fa3b981b9fc9"
-					(reference "#PWR059")
+					(reference "#PWR064")
 					(unit 1)
 				)
@@
 		(dnp no)
 		(fields_autoplaced yes)
-		(property "Reference" "#PWR054"
+		(property "Reference" "#PWR059"
 			(at 121.92 96.52 0)
 			(effects
@@
 			(project ""
 				(path "/fd7503bc-e7fc-4766-b224-3d1c3d7de5ff/01163162-2dd3-462f-91a6-fa3b981b9fc9"
-					(reference "#PWR054")
+					(reference "#PWR059")
 					(unit 1)
 				)

Commit message: exported stuff
Parts:
- D10, D9: footprint WLIB_DO:LED_0603_1608Metric -> LED_SMD:LED_0603_1608Metric
- renumbered R33 to R45, R34 to R46, R35 to R47, R36 to R48
Changed lines of the file:
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@@
 		(dnp no)
 		(fields_autoplaced yes)
-		(property "Reference" "R36"
+		(property "Reference" "R48"
 			(at 193.04 78.7399 0)
 			(effects
@@
 			(project "FPGA_Board_BA"
 				(path "/fd7503bc-e7fc-4766-b224-3d1c3d7de5ff/01163162-2dd3-462f-91a6-fa3b981b9fc9"
-					(reference "R36")
+					(reference "R48")
 					(unit 1)
 				)
@@
 			)
 		)
-		(property "Footprint" "WLIB_DO:LED_0603_1608Metric"
+		(property "Footprint" "LED_SMD:LED_0603_1608Metric"
 			(at 161.29 142.24 0)
 			(effects
@@
 		(dnp no)
 		(fields_autoplaced yes)
-		(property "Reference" "#PWR060"
+		(property "Reference" "#PWR065"
 			(at 129.54 152.4 0)
 			(effects
@@
 			(project ""
 				(path "/fd7503bc-e7fc-4766-b224-3d1c3d7de5ff/01163162-2dd3-462f-91a6-fa3b981b9fc9"
-					(reference "#PWR060")
+					(reference "#PWR065")
 					(unit 1)
 				)
@@
 			)
 		)
-		(property "Footprint" "WLIB_DO:LED_0603_1608Metric"
+		(property "Footprint" "LED_SMD:LED_0603_1608Metric"
 			(at 180.34 88.9 0)
 			(effects
@@
 		(dnp no)
 		(fields_autoplaced yes)
-		(property "Reference" "#PWR058"
+		(property "Reference" "#PWR063"
 			(at 67.31 92.71 0)
 			(effects
@@
 			(project "FPGA_Board_BA"
 				(path "/fd7503bc-e7fc-4766-b224-3d1c3d7de5ff/01163162-2dd3-462f-91a6-fa3b981b9fc9"
-					(reference "#PWR058")
+					(reference "#PWR063")
 					(unit 1)
 				)
@@
 		(dnp no)
 		(fields_autoplaced yes)
-		(property "Reference" "R33"
+		(property "Reference" "R45"
 			(at 147.32 76.1999 0)
 			(effects
@@
 			(project ""
 				(path "/fd7503bc-e7fc-4766-b224-3d1c3d7de5ff/01163162-2dd3-462f-91a6-fa3b981b9fc9"
-					(reference "R33")
+					(reference "R45")
 					(unit 1)
 				)
@@
 		(dnp no)
 		(fields_autoplaced yes)
-		(property "Reference" "R35"
+		(property "Reference" "R47"
 			(at 173.99 132.0799 0)
 			(effects
@@
 			(project ""
 				(path "/fd7503bc-e7fc-4766-b224-3d1c3d7de5ff/01163162-2dd3-462f-91a6-fa3b981b9fc9"
-					(reference "R35")
+					(reference "R47")
 					(unit 1)
 				)
@@
 		(dnp no)
 		(fields_autoplaced yes)
-		(property "Reference" "#PWR063"
+		(property "Reference" "#PWR068"
 			(at 171.45 154.94 0)
 			(effects
@@
 			(project "FPGA_Board_BA"
 				(path "/fd7503bc-e7fc-4766-b224-3d1c3d7de5ff/01163162-2dd3-462f-91a6-fa3b981b9fc9"
-					(reference "#PWR063")
+					(reference "#PWR068")
 					(unit 1)
 				)
@@
 		(dnp no)
 		(fields_autoplaced yes)
-		(property "Reference" "#PWR061"
+		(property "Reference" "#PWR066"
 			(at 144.78 102.87 0)
 			(effects
@@
 			(project "FPGA_Board_BA"
 				(path "/fd7503bc-e7fc-4766-b224-3d1c3d7de5ff/01163162-2dd3-462f-91a6-fa3b981b9fc9"
-					(reference "#PWR061")
+					(reference "#PWR066")
 					(unit 1)
 				)
@@
 		(dnp no)
 		(fields_autoplaced yes)
-		(property "Reference" "#PWR062"
+		(property "Reference" "#PWR067"
 			(at 153.67 123.19 0)
 			(effects
@@
 			(project ""
 				(path "/fd7503bc-e7fc-4766-b224-3d1c3d7de5ff/01163162-2dd3-462f-91a6-fa3b981b9fc9"
-					(reference "#PWR062")
+					(reference "#PWR067")
 					(unit 1)
 				)
@@
 		(dnp no)
 		(fields_autoplaced yes)
-		(property "Reference" "R34"
+		(property "Reference" "R46"
 			(at 147.32 88.8999 0)
 			(effects
@@
 			(project ""
 				(path "/fd7503bc-e7fc-4766-b224-3d1c3d7de5ff/01163162-2dd3-462f-91a6-fa3b981b9fc9"
-					(reference "R34")
+					(reference "R46")
 					(unit 1)
 				)
@@
 		(dnp no)
 		(fields_autoplaced yes)
-		(property "Reference" "#PWR065"
+		(property "Reference" "#PWR070"
 			(at 190.5 101.6 0)
 			(effects
@@
 			(project "FPGA_Board_BA"
 				(path "/fd7503bc-e7fc-4766-b224-3d1c3d7de5ff/01163162-2dd3-462f-91a6-fa3b981b9fc9"
-					(reference "#PWR065")
+					(reference "#PWR070")
 					(unit 1)
 				)
@@
 		(dnp no)
 		(fields_autoplaced yes)
-		(property "Reference" "#PWR064"
+		(property "Reference" "#PWR069"
 			(at 173.99 96.52 0)
 			(effects
@@
 			(project "FPGA_Board_BA"
 				(path "/fd7503bc-e7fc-4766-b224-3d1c3d7de5ff/01163162-2dd3-462f-91a6-fa3b981b9fc9"
-					(reference "#PWR064")
+					(reference "#PWR069")
 					(unit 1)
 				)
@@
 		(dnp no)
 		(fields_autoplaced yes)
-		(property "Reference" "#PWR059"
+		(property "Reference" "#PWR064"
 			(at 121.92 96.52 0)
 			(effects
@@
 			(project ""
 				(path "/fd7503bc-e7fc-4766-b224-3d1c3d7de5ff/01163162-2dd3-462f-91a6-fa3b981b9fc9"
-					(reference "#PWR059")
-					(unit 1)
-				)
+					(reference "#PWR064")
+					(unit 1)
+				)

Commit message: schematic fixes after Leo Meeting
Parts:
- removed C50, C51: 1u_0603, WLIB_Capacitor:C_0603, symbol WLIB_C:1u_0603
- removed D9: LED_G_0603, LED_SMD:LED_0603_1608Metric, symbol WLIB_D:LED_G_0603
- removed R47: 10k_0603, Resistor_SMD:R_0603_1608Metric, symbol WLIB_R:10k_0603
- removed U9: MCP1703AT-5002EDB, Package_TO_SOT_SMD:SOT-223, symbol MYLIB_Misc:MCP1703AT_5002
Other:
- added sheet 5VA-1 (5va.kicad_sch)
- added sheet 5VA-2 (5va.kicad_sch)
- note added: "Driven loads: - Tamura Current Sensor 50mA - 150mA (4x, typ:12.5mA, max:37.5mA) - HV-Probe (4x, (TLV197 typ:1mA)) 4mA - ADC (2x, typ: 31mA) 62mA - OpAmp for ADC (16x, Typ:9mA) 144mA - Potentiometer (2x, max:1.5mA) 3mA Sum: 263mA - 363mA Maximal Current: 250mA"
- note removed: "Driven loads: - Tamura Current Sensor 50mA - 150mA (4x, typ:12.5mA, max:37.5mA) - HV-Probe (4x, (TLV197 typ:1mA)) 4mA - ADC (2x, typ: 31mA) 62mA - OpAmp for ADC (16x, Typ:9mA) 144mA - Potentiometer (2x, max:1.5mA) 3mA Sum: 263mA - 363mA Maximal Current: 250mA Frage: sollte der Tamura auch von 5VA versorgt werden?"
- note removed: "Status LED for active low-noise 5V"
- moved on the sheet: C48, C49, C52, C53, D10, L3, R45, R46, R48, U8

Commit message: Component placement ready. Waiting to meet with Leo
Parts:
- L3: footprint (none) -> MYLIB_Misc:74404043010A
Changed lines of the file:
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@@
 			)
 		)
-		(property "Footprint" ""
+		(property "Footprint" "MYLIB_Misc:74404043010A"
 			(at 82.55 24.13 0)
 			(effects
