File: FPGA_Board_BA/PCB/encoder.kicad_sch (KiCad schematic)
At the start: 1 part, among them J20 JST_XH_05_vertical

Commit message: layout ready to be reviewed by Leo
Connections:
- net +5V renamed +5V_Zynq
