File: FPGA_Board_BA/PCB/ls_encoder.kicad_sch (KiCad schematic)
At the start: 5 parts, among them U36 SN74LXC2T45Q1

Commit message: 22.11
Parts:
- removed C148, C149: 100n_0603, WLIB_Capacitor:C_0603, symbol WLIB_C:100n_0603
- removed R179, R180: 10k_0603, Resistor_SMD:R_0603_1608Metric, symbol WLIB_R:10k_0603
- removed U36: SN74LXC2T45Q1, MYLIB_Misc:SN74LXC2T45QDCURQ1, symbol MYLIB_Misc:SN74LXC2T45Q1
- added C150, C151: 100n_0603, WLIB_Capacitor:C_0603, symbol WLIB_C:100n_0603
- added R181, R182: 0R_0603, Resistor_SMD:R_0603_1608Metric, symbol WLIB_R:0R_0603
- added U37: SN74LXC2T45Q1, MYLIB_Misc:SN74LXC2T45QDCURQ1, symbol MYLIB_Misc:SN74LXC2T45Q1
Connections:
- net +3.3V: now also C151.1, U37.8 (VCCB)
- net A1: now also U37.2 (A1)
- net A2: now also U37.3 (A2)
- net B1: now also U37.7 (B1)
- net B2: now also U37.6 (B2)
- net GND: now also C150.1, C151.2, R182.1, U37.4 (GND)
- new net: R181.2, R182.2, U37.5 (DIR)
- new net +5V: C150.2, R181.1, U37.1 (VCCA)
Other:
- note added: "Only Pull-down populated: direction is B->A Only pull-up populated: direction is A->B"

Commit message: exported stuff
Parts:
- renumbered C150 to C145, C151 to C146, R181 to R220, R182 to R221, U37 to U36
Changed lines of the file:
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@@
 		(dnp no)
 		(fields_autoplaced yes)
-		(property "Reference" "#PWR0226"
+		(property "Reference" "#PWR0238"
 			(at 166.37 95.25 0)
 			(effects
@@
 			(project "FPGA_Board_BA"
 				(path "/fd7503bc-e7fc-4766-b224-3d1c3d7de5ff/81c9b981-9c9c-474d-998d-986f60c2f16d/01c0a5e1-90db-4782-afb3-2d55d15a02b0"
-					(reference "#PWR0260")
-					(unit 1)
-				)
-				(path "/fd7503bc-e7fc-4766-b224-3d1c3d7de5ff/81c9b981-9c9c-474d-998d-986f60c2f16d/d2b4a720-02d4-4b22-8ca6-78ca6e0e04d1"
-					(reference "#PWR0226")
+					(reference "#PWR0272")
+					(unit 1)
+				)
+				(path "/fd7503bc-e7fc-4766-b224-3d1c3d7de5ff/81c9b981-9c9c-474d-998d-986f60c2f16d/d2b4a720-02d4-4b22-8ca6-78ca6e0e04d1"
+					(reference "#PWR0238")
 					(unit 1)
 				)
@@
 		(dnp no)
 		(fields_autoplaced yes)
-		(property "Reference" "U37"
+		(property "Reference" "U36"
 			(at 134.2233 111.76 0)
 			(effects
@@
 			(project "FPGA_Board_BA"
 				(path "/fd7503bc-e7fc-4766-b224-3d1c3d7de5ff/81c9b981-9c9c-474d-998d-986f60c2f16d/01c0a5e1-90db-4782-afb3-2d55d15a02b0"
-					(reference "U43")
-					(unit 1)
-				)
-				(path "/fd7503bc-e7fc-4766-b224-3d1c3d7de5ff/81c9b981-9c9c-474d-998d-986f60c2f16d/d2b4a720-02d4-4b22-8ca6-78ca6e0e04d1"
-					(reference "U37")
+					(reference "U42")
+					(unit 1)
+				)
+				(path "/fd7503bc-e7fc-4766-b224-3d1c3d7de5ff/81c9b981-9c9c-474d-998d-986f60c2f16d/d2b4a720-02d4-4b22-8ca6-78ca6e0e04d1"
+					(reference "U36")
 					(unit 1)
 				)
@@
 		(dnp no)
 		(fields_autoplaced yes)
-		(property "Reference" "#PWR0224"
+		(property "Reference" "#PWR0236"
 			(at 132.08 120.65 0)
 			(effects
@@
 			(project "FPGA_Board_BA"
 				(path "/fd7503bc-e7fc-4766-b224-3d1c3d7de5ff/81c9b981-9c9c-474d-998d-986f60c2f16d/01c0a5e1-90db-4782-afb3-2d55d15a02b0"
-					(reference "#PWR0258")
-					(unit 1)
-				)
-				(path "/fd7503bc-e7fc-4766-b224-3d1c3d7de5ff/81c9b981-9c9c-474d-998d-986f60c2f16d/d2b4a720-02d4-4b22-8ca6-78ca6e0e04d1"
-					(reference "#PWR0224")
+					(reference "#PWR0270")
+					(unit 1)
+				)
+				(path "/fd7503bc-e7fc-4766-b224-3d1c3d7de5ff/81c9b981-9c9c-474d-998d-986f60c2f16d/d2b4a720-02d4-4b22-8ca6-78ca6e0e04d1"
+					(reference "#PWR0236")
 					(unit 1)
 				)
@@
 		(dnp no)
 		(fields_autoplaced yes)
-		(property "Reference" "#PWR0221"
+		(property "Reference" "#PWR0233"
 			(at 100.33 93.98 0)
 			(effects
@@
 			(project "FPGA_Board_BA"
 				(path "/fd7503bc-e7fc-4766-b224-3d1c3d7de5ff/81c9b981-9c9c-474d-998d-986f60c2f16d/01c0a5e1-90db-4782-afb3-2d55d15a02b0"
-					(reference "#PWR0255")
-					(unit 1)
-				)
-				(path "/fd7503bc-e7fc-4766-b224-3d1c3d7de5ff/81c9b981-9c9c-474d-998d-986f60c2f16d/d2b4a720-02d4-4b22-8ca6-78ca6e0e04d1"
-					(reference "#PWR0221")
+					(reference "#PWR0267")
+					(unit 1)
+				)
+				(path "/fd7503bc-e7fc-4766-b224-3d1c3d7de5ff/81c9b981-9c9c-474d-998d-986f60c2f16d/d2b4a720-02d4-4b22-8ca6-78ca6e0e04d1"
+					(reference "#PWR0233")
 					(unit 1)
 				)
@@
 		(dnp no)
 		(fields_autoplaced yes)
-		(property "Reference" "R181"
+		(property "Reference" "R220"
 			(at 95.25 100.33 90)
 			(effects
@@
 			(project "FPGA_Board_BA"
 				(path "/fd7503bc-e7fc-4766-b224-3d1c3d7de5ff/81c9b981-9c9c-474d-998d-986f60c2f16d/01c0a5e1-90db-4782-afb3-2d55d15a02b0"
-					(reference "R201")
-					(unit 1)
-				)
-				(path "/fd7503bc-e7fc-4766-b224-3d1c3d7de5ff/81c9b981-9c9c-474d-998d-986f60c2f16d/d2b4a720-02d4-4b22-8ca6-78ca6e0e04d1"
-					(reference "R181")
+					(reference "R240")
+					(unit 1)
+				)
+				(path "/fd7503bc-e7fc-4766-b224-3d1c3d7de5ff/81c9b981-9c9c-474d-998d-986f60c2f16d/d2b4a720-02d4-4b22-8ca6-78ca6e0e04d1"
+					(reference "R220")
 					(unit 1)
 				)
@@
 		(dnp no)
 		(fields_autoplaced yes)
-		(property "Reference" "#PWR0220"
+		(property "Reference" "#PWR0232"
 			(at 83.82 107.95 0)
 			(effects
@@
 			(project "FPGA_Board_BA"
 				(path "/fd7503bc-e7fc-4766-b224-3d1c3d7de5ff/81c9b981-9c9c-474d-998d-986f60c2f16d/01c0a5e1-90db-4782-afb3-2d55d15a02b0"
-					(reference "#PWR0254")
-					(unit 1)
-				)
-				(path "/fd7503bc-e7fc-4766-b224-3d1c3d7de5ff/81c9b981-9c9c-474d-998d-986f60c2f16d/d2b4a720-02d4-4b22-8ca6-78ca6e0e04d1"
-					(reference "#PWR0220")
+					(reference "#PWR0266")
+					(unit 1)
+				)
+				(path "/fd7503bc-e7fc-4766-b224-3d1c3d7de5ff/81c9b981-9c9c-474d-998d-986f60c2f16d/d2b4a720-02d4-4b22-8ca6-78ca6e0e04d1"
+					(reference "#PWR0232")
 					(unit 1)
 				)
@@
 		(dnp yes)
 		(fields_autoplaced yes)
-		(property "Reference" "R182"
+		(property "Reference" "R221"
 			(at 106.68 113.0299 0)
 			(effects
@@
 			(project "FPGA_Board_BA"
 				(path "/fd7503bc-e7fc-4766-b224-3d1c3d7de5ff/81c9b981-9c9c-474d-998d-986f60c2f16d/01c0a5e1-90db-4782-afb3-2d55d15a02b0"
-					(reference "R202")
-					(unit 1)
-				)
-				(path "/fd7503bc-e7fc-4766-b224-3d1c3d7de5ff/81c9b981-9c9c-474d-998d-986f60c2f16d/d2b4a720-02d4-4b22-8ca6-78ca6e0e04d1"
-					(reference "R182")
+					(reference "R241")
+					(unit 1)
+				)
+				(path "/fd7503bc-e7fc-4766-b224-3d1c3d7de5ff/81c9b981-9c9c-474d-998d-986f60c2f16d/d2b4a720-02d4-4b22-8ca6-78ca6e0e04d1"
+					(reference "R221")
 					(unit 1)
 				)
@@
 		(dnp no)
 		(fields_autoplaced yes)
-		(property "Reference" "#PWR0223"
+		(property "Reference" "#PWR0235"
 			(at 123.19 86.36 0)
 			(effects
@@
 			(project "FPGA_Board_BA"
 				(path "/fd7503bc-e7fc-4766-b224-3d1c3d7de5ff/81c9b981-9c9c-474d-998d-986f60c2f16d/01c0a5e1-90db-4782-afb3-2d55d15a02b0"
-					(reference "#PWR0257")
-					(unit 1)
-				)
-				(path "/fd7503bc-e7fc-4766-b224-3d1c3d7de5ff/81c9b981-9c9c-474d-998d-986f60c2f16d/d2b4a720-02d4-4b22-8ca6-78ca6e0e04d1"
-					(reference "#PWR0223")
+					(reference "#PWR0269")
+					(unit 1)
+				)
+				(path "/fd7503bc-e7fc-4766-b224-3d1c3d7de5ff/81c9b981-9c9c-474d-998d-986f60c2f16d/d2b4a720-02d4-4b22-8ca6-78ca6e0e04d1"
+					(reference "#PWR0235")
 					(unit 1)
 				)
@@
 		(dnp no)
 		(fields_autoplaced yes)
-		(property "Reference" "C150"
+		(property "Reference" "C145"
 			(at 110.49 76.2 90)
 			(effects
@@
 			(project "FPGA_Board_BA"
 				(path "/fd7503bc-e7fc-4766-b224-3d1c3d7de5ff/81c9b981-9c9c-474d-998d-986f60c2f16d/01c0a5e1-90db-4782-afb3-2d55d15a02b0"
-					(reference "C160")
-					(unit 1)
-				)
-				(path "/fd7503bc-e7fc-4766-b224-3d1c3d7de5ff/81c9b981-9c9c-474d-998d-986f60c2f16d/d2b4a720-02d4-4b22-8ca6-78ca6e0e04d1"
-					(reference "C150")
+					(reference "C155")
+					(unit 1)
+				)
+				(path "/fd7503bc-e7fc-4766-b224-3d1c3d7de5ff/81c9b981-9c9c-474d-998d-986f60c2f16d/d2b4a720-02d4-4b22-8ca6-78ca6e0e04d1"
+					(reference "C145")
 					(unit 1)
 				)
@@
 		(dnp no)
 		(fields_autoplaced yes)
-		(property "Reference" "#PWR0225"
+		(property "Reference" "#PWR0237"
 			(at 140.97 86.36 0)
 			(effects
@@
 			(project "FPGA_Board_BA"
 				(path "/fd7503bc-e7fc-4766-b224-3d1c3d7de5ff/81c9b981-9c9c-474d-998d-986f60c2f16d/01c0a5e1-90db-4782-afb3-2d55d15a02b0"
-					(reference "#PWR0259")
-					(unit 1)
-				)
-				(path "/fd7503bc-e7fc-4766-b224-3d1c3d7de5ff/81c9b981-9c9c-474d-998d-986f60c2f16d/d2b4a720-02d4-4b22-8ca6-78ca6e0e04d1"
-					(reference "#PWR0225")
+					(reference "#PWR0271")
+					(unit 1)
+				)
+				(path "/fd7503bc-e7fc-4766-b224-3d1c3d7de5ff/81c9b981-9c9c-474d-998d-986f60c2f16d/d2b4a720-02d4-4b22-8ca6-78ca6e0e04d1"
+					(reference "#PWR0237")
 					(unit 1)
 				)
@@
 		(dnp no)
 		(fields_autoplaced yes)
-		(property "Reference" "C151"
+		(property "Reference" "C146"
 			(at 153.67 76.2 90)
 			(effects
@@
 			(project "FPGA_Board_BA"
 				(path "/fd7503bc-e7fc-4766-b224-3d1c3d7de5ff/81c9b981-9c9c-474d-998d-986f60c2f16d/01c0a5e1-90db-4782-afb3-2d55d15a02b0"
-					(reference "C161")
-					(unit 1)
-				)
-				(path "/fd7503bc-e7fc-4766-b224-3d1c3d7de5ff/81c9b981-9c9c-474d-998d-986f60c2f16d/d2b4a720-02d4-4b22-8ca6-78ca6e0e04d1"
-					(reference "C151")
+					(reference "C156")
+					(unit 1)
+				)
+				(path "/fd7503bc-e7fc-4766-b224-3d1c3d7de5ff/81c9b981-9c9c-474d-998d-986f60c2f16d/d2b4a720-02d4-4b22-8ca6-78ca6e0e04d1"
+					(reference "C146")
 					(unit 1)
 				)
@@
 		(dnp no)
 		(fields_autoplaced yes)
-		(property "Reference" "#PWR0222"
+		(property "Reference" "#PWR0234"
 			(at 104.14 127 0)
 			(effects
@@
 			(project "FPGA_Board_BA"
 				(path "/fd7503bc-e7fc-4766-b224-3d1c3d7de5ff/81c9b981-9c9c-474d-998d-986f60c2f16d/01c0a5e1-90db-4782-afb3-2d55d15a02b0"
-					(reference "#PWR0256")
-					(unit 1)
-				)
-				(path "/fd7503bc-e7fc-4766-b224-3d1c3d7de5ff/81c9b981-9c9c-474d-998d-986f60c2f16d/d2b4a720-02d4-4b22-8ca6-78ca6e0e04d1"
-					(reference "#PWR0222")
-					(unit 1)
-				)
+					(reference "#PWR0268")
+					(unit 1)
+				)
+				(path "/fd7503bc-e7fc-4766-b224-3d1c3d7de5ff/81c9b981-9c9c-474d-998d-986f60c2f16d/d2b4a720-02d4-4b22-8ca6-78ca6e0e04d1"
+					(reference "#PWR0234")
+					(unit 1)
+				)

Commit message: layout 99% ready
Connections:
- net +5V renamed +5VA
Changed lines of the file:
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@@
-		)
-	)
-	(label "+5V"
-		(at 129.54 83.82 180)
-		(effects
-			(font
-				(size 1.27 1.27)
-			)
-			(justify right bottom)
 		)
 	)
@@
 	)
 	(symbol
+		(lib_id "power:+5VA")
+		(at 123.19 82.55 0)
+		(unit 1)
+		(exclude_from_sim no)
+		(in_bom yes)
+		(on_board yes)
+		(dnp no)
+		(fields_autoplaced yes)
+		(property "Reference" "#PWR0159"
+			(at 123.19 86.36 0)
+			(effects
+				(font
+					(size 1.27 1.27)
+				)
+				(hide yes)
+			)
+		)
+		(property "Value" "+5VA"
+			(at 123.19 77.47 0)
+			(effects
+				(font
+					(size 1.27 1.27)
+				)
+			)
+		)
+		(property "Footprint" ""
+			(at 123.19 82.55 0)
+			(effects
+				(font
+					(size 1.27 1.27)
+				)
+				(hide yes)
+			)
+		)
+		(property "Datasheet" ""
+			(at 123.19 82.55 0)
+			(effects
+				(font
+					(size 1.27 1.27)
+				)
+				(hide yes)
+			)
+		)
+		(property "Description" "Power symbol creates a global label with name \"+5VA\""
+			(at 123.19 82.55 0)
+			(effects
+				(font
+					(size 1.27 1.27)
+				)
+				(hide yes)
+			)
+		)
+		(pin "1"
+		)
+		(instances
+			(project ""
+				(path "/fd7503bc-e7fc-4766-b224-3d1c3d7de5ff/81c9b981-9c9c-474d-998d-986f60c2f16d/01c0a5e1-90db-4782-afb3-2d55d15a02b0"
+					(reference "#PWR0164")
+					(unit 1)
+				)
+				(path "/fd7503bc-e7fc-4766-b224-3d1c3d7de5ff/81c9b981-9c9c-474d-998d-986f60c2f16d/d2b4a720-02d4-4b22-8ca6-78ca6e0e04d1"
+					(reference "#PWR0159")
+					(unit 1)
+				)
+			)
+		)
+	)
+	(symbol
 		(lib_id "WLIB_R:0R_0603")
 		(at 95.25 106.68 90)
@@
 	)
 	(symbol
-		(lib_id "power:+5V")
+		(lib_id "WLIB_R:0R_0603")
+		(at 104.14 114.3 180)
+		(unit 1)
+		(exclude_from_sim no)
+		(in_bom yes)
+		(on_board yes)
+		(dnp yes)
+		(fields_autoplaced yes)
+		(property "Reference" "R221"
+			(at 106.68 113.0299 0)
+			(effects
+				(font
+					(size 1.27 1.27)
+				)
+				(justify right)
+			)
+		)
+		(property "Value" "0R_0603"
+			(at 106.68 115.5699 0)
+			(effects
+				(font
+					(size 1.27 1.27)
+				)
+				(justify right)
+			)
+		)
+		(property "Footprint" "Resistor_SMD:R_0603_1608Metric"
+			(at 104.14 130.81 0)
+			(effects
+				(font
+					(size 1.27 1.27)
+				)
+				(hide yes)
+			)
+		)
+		(property "Datasheet" "https://www.farnell.com/datasheets/2869757.pdf"
+			(at 104.14 133.35 0)
+			(effects
+				(font
+					(size 1.27 1.27)
+				)
+				(hide yes)
+			)
+		)
+		(property "Description" "Jumper Resistor"
+			(at 104.14 114.3 0)
+			(effects
+				(font
+					(size 1.27 1.27)
+				)
+				(hide yes)
+			)
+		)
+		(property "FARNELL" "2309111"
+			(at 104.14 128.27 0)
+			(effects
+				(font
+					(size 1.27 1.27)
+				)
+				(hide yes)
+			)
+		)
+		(property "Rated Power" "100mW"
+			(at 104.14 125.73 0)
+			(effects
+				(font
+					(size 1.27 1.27)
+				)
+				(hide yes)
+			)
+		)
+		(pin "2"
+		)
+		(pin "1"
+		)
+		(instances
+			(project "FPGA_Board_BA"
+				(path "/fd7503bc-e7fc-4766-b224-3d1c3d7de5ff/81c9b981-9c9c-474d-998d-986f60c2f16d/01c0a5e1-90db-4782-afb3-2d55d15a02b0"
+					(reference "R241")
+					(unit 1)
+				)
+				(path "/fd7503bc-e7fc-4766-b224-3d1c3d7de5ff/81c9b981-9c9c-474d-998d-986f60c2f16d/d2b4a720-02d4-4b22-8ca6-78ca6e0e04d1"
+					(reference "R221")
+					(unit 1)
+				)
+			)
+		)
+	)
+	(symbol
+		(lib_id "power:+5VA")
 		(at 83.82 104.14 0)
 		(unit 1)
@@
 		(dnp no)
 		(fields_autoplaced yes)
-		(property "Reference" "#PWR0232"
+		(property "Reference" "#PWR0165"
 			(at 83.82 107.95 0)
 			(effects
@@
 			)
 		)
-		(property "Value" "+5V"
+		(property "Value" "+5VA"
 			(at 83.82 99.06 0)
 			(effects
@@
 			)
 		)
-		(property "Description" "Power symbol creates a global label with name \"+5V\""
+		(property "Description" "Power symbol creates a global label with name \"+5VA\""
 			(at 83.82 104.14 0)
 			(effects
@@
 			(project "FPGA_Board_BA"
 				(path "/fd7503bc-e7fc-4766-b224-3d1c3d7de5ff/81c9b981-9c9c-474d-998d-986f60c2f16d/01c0a5e1-90db-4782-afb3-2d55d15a02b0"
-					(reference "#PWR0266")
-					(unit 1)
-				)
-				(path "/fd7503bc-e7fc-4766-b224-3d1c3d7de5ff/81c9b981-9c9c-474d-998d-986f60c2f16d/d2b4a720-02d4-4b22-8ca6-78ca6e0e04d1"
-					(reference "#PWR0232")
-					(unit 1)
-				)
-			)
-		)
-	)
-	(symbol
-		(lib_id "WLIB_R:0R_0603")
-		(at 104.14 114.3 180)
-		(unit 1)
-		(exclude_from_sim no)
-		(in_bom yes)
-		(on_board yes)
-		(dnp yes)
-		(fields_autoplaced yes)
-		(property "Reference" "R221"
-			(at 106.68 113.0299 0)
-			(effects
-				(font
-					(size 1.27 1.27)
-				)
-				(justify right)
-			)
-		)
-		(property "Value" "0R_0603"
-			(at 106.68 115.5699 0)
-			(effects
-				(font
-					(size 1.27 1.27)
-				)
-				(justify right)
-			)
-		)
-		(property "Footprint" "Resistor_SMD:R_0603_1608Metric"
-			(at 104.14 130.81 0)
-			(effects
-				(font
-					(size 1.27 1.27)
-				)
-				(hide yes)
-			)
-		)
-		(property "Datasheet" "https://www.farnell.com/datasheets/2869757.pdf"
-			(at 104.14 133.35 0)
-			(effects
-				(font
-					(size 1.27 1.27)
-				)
-				(hide yes)
-			)
-		)
-		(property "Description" "Jumper Resistor"
-			(at 104.14 114.3 0)
-			(effects
-				(font
-					(size 1.27 1.27)
-				)
-				(hide yes)
-			)
-		)
-		(property "FARNELL" "2309111"
-			(at 104.14 128.27 0)
-			(effects
-				(font
-					(size 1.27 1.27)
-				)
-				(hide yes)
-			)
-		)
-		(property "Rated Power" "100mW"
-			(at 104.14 125.73 0)
-			(effects
-				(font
-					(size 1.27 1.27)
-				)
-				(hide yes)
-			)
-		)
-		(pin "2"
-		)
-		(pin "1"
-		)
-		(instances
-			(project "FPGA_Board_BA"
-				(path "/fd7503bc-e7fc-4766-b224-3d1c3d7de5ff/81c9b981-9c9c-474d-998d-986f60c2f16d/01c0a5e1-90db-4782-afb3-2d55d15a02b0"
-					(reference "R241")
-					(unit 1)
-				)
-				(path "/fd7503bc-e7fc-4766-b224-3d1c3d7de5ff/81c9b981-9c9c-474d-998d-986f60c2f16d/d2b4a720-02d4-4b22-8ca6-78ca6e0e04d1"
-					(reference "R221")
-					(unit 1)
-				)
-			)
-		)
-	)
-	(symbol
-		(lib_id "power:+5V")
-		(at 123.19 82.55 0)
-		(unit 1)
-		(exclude_from_sim no)
-		(in_bom yes)
-		(on_board yes)
-		(dnp no)
-		(fields_autoplaced yes)
-		(property "Reference" "#PWR0235"
-			(at 123.19 86.36 0)
-			(effects
-				(font
-					(size 1.27 1.27)
-				)
-				(hide yes)
-			)
-		)
-		(property "Value" "+5V"
-			(at 123.19 77.47 0)
-			(effects
-				(font
-					(size 1.27 1.27)
-				)
-			)
-		)
-		(property "Footprint" ""
-			(at 123.19 82.55 0)
-			(effects
-				(font
-					(size 1.27 1.27)
-				)
-				(hide yes)
-			)
-		)
-		(property "Datasheet" ""
-			(at 123.19 82.55 0)
-			(effects
-				(font
-					(size 1.27 1.27)
-				)
-				(hide yes)
-			)
-		)
-		(property "Description" "Power symbol creates a global label with name \"+5V\""
-			(at 123.19 82.55 0)
-			(effects
-				(font
-					(size 1.27 1.27)
-				)
-				(hide yes)
-			)
-		)
-		(pin "1"
-		)
-		(instances
-			(project "FPGA_Board_BA"
-				(path "/fd7503bc-e7fc-4766-b224-3d1c3d7de5ff/81c9b981-9c9c-474d-998d-986f60c2f16d/01c0a5e1-90db-4782-afb3-2d55d15a02b0"
-					(reference "#PWR0269")
-					(unit 1)
-				)
-				(path "/fd7503bc-e7fc-4766-b224-3d1c3d7de5ff/81c9b981-9c9c-474d-998d-986f60c2f16d/d2b4a720-02d4-4b22-8ca6-78ca6e0e04d1"
-					(reference "#PWR0235")
-					(unit 1)
-				)
+					(reference "#PWR0168")
+					(unit 1)
+				)
+				(path "/fd7503bc-e7fc-4766-b224-3d1c3d7de5ff/81c9b981-9c9c-474d-998d-986f60c2f16d/d2b4a720-02d4-4b22-8ca6-78ca6e0e04d1"
+					(reference "#PWR0165")
+					(unit 1)
+				)
